File: A2630-New-KiCAD/N2360.sch (KiCad schematic (older format))
At the start: 0 parts

Commit message: Add files via upload
Changed lines of the file:
@@
 $Descr A4 11693 8268
 encoding utf-8
-Sheet 1 5
+Sheet 1 6
 Title ""
 Date ""
@@
 F1 "Card Edge.sch" 50
 $EndSheet
+$Sheet
+S 1025 1425 1100 400
+U 634ECC15
+F0 "Logic" 51
+F1 "Logic.sch" 51
+$EndSheet
 $EndSCHEMATC

Commit message: Add files via upload
Changed lines of the file:
@@
 $Descr A4 11693 8268
 encoding utf-8
-Sheet 1 6
+Sheet 1 8
 Title ""
 Date ""
@@
 F1 "Logic.sch" 51
 $EndSheet
+$Sheet
+S 2475 1400 1000 400
+U 61EF4CC7
+F0 "Xilinx" 50
+F1 "Xilinx.sch" 50
+$EndSheet
+$Sheet
+S 3775 1450 875  350
+U 61FBE594
+F0 "Base Memory" 51
+F1 "BaseMemory.sch" 51
+$EndSheet
 $EndSCHEMATC

Commit message: Add files via upload
Changed lines of the file:
@@
+$EndSheet
+$Sheet
+S 3775 1450 875  350
+U 61FBE594
+F0 "Base Memory" 51
+F1 "BaseMemory.sch" 51
 $EndSheet
 $Sheet
 S 2475 775  1050 350
 U 61D9C8DC
-F0 "Memory" 50
-F1 "Memory.sch" 50
+F0 "Expansion Memory" 50
+F1 "ExpansionMemory.sch" 50
+$EndSheet
+$Sheet
+S 3750 775  900  350
+U 61DF74A0
+F0 "Card Edge" 50
+F1 "Card Edge.sch" 50
 $EndSheet
 $Sheet
@@
 F0 "Power and Spares" 50
 F1 "Power.sch" 50
-$EndSheet
-$Sheet
-S 3750 775  900  350
-U 61DF74A0
-F0 "Card Edge" 50
-F1 "Card Edge.sch" 50
 $EndSheet
 $Sheet
@@
 F1 "Xilinx.sch" 50
 $EndSheet
-$Sheet
-S 3775 1450 875  350
-U 61FBE594
-F0 "Base Memory" 51
-F1 "BaseMemory.sch" 51
-$EndSheet
 $EndSCHEMATC

Commit message: Add files via upload
Changed lines of the file:
@@
 $Descr A4 11693 8268
 encoding utf-8
-Sheet 1 8
+Sheet 1 9
 Title ""
 Date ""
@@
 F1 "Xilinx.sch" 50
 $EndSheet
+$Sheet
+S 4875 1450 925  350
+U 62089831
+F0 "CPLD 1" 50
+F1 "CPLD1.sch" 50
+$EndSheet
 $EndSCHEMATC

Commit message: Add files via upload
Changed lines of the file:
@@
 $Descr A4 11693 8268
 encoding utf-8
-Sheet 1 9
+Sheet 1 8
 Title ""
 Date ""
@@
 $EndSheet
 $Sheet
-S 2475 1400 1000 400
-U 61EF4CC7
-F0 "Xilinx" 50
-F1 "Xilinx.sch" 50
-$EndSheet
-$Sheet
