File: A2630-New-KiCAD/Card Edge.sch (KiCad schematic (older format))
At the start: 13 parts, among them CN700 Amiga-2000-CPU-Slot, U300 74HCT05, U307 74HCT04, U700 74HCT174, U701 74FCT646, U702 74FCT646, U703 74HCT245, U704 74HCT245, U705 74HCT245, U706 74HCT245, U707 74HCT245

Commit message: Add files via upload
Parts:
- added C701, C702, C703, C704, C705, C706, C707: 0.22uF, Capacitor_SMD:C_0805_2012Metric, symbol Device:C
- added C712, C714, C718: 10uF, symbol Device:CP1
- added C713: 47uF, symbol Device:CP1
- added J301, J302, J303, J304: Jumper_NO_Small, Connector_PinHeader_2.54mm:PinHeader_1x02_P2.54mm_Vertical, symbol Device:Jumper_NO_Small
- added RN300: 3.3K, Resistor_THT:R_Array_SIP5, symbol Device:R_Network04
Connections:
- net +5V: now also U701.24 (Vcc), U702.24 (Vcc), U703.20 (Vcc), U704.20 (Vcc), U705.20 (Vcc), U706.20 (Vcc), U707.20 (Vcc), C701.1, C702.1, C703.1, C704.1, C705.1, C706.1, C707.1, C712.1, C713.1, C714.1, C718.1, RN300.1 (common)
- net GND: now also U701.12 (GND), U702.12 (GND), U703.10 (GND), U704.10 (GND), U705.10 (GND), U706.10 (GND), U707.10 (GND), C701.2, C702.2, C703.2, C704.2, C705.2, C706.2, C707.2, C712.2, C713.2, C714.2, C718.2, J301.1, J302.1, J303.1, J304.1
- new net B2000: J302.2, RN300.3 (R2)
- new net MEG4: J301.2, RN300.2 (R1)
- new net OSMODE: J304.2, RN300.5 (R4)
- new net RAM_AUTO: J303.2, RN300.4 (R3)
Other:
- note added: "Not all these jumpers will make it to the final version.\nJ301 - 2MEG Shorted/4MEG Open\nJ302 - A2000 Shorted/B2000 Open\nJ303 - Do not configure RAM Shorted/Autoconfigure RAM Open\nJ404 - AMIX Shorted/AmigaOS Open"
- moved on the sheet: U701B, U702B, U703B, U704B, U705B, U706B, U707B

Commit message: Add files via upload
Connections:
- net _BERR: now also U300.8; no longer U300.9
- net at U307.6: now also U300.9; no longer U300.8
Changed lines of the file:
@@
 $Descr B 17000 11000
 encoding utf-8
-Sheet 5 6
+Sheet 5 8
 Title ""
 Date ""
@@
 Wire Wire Line
 	4125 7350 2975 7350
-Text GLabel 950  7450 0    39   BiDi ~ 0
+Text GLabel 950  7450 0    50   BiDi ~ 0
 _VPA
 Wire Wire Line
@@
 Wire Wire Line
 	4025 7900 950  7900
-Text GLabel 925  7575 0    39   BiDi ~ 0
+Text GLabel 925  7575 0    50   BiDi ~ 0
 E
-Text GLabel 950  7700 0    39   BiDi ~ 0
+Text GLabel 950  7700 0    50   BiDi ~ 0
 _VMA
-Text GLabel 950  7800 0    39   BiDi ~ 0
+Text GLabel 950  7800 0    50   BiDi ~ 0
 _RESET
-Text GLabel 950  7900 0    39   Output ~ 0
+Text GLabel 950  7900 0    50   Output ~ 0
 _HALT
 Wire Wire Line
@@
 U 4 1 6234EB07
 P 1675 7225
-F 0 "U300" H 1675 7542 50  0000 C CNN
-F 1 "74HCT05" H 1675 7451 50  0000 C CNN
+F 0 "U300" H 1700 6925 50  0000 C CNN
+F 1 "74HCT05" H 1675 7000 50  0000 C CNN
 F 2 "Package_SO:SOIC-14_3.9x8.7mm_P1.27mm" H 1675 7225 50  0001 C CNN
 F 3 "http://www.ti.com/lit/gpn/sn74LS05" H 1675 7225 50  0001 C CNN
 	4    1675 7225
-	1    0    0    -1
+	-1   0    0    1
 $EndComp
 Wire Wire Line
@@
 Wire Wire Line
 	14350 2825 14350 3575
+Connection ~ 14350 3575
+Wire Wire Line
+	14350 3575 15025 3575
+$Comp
+L power:+5V #PWR?
+U 1 1 634E5D41
+P 14050 2425
+F 0 "#PWR?" H 14050 2275 50  0001 C CNN
+F 1 "+5V" H 14065 2598 50  0000 C CNN
+F 2 "" H 14050 2425 50  0001 C CNN
+F 3 "" H 14050 2425 50  0001 C CNN
+	1    14050 2425
+	1    0    0    -1
+$EndComp
+Text Notes 13675 4300 0    51   ~ 0
+Not all these jumpers will make it to the final version.\nJ301 - 2MEG Shorted/4MEG Open\nJ302 - A2000 Shorted/B2000 Open\nJ303 - Do not configure RAM Shorted/Autoconfigure RAM Open\nJ404 - AMIX Shorted/AmigaOS Open
 Wire Bus Line
 	1250 3825 1250 4075
@@
 Wire Bus Line
 	8100 2575 8100 10025
-Connection ~ 14350 3575
-Wire Wire Line
-	14350 3575 15025 3575
-$Comp
-L power:+5V #PWR?
-U 1 1 634E5D41
-P 14050 2425
-F 0 "#PWR?" H 14050 2275 50  0001 C CNN
-F 1 "+5V" H 14065 2598 50  0000 C CNN
-F 2 "" H 14050 2425 50  0001 C CNN
-F 3 "" H 14050 2425 50  0001 C CNN
-	1    14050 2425
-	1    0    0    -1
-$EndComp
-Text Notes 13675 4300 0    51   ~ 0
-Not all these jumpers will make it to the final version.\nJ301 - 2MEG Shorted/4MEG Open\nJ302 - A2000 Shorted/B2000 Open\nJ303 - Do not configure RAM Shorted/Autoconfigure RAM Open\nJ404 - AMIX Shorted/AmigaOS Open
 $EndSCHEMATC

Commit message: Add files via upload
Parts:
- C712, C713, C714, C718: footprint (none) -> Capacitor_THT:CP_Radial_D5.0mm_P2.00mm
Changed lines of the file:
@@
 	9350 8825 9450 8825
 $Comp
-L power:+5V #PWR?
+L power:+5V #PWR0139
 U 1 1 6223A134
 P 8975 7650
-F 0 "#PWR?" H 8975 7500 50  0001 C CNN
+F 0 "#PWR0139" H 8975 7500 50  0001 C CNN
 F 1 "+5V" H 8990 7823 50  0000 C CNN
 F 2 "" H 8975 7650 50  0001 C CNN
@@
 Connection ~ 8975 7650
 $Comp
-L power:GND #PWR?
+L power:GND #PWR0140
 U 1 1 6223E02F
 P 14725 8825
-F 0 "#PWR?" H 14725 8575 50  0001 C CNN
+F 0 "#PWR0140" H 14725 8575 50  0001 C CNN
 F 1 "GND" H 14730 8652 50  0000 C CNN
 F 2 "" H 14725 8825 50  0001 C CNN
@@
 F 0 "C713" H 8860 9154 50  0000 R CNN
 F 1 "47uF" H 8860 9245 50  0000 R CNN
-F 2 "" H 8975 9200 50  0001 C CNN
+F 2 "Capacitor_THT:CP_Radial_D5.0mm_P2.00mm" H 8975 9200 50  0001 C CNN
 F 3 "~" H 8975 9200 50  0001 C CNN
 	1    8975 9200
@@
 F 0 "C714" H 9335 9154 50  0000 R CNN
 F 1 "10uF" H 9335 9245 50  0000 R CNN
-F 2 "" H 9450 9200 50  0001 C CNN
+F 2 "Capacitor_THT:CP_Radial_D5.0mm_P2.00mm" H 9450 9200 50  0001 C CNN
 F 3 "~" H 9450 9200 50  0001 C CNN
 	1    9450 9200
@@
 F 0 "C718" H 9810 9154 50  0000 R CNN
 F 1 "10uF" H 9810 9245 50  0000 R CNN
-F 2 "" H 9925 9200 50  0001 C CNN
+F 2 "Capacitor_THT:CP_Radial_D5.0mm_P2.00mm" H 9925 9200 50  0001 C CNN
 F 3 "~" H 9925 9200 50  0001 C CNN
 	1    9925 9200
@@
 F 0 "C712" H 10260 9154 50  0000 R CNN
 F 1 "10uF" H 10260 9245 50  0000 R CNN
-F 2 "" H 10375 9200 50  0001 C CNN
+F 2 "Capacitor_THT:CP_Radial_D5.0mm_P2.00mm" H 10375 9200 50  0001 C CNN
 F 3 "~" H 10375 9200 50  0001 C CNN
 	1    10375 9200
@@
 	13400 3225 13400 3400
 $Comp
-L power:GND #PWR?
+L power:GND #PWR0141
 U 1 1 63340664
 P 13400 3875
-F 0 "#PWR?" H 13400 3625 50  0001 C CNN
+F 0 "#PWR0141" H 13400 3625 50  0001 C CNN
 F 1 "GND" H 13405 3702 50  0000 C CNN
 F 2 "" H 13400 3875 50  0001 C CNN
@@
 	14350 3575 15025 3575
 $Comp
-L power:+5V #PWR?
+L power:+5V #PWR0142
 U 1 1 634E5D41
 P 14050 2425
-F 0 "#PWR?" H 14050 2275 50  0001 C CNN
+F 0 "#PWR0142" H 14050 2275 50  0001 C CNN
 F 1 "+5V" H 14065 2598 50  0000 C CNN
 F 2 "" H 14050 2425 50  0001 C CNN

Commit message: Add files via upload
Connections:
- net A3: now also U707.6 (A4); no longer U707.5 (A3)
- net A4: now also U707.5 (A3); no longer U707.6 (A4)
- net AA3: now also U707.14 (B4); no longer U707.15 (B3)
- net AA4: now also U707.15 (B3); no longer U707.14 (B4)
- net _AAS: now also CN700.74
- net _LDS: now also CN700.70
Changed lines of the file:
@@
 	4125 8550 950  8550
 Wire Wire Line
-	4100 8650 950  8650
+	4125 8650 950  8650
 Wire Wire Line
 	4125 8750 950  8750
 Wire Wire Line
-	4100 8850 950  8850
+	4125 8850 950  8850
 Text GLabel 950  8350 0    50   BiDi ~ 0
 _ABG
@@
 Text Label 12125 5400 2    51   ~ 0
 A2
-Text Label 12125 5300 2    51   ~ 0
+Text Label 12100 5200 2    51   ~ 0
 A3
-Text Label 12125 5200 2    51   ~ 0
+Text Label 12100 5300 2    51   ~ 0
 A4
 Text Label 12125 5100 2    51   ~ 0
@@
 Text Label 10450 5400 0    51   ~ 0
 AA2
+Text Label 10450 5200 0    51   ~ 0
+AA3
 Text Label 10450 5300 0    51   ~ 0
-AA3
-Text Label 10450 5200 0    51   ~ 0
 AA4
 Text Label 10450 5100 0    51   ~ 0

Commit message: Add files via upload
Connections:
- net A1: now also U707.8 (A6); no longer U707.3 (A1)
- net A14: now also U706.9 (A7); no longer U706.8 (A6)
- net A15: now also U706.8 (A6); no longer U706.9 (A7)
- net A2: now also U707.9 (A7); no longer U707.4 (A2)
- net A22: now also U705.9 (A7); no longer U705.8 (A6)
- net A23: now also U705.8 (A6); no longer U705.9 (A7)
- net A5: now also U707.3 (A1); no longer U707.7 (A5)
- net A6: now also U707.4 (A2); no longer U707.8 (A6)
- net A7: now also U707.7 (A5); no longer U707.9 (A7)
- net AA1: now also U707.12 (B6); no longer U707.17 (B1)
- net AA14: now also U706.11 (B7); no longer U706.12 (B6)
- net AA15: now also U706.12 (B6); no longer U706.11 (B7)
- net AA2: now also U707.11 (B7); no longer U707.16 (B2)
- net AA22: now also U705.11 (B7); no longer U705.12 (B6)
- net AA23: now also U705.12 (B6); no longer U705.11 (B7)
- net AA5: now also U707.17 (B1); no longer U707.13 (B5)
- net AA6: now also U707.16 (B2); no longer U707.12 (B6)
- net AA7: now also U707.13 (B5); no longer U707.11 (B7)
- net CLK7M: now reaches U700.9 (Cp)
- net A0: no longer names the net of U707.2 (A0)
- net AA0: no longer names the net of U707.18 (B0)
- no-connect marks 3 -> 5
Other:
- note added: "There is no A0 on the 68000 (Amiga 2000)\nThus, it is not connected here."
- note removed: "PAL HERE"
Changed lines of the file:
@@
 Wire Wire Line
 	2525 3475 3025 3475
-Wire Wire Line
-	3025 3475 3025 1175
 $Comp
 L power:GND #PWR0128
@@
 Wire Wire Line
 	3575 7575 925  7575
-Text Notes 2625 1175 0    157  ~ 0
-PAL HERE
 $Comp
 L N2630:74FCT646 U701
@@
 	6250 10225 975  10225
 Text GLabel 975  10225 0    51   BiDi ~ 0
-D(31:0)
+D[31..0]
 Entry Wire Line
 	6250 2575 6350 2475
@@
 Wire Bus Line
 	15925 975  12225 975
-Entry Wire Line
-	12225 5500 12125 5600
 Wire Wire Line
 	12125 5600 11775 5600
@@
 	12125 3975 12225 3875
 Text GLabel 15925 975  2    51   BiDi ~ 0
-A(31:0)
-Text Label 12125 5600 2    51   ~ 0
-A0
+A[31..0]
+Text Label 12125 4900 2    51   ~ 0
+A2
+Text Label 12125 5200 2    51   ~ 0
+A3
+Text Label 12125 5300 2    51   ~ 0
+A4
 Text Label 12125 5500 2    51   ~ 0
-A1
+A5
 Text Label 12125 5400 2    51   ~ 0
-A2
-Text Label 12100 5200 2    51   ~ 0
-A3
-Text Label 12100 5300 2    51   ~ 0
-A4
+A6
 Text Label 12125 5100 2    51   ~ 0
-A5
-Text Label 12125 5000 2    51   ~ 0
-A6
-Text Label 12125 4900 2    51   ~ 0
 A7
 Text Label 12125 4075 2    51   ~ 0
@@
 Text Label 12125 3575 2    51   ~ 0
 A13
+Text Label 12125 3375 2    51   ~ 0
+A14
 Text Label 12125 3475 2    51   ~ 0
-A14
-Text Label 12125 3375 2    51   ~ 0
 A15
 Text Label 12125 2525 2    51   ~ 0
@@
 Text Label 12125 2025 2    51   ~ 0
 A21
+Text Label 12125 1825 2    51   ~ 0
+A22
 Text Label 12125 1925 2    51   ~ 0
-A22
-Text Label 12125 1825 2    51   ~ 0
 A23
 $Comp
@@
 Entry Wire Line
 	10450 5500 10350 5400
-Entry Wire Line
-	10450 5600 10350 5500
 Wire Bus Line
 	10350 1300 5300 1300
@@
 Entry Wire Line
 	10450 2425 10350 2325
-Text Label 10450 5600 0    51   ~ 0
-AA0
-Text Label 10450 5500 0    51   ~ 0
+Text Label 10450 5000 0    51   ~ 0
 AA1
-Text Label 10450 5400 0    51   ~ 0
+Text Label 10450 4900 0    51   ~ 0
 AA2
 Text Label 10450 5200 0    51   ~ 0
@@
 Text Label 10450 5300 0    51   ~ 0
 AA4
+Text Label 10450 5500 0    51   ~ 0
+AA5
+Text Label 10450 5400 0    51   ~ 0
+AA6
 Text Label 10450 5100 0    51   ~ 0
-AA5
-Text Label 10450 5000 0    51   ~ 0
-AA6
-Text Label 10450 4900 0    51   ~ 0
 AA7
 Text Label 10450 4075 0    51   ~ 0
@@
 Text Label 10450 3575 0    51   ~ 0
 AA13
+Text Label 10450 3375 0    51   ~ 0
+AA14
 Text Label 10450 3475 0    51   ~ 0
-AA14
-Text Label 10450 3375 0    51   ~ 0
 AA15
 Text Label 10450 2525 0    51   ~ 0
@@
 Text Label 10450 2025 0    51   ~ 0
 AA21
+Text Label 10450 1825 0    51   ~ 0
+AA22
 Text Label 10450 1925 0    51   ~ 0
-AA22
-Text Label 10450 1825 0    51   ~ 0
 AA23
 Wire Wire Line
@@
 Text Notes 13675 4300 0    51   ~ 0
 Not all these jumpers will make it to the final version.\nJ301 - 2MEG Shorted/4MEG Open\nJ302 - A2000 Shorted/B2000 Open\nJ303 - Do not configure RAM Shorted/Autoconfigure RAM Open\nJ404 - AMIX Shorted/AmigaOS Open
+NoConn ~ 10450 5600
+Text Label 12125 5000 2    51   ~ 0
+A1
+NoConn ~ 12125 5600
+Text Notes 12400 5600 0    50   ~ 0
+There is no A0 on the 68000 (Amiga 2000)\nThus, it is not connected here.
 Wire Bus Line
 	1250 3825 1250 4075
@@
 	4650 8400 4650 10025
 Wire Bus Line
-	12225 975  12225 5500
+	12225 975  12225 5400
 Wire Bus Line
-	10350 1300 10350 5500
+	10350 1300 10350 5400
 Wire Bus Line
 	6250 2575 6250 10225
 Wire Bus Line
 	8100 2575 8100 10025
+Text Label 3025 3475 2    50   ~ 0
+CLK7M
 $EndSCHEMATC

Commit message: Add files via upload
Connections:
- net 28M: now reaches CN700.9
- net CLK7M renamed _CLK7M
Changed lines of the file:
@@
 $Descr B 17000 11000
 encoding utf-8
-Sheet 5 8
+Sheet 5 9
 Title ""
 Date ""
@@
 	4125 5850 3550 5850
 Wire Wire Line
-	4025 5900 3550 5900
-Wire Wire Line
-	4125 5950 3550 5950
-Wire Wire Line
 	4025 6000 925  6000
-Text Label 3550 5850 2    39   ~ 0
-_C3
-Text Label 3550 5900 2    39   ~ 0
-_CDAC
-Text Label 3550 5950 2    39   ~ 0
-_C1
 Text GLabel 925  6000 0    50   Input ~ 0
 _OVR
@@
 Text Notes 12400 5600 0    50   ~ 0
 There is no A0 on the 68000 (Amiga 2000)\nThus, it is not connected here.
+Text GLabel 925  5625 0    50   Output ~ 0
+_C3
+Text GLabel 925  5725 0    50   Output ~ 0
+_CDAC
+Text GLabel 925  5825 0    50   Output ~ 0
+_C1
+Wire Wire Line
+	925  5625 3550 5625
+Wire Wire Line
+	3550 5625 3550 5850
+Wire Wire Line
+	3425 5900 3425 5725
+Wire Wire Line
+	3425 5725 925  5725
+Wire Wire Line
+	3425 5900 4025 5900
+Wire Wire Line
+	1475 5950 1475 5825
+Wire Wire Line
+	1475 5825 925  5825
+Wire Wire Line
+	1475 5950 4125 5950
+Text GLabel 1075 2225 0    50   Input ~ 0
+_CLK7M
+Wire Wire Line
+	1075 2225 3025 2225
+Wire Wire Line
+	3025 2225 3025 3475
+Wire Wire Line
+	4025 5600 3600 5600
+Wire Wire Line
+	3600 5600 3600 5450
+Wire Wire Line
+	3600 5450 925  5450
+Text GLabel 925  5450 0    50   Output ~ 0
+28M
 Wire Bus Line
 	1250 3825 1250 4075
@@
 Wire Bus Line
 	8100 2575 8100 10025
-Text Label 3025 3475 2    50   ~ 0
-CLK7M
 $EndSCHEMATC

Commit message: Add files via upload
Connections:
- net ARW renamed AR_W
- net MEG4 renamed TWOMB
- net RAM_AUTO renamed AUTO
Changed lines of the file:
@@
 $Descr B 17000 11000
 encoding utf-8
-Sheet 5 9
+Sheet 5 8
 Title ""
 Date ""
@@
 _DTACK
 Text GLabel 950  8550 0    50   BiDi ~ 0
-ARW
+AR_W
 Text GLabel 950  8650 0    50   BiDi ~ 0
 _LDS
@@
 	13850 3400 14250 3400
 Text GLabel 15025 3050 2    51   Output ~ 0
-MEG4
+TWOMB
 Text GLabel 15025 3225 2    51   Output ~ 0
 B2000
 Text GLabel 15025 3400 2    51   Output ~ 0
-RAM_AUTO
+AUTO
 Text GLabel 15025 3575 2    51   Output ~ 0
 OSMODE

Commit message: Add files via upload
Parts:
- removed RN300: 3.3K, Resistor_THT:R_Array_SIP5, symbol Device:R_Network04
- added J305: Jumper_NO_Small, Connector_PinHeader_2.54mm:PinHeader_1x02_P2.54mm_Vertical, symbol Device:Jumper_NO_Small
- added RN300: 3.3K, Resistor_THT:R_Array_SIP6, symbol Device:R_Network05
Connections:
- net +5V: now also RN300.1 (common)
- net AD0: now also U702.14 (B7); no longer U702.13 (B8)
- net AD1: now also U702.13 (B8); no longer U702.14 (B7)
- net AD2: now also U702.17 (B4), U704.15 (B3); no longer U702.15 (B6), U704.13 (B5)
- net AD4: now also U702.15 (B6), U704.13 (B5); no longer U702.17 (B4), U704.15 (B3)
- net AD8: now also U703.12 (B6); no longer U703.11 (B7)
- net AD9: now also U703.11 (B7); no longer U703.12 (B6)
- net B2000: now also RN300.3 (R2)
- net D16: now also U702.10 (A7); no longer U702.11 (A8)
- net D17: now also U702.11 (A8); no longer U702.10 (A7)
- net D18: now also U702.7 (A4); no longer U702.9 (A6)
- net D2: now also U704.5 (A3); no longer U704.7 (A5)
- net D20: now also U702.9 (A6); no longer U702.7 (A4)
- net D4: now also U704.7 (A5); no longer U704.5 (A3)
- net D8: now also U703.8 (A6); no longer U703.9 (A7)
- net D9: now also U703.9 (A7); no longer U703.8 (A6)
- net GND: now also J305.1
- net OSMODE: now also RN300.5 (R4)
- net TWOMB: now also RN300.2 (R1)
- net AUTO renamed Z2AUTO
- net Z2AUTO: now also RN300.4 (R3)
- new net Z3AUTO: J305.2, RN300.6 (R5)
Other:
- note added: "Not all these jumpers will make it to the final version.\nJ301 - 2MEG Shorted/4MEG Open\nJ302 - A2000 Shorted/B2000 Open\nJ303 - Do not configure Z2 RAM Shorted/Autoconfigure Z2 RAM Open\nJ304 - AMIX Shorted/AmigaOS Open\nJ305 - Do not configure Z3 RAM Shorted/Autoconfigure Z3 RAM Open"
- note removed: "Not all these jumpers will make it to the final version.\nJ301 - 2MEG Shorted/4MEG Open\nJ302 - A2000 Shorted/B2000 Open\nJ303 - Do not configure RAM Shorted/Autoconfigure RAM Open\nJ404 - AMIX Shorted/AmigaOS Open"
Changed lines of the file:
@@
 Text Label 8000 9175 2    51   ~ 0
 AD1
-Text Label 8000 9075 2    51   ~ 0
+Text Label 8000 8875 2    51   ~ 0
 AD2
 Text Label 8000 8975 2    51   ~ 0
 AD3
-Text Label 8000 8875 2    51   ~ 0
+Text Label 8000 9075 2    51   ~ 0
 AD4
 Text Label 8000 8775 2    51   ~ 0
@@
 Text Label 8000 8575 2    51   ~ 0
 AD7
+Text Label 8000 7550 2    51   ~ 0
+AD8
 Text Label 8000 7650 2    51   ~ 0
-AD8
-Text Label 8000 7550 2    51   ~ 0
 AD9
 Text Label 8000 7450 2    51   ~ 0
@@
 Entry Wire Line
 	6350 5650 6250 5750
+Text Label 8000 5550 2    51   ~ 0
+AD0
 Text Label 8000 5650 2    51   ~ 0
-AD0
-Text Label 8000 5550 2    51   ~ 0
 AD1
-Text Label 8000 5450 2    51   ~ 0
+Text Label 8000 5050 2    51   ~ 0
 AD2
 Text Label 8000 5350 2    51   ~ 0
 AD3
-Text Label 8000 5050 2    51   ~ 0
+Text Label 8000 5450 2    51   ~ 0
 AD4
 Text Label 8000 4950 2    51   ~ 0
@@
 Text Label 6350 9175 0    51   ~ 0
 D1
-Text Label 6350 9075 0    51   ~ 0
+Text Label 6350 8875 0    51   ~ 0
 D2
 Text Label 6350 8975 0    51   ~ 0
 D3
-Text Label 6350 8875 0    51   ~ 0
+Text Label 6350 9075 0    51   ~ 0
 D4
 Text Label 6350 8775 0    51   ~ 0
@@
 Text Label 6350 8575 0    51   ~ 0
 D7
+Text Label 6350 7550 0    51   ~ 0
+D8
 Text Label 6350 7650 0    51   ~ 0
-D8
-Text Label 6350 7550 0    51   ~ 0
 D9
 Text Label 6350 7450 0    51   ~ 0
@@
 Text Label 6350 6950 0    51   ~ 0
 D15
+Text Label 6350 5550 0    51   ~ 0
+D16
 Text Label 6350 5650 0    51   ~ 0
-D16
-Text Label 6350 5550 0    51   ~ 0
 D17
-Text Label 6350 5450 0    51   ~ 0
+Text Label 6350 5050 0    51   ~ 0
 D18
 Text Label 6350 5350 0    51   ~ 0
 D19
-Text Label 6350 5050 0    51   ~ 0
+Text Label 6350 5450 0    51   ~ 0
 D20
 Text Label 6350 4950 0    51   ~ 0
@@
 Connection ~ 13400 3575
 Wire Wire Line
-	13400 3575 13400 3875
+	13400 3575 13400 3750
 Wire Wire Line
 	13650 3400 13400 3400
@@
 	1    0    0    -1
 $EndComp
-$Comp
-L Device:R_Network04 RN300
-U 1 1 63340B2B
-P 14250 2625
-F 0 "RN300" H 14438 2671 50  0000 L CNN
-F 1 "3.3K" H 14438 2580 50  0000 L CNN
-F 2 "Resistor_THT:R_Array_SIP5" V 14525 2625 50  0001 C CNN
-F 3 "http://www.vishay.com/docs/31509/csc.pdf" H 14250 2625 50  0001 C CNN
-	1    14250 2625
-	1    0    0    -1
-$EndComp
 Wire Wire Line
 	13850 3050 14050 3050
@@
 B2000
 Text GLabel 15025 3400 2    51   Output ~ 0
-AUTO
+Z2AUTO
 Text GLabel 15025 3575 2    51   Output ~ 0
 OSMODE
@@
 	1    0    0    -1
 $EndComp
-Text Notes 13675 4300 0    51   ~ 0
-Not all these jumpers will make it to the final version.\nJ301 - 2MEG Shorted/4MEG Open\nJ302 - A2000 Shorted/B2000 Open\nJ303 - Do not configure RAM Shorted/Autoconfigure RAM Open\nJ404 - AMIX Shorted/AmigaOS Open
+Text Notes 13675 4475 0    51   ~ 0
+Not all these jumpers will make it to the final version.\nJ301 - 2MEG Shorted/4MEG Open\nJ302 - A2000 Shorted/B2000 Open\nJ303 - Do not configure Z2 RAM Shorted/Autoconfigure Z2 RAM Open\nJ304 - AMIX Shorted/AmigaOS Open\nJ305 - Do not configure Z3 RAM Shorted/Autoconfigure Z3 RAM Open
 NoConn ~ 10450 5600
 Text Label 12125 5000 2    51   ~ 0
@@
 Text GLabel 925  5450 0    50   Output ~ 0
 28M
+$Comp
+L Device:Jumper_NO_Small J305
+U 1 1 622A3FB8
+P 13750 3750
+F 0 "J305" H 13750 3843 50  0000 C CNN
+F 1 "Jumper_NO_Small" H 13750 3844 50  0001 C CNN
+F 2 "Connector_PinHeader_2.54mm:PinHeader_1x02_P2.54mm_Vertical" H 13750 3750 50  0001 C CNN
+F 3 "~" H 13750 3750 50  0001 C CNN
+	1    13750 3750
+	1    0    0    -1
+$EndComp
+Wire Wire Line
+	13650 3750 13400 3750
+Connection ~ 13400 3750
+Wire Wire Line
+	13400 3750 13400 3875
+Wire Wire Line
+	13850 3750 14450 3750
+Text GLabel 15025 3750 2    51   Output ~ 0
+Z3AUTO
+$Comp
+L Device:R_Network05 RN300
+U 1 1 623007A9
+P 14250 2625
+F 0 "RN300" H 14538 2671 50  0000 L CNN
+F 1 "3.3K" H 14538 2580 50  0000 L CNN
+F 2 "Resistor_THT:R_Array_SIP6" V 14625 2625 50  0001 C CNN
+F 3 "http://www.vishay.com/docs/31509/csc.pdf" H 14250 2625 50  0001 C CNN
+	1    14250 2625
+	1    0    0    -1
+$EndComp
+Wire Wire Line
+	14450 2825 14450 3750
+Connection ~ 14450 3750
+Wire Wire Line
+	14450 3750 15025 3750
 Wire Bus Line
 	1250 3825 1250 4075
