File: A2630-New-KiCAD/Power.sch (KiCad schematic (older format))
At the start: 1 part, among them U204 74HCT04

Commit message: Add files via upload
Parts:
- added U307: 74HCT04, Package_SO:SOIC-14_3.9x8.7mm_P1.27mm, symbol 74xx:74LS04
- added U606: 74HCT244, Package_SO:SOIC-20W_7.5x12.8mm_P1.27mm, symbol 74xx:74LS244_Split
Connections:
- net GND: now also U606.11, U606.13, U606.15, U606.17, U606.19
- no-connect marks 1 -> 5
Changed lines of the file:
@@
 $Descr A4 11693 8268
 encoding utf-8
-Sheet 4 5
+Sheet 4 6
 Title ""
 Date ""
@@
 L power:GND #PWR0123
 U 1 1 620AFB56
-P 1025 1600
-F 0 "#PWR0123" H 1025 1350 50  0001 C CNN
-F 1 "GND" H 1030 1427 50  0000 C CNN
-F 2 "" H 1025 1600 50  0001 C CNN
-F 3 "" H 1025 1600 50  0001 C CNN
-	1    1025 1600
+P 1025 4025
+F 0 "#PWR0123" H 1025 3775 50  0001 C CNN
+F 1 "GND" H 1030 3852 50  0000 C CNN
+F 2 "" H 1025 4025 50  0001 C CNN
+F 3 "" H 1025 4025 50  0001 C CNN
+	1    1025 4025
 	1    0    0    -1
 $EndComp
 NoConn ~ 1625 1300
 Wire Wire Line
-	1025 1600 1025 1300
+	1025 4025 1025 3575
+$Comp
+L 74xx:74LS244_Split U?
+U 5 1 63502654
+P 1325 1850
+AR Path="/634ECC15/63502654" Ref="U?"  Part="1"
+AR Path="/6209FB19/63502654" Ref="U606"  Part="5"
+F 0 "U606" H 1325 2167 50  0000 C CNN
+F 1 "74HCT244" H 1325 2076 50  0000 C CNN
+F 2 "Package_SO:SOIC-20W_7.5x12.8mm_P1.27mm" H 1325 1850 50  0001 C CNN
+F 3 "http://www.ti.com/lit/ds/symlink/sn74ls241.pdf" H 1325 1850 50  0001 C CNN
+	5    1325 1850
+	1    0    0    -1
+$EndComp
+$Comp
+L 74xx:74LS244_Split U?
+U 6 1 6350265A
+P 1325 2500
+AR Path="/634ECC15/6350265A" Ref="U?"  Part="2"
+AR Path="/6209FB19/6350265A" Ref="U606"  Part="6"
+F 0 "U606" H 1325 2817 50  0000 C CNN
+F 1 "74HCT244" H 1325 2726 50  0000 C CNN
+F 2 "Package_SO:SOIC-20W_7.5x12.8mm_P1.27mm" H 1325 2500 50  0001 C CNN
+F 3 "http://www.ti.com/lit/ds/symlink/sn74ls241.pdf" H 1325 2500 50  0001 C CNN
+	6    1325 2500
+	1    0    0    -1
+$EndComp
+$Comp
+L 74xx:74LS244_Split U?
+U 7 1 63502660
+P 1325 3025
+AR Path="/634ECC15/63502660" Ref="U?"  Part="3"
+AR Path="/6209FB19/63502660" Ref="U606"  Part="7"
+F 0 "U606" H 1325 3342 50  0000 C CNN
+F 1 "74HCT244" H 1325 3251 50  0000 C CNN
+F 2 "Package_SO:SOIC-20W_7.5x12.8mm_P1.27mm" H 1325 3025 50  0001 C CNN
+F 3 "http://www.ti.com/lit/ds/symlink/sn74ls241.pdf" H 1325 3025 50  0001 C CNN
+	7    1325 3025
+	1    0    0    -1
+$EndComp
+$Comp
+L 74xx:74LS244_Split U?
+U 8 1 63502666
+P 1325 3575
+AR Path="/634ECC15/63502666" Ref="U?"  Part="4"
+AR Path="/6209FB19/63502666" Ref="U606"  Part="8"
+F 0 "U606" H 1325 3892 50  0000 C CNN
+F 1 "74HCT244" H 1325 3801 50  0000 C CNN
+F 2 "Package_SO:SOIC-20W_7.5x12.8mm_P1.27mm" H 1325 3575 50  0001 C CNN
+F 3 "http://www.ti.com/lit/ds/symlink/sn74ls241.pdf" H 1325 3575 50  0001 C CNN
+	8    1325 3575
+	1    0    0    -1
+$EndComp
+Connection ~ 1025 1850
+Wire Wire Line
+	1025 1850 1025 1300
+Wire Wire Line
+	1325 2100 1025 2100
+Connection ~ 1025 2100
+Wire Wire Line
+	1025 2100 1025 1850
+Connection ~ 1025 2500
+Wire Wire Line
+	1025 2500 1025 2100
+Connection ~ 1025 3025
+Wire Wire Line
+	1025 3025 1025 2500
+Connection ~ 1025 3575
+Wire Wire Line
+	1025 3575 1025 3025
+NoConn ~ 1625 1850
+NoConn ~ 1625 2500
+NoConn ~ 1625 3025
+NoConn ~ 1625 3575
+$Comp
+L 74xx:74LS04 U?
+U 1 1 63633FBA
+P 2275 1275
+AR Path="/61DF74A0/63633FBA" Ref="U?"  Part="3"
+AR Path="/6209FB19/63633FBA" Ref="U307"  Part="1"
+F 0 "U307" H 2275 958 50  0000 C CNN
+F 1 "74HCT04" H 2275 1049 50  0000 C CNN
+F 2 "Package_SO:SOIC-14_3.9x8.7mm_P1.27mm" H 2275 1275 50  0001 C CNN
+F 3 "http://www.ti.com/lit/gpn/sn74LS04" H 2275 1275 50  0001 C CNN
+	1    2275 1275
+	1    0    0    -1
+$EndComp
+$Comp
+L 74xx:74LS04 U?
+U 2 1 6363485A
+P 2275 1825
+AR Path="/61DF74A0/6363485A" Ref="U?"  Part="3"
+AR Path="/6209FB19/6363485A" Ref="U307"  Part="2"
+F 0 "U307" H 2275 1508 50  0000 C CNN
+F 1 "74HCT04" H 2275 1599 50  0000 C CNN
+F 2 "Package_SO:SOIC-14_3.9x8.7mm_P1.27mm" H 2275 1825 50  0001 C CNN
+F 3 "http://www.ti.com/lit/gpn/sn74LS04" H 2275 1825 50  0001 C CNN
+	2    2275 1825
+	1    0    0    -1
+$EndComp
+$Comp
+L 74xx:74LS04 U?
+U 4 1 636358AA
+P 2275 2425
+AR Path="/61DF74A0/636358AA" Ref="U?"  Part="3"
+AR Path="/6209FB19/636358AA" Ref="U307"  Part="4"
+F 0 "U307" H 2275 2108 50  0000 C CNN
+F 1 "74HCT04" H 2275 2199 50  0000 C CNN
+F 2 "Package_SO:SOIC-14_3.9x8.7mm_P1.27mm" H 2275 2425 50  0001 C CNN
+F 3 "http://www.ti.com/lit/gpn/sn74LS04" H 2275 2425 50  0001 C CNN
+	4    2275 2425
+	1    0    0    -1
+$EndComp
 $EndSCHEMATC

Commit message: Add files via upload
Parts:
- removed unit 2 of U307
- added U300: 74HCT05, Package_SO:SOIC-14_3.9x8.7mm_P1.27mm, symbol 74xx:74LS05
Changed lines of the file:
@@
 $Descr A4 11693 8268
 encoding utf-8
-Sheet 4 6
+Sheet 4 8
 Title ""
 Date ""
@@
 $Comp
 L 74xx:74LS04 U?
-U 2 1 6363485A
-P 2275 1825
-AR Path="/61DF74A0/6363485A" Ref="U?"  Part="3"
-AR Path="/6209FB19/6363485A" Ref="U307"  Part="2"
-F 0 "U307" H 2275 1508 50  0000 C CNN
-F 1 "74HCT04" H 2275 1599 50  0000 C CNN
-F 2 "Package_SO:SOIC-14_3.9x8.7mm_P1.27mm" H 2275 1825 50  0001 C CNN
-F 3 "http://www.ti.com/lit/gpn/sn74LS04" H 2275 1825 50  0001 C CNN
-	2    2275 1825
-	1    0    0    -1
-$EndComp
-$Comp
-L 74xx:74LS04 U?
 U 4 1 636358AA
 P 2275 2425
@@
 	1    0    0    -1
 $EndComp
+$Comp
+L 74xx:74LS05 U?
+U 2 1 61F394C8
+P 3250 1275
+AR Path="/61DF74A0/61F394C8" Ref="U?"  Part="4"
+AR Path="/634ECC15/61F394C8" Ref="U?"  Part="1"
+AR Path="/6209FB19/61F394C8" Ref="U300"  Part="2"
+F 0 "U300" H 3250 1592 50  0000 C CNN
+F 1 "74HCT05" H 3250 1501 50  0000 C CNN
+F 2 "Package_SO:SOIC-14_3.9x8.7mm_P1.27mm" H 3250 1275 50  0001 C CNN
+F 3 "http://www.ti.com/lit/gpn/sn74LS05" H 3250 1275 50  0001 C CNN
+	2    3250 1275
+	1    0    0    -1
+$EndComp
+$Comp
+L 74xx:74LS05 U?
+U 5 1 61F3D66D
+P 3250 2300
+AR Path="/61DF74A0/61F3D66D" Ref="U?"  Part="4"
+AR Path="/634ECC15/61F3D66D" Ref="U?"  Part="1"
+AR Path="/6209FB19/61F3D66D" Ref="U300"  Part="5"
+F 0 "U300" H 3250 2617 50  0000 C CNN
+F 1 "74HCT05" H 3250 2526 50  0000 C CNN
+F 2 "Package_SO:SOIC-14_3.9x8.7mm_P1.27mm" H 3250 2300 50  0001 C CNN
+F 3 "http://www.ti.com/lit/gpn/sn74LS05" H 3250 2300 50  0001 C CNN
+	5    3250 2300
+	1    0    0    -1
+$EndComp
+$Comp
+L 74xx:74LS05 U?
+U 6 1 61F3E9BB
+P 3250 2850
+AR Path="/61DF74A0/61F3E9BB" Ref="U?"  Part="4"
+AR Path="/634ECC15/61F3E9BB" Ref="U?"  Part="1"
+AR Path="/6209FB19/61F3E9BB" Ref="U300"  Part="6"
+F 0 "U300" H 3250 3167 50  0000 C CNN
+F 1 "74HCT05" H 3250 3076 50  0000 C CNN
+F 2 "Package_SO:SOIC-14_3.9x8.7mm_P1.27mm" H 3250 2850 50  0001 C CNN
+F 3 "http://www.ti.com/lit/gpn/sn74LS05" H 3250 2850 50  0001 C CNN
+	6    3250 2850
+	1    0    0    -1
+$EndComp

Commit message: Add files via upload
Parts:
- removed unit 2 of U300
Changed lines of the file:
@@
-$Comp
-L 74xx:74LS05 U?
-U 2 1 61F394C8
-P 3250 1275
-AR Path="/61DF74A0/61F394C8" Ref="U?"  Part="4"
-AR Path="/634ECC15/61F394C8" Ref="U?"  Part="1"
-AR Path="/6209FB19/61F394C8" Ref="U300"  Part="2"
-F 0 "U300" H 3250 1592 50  0000 C CNN
-F 1 "74HCT05" H 3250 1501 50  0000 C CNN
-F 2 "Package_SO:SOIC-14_3.9x8.7mm_P1.27mm" H 3250 1275 50  0001 C CNN
-F 3 "http://www.ti.com/lit/gpn/sn74LS05" H 3250 1275 50  0001 C CNN
-	2    3250 1275
-	1    0    0    -1
-$EndComp
 $Comp
 L 74xx:74LS05 U?

Commit message: Add files via upload
Parts:
- added C200, C201, C202, C210, C215, C217, C219: 0.01uF, Capacitor_SMD:C_0805_2012Metric, symbol Device:C
- added C204, C206, C208, C214, C216, C218, C220: 0.1uF, Capacitor_SMD:C_0805_2012Metric, symbol Device:C
- added C205: 330pF, Capacitor_SMD:C_0805_2012Metric, symbol Device:C
- added C209: 0.22uF, Capacitor_SMD:C_0805_2012Metric, symbol Device:C
- added unit 7 of U204
Connections:
- net GND: now also C200.2, C201.2, C202.2, C204.2, C205.2, C206.2, C208.2, C209.2, C210.2, C214.2, C215.2, C216.2, C217.2, C218.2, C219.2, C220.2, U204.7 (GND)
- new net +5V: C200.1, C201.1, C202.1, C204.1, C205.1, C206.1, C208.1, C209.1, C210.1, C214.1, C215.1, C216.1, C217.1, C218.1, C219.1, C220.1, U204.14 (VCC)
