File: A2630-New-KiCAD/ExpansionMemory.sch (KiCad schematic (older format))
At the start: 12 parts, among them U102 27C256, U103 27C256, U406 SDRAM_512Mb(32Mx16), U407 SDRAM_512Mb(32Mx16), U408 SDRAM_512Mb(32Mx16), U409 SDRAM_512Mb(32Mx16)

Commit message: Add files via upload
Parts:
- U406, U407, U408, U409: footprint TSOPII-54 -> Package_SO:TSOP-II-54_22.2x10.16mm_P0.8mm
Connections:
- net CPUCLK_A: now also U406.38 (CLK), U407.38 (CLK), U408.38 (CLK), U409.38 (CLK)
- net _EM0LLBE: now reaches U406.15 (LDQM)
- net EM0R_W: now reaches U406.16 (WE)
- net EM0R_W: now also U407.16 (WE)
- net _CAS0: now reaches U406.17 (CAS)
- net _CAS0: now also U407.17 (CAS)
- net _RAS0: now reaches U406.18 (RAS)
- net _RAS0: now also U407.18 (RAS)
- net _EM0CS: now reaches U406.19 (CS)
- net _EM0CS: now also U407.19 (CS)
- net EM0B0: now reaches U406.20 (BA0)
- net EM0B0: now also U407.20 (BA0)
- net EM0B1: now reaches U406.21 (BA1)
- net EM0B1: now also U407.21 (BA1)
- net EM0CLKE: now reaches U406.37 (CKE)
- net EM0CLKE: now also U407.37 (CKE)
- net _EM0LMBE: now reaches U406.39 (UDQM)
- net _EM0UUBE: now reaches U407.15 (LDQM)
- net _EM0UMBE: now reaches U407.39 (UDQM)
- net _EM1LLBE: now reaches U408.15 (LDQM)
- net EM1R_W: now reaches U408.16 (WE)
- net EM1R_W: now also U409.16 (WE)
- net _CAS1: now reaches U408.17 (CAS)
- net _CAS1: now also U409.17 (CAS)
- net _RAS1: now reaches U408.18 (RAS)
- net _RAS1: now also U409.18 (RAS)
- net _EM1CS: now reaches U408.19 (CS)
- net _EM1CS: now also U409.19 (CS)
- net EM1B0: now reaches U408.20 (BA0)
- net EM1B0: now also U409.20 (BA0)
- net EM1B1: now reaches U408.21 (BA1)
- net EM1B1: now also U409.21 (BA1)
- net EM1CLKE: now reaches U408.37 (CKE)
- net EM1CLKE: now also U409.37 (CKE)
- net _EM1LMBE: now reaches U408.39 (UDQM)
- net _EM1UMBE: now reaches U409.15 (LDQM)
- net _EM1UUBE: now reaches U409.39 (UDQM)
Other:
- note added: "BANK0"
- note added: "BANK0 = First 64MB\nBANK1 = Second 64MB"
- note added: "BANK1"
- note added: "CKE..The next rising edge of the CLK signal is valid \nwhen CKE is high and invalid when it is low. When \nCKE is LOW, the device will be in power-down mode, \nclock suspend mode or self-refresh mode\nJN: Might be able to refresh one bank when the other is\nbeing accessed?"
- note added: "JN Notes: put row address on the EMA bus \nand signal RAS. This is 68030 addresses A14:2. \nPut column address on the EMA bus and signal \nCAS. These are 68030 addresses A24:15."
- moved on the sheet: U102, U103

Commit message: Add files via upload
Changed lines of the file:
@@
 CPUCLK_A
 Text GLabel 1350 900  0    50   BiDi ~ 0
-D(31..0)
+D[31..0]
 Text GLabel 1300 4650 0    50   Input ~ 0
 EM0R_W
@@
 	12225 4350 12325 4250
 Text GLabel 11425 4350 0    50   BiDi ~ 0
-D(31:0)
+D[31..0]
 Text GLabel 11500 1150 0    50   Input ~ 0
-A(31:0)
+A[31..0]
 Wire Wire Line
 	14425 3675 14300 3675
@@
 	5400 1000 5300 900
 Text GLabel 1350 1100 0    50   BiDi ~ 0
-EM(12..0)
+EMA(12..0)
 Entry Bus Bus
 	3100 1200 3000 1100
@@
 Text Notes 8000 1800 0    118  ~ 0
 BANK1
+Text Notes 10850 5500 0    118  ~ 0
+JN Notes: put row address on the EMA bus \nand signal RAS. This is 68030 addresses A14:2. \nPut column address on the EMA bus and signal \nCAS. These are 68030 addresses A24:15.
+Text GLabel 1300 4300 0    50   Input ~ 0
+EM0CLKE
+Text GLabel 15600 7300 2    50   Input ~ 0
+EM1CLKE
+Text Notes 750  2150 0    118  ~ 0
+BANK0 = First 64MB\nBANK1 = Second 64MB
 Wire Bus Line
 	1350 1100 7100 1100
@@
 Wire Bus Line
 	5400 1000 5400 7600
-Text Notes 10850 5500 0    118  ~ 0
-JN Notes: put row address on the EMA bus \nand signal RAS. This is 68030 addresses A14:2. \nPut column address on the EMA bus and signal \nCAS. These are 68030 addresses A24:15.
-Text GLabel 1300 4300 0    50   Input ~ 0
-EM0CLKE
-Text GLabel 15600 7300 2    50   Input ~ 0
-EM1CLKE
-Text Notes 750  2150 0    118  ~ 0
-BANK0 = First 64MB\nBANK1 = Second 64MB
 $EndSCHEMATC

Commit message: Add files via upload
Other:
- note added: "HIGH_BYTE"
- note added: "LOW_BYTE"
Changed lines of the file:
@@
 Entry Bus Bus
 	5400 1000 5300 900
-Text GLabel 1350 1100 0    50   BiDi ~ 0
+Text GLabel 1350 1100 0    50   Input ~ 0
 EMA(12..0)
 Entry Bus Bus
@@
 Text GLabel 15600 7300 2    50   Input ~ 0
 EM1CLKE
-Text Notes 750  2150 0    118  ~ 0
+Text Notes 7725 10225 0    118  ~ 0
 BANK0 = First 64MB\nBANK1 = Second 64MB
 Wire Bus Line
@@
 Wire Bus Line
 	5400 1000 5400 7600
+Text Notes 950  3200 0    118  ~ 0
+LOW_BYTE
+Text Notes 950  7125 0    118  ~ 0
+HIGH_BYTE
 $EndSCHEMATC

Commit message: Add files via upload
Parts:
- added C410, C411, C412, C413: 0.33uF, Capacitor_SMD:C_0805_2012Metric, symbol Device:C
Connections:
- net +3V3: now also C410.1, C411.1, C412.1, C413.1
- net GND: now also C410.2, C411.2, C412.2, C413.2
Other:
- moved on the sheet: C102, C103, C406, C407, C408, C409
Changed lines of the file:
@@
 L Device:C C406
 U 1 1 62F57967
-P 14450 8125
-F 0 "C406" H 14565 8171 50  0000 L CNN
-F 1 "0.33uF" H 14565 8080 50  0000 L CNN
-F 2 "Capacitor_SMD:C_0805_2012Metric" H 14488 7975 50  0001 C CNN
-F 3 "~" H 14450 8125 50  0001 C CNN
-	1    14450 8125
+P 13750 8125
+F 0 "C406" H 13650 8350 50  0000 L CNN
+F 1 "0.33uF" H 13625 7875 50  0000 L CNN
+F 2 "Capacitor_SMD:C_0805_2012Metric" H 13788 7975 50  0001 C CNN
+F 3 "~" H 13750 8125 50  0001 C CNN
+	1    13750 8125
 	1    0    0    -1
 $EndComp
@@
 L Device:C C407
 U 1 1 62F59277
-P 14875 8125
-F 0 "C407" H 14990 8171 50  0000 L CNN
-F 1 "0.33uF" H 14990 8080 50  0000 L CNN
-F 2 "Capacitor_SMD:C_0805_2012Metric" H 14913 7975 50  0001 C CNN
-F 3 "~" H 14875 8125 50  0001 C CNN
-	1    14875 8125
+P 14075 8125
+F 0 "C407" H 13975 8350 50  0000 L CNN
+F 1 "0.33uF" H 13950 7875 50  0000 L CNN
+F 2 "Capacitor_SMD:C_0805_2012Metric" H 14113 7975 50  0001 C CNN
+F 3 "~" H 14075 8125 50  0001 C CNN
+	1    14075 8125
 	1    0    0    -1
 $EndComp
@@
 L Device:C C408
 U 1 1 62F59AAD
-P 15300 8125
-F 0 "C408" H 15415 8171 50  0000 L CNN
-F 1 "0.33uF" H 15415 8080 50  0000 L CNN
-F 2 "Capacitor_SMD:C_0805_2012Metric" H 15338 7975 50  0001 C CNN
-F 3 "~" H 15300 8125 50  0001 C CNN
-	1    15300 8125
+P 14375 8125
+F 0 "C408" H 14275 8350 50  0000 L CNN
+F 1 "0.33uF" H 14250 7875 50  0000 L CNN
+F 2 "Capacitor_SMD:C_0805_2012Metric" H 14413 7975 50  0001 C CNN
+F 3 "~" H 14375 8125 50  0001 C CNN
+	1    14375 8125
 	1    0    0    -1
 $EndComp
@@
 L Device:C C409
 U 1 1 62F5A38E
-P 15725 8125
-F 0 "C409" H 15840 8171 50  0000 L CNN
-F 1 "0.33uF" H 15840 8080 50  0000 L CNN
-F 2 "Capacitor_SMD:C_0805_2012Metric" H 15763 7975 50  0001 C CNN
-F 3 "~" H 15725 8125 50  0001 C CNN
-	1    15725 8125
-	1    0    0    -1
-$EndComp
-Wire Wire Line
-	14450 8500 14450 8275
-Wire Wire Line
-	14450 7975 14450 7750
-Wire Wire Line
-	14450 7750 14875 7750
-Wire Wire Line
-	15725 7975 15725 7750
-Wire Wire Line
-	15725 8275 15725 8500
-Wire Wire Line
-	15725 8500 15300 8500
-Wire Wire Line
-	15300 7975 15300 7750
-Connection ~ 15300 7750
-Wire Wire Line
-	15300 7750 15725 7750
-Wire Wire Line
-	14875 7975 14875 7750
-Connection ~ 14875 7750
-Wire Wire Line
-	14875 7750 15300 7750
-Wire Wire Line
-	14875 8275 14875 8500
-Connection ~ 14875 8500
-Wire Wire Line
-	14875 8500 14450 8500
-Wire Wire Line
-	15300 8275 15300 8500
-Connection ~ 15300 8500
-Wire Wire Line
-	15300 8500 14875 8500
+P 14675 8125
+F 0 "C409" H 14575 8350 50  0000 L CNN
+F 1 "0.33uF" H 14550 7875 50  0000 L CNN
+F 2 "Capacitor_SMD:C_0805_2012Metric" H 14713 7975 50  0001 C CNN
+F 3 "~" H 14675 8125 50  0001 C CNN
+	1    14675 8125
+	1    0    0    -1
+$EndComp
 $Comp
 L power:GND #PWR0111
 U 1 1 63373380
-P 14450 8500
-F 0 "#PWR0111" H 14450 8250 50  0001 C CNN
-F 1 "GND" H 14455 8327 50  0000 C CNN
-F 2 "" H 14450 8500 50  0001 C CNN
-F 3 "" H 14450 8500 50  0001 C CNN
-	1    14450 8500
-	1    0    0    -1
-$EndComp
-Connection ~ 14450 8500
+P 13375 8450
+F 0 "#PWR0111" H 13375 8200 50  0001 C CNN
+F 1 "GND" H 13380 8277 50  0000 C CNN
+F 2 "" H 13375 8450 50  0001 C CNN
+F 3 "" H 13375 8450 50  0001 C CNN
+	1    13375 8450
+	1    0    0    -1
+$EndComp
 $Comp
 L power:+3.3V #PWR0116
 U 1 1 6337477A
-P 14450 7750
-F 0 "#PWR0116" H 14450 7600 50  0001 C CNN
-F 1 "+3.3V" H 14465 7923 50  0000 C CNN
-F 2 "" H 14450 7750 50  0001 C CNN
-F 3 "" H 14450 7750 50  0001 C CNN
-	1    14450 7750
-	1    0    0    -1
-$EndComp
-Connection ~ 14450 7750
+P 13375 7850
+F 0 "#PWR0116" H 13375 7700 50  0001 C CNN
+F 1 "+3.3V" H 13390 8023 50  0000 C CNN
+F 2 "" H 13375 7850 50  0001 C CNN
+F 3 "" H 13375 7850 50  0001 C CNN
+	1    13375 7850
+	1    0    0    -1
+$EndComp
 Text GLabel 1300 4450 0    50   Input ~ 0
 _RAS0
@@
 L Device:C C102
 U 1 1 62B32A4C
-P 12955 8135
-F 0 "C102" H 13070 8181 50  0000 L CNN
-F 1 "0.22uF" H 13070 8090 50  0000 L CNN
-F 2 "Capacitor_SMD:C_0805_2012Metric" H 12993 7985 50  0001 C CNN
-F 3 "~" H 12955 8135 50  0001 C CNN
-	1    12955 8135
+P 11630 8160
+F 0 "C102" H 11745 8206 50  0000 L CNN
+F 1 "0.22uF" H 11745 8115 50  0000 L CNN
+F 2 "Capacitor_SMD:C_0805_2012Metric" H 11668 8010 50  0001 C CNN
+F 3 "~" H 11630 8160 50  0001 C CNN
+	1    11630 8160
 	1    0    0    -1
 $EndComp
@@
 L Device:C C103
 U 1 1 62B330BE
-P 13455 8135
-F 0 "C103" H 13570 8181 50  0000 L CNN
-F 1 "0.22uF" H 13570 8090 50  0000 L CNN
-F 2 "Capacitor_SMD:C_0805_2012Metric" H 13493 7985 50  0001 C CNN
-F 3 "~" H 13455 8135 50  0001 C CNN
-	1    13455 8135
-	1    0    0    -1
-$EndComp
-Wire Wire Line
-	12955 8285 12955 8435
-Wire Wire Line
-	12955 8435 13455 8435
-Wire Wire Line
-	13455 8435 13455 8285
-Wire Wire Line
-	12955 7985 12955 7785
-Wire Wire Line
-	12955 7785 13455 7785
-Wire Wire Line
-	13455 7785 13455 7985
+P 12130 8160
+F 0 "C103" H 12245 8206 50  0000 L CNN
+F 1 "0.22uF" H 12245 8115 50  0000 L CNN
+F 2 "Capacitor_SMD:C_0805_2012Metric" H 12168 8010 50  0001 C CNN
+F 3 "~" H 12130 8160 50  0001 C CNN
+	1    12130 8160
+	1    0    0    -1
+$EndComp
+Wire Wire Line
+	11630 8310 11630 8460
+Wire Wire Line
+	11630 8460 12130 8460
+Wire Wire Line
+	12130 8460 12130 8310
+Wire Wire Line
+	11630 8010 11630 7810
+Wire Wire Line
+	11630 7810 12130 7810
+Wire Wire Line
+	12130 7810 12130 8010
 $Comp
 L power:GND #PWR0133
 U 1 1 62B75BE7
-P 12955 8435
-F 0 "#PWR0133" H 12955 8185 50  0001 C CNN
-F 1 "GND" H 12960 8262 50  0000 C CNN
-F 2 "" H 12955 8435 50  0001 C CNN
-F 3 "" H 12955 8435 50  0001 C CNN
-	1    12955 8435
-	1    0    0    -1
-$EndComp
-Connection ~ 12955 8435
+P 11630 8460
+F 0 "#PWR0133" H 11630 8210 50  0001 C CNN
+F 1 "GND" H 11635 8287 50  0000 C CNN
+F 2 "" H 11630 8460 50  0001 C CNN
+F 3 "" H 11630 8460 50  0001 C CNN
+	1    11630 8460
+	1    0    0    -1
+$EndComp
+Connection ~ 11630 8460
 $Comp
 L power:+5V #PWR0134
 U 1 1 62B765FC
-P 12955 7785
-F 0 "#PWR0134" H 12955 7635 50  0001 C CNN
-F 1 "+5V" H 12970 7958 50  0000 C CNN
-F 2 "" H 12955 7785 50  0001 C CNN
-F 3 "" H 12955 7785 50  0001 C CNN
-	1    12955 7785
-	1    0    0    -1
-$EndComp
-Connection ~ 12955 7785
+P 11630 7810
+F 0 "#PWR0134" H 11630 7660 50  0001 C CNN
+F 1 "+5V" H 11645 7983 50  0000 C CNN
+F 2 "" H 11630 7810 50  0001 C CNN
+F 3 "" H 11630 7810 50  0001 C CNN
+	1    11630 7810
+	1    0    0    -1
+$EndComp
+Connection ~ 11630 7810
 $Comp
 L power:+5V #PWR0135
@@
 Text Notes 7725 10225 0    118  ~ 0
 BANK0 = First 64MB\nBANK1 = Second 64MB
+Text Notes 950  3200 0    118  ~ 0
+LOW_BYTE
+Text Notes 950  7125 0    118  ~ 0
+HIGH_BYTE
+Wire Wire Line
+	13750 8275 14075 8275
+Connection ~ 14075 8275
+Wire Wire Line
+	14075 8275 14375 8275
+Connection ~ 14375 8275
+Wire Wire Line
+	14375 8275 14675 8275
+Wire Wire Line
+	13750 7975 14075 7975
+Connection ~ 14075 7975
+Wire Wire Line
+	14075 7975 14375 7975
+Connection ~ 14375 7975
+Wire Wire Line
+	14375 7975 14675 7975
+$Comp
+L Device:C C410
+U 1 1 6329FA61
+P 14975 8125
+F 0 "C410" H 14875 8350 50  0000 L CNN
+F 1 "0.33uF" H 14850 7875 50  0000 L CNN
+F 2 "Capacitor_SMD:C_0805_2012Metric" H 15013 7975 50  0001 C CNN
+F 3 "~" H 14975 8125 50  0001 C CNN
+	1    14975 8125
+	1    0    0    -1
+$EndComp
+$Comp
+L Device:C C411
+U 1 1 6329FEA9
+P 15275 8125
+F 0 "C411" H 15175 8350 50  0000 L CNN
+F 1 "0.33uF" H 15150 7875 50  0000 L CNN
+F 2 "Capacitor_SMD:C_0805_2012Metric" H 15313 7975 50  0001 C CNN
+F 3 "~" H 15275 8125 50  0001 C CNN
+	1    15275 8125
+	1    0    0    -1
+$EndComp
+$Comp
+L Device:C C412
+U 1 1 632A03C7
+P 15600 8125
+F 0 "C412" H 15500 8350 50  0000 L CNN
+F 1 "0.33uF" H 15475 7875 50  0000 L CNN
+F 2 "Capacitor_SMD:C_0805_2012Metric" H 15638 7975 50  0001 C CNN
+F 3 "~" H 15600 8125 50  0001 C CNN
+	1    15600 8125
+	1    0    0    -1
+$EndComp
+$Comp
+L Device:C C413
+U 1 1 632A07B3
+P 15900 8125
+F 0 "C413" H 15800 8350 50  0000 L CNN
+F 1 "0.33uF" H 15775 7875 50  0000 L CNN
+F 2 "Capacitor_SMD:C_0805_2012Metric" H 15938 7975 50  0001 C CNN
+F 3 "~" H 15900 8125 50  0001 C CNN
+	1    15900 8125
+	1    0    0    -1
+$EndComp
+Wire Wire Line
+	15900 7975 15600 7975
+Connection ~ 14675 7975
+Connection ~ 14975 7975
+Wire Wire Line
+	14975 7975 14675 7975
+Connection ~ 15275 7975
+Wire Wire Line
+	15275 7975 14975 7975
+Connection ~ 15600 7975
+Wire Wire Line
+	15600 7975 15275 7975
+Wire Wire Line
+	14675 8275 14975 8275
+Connection ~ 14675 8275
+Connection ~ 14975 8275
+Wire Wire Line
+	14975 8275 15275 8275
+Connection ~ 15275 8275
+Wire Wire Line
+	15275 8275 15600 8275
+Connection ~ 15600 8275
+Wire Wire Line
+	15600 8275 15900 8275
+Wire Wire Line
+	13750 8275 13375 8275
+Wire Wire Line
+	13375 8275 13375 8450
+Connection ~ 13750 8275
+Wire Wire Line
+	13750 7975 13375 7975
+Wire Wire Line
+	13375 7975 13375 7850
 Wire Bus Line
 	1350 1100 7100 1100
@@
 Wire Bus Line
 	5400 1000 5400 7600
-Text Notes 950  3200 0    118  ~ 0
-LOW_BYTE
-Text Notes 950  7125 0    118  ~ 0
-HIGH_BYTE
+Connection ~ 13750 7975
 $EndSCHEMATC
