File: A2630-New-KiCAD/Logic.sch (KiCad schematic (older format))
At the start: 6 parts, among them U302 74HCT174, U303 74HCT174, U307 74HCT04, U503 74HCT74, U606 74HCT244, U999 XC9572XL-TQ100

Commit message: Add files via upload
Parts:
- removed U999: XC9572XL-TQ100, Package_QFP:TQFP-100_14x14mm_P0.5mm, symbol CPLD_Xilinx:XC9572XL-TQ100
- added R500, R501, R502: 1K, Resistor_SMD:R_0805_2012Metric, symbol Device:R
- added U300 (x2): 74HCT05, Package_SO:SOIC-14_3.9x8.7mm_P1.27mm, symbol 74xx:74LS05
- added unit 2 of U307
- added U502: 74HCT74, Package_SO:SOIC-14_3.9x8.7mm_P1.27mm, symbol 74xx:74LS74
Connections:
- net labels added: 7M, BG, BGDIS, _ABG, _BOSS, _CPURESET, _DTACK, _VPA
- net labels removed: +3.3V, A7M, B2000, CDAC, S_7MDIS, _C1, _C3
- wire segments 106 -> 96
- no-connect marks 4 -> 6
Other:
- note removed: "TO U505-2"
- note removed: "TO U606"
- note removed: "U503"
- note removed: "U708"

Commit message: Add files via upload
Changed lines of the file:
@@
 	4125 4950 4125 4725
 $Comp
-L power:+5V #PWR?
+L power:+5V #PWR0143
 U 1 1 6357ECC4
 P 4125 4725
-F 0 "#PWR?" H 4125 4575 50  0001 C CNN
+F 0 "#PWR0143" H 4125 4575 50  0001 C CNN
 F 1 "+5V" H 4140 4898 50  0000 C CNN
 F 2 "" H 4125 4725 50  0001 C CNN
@@
 $EndComp
 $Comp
-L power:+5V #PWR?
+L power:+5V #PWR0144
 U 1 1 6357ED6E
 P 2800 4725
-F 0 "#PWR?" H 2800 4575 50  0001 C CNN
+F 0 "#PWR0144" H 2800 4575 50  0001 C CNN
 F 1 "+5V" H 2815 4898 50  0000 C CNN
 F 2 "" H 2800 4725 50  0001 C CNN
@@
 	1225 6850 1225 6725
 $Comp
-L power:+5V #PWR?
+L power:+5V #PWR0145
 U 1 1 635DF0C9
 P 1225 6725
-F 0 "#PWR?" H 1225 6575 50  0001 C CNN
+F 0 "#PWR0145" H 1225 6575 50  0001 C CNN
 F 1 "+5V" H 1240 6898 50  0000 C CNN
 F 2 "" H 1225 6725 50  0001 C CNN
@@
 TO u304
 $Comp
-L power:+5V #PWR?
+L power:+5V #PWR0146
 U 1 1 63609F5E
 P 2275 6300
-F 0 "#PWR?" H 2275 6150 50  0001 C CNN
+F 0 "#PWR0146" H 2275 6150 50  0001 C CNN
 F 1 "+5V" H 2290 6473 50  0000 C CNN
 F 2 "" H 2275 6300 50  0001 C CNN
@@
 $EndComp
 $Comp
-L power:+5V #PWR?
+L power:+5V #PWR0147
 U 1 1 6360A387
 P 4075 6300
-F 0 "#PWR?" H 4075 6150 50  0001 C CNN
+F 0 "#PWR0147" H 4075 6150 50  0001 C CNN
 F 1 "+5V" H 4090 6473 50  0000 C CNN
 F 2 "" H 4075 6300 50  0001 C CNN
@@
 $EndComp
 $Comp
-L power:GND #PWR?
+L power:GND #PWR0148
 U 1 1 6360AB27
 P 4075 7800
-F 0 "#PWR?" H 4075 7550 50  0001 C CNN
+F 0 "#PWR0148" H 4075 7550 50  0001 C CNN
 F 1 "GND" H 4080 7627 50  0000 C CNN
 F 2 "" H 4075 7800 50  0001 C CNN
@@
 $EndComp
 $Comp
-L power:GND #PWR?
+L power:GND #PWR0149
 U 1 1 6360ABD4
 P 2275 7800
-F 0 "#PWR?" H 2275 7550 50  0001 C CNN
+F 0 "#PWR0149" H 2275 7550 50  0001 C CNN
 F 1 "GND" H 2280 7627 50  0000 C CNN
 F 2 "" H 2275 7800 50  0001 C CNN
@@
 	13375 1950 13375 1700
 $Comp
-L power:+5V #PWR?
+L power:+5V #PWR0150
 U 1 1 61F175E8
 P 13375 1700
-F 0 "#PWR?" H 13375 1550 50  0001 C CNN
+F 0 "#PWR0150" H 13375 1550 50  0001 C CNN
 F 1 "+5V" H 13390 1873 50  0000 C CNN
 F 2 "" H 13375 1700 50  0001 C CNN
@@
 $Comp
 L 74xx:74LS05 U?
-U 1 1 61F6E714
+U 2 1 61F6E714
 P 12525 3150
 AR Path="/61DF74A0/61F6E714" Ref="U?"  Part="4"
-AR Path="/634ECC15/61F6E714" Ref="U300"  Part="1"
+AR Path="/634ECC15/61F6E714" Ref="U300"  Part="2"
 AR Path="/6209FB19/61F6E714" Ref="U?"  Part="3"
 F 0 "U300" H 12525 3467 50  0000 C CNN
@@
 F 2 "Package_SO:SOIC-14_3.9x8.7mm_P1.27mm" H 12525 3150 50  0001 C CNN
 F 3 "http://www.ti.com/lit/gpn/sn74LS05" H 12525 3150 50  0001 C CNN
-	1    12525 3150
+	2    12525 3150
 	1    0    0    -1
 $EndComp
@@
 	13475 3150 14375 3150
 $Comp
-L power:+5V #PWR?
+L power:+5V #PWR0151
 U 1 1 61F847B3
 P 13475 2850
-F 0 "#PWR?" H 13475 2700 50  0001 C CNN
+F 0 "#PWR0151" H 13475 2700 50  0001 C CNN
 F 1 "+5V" H 13490 3023 50  0000 C CNN
 F 2 "" H 13475 2850 50  0001 C CNN
@@
 $EndComp
 $Comp
-L power:+5V #PWR?
+L power:+5V #PWR0152
 U 1 1 61F941E9
 P 15375 2525
-F 0 "#PWR?" H 15375 2375 50  0001 C CNN
+F 0 "#PWR0152" H 15375 2375 50  0001 C CNN
 F 1 "+5V" H 15390 2698 50  0000 C CNN
 F 2 "" H 15375 2525 50  0001 C CNN
@@
 $EndComp
 $Comp
-L power:+5V #PWR?
+L power:+5V #PWR0153
 U 1 1 61FA2CD6
 P 15375 3350
-F 0 "#PWR?" H 15375 3200 50  0001 C CNN
+F 0 "#PWR0153" H 15375 3200 50  0001 C CNN
 F 1 "+5V" H 15390 3523 50  0000 C CNN
 F 2 "" H 15375 3350 50  0001 C CNN

Commit message: Add files via upload
Connections:
- net labels added: D[31..0], _S7MDIS_DFF
- net labels removed: D(31:0)
Other:
- note added: "STATE MACHINE"
- note added: "THESE ARE IN THE CPLD!"
- note removed: "PAL HERE"
Changed lines of the file:
@@
 Wire Wire Line
 	3200 4400 3200 5475
-Text Notes 2475 5550 0    236  ~ 0
-PAL HERE
 $Comp
 L 74xx:74LS174 U302
@@
 	1625 7100 1525 7000
 Text GLabel 1175 5875 0    51   Input ~ 0
-D(31:0)
+D[31..0]
 Entry Bus Bus
 	1425 5875 1525 5975
@@
 Wire Bus Line
 	3325 5875 3325 6900
+Text Label 3200 5475 1    50   ~ 0
+_S7MDIS_DFF
+Text Notes 5025 4050 2    118  ~ 0
+STATE MACHINE
+Text Notes 5650 6075 2    118  ~ 0
+THESE ARE IN THE CPLD!
 $EndSCHEMATC

Commit message: Add files via upload
Parts:
- removed U302: 74HCT174, Package_SO:SOIC-16_3.9x9.9mm_P1.27mm, symbol 74xx:74LS174
- removed unit 5 of U307
- removed unit 6 of U307
Connections:
- net ROMCLK: now reaches U303.9 (Cp)
- no-connect marks 6 -> 4
Other:
- note removed: "FROM U301"
- note removed: "THESE ARE IN THE CPLD!"
- note removed: "TO u304"
Changed lines of the file:
@@
 $Descr B 17000 11000
 encoding utf-8
-Sheet 7 9
+Sheet 7 8
 Title ""
 Date ""
@@
 	3200 4400 3200 5475
 $Comp
-L 74xx:74LS174 U302
-U 1 1 635AD4A3
-P 4075 7000
-F 0 "U302" H 4200 7625 50  0000 C CNN
-F 1 "74HCT174" H 4300 7550 50  0000 C CNN
-F 2 "Package_SO:SOIC-16_3.9x9.9mm_P1.27mm" H 4075 7000 50  0001 C CNN
-F 3 "http://www.ti.com/lit/gpn/sn74LS174" H 4075 7000 50  0001 C CNN
-	1    4075 7000
-	1    0    0    -1
-$EndComp
-Wire Wire Line
-	3575 6600 3425 6600
-Wire Wire Line
-	3575 6700 3425 6700
-Wire Wire Line
-	3575 6800 3425 6800
-Wire Wire Line
-	3575 6900 3425 6900
-Wire Wire Line
-	3575 7000 3425 7000
-Wire Wire Line
-	4575 6600 4775 6600
-Wire Wire Line
-	4575 6700 4775 6700
-Wire Wire Line
-	4575 6800 4775 6800
-Wire Wire Line
-	4575 6900 4775 6900
-Wire Wire Line
-	4575 7000 4775 7000
-Wire Wire Line
-	4575 7100 4775 7100
-Entry Wire Line
-	3425 6600 3325 6500
-Entry Wire Line
-	3425 6700 3325 6600
-Entry Wire Line
-	3425 6800 3325 6700
-Entry Wire Line
-	3425 6900 3325 6800
-Entry Wire Line
-	3425 7000 3325 6900
-$Comp
 L 74xx:74LS174 U303
 U 1 1 635CAE10
@@
 	1775 7100 1625 7100
 Wire Wire Line
-	2775 6600 2800 6600
-Wire Wire Line
-	2775 6700 2800 6700
-Wire Wire Line
-	2775 6900 2800 6900
-Wire Wire Line
-	2775 7000 2800 7000
-Wire Wire Line
-	2775 7100 2800 7100
+	2775 6600 3400 6600
+Wire Wire Line
+	2775 6700 3400 6700
+Wire Wire Line
+	2775 6900 3400 6900
+Wire Wire Line
+	2775 7000 3400 7000
+Wire Wire Line
+	2775 7100 3400 7100
 Entry Wire Line
 	1625 6600 1525 6500
@@
 	1    0    0    -1
 $EndComp
-Text Label 3425 6600 0    51   ~ 0
-D31
-Text Label 3425 6700 0    51   ~ 0
-D30
-Text Label 3425 6800 0    51   ~ 0
-D29
-Text Label 3425 6900 0    51   ~ 0
-D28
-Text Label 3425 7000 0    51   ~ 0
-D27
-Wire Wire Line
-	3275 6800 3275 7100
-Wire Wire Line
-	3275 7100 3575 7100
 Wire Wire Line
 	2775 6800 3275 6800
 Text Label 2800 6800 0    51   ~ 0
 ROMCONF
-Text GLabel 2800 7100 2    51   Output ~ 0
+Text GLabel 3400 7100 2    51   Output ~ 0
 68KMODE
-Text GLabel 2800 7000 2    51   Output ~ 0
+Text GLabel 3400 7000 2    51   Output ~ 0
 JMODE
-Text Label 2800 6600 0    51   ~ 0
-PHANTOMLO
-Text Label 2800 6700 0    51   ~ 0
-PHANTOMHI
-Text Label 2800 6900 0    51   ~ 0
-RSTENB
-Text Label 4775 7100 0    51   ~ 0
-RAMCONF
-NoConn ~ 4775 6900
-NoConn ~ 4775 7000
-Text Label 4775 6600 0    51   ~ 0
-RA2
-Text Label 4775 6700 0    51   ~ 0
-RA1
-Text Label 4775 6800 0    51   ~ 0
-RA0
-Text Notes 5275 6725 2    51   ~ 0
-TO u304
 $Comp
 L power:+5V #PWR0146
@@
 $EndComp
 $Comp
-L power:+5V #PWR0147
-U 1 1 6360A387
-P 4075 6300
-F 0 "#PWR0147" H 4075 6150 50  0001 C CNN
-F 1 "+5V" H 4090 6473 50  0000 C CNN
-F 2 "" H 4075 6300 50  0001 C CNN
-F 3 "" H 4075 6300 50  0001 C CNN
-	1    4075 6300
-	1    0    0    -1
-$EndComp
-$Comp
-L power:GND #PWR0148
-U 1 1 6360AB27
-P 4075 7800
-F 0 "#PWR0148" H 4075 7550 50  0001 C CNN
-F 1 "GND" H 4080 7627 50  0000 C CNN
-F 2 "" H 4075 7800 50  0001 C CNN
-F 3 "" H 4075 7800 50  0001 C CNN
-	1    4075 7800
-	1    0    0    -1
-$EndComp
-$Comp
 L power:GND #PWR0149
 U 1 1 6360ABD4
@@
 $EndComp
 Wire Wire Line
-	1775 7300 1450 7300
-Wire Wire Line
-	1450 7300 1450 8200
-Wire Wire Line
-	3575 7300 3325 7300
-Wire Wire Line
-	3325 7300 3325 8325
+	1775 7300 1225 7300
 Wire Wire Line
 	1775 7500 1225 7500
 Text GLabel 1225 7500 0    51   Input ~ 0
 _REGRESET
-Wire Wire Line
-	3600 7500 3575 7500
-Wire Wire Line
-	3475 7500 3475 8325
-Connection ~ 3575 7500
-Wire Wire Line
-	3575 7500 3475 7500
-Text Notes 3850 8400 2    51   ~ 0
-FROM U301
-$Comp
-L 74xx:74LS04 U?
-U 5 1 636212F5
-P 1450 8500
-AR Path="/61DF74A0/636212F5" Ref="U?"  Part="3"
-AR Path="/634ECC15/636212F5" Ref="U307"  Part="5"
-F 0 "U307" H 1450 8183 50  0000 C CNN
-F 1 "74HCT04" H 1450 8274 50  0000 C CNN
-F 2 "Package_SO:SOIC-14_3.9x8.7mm_P1.27mm" H 1450 8500 50  0001 C CNN
-F 3 "http://www.ti.com/lit/gpn/sn74LS04" H 1450 8500 50  0001 C CNN
-	5    1450 8500
-	0    -1   -1   0
-$EndComp
-$Comp
-L 74xx:74LS04 U?
-U 6 1 636251C6
-P 3325 8625
-AR Path="/61DF74A0/636251C6" Ref="U?"  Part="3"
-AR Path="/634ECC15/636251C6" Ref="U307"  Part="6"
-F 0 "U307" H 3325 8308 50  0000 C CNN
-F 1 "74HCT04" H 3325 8399 50  0000 C CNN
-F 2 "Package_SO:SOIC-14_3.9x8.7mm_P1.27mm" H 3325 8625 50  0001 C CNN
-F 3 "http://www.ti.com/lit/gpn/sn74LS04" H 3325 8625 50  0001 C CNN
-	6    3325 8625
-	0    -1   -1   0
-$EndComp
-Text Notes 3525 9000 2    51   ~ 0
-FROM U301
-Text Notes 1675 8900 2    51   ~ 0
-FROM U301
 $Comp
 L 74xx:74LS74 U502
@@
 Text Notes 5025 4050 2    118  ~ 0
 STATE MACHINE
-Text Notes 5650 6075 2    118  ~ 0
-THESE ARE IN THE CPLD!
 Wire Bus Line
-	1175 5875 3325 5875
+	1175 5875 1425 5875
+Text GLabel 1225 7300 0    50   Input ~ 0
+ROMCLK
+Text GLabel 3400 6700 2    50   Output ~ 0
+PHANTOMHI
+Text GLabel 3400 6600 2    50   Output ~ 0
+PHANTOMLO
+Text GLabel 3400 6900 2    50   Output ~ 0
+RSTENB
 Wire Bus Line
 	1525 5975 1525 7000
-Wire Bus Line
-	3325 5875 3325 6900
 $EndSCHEMATC

Commit message: Add files via upload
Parts:
- added C300, C503, C606: 0.22, Capacitor_SMD:C_0805_2012Metric, symbol Device:C
Connections:
- net +5V: now also U300.14 (VCC), U503.14 (VCC), U606.20 (VCC), C300.1, C503.1, C606.1
- net GND: now also U300.7 (GND), U503.7 (GND), U606.10 (GND), C300.2, C503.2, C606.2
Other:
- moved on the sheet: U503C, U606I
Changed lines of the file:
@@
 L 74xx:74LS244_Split U606
 U 9 1 634F66F6
-P 14600 8400
-F 0 "U606" V 14725 8300 50  0000 L CNN
-F 1 "74HCT244" V 14500 8225 50  0000 L CNN
-F 2 "Package_SO:SOIC-20W_7.5x12.8mm_P1.27mm" H 14600 8400 50  0001 C CNN
-F 3 "http://www.ti.com/lit/ds/symlink/sn74ls241.pdf" H 14600 8400 50  0001 C CNN
-	9    14600 8400
+P 14675 8350
+F 0 "U606" V 14800 8250 50  0000 L CNN
+F 1 "74HCT244" V 14575 8175 50  0000 L CNN
+F 2 "Package_SO:SOIC-20W_7.5x12.8mm_P1.27mm" H 14675 8350 50  0001 C CNN
+F 3 "http://www.ti.com/lit/ds/symlink/sn74ls241.pdf" H 14675 8350 50  0001 C CNN
+	9    14675 8350
 	1    0    0    -1
 $EndComp
@@
 L 74xx:74LS74 U503
 U 3 1 6356B308
-P 15750 8400
-F 0 "U503" V 15850 8275 50  0000 L CNN
-F 1 "74HCT74" V 15625 8250 50  0000 L CNN
-F 2 "Package_SO:SOIC-14_3.9x8.7mm_P1.27mm" H 15750 8400 50  0001 C CNN
-F 3 "74xx/74hc_hct74.pdf" H 15750 8400 50  0001 C CNN
-	3    15750 8400
+P 15650 8350
+F 0 "U503" V 15750 8225 50  0000 L CNN
+F 1 "74HCT74" V 15525 8200 50  0000 L CNN
+F 2 "Package_SO:SOIC-14_3.9x8.7mm_P1.27mm" H 15650 8350 50  0001 C CNN
+F 3 "74xx/74hc_hct74.pdf" H 15650 8350 50  0001 C CNN
+	3    15650 8350
 	1    0    0    -1
 $EndComp
@@
 Text GLabel 3400 6900 2    50   Output ~ 0
 RSTENB
+$Comp
+L Device:C C300
+U 1 1 6353B771
+P 14125 8325
+F 0 "C300" H 14240 8371 50  0000 L CNN
+F 1 "0.22" H 14240 8280 50  0000 L CNN
+F 2 "Capacitor_SMD:C_0805_2012Metric" H 14163 8175 50  0001 C CNN
+F 3 "~" H 14125 8325 50  0001 C CNN
+	1    14125 8325
+	1    0    0    -1
+$EndComp
+$Comp
+L Device:C C606
+U 1 1 6353D849
+P 15050 8325
+F 0 "C606" H 15165 8371 50  0000 L CNN
+F 1 "0.22" H 15165 8280 50  0000 L CNN
+F 2 "Capacitor_SMD:C_0805_2012Metric" H 15088 8175 50  0001 C CNN
+F 3 "~" H 15050 8325 50  0001 C CNN
+	1    15050 8325
+	1    0    0    -1
+$EndComp
+$Comp
+L Device:C C503
+U 1 1 6353FA52
+P 16050 8325
+F 0 "C503" H 16165 8371 50  0000 L CNN
+F 1 "0.22" H 16165 8280 50  0000 L CNN
+F 2 "Capacitor_SMD:C_0805_2012Metric" H 16088 8175 50  0001 C CNN
+F 3 "~" H 16050 8325 50  0001 C CNN
+	1    16050 8325
+	1    0    0    -1
+$EndComp
+Wire Wire Line
+	16050 8175 16050 7850
+Wire Wire Line
+	16050 7850 15650 7850
+Connection ~ 14675 7850
+Wire Wire Line
+	14675 7850 14125 7850
+Wire Wire Line
+	13750 8850 14125 8850
+Wire Wire Line
+	16050 8850 16050 8475
+Wire Wire Line
+	15650 8750 15650 8850
+Connection ~ 15650 8850
+Wire Wire Line
+	15650 8850 16050 8850
+Wire Wire Line
+	15650 7950 15650 7850
+Connection ~ 15650 7850
+Wire Wire Line
+	15650 7850 15050 7850
+$Comp
+L power:+5V #PWR0103
+U 1 1 635487F0
+P 16050 7850
+F 0 "#PWR0103" H 16050 7700 50  0001 C CNN
+F 1 "+5V" H 16065 8023 50  0000 C CNN
+F 2 "" H 16050 7850 50  0001 C CNN
+F 3 "" H 16050 7850 50  0001 C CNN
+	1    16050 7850
+	1    0    0    -1
+$EndComp
+Connection ~ 16050 7850
+$Comp
+L power:GND #PWR0183
+U 1 1 63548D8D
+P 16050 8850
+F 0 "#PWR0183" H 16050 8600 50  0001 C CNN
+F 1 "GND" H 16055 8677 50  0000 C CNN
+F 2 "" H 16050 8850 50  0001 C CNN
+F 3 "" H 16050 8850 50  0001 C CNN
+	1    16050 8850
+	1    0    0    -1
+$EndComp
+Connection ~ 16050 8850
+Wire Wire Line
+	15050 8175 15050 7850
+Connection ~ 15050 7850
+Wire Wire Line
+	15050 7850 14675 7850
+Wire Wire Line
+	15050 8475 15050 8850
+Connection ~ 15050 8850
+Wire Wire Line
+	15050 8850 15650 8850
+Connection ~ 14675 8850
+Wire Wire Line
+	14675 8850 15050 8850
+Wire Wire Line
+	14125 8175 14125 7850
+Connection ~ 14125 7850
+Wire Wire Line
+	14125 7850 13750 7850
+Wire Wire Line
+	14125 8475 14125 8850
 Wire Bus Line
 	1525 5975 1525 7000
+Connection ~ 14125 8850
+Wire Wire Line
+	14125 8850 14675 8850
 $EndSCHEMATC

Commit message: Add files via upload
Parts:
- added R300: 1K, Resistor_SMD:R_0805_2012Metric, symbol Device:R
- added R301: 470, Resistor_SMD:R_0805_2012Metric, symbol Device:R
- added R302: 3.3K, Resistor_SMD:R_0805_2012Metric, symbol Device:R
- added unit 5 of U300
- added U507: 74HCT74, Package_SO:SOIC-14_3.9x8.7mm_P1.27mm, symbol 74xx:74LS74
Connections:
- net +5V: now also R301.1, R302.1, U507.4 (~S)
- net GND: now also R300.2
- net ROMCONF: no longer names the net of U303.7 (Q2)
- net _S7MDIS_DFF renamed _S7MDISD
- new net: U300.11, U507.5 (Q)
- new net DSCLK: U507.3 (C)
- new net _AS: R302.2
- new net _DSACK1: U300.10
- new net _DSACKDIS: U507.1 (~R)
- new net _DSACKEN: U507.2 (D)
- new net _EXTSEL: R300.1
- new net _MEMSEL: R301.2
- no-connect marks 4 -> 6
Other:
- note added: "BUS GRANT ENABLE/DISABLE"
- note added: "DISCRETE LOGIC BITS"
- note added: "DSACK FOR 16 BIT CYCLES"
- note added: "OUTPUT TO AMIGA BUFFER"
- note added: "PULL UP/DOWN"
- note added: "RESET CONFIGURE"
- note added: "STARTUP ROM CONFIG"
- note added: "Summer turns me upside down"
- note removed: "_IVMA (U506)\nTRISTATE (U305)\nClocks (U708)"
- moved on the sheet: C300, C503, C606, R500, R501, R502, U300A, U300B, U300G, U303, U307B, U502A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
