File: A2630-New-KiCAD/Logic.kicad_sch (KiCad schematic)
At the start: 24 parts, among them U300 74HCT05, U303 74HCT174, U307 74HCT04, U414 74LVC257, U415 74LVC257, U416 74LVC257, U417 74LVC257, U502 74HCT74, U503 74HCT74, U507 74HCT74, U606 74HCT244

Commit message: Add files via upload
Parts:
- removed R302: 3.3K, Resistor_SMD:R_0805_2012Metric, symbol Device:R
Other:
- moved on the sheet: R300
Changed lines of the file:
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@@
-    (stroke (width 0) (type default) (color 0 0 0 0))
-  )
-  (wire (pts (xy 262.89 133.985) (xy 255.27 133.985))
     (stroke (width 0) (type default) (color 0 0 0 0))
   )
@@
     (stroke (width 0) (type default) (color 0 0 0 0))
   )
-  (wire (pts (xy 274.32 140.97) (xy 266.7 140.97))
+  (wire (pts (xy 263.906 123.571) (xy 256.286 123.571))
     (stroke (width 0) (type default) (color 0 0 0 0))
   )
@@
     (stroke (width 0) (type default) (color 0 0 0 0))
   )
-  (polyline (pts (xy 248.92 156.21) (xy 300.99 156.21))
+  (polyline (pts (xy 248.92 139.7) (xy 300.99 139.7))
     (stroke (width 0) (type default) (color 0 0 0 0))
   )
@@
     (stroke (width 0) (type default) (color 0 0 0 0))
   )
-  (polyline (pts (xy 300.99 156.21) (xy 300.99 90.17))
+  (polyline (pts (xy 300.99 139.7) (xy 300.99 90.17))
     (stroke (width 0) (type default) (color 0 0 0 0))
   )
@@
     (stroke (width 0) (type default) (color 0 0 0 0))
   )
-  (polyline (pts (xy 248.92 90.17) (xy 248.92 156.21))
+  (polyline (pts (xy 248.92 90.17) (xy 248.92 139.7))
     (stroke (width 0) (type default) (color 0 0 0 0))
   )
@@
   )
   (global_label "_DTACK" (shape input) (at 290.83 133.985 0) (fields_autoplaced)
-    (effects (font (size 1.27 1.27)) (justify left))
-    (property "Intersheet References" "${INTERSHEET_REFS}" (id 0) (at -33.655 59.055 0)
-      (effects (font (size 1.27 1.27)) hide)
-    )
-  )
-  (global_label "_AS" (shape input) (at 262.89 133.985 0) (fields_autoplaced)
     (effects (font (size 1.27 1.27)) (justify left))
     (property "Intersheet References" "${INTERSHEET_REFS}" (id 0) (at -33.655 59.055 0)
@@
     )
   )
-  (global_label "EXTSEL" (shape input) (at 274.32 140.97 0) (fields_autoplaced)
+  (global_label "EXTSEL" (shape input) (at 263.906 123.571 0) (fields_autoplaced)
     (effects (font (size 1.2954 1.2954)) (justify left))
-    (property "Intersheet References" "${INTERSHEET_REFS}" (id 0) (at -33.655 59.055 0)
+    (property "Intersheet References" "${INTERSHEET_REFS}" (id 0) (at -44.069 41.656 0)
       (effects (font (size 1.27 1.27)) hide)
     )
@@
     (pin "11")
   )
-  (symbol (lib_id "Device:R") (at 266.7 144.78 0) (unit 1)
-    (in_bom yes) (on_board yes)
-    (property "Reference" "R300" (id 0) (at 268.478 143.6116 0)
+  (symbol (lib_id "Device:R") (at 256.286 127.381 0) (unit 1)
+    (in_bom yes) (on_board yes)
+    (property "Reference" "R300" (id 0) (at 258.064 126.2126 0)
       (effects (font (size 1.27 1.27)) (justify left))
     )
-    (property "Value" "1K" (id 1) (at 268.478 145.923 0)
+    (property "Value" "1K" (id 1) (at 258.064 128.524 0)
       (effects (font (size 1.27 1.27)) (justify left))
     )
-    (property "Footprint" "Resistor_SMD:R_0805_2012Metric" (id 2) (at 264.922 144.78 90)
-      (effects (font (size 1.27 1.27)) hide)
-    )
-    (property "Datasheet" "~" (id 3) (at 266.7 144.78 0)
+    (property "Footprint" "Resistor_SMD:R_0805_2012Metric" (id 2) (at 254.508 127.381 90)
+      (effects (font (size 1.27 1.27)) hide)
+    )
+    (property "Datasheet" "~" (id 3) (at 256.286 127.381 0)
       (effects (font (size 1.27 1.27)) hide)
     )
@@
     (pin "2")
   )
-  (symbol (lib_id "power:GND") (at 266.7 148.59 0) (unit 1)
-    (in_bom yes) (on_board yes)
-    (property "Reference" "#PWR04" (id 0) (at 266.7 154.94 0)
-      (effects (font (size 1.27 1.27)) hide)
-    )
-    (property "Value" "GND" (id 1) (at 266.827 152.9842 0))
-    (property "Footprint" "" (id 2) (at 266.7 148.59 0)
-      (effects (font (size 1.27 1.27)) hide)
-    )
-    (property "Datasheet" "" (id 3) (at 266.7 148.59 0)
+  (symbol (lib_id "power:GND") (at 256.286 131.191 0) (unit 1)
+    (in_bom yes) (on_board yes)
+    (property "Reference" "#PWR04" (id 0) (at 256.286 137.541 0)
+      (effects (font (size 1.27 1.27)) hide)
+    )
+    (property "Value" "GND" (id 1) (at 256.413 135.5852 0))
+    (property "Footprint" "" (id 2) (at 256.286 131.191 0)
+      (effects (font (size 1.27 1.27)) hide)
+    )
+    (property "Datasheet" "" (id 3) (at 256.286 131.191 0)
       (effects (font (size 1.27 1.27)) hide)
     )
@@
       (effects (font (size 1.27 1.27)) hide)
     )
-    (pin "1")
-  )
-  (symbol (lib_id "Device:R") (at 255.27 130.175 0) (unit 1)
-    (in_bom yes) (on_board yes)
-    (property "Reference" "R302" (id 0) (at 257.048 129.0066 0)
-      (effects (font (size 1.27 1.27)) (justify left))
-    )
-    (property "Value" "3.3K" (id 1) (at 257.048 131.318 0)
-      (effects (font (size 1.27 1.27)) (justify left))
-    )
-    (property "Footprint" "Resistor_SMD:R_0805_2012Metric" (id 2) (at 253.492 130.175 90)
-      (effects (font (size 1.27 1.27)) hide)
-    )
-    (property "Datasheet" "~" (id 3) (at 255.27 130.175 0)
-      (effects (font (size 1.27 1.27)) hide)
-    )
-    (pin "1")
-    (pin "2")
-  )
-  (symbol (lib_id "power:+5V") (at 255.27 126.365 0) (unit 1)
-    (in_bom yes) (on_board yes)
-    (property "Reference" "#PWR02" (id 0) (at 255.27 130.175 0)
-      (effects (font (size 1.27 1.27)) hide)
-    )
-    (property "Value" "+5V" (id 1) (at 255.651 121.9708 0))
-    (property "Footprint" "" (id 2) (at 255.27 126.365 0)
-      (effects (font (size 1.27 1.27)) hide)
-    )
-    (property "Datasheet" "" (id 3) (at 255.27 126.365 0)
-      (effects (font (size 1.27 1.27)) hide)
-    )

Commit message: Add files via upload
Parts:
- added C307, C502, C507: 0.22uf, Capacitor_SMD:C_0805_2012Metric, symbol Device:C
- added R503, R504, R505, R506: 1K, Resistor_SMD:R_0805_2012Metric, symbol Device:R
- added unit 7 of U307
- added unit 3 of U502
- added unit 3 of U507
- C300, C414, C415, C416, C417, C503, C606: value 0.22 -> 0.22uf
Connections:
- net +5V: now also C307.1, C502.1, C507.1, R503.1, R504.1, R505.1, R506.1, U307.14 (VCC), U502.14 (VCC), U507.14 (VCC); no longer U502.13 (~{R}), U503.1 (~{R}), U503.13 (~{R}), U503.14 (VCC), U507.4 (~{S})
- net GND: now also C307.2, C502.2, C507.2, U307.7 (GND), U502.7 (GND), U507.7 (GND)
- new net: R503.2, U502.13 (~{R})
- new net: R504.2, U507.4 (~{S})
- new net: R505.2, U503.1 (~{R})
- new net: R506.2, U503.13 (~{R})
Other:
- moved on the sheet: C300, C414, C415, C416, C417, C503, C606, U300G, U303, U414B, U415B, U416B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

Commit message: Add files via upload
Connections:
- net D18 is gone; now on net GND: U303.6 (D2)
Changed lines of the file:
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@@
   (junction (at 160.401 229.87) (diameter 0) (color 0 0 0 0)
+  )
+  (junction (at 79.375 215.9) (diameter 0) (color 0 0 0 0)
   )
   (junction (at 213.487 229.87) (diameter 0) (color 0 0 0 0)
@@
     (stroke (width 0) (type default) (color 0 0 0 0))
   )
-  (bus_entry (at 62.865 190.5) (size -2.54 -2.54)
-    (stroke (width 0) (type default) (color 0 0 0 0))
-  )
   (bus_entry (at 340.36 85.09) (size -2.54 -2.54)
     (stroke (width 0) (type default) (color 0 0 0 0))
@@
     (stroke (width 0) (type default) (color 0 0 0 0))
   )
-  (bus (pts (xy 60.325 187.96) (xy 60.325 193.04))
+  (bus (pts (xy 60.325 185.42) (xy 60.325 193.04))
     (stroke (width 0) (type default) (color 0 0 0 0))
   )
@@
     (stroke (width 0) (type default) (color 0 0 0 0))
   )
+  (wire (pts (xy 66.675 190.5) (xy 57.15 190.5))
+    (stroke (width 0) (type default) (color 0 0 0 0))
+  )
   (wire (pts (xy 75.565 94.615) (xy 46.99 94.615))
     (stroke (width 0) (type default) (color 0 0 0 0))
@@
     (stroke (width 0) (type default) (color 0 0 0 0))
   )
+  (wire (pts (xy 57.15 190.5) (xy 57.15 215.9))
+    (stroke (width 0) (type default) (color 0 0 0 0))
+  )
   (wire (pts (xy 282.067 255.27) (xy 292.227 255.27))
     (stroke (width 0) (type default) (color 0 0 0 0))
@@
     (stroke (width 0) (type default) (color 0 0 0 0))
   )
-  (wire (pts (xy 66.675 190.5) (xy 62.865 190.5))
-    (stroke (width 0) (type default) (color 0 0 0 0))
-  )
   (bus (pts (xy 337.82 80.01) (xy 337.82 82.55))
     (stroke (width 0) (type default) (color 0 0 0 0))
@@
     (stroke (width 0) (type default) (color 0 0 0 0))
   )
-  (bus (pts (xy 60.325 185.42) (xy 60.325 187.96))
+  (wire (pts (xy 79.375 215.9) (xy 57.15 215.9))
     (stroke (width 0) (type default) (color 0 0 0 0))
   )
@@
     (effects (font (size 1.27 1.27)) (justify right bottom))
   )
-  (label "D18" (at 62.865 190.5 0)
-    (effects (font (size 1.2954 1.2954)) (justify left bottom))
-  )
   (label "A20" (at 340.36 92.71 0)

Commit message: Add files via upload
Connections:
- net A15: now also U417.5 (I0b), U417.6 (I1b); no longer U414.3 (I1a)
- net A16: now also U417.13 (I1c), U417.14 (I0c); no longer U414.6 (I1b)
- net A17: now also U414.3 (I1a); no longer U414.13 (I1c)
- net A18: now also U414.6 (I1b); no longer U414.10 (I1d)
- net A19: now also U414.13 (I1c); no longer U415.3 (I1a)
- net A20: now also U414.10 (I1d); no longer U415.6 (I1b)
- net A21: now also U415.3 (I1a); no longer U415.13 (I1c)
- net A22: now also U415.6 (I1b); no longer U415.10 (I1d)
- net A23: now also U415.13 (I1c); no longer U416.3 (I1a)
- net A24: now also U415.10 (I1d); no longer U416.6 (I1b)
- net GND: now also U416.6 (I1b); no longer U417.13 (I1c), U417.14 (I0c), U417.5 (I0b), U417.6 (I1b)
- net BANK1: now reaches U417.12 (Zc)
- net BANK0: now reaches U417.7 (Zb)
- new net A25: U416.3 (I1a)
- no-connect marks 9 -> 7

Commit message: Add files via upload
Parts:
- added C418, C419, C420, C421: 0.22uf, Capacitor_SMD:C_0805_2012Metric, symbol Device:C
- added U418, U419, U420, U421: 74LVC245, Package_SO:TSSOP-20_4.4x6.5mm_P0.65mm, symbol N2630:74LVC245
Connections:
- net +3V3: now also C418.1, C419.1, C420.1, C421.1, U418.20 (VCC), U419.20 (VCC), U420.20 (VCC), U421.20 (VCC)
- net D16: now also U420.9 (A7)
- net D17: now also U420.8 (A6)
- net D19: now also U420.6 (A4)
- net D20: now also U420.5 (A3)
- net GND: now also C418.2, C419.2, C420.2, C421.2, U418.10 (GND), U418.19 (CE), U419.10 (GND), U419.19 (CE), U420.10 (GND), U420.19 (CE), U421.10 (GND), U421.19 (CE)
- new net D0: U418.9 (A7)
- new net D1: U418.8 (A6)
- new net D10: U419.7 (A5)
- new net D11: U419.6 (A4)
- new net D12: U419.5 (A3)
- new net D13: U419.4 (A2)
- new net D14: U419.3 (A1)
- new net D15: U419.2 (A0)
- new net D18: U420.7 (A5)
- new net D2: U418.7 (A5)
- new net D21: U420.4 (A2)
- new net D22: U420.3 (A1)
- new net D23: U420.2 (A0)
- new net D24: U421.9 (A7)
- new net D25: U421.8 (A6)
- new net D26: U421.7 (A5)
- new net D27: U421.6 (A4)
- new net D28: U421.5 (A3)
- new net D29: U421.4 (A2)
- new net D3: U418.6 (A4)
- new net D30: U421.3 (A1)
- new net D31: U421.2 (A0)
- new net D4: U418.5 (A3)
- new net D5: U418.4 (A2)
- new net D6: U418.3 (A1)
- new net D7: U418.2 (A0)
- new net D8: U419.9 (A7)
- new net D9: U419.8 (A6)
- new net EMD0: U418.11 (B7)
- new net EMD1: U418.12 (B6)
- new net EMD10: U419.13 (B5)
- new net EMD11: U419.14 (B4)
- new net EMD12: U419.15 (B3)
- new net EMD13: U419.16 (B2)
- new net EMD14: U419.17 (B1)
- new net EMD15: U419.18 (B0)
- new net EMD16: U420.11 (B7)
- new net EMD17: U420.12 (B6)
- new net EMD18: U420.13 (B5)
- new net EMD19: U420.14 (B4)
- new net EMD2: U418.13 (B5)
- new net EMD20: U420.15 (B3)
- new net EMD21: U420.16 (B2)
- new net EMD22: U420.17 (B1)
- new net EMD23: U420.18 (B0)
- new net EMD24: U421.11 (B7)
- new net EMD25: U421.12 (B6)
- new net EMD26: U421.13 (B5)
- new net EMD27: U421.14 (B4)
- new net EMD28: U421.15 (B3)
- new net EMD29: U421.16 (B2)
- new net EMD3: U418.14 (B4)
- new net EMD30: U421.17 (B1)
- new net EMD31: U421.18 (B0)
- new net EMD4: U418.15 (B3)
- new net EMD5: U418.16 (B2)
- new net EMD6: U418.17 (B1)
- new net EMD7: U418.18 (B0)
- new net EMD8: U419.11 (B7)
- new net EMD9: U419.12 (B6)
- new net EMDDIR: U418.1 (A->B), U419.1 (A->B), U420.1 (A->B), U421.1 (A->B)
Other:
- moved on the sheet: R300, R301, R500, R501, R502, R503, R504, R505, R506, U300A, U300B, U300E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

Commit message: Add files via upload
Parts:
- added C303: 0.22uf, Capacitor_SMD:C_0805_2012Metric, symbol Device:C
- added R307: 1K, Resistor_SMD:R_0805_2012Metric, symbol Device:R
Connections:
- net +5V: now also U503.14 (VCC), C303.1, R307.1; no longer U303.11 (D3)
- net GND: now also C303.2
- net 68KMODE renamed MODE68K
- new net: R307.2, U303.11 (D3)
Changed lines of the file:
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@@
   (junction (at 205.105 255.27) (diameter 0) (color 0 0 0 0)
   )
+  (junction (at 205.105 229.87) (diameter 0) (color 0 0 0 0)
+  )
   (junction (at 195.834 229.87) (diameter 0) (color 0 0 0 0)
   )
@@
   (junction (at 242.697 255.27) (diameter 0) (color 0 0 0 0)
   )
-  (junction (at 203.327 229.87) (diameter 0) (color 0 0 0 0)
-  )
   (junction (at 151.765 255.27) (diameter 0) (color 0 0 0 0)
   )
@@
   (junction (at 160.401 229.87) (diameter 0) (color 0 0 0 0)
   )
+  (junction (at 62.865 154.94) (diameter 0) (color 0 0 0 0)
+  )
   (junction (at 62.865 197.485) (diameter 0) (color 0 0 0 0)
   )
@@
     (stroke (width 0) (type default) (color 0 0 0 0))
   )
-  (wire (pts (xy 203.327 229.87) (xy 195.834 229.87))
+  (wire (pts (xy 195.834 229.87) (xy 205.105 229.87))
     (stroke (width 0) (type default) (color 0 0 0 0))
   )
@@
     (stroke (width 0) (type default) (color 0 0 0 0))
   )
+  (wire (pts (xy 205.105 229.87) (xy 205.105 232.41))
+    (stroke (width 0) (type default) (color 0 0 0 0))
+  )
   (wire (pts (xy 289.56 156.845) (xy 296.545 156.845))
     (stroke (width 0) (type default) (color 0 0 0 0))
@@
     (stroke (width 0) (type default) (color 0 0 0 0))
   )
+  (wire (pts (xy 62.865 152.4) (xy 62.865 154.94))
+    (stroke (width 0) (type default) (color 0 0 0 0))
+  )
   (wire (pts (xy 292.227 255.27) (xy 301.117 255.27))
     (stroke (width 0) (type default) (color 0 0 0 0))
@@
     (stroke (width 0) (type default) (color 0 0 0 0))
   )
+  (wire (pts (xy 62.865 154.94) (xy 71.12 154.94))
+    (stroke (width 0) (type default) (color 0 0 0 0))
+  )
   (wire (pts (xy 258.445 164.465) (xy 264.16 164.465))
     (stroke (width 0) (type default) (color 0 0 0 0))
@@
     (stroke (width 0) (type default) (color 0 0 0 0))
   )
+  (wire (pts (xy 62.865 154.94) (xy 62.865 159.385))
+    (stroke (width 0) (type default) (color 0 0 0 0))
+  )
   (bus (pts (xy 337.82 38.1) (xy 337.82 43.18))
     (stroke (width 0) (type default) (color 0 0 0 0))
@@
     (stroke (width 0) (type default) (color 0 0 0 0))
   )
-  (wire (pts (xy 213.487 229.87) (xy 203.327 229.87))
+  (wire (pts (xy 213.487 229.87) (xy 205.105 229.87))
     (stroke (width 0) (type default) (color 0 0 0 0))
   )
@@
     (stroke (width 0) (type default) (color 0 0 0 0))
   )
-  (wire (pts (xy 203.327 232.41) (xy 203.327 229.87))
-    (stroke (width 0) (type default) (color 0 0 0 0))
-  )
   (wire (pts (xy 340.36 180.34) (xy 350.52 180.34))
     (stroke (width 0) (type default) (color 0 0 0 0))
@@
     (stroke (width 0) (type default) (color 0 0 0 0))
   )
+  (wire (pts (xy 78.74 154.94) (xy 83.82 154.94))
+    (stroke (width 0) (type default) (color 0 0 0 0))
+  )
   (wire (pts (xy 137.795 195.58) (xy 137.795 203.835))
     (stroke (width 0) (type default) (color 0 0 0 0))
@@
     )
   )
-  (global_label "68KMODE" (shape output) (at 91.44 179.705 0) (fields_autoplaced)
+  (global_label "MODE68K" (shape output) (at 91.44 179.705 0) (fields_autoplaced)
     (effects (font (size 1.2954 1.2954)) (justify left))
-    (property "Intersheet References" "${INTERSHEET_REFS}" (id 0) (at -16.51 -25.4 0)
-      (effects (font (size 1.27 1.27)) hide)
+    (property "Intersheet References" "${INTERSHEET_REFS}" (id 0) (at 102.8783 179.6241 0)
+      (effects (font (size 1.2954 1.2954)) (justify left) hide)
     )
   )
@@
     (pin "9")
   )
-  (symbol (lib_id "power:+5V") (at 36.195 170.18 0) (unit 1)
+  (symbol (lib_id "power:+5V") (at 36.195 162.56 0) (unit 1)
     (in_bom yes) (on_board yes)
-    (property "Reference" "#PWR0145" (id 0) (at 36.195 173.99 0)
+    (property "Reference" "#PWR0145" (id 0) (at 36.195 166.37 0)
       (effects (font (size 1.27 1.27)) hide)
     )
-    (property "Value" "+5V" (id 1) (at 36.576 165.7858 0))
-    (property "Footprint" "" (id 2) (at 36.195 170.18 0)
+    (property "Value" "+5V" (id 1) (at 36.576 158.1658 0))
+    (property "Footprint" "" (id 2) (at 36.195 162.56 0)
       (effects (font (size 1.27 1.27)) hide)
     )
-    (property "Datasheet" "" (id 3) (at 36.195 170.18 0)
+    (property "Datasheet" "" (id 3) (at 36.195 162.56 0)
       (effects (font (size 1.27 1.27)) hide)
     )
     (pin "1")
   )
-  (symbol (lib_id "power:+5V") (at 62.865 159.385 0) (unit 1)
+  (symbol (lib_id "power:+5V") (at 62.865 152.4 0) (unit 1)
     (in_bom yes) (on_board yes)
-    (property "Reference" "#PWR0146" (id 0) (at 62.865 163.195 0)
+    (property "Reference" "#PWR0146" (id 0) (at 62.865 156.21 0)
       (effects (font (size 1.27 1.27)) hide)
     )
-    (property "Value" "+5V" (id 1) (at 63.246 154.9908 0))
-    (property "Footprint" "" (id 2) (at 62.865 159.385 0)
+    (property "Value" "+5V" (id 1) (at 63.246 148.0058 0))
+    (property "Footprint" "" (id 2) (at 62.865 152.4 0)
       (effects (font (size 1.27 1.27)) hide)
     )
-    (property "Datasheet" "" (id 3) (at 62.865 159.385 0)
+    (property "Datasheet" "" (id 3) (at 62.865 152.4 0)
       (effects (font (size 1.27 1.27)) hide)
     )
@@
     (pin "2")
   )
+  (symbol (lib_id "Device:C") (at 74.93 154.94 90) (unit 1)
+    (in_bom yes) (on_board yes)
+    (property "Reference" "C303" (id 0) (at 73.025 153.543 90)
+      (effects (font (size 1.27 1.27)) (justify left))
+    )
+    (property "Value" "0.22uf" (id 1) (at 83.312 153.543 90)
+      (effects (font (size 1.27 1.27)) (justify left))
+    )
+    (property "Footprint" "Capacitor_SMD:C_0805_2012Metric" (id 2) (at 78.74 153.9748 0)
+      (effects (font (size 1.27 1.27)) hide)
+    )
+    (property "Datasheet" "~" (id 3) (at 74.93 154.94 0)
+      (effects (font (size 1.27 1.27)) hide)
+    )
+    (pin "1")
+    (pin "2")
+  )
   (symbol (lib_id "power:GND") (at 346.71 208.915 0) (unit 1)
     (in_bom yes) (on_board yes) (fields_autoplaced)
@@
     (pin "1")
   )
+  (symbol (lib_id "power:GND") (at 83.82 154.94 0) (unit 1)
+    (in_bom yes) (on_board yes) (fields_autoplaced)
+    (property "Reference" "#PWR0169" (id 0) (at 83.82 161.29 0)
+      (effects (font (size 1.27 1.27)) hide)
+    )
+    (property "Value" "GND" (id 1) (at 83.82 159.3834 0))
+    (property "Footprint" "" (id 2) (at 83.82 154.94 0)
+      (effects (font (size 1.27 1.27)) hide)
+    )
+    (property "Datasheet" "" (id 3) (at 83.82 154.94 0)
+      (effects (font (size 1.27 1.27)) hide)
+    )
+    (pin "1")
+  )
   (symbol (lib_id "power:GND") (at 350.52 119.38 0) (unit 1)
     (in_bom yes) (on_board yes) (fields_autoplaced)
@@
     (pin "1")
   )
+  (symbol (lib_id "Device:R") (at 36.195 166.37 0) (unit 1)
+    (in_bom yes) (on_board yes)
+    (property "Reference" "R307" (id 0) (at 38.735 168.91 90)
+      (effects (font (size 1.27 1.27)) (justify left))
+    )
+    (property "Value" "1K" (id 1) (at 36.195 167.64 90)
+      (effects (font (size 1.27 1.27)) (justify left))
+    )
+    (property "Footprint" "Resistor_SMD:R_0805_2012Metric" (id 2) (at 34.417 166.37 90)
+      (effects (font (size 1.27 1.27)) hide)
+    )
+    (property "Datasheet" "~" (id 3) (at 36.195 166.37 0)
+      (effects (font (size 1.27 1.27)) hide)
+    )
+    (pin "1")
+    (pin "2")
+  )
   (symbol (lib_id "N2630:74LVC245") (at 147.32 208.28 0) (unit 2)

Commit message: Add files via upload
Connections:
- net D17: now also U303.14 (D5); no longer U303.4 (D1)
- net D20: now also U303.4 (D1); no longer U303.14 (D5)
- net MODE68K: now also U303.5 (Q1); no longer U303.15 (Q5)
- net PHANTOMHI: now also U303.15 (Q5); no longer U303.5 (Q1)
Other:
- note added: "RESET"
- note added: "When we are not BOSS, the 2630 is held in reset. This tristates the 68030 and other devices. This also serves as the power up reset."
- note removed: "RESET CONFIGURE"
Changed lines of the file:
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@@
     (effects (font (size 2.9972 2.9972)) (justify left bottom))
   )
-  (text "RESET CONFIGURE" (at 175.895 147.955 180)
+  (text "RESET" (at 153.035 147.32 180)
     (effects (font (size 2.9972 2.9972)) (justify right bottom))
   )
@@
     (effects (font (size 5.9944 5.9944)) (justify left bottom))
   )
+  (text "When we are not BOSS, the 2630\nis held in reset. This tristates \nthe 68030 and other devices. This\nalso serves as the power up reset."
+    (at 152.4 182.88 0)
+    (effects (font (size 1.27 1.27)) (justify left bottom))
+  )
   (text "OUTPUT TO AMIGA BUFFER" (at 33.655 24.765 0)
     (effects (font (size 2.9972 2.9972)) (justify left bottom))
@@
     (effects (font (size 1.27 1.27)) (justify right bottom))
   )
-  (label "D17" (at 46.355 169.545 0)
+  (label "D17" (at 46.355 179.705 0)
     (effects (font (size 1.2954 1.2954)) (justify left bottom))
   )
@@
     (effects (font (size 1.27 1.27)) (justify left bottom))
   )
-  (label "D20" (at 46.355 179.705 0)
+  (label "D20" (at 46.355 169.545 0)
     (effects (font (size 1.2954 1.2954)) (justify left bottom))
   )
@@
     )
   )
-  (global_label "MODE68K" (shape output) (at 91.44 179.705 0) (fields_autoplaced)
+  (global_label "MODE68K" (shape output) (at 91.44 169.545 0) (fields_autoplaced)
     (effects (font (size 1.2954 1.2954)) (justify left))
-    (property "Intersheet References" "${INTERSHEET_REFS}" (id 0) (at 102.8783 179.6241 0)
+    (property "Intersheet References" "${INTERSHEET_REFS}" (id 0) (at 102.8783 169.4641 0)
       (effects (font (size 1.2954 1.2954)) (justify left) hide)
     )
@@
     )
   )
-  (global_label "PHANTOMHI" (shape output) (at 91.44 169.545 0) (fields_autoplaced)
-    (effects (font (size 1.27 1.27)) (justify left))
-    (property "Intersheet References" "${INTERSHEET_REFS}" (id 0) (at -16.51 -25.4 0)
-      (effects (font (size 1.27 1.27)) hide)
-    )
+  (global_label "PHANTOMHI" (shape output) (at 91.44 179.705 0) (fields_autoplaced)
+    (effects (font (size 1.27 1.27)) (justify left))
+    (property "Intersheet References" "${INTERSHEET_REFS}" (id 0) (at -16.51 -15.24 0)
+      (effects (font (size 1.27 1.27)) hide)
+    )
