File: A2630-New-KiCAD/ExpansionMemory.kicad_sch (KiCad schematic)
At the start: 16 parts, among them U102 27C256, U103 27C256, U406 SDRAM_512Mb(32Mx16), U407 SDRAM_512Mb(32Mx16), U408 SDRAM_512Mb(32Mx16), U409 SDRAM_512Mb(32Mx16)

Commit message: Add files via upload
Changed lines of the file:
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@@
   )
   (text "This is Zorro 3 memory, so it is always\ntreated as 32 bit memory and cannot be \nused by the Amiga 2000 chip set and cannot\nbe used by anything on the Zoroo 2 bus.\nIt can only be used by the 68030."
-    (at 274.955 153.67 0)
+    (at 274.955 155.575 0)
     (effects (font (size 3 3)) (justify left bottom))
   )
@@
   )
   (text "JN Notes: put row address on the EMA bus \nand signal RAS. This is 68030 addresses A14:2. \nPut column address on the EMA bus and signal \nCAS. These are 68030 addresses A24:15."
-    (at 275.59 139.7 0)
+    (at 274.32 132.08 0)
     (effects (font (size 2.9972 2.9972)) (justify left bottom))
   )

Commit message: Add files via upload
Other:
- note removed: "TRIVIA: A31..24 is the autoconfig base address A1..0 are part of the sizing system for mem This leaves A23..A2 for actual addressing...22 bits. This is why the Amiga can only address 128 megabytes!"
Changed lines of the file:
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@@
     (effects (font (size 3.9878 3.9878)) (justify left bottom))
-  )
-  (text "TRIVIA:\nA31..24 is the autoconfig base address\nA1..0 are part of the sizing system for mem\nThis leaves A23..A2 for actual addressing...22 bits.\nThis is why the Amiga can only address 128 megabytes!"
-    (at 144.78 37.465 0)
-    (effects (font (size 3 3)) (justify left bottom))
   )
   (text "JN Notes: put row address on the EMA bus \nand signal RAS. This is 68030 addresses A14:2. \nPut column address on the EMA bus and signal \nCAS. These are 68030 addresses A24:15."

Commit message: Add files via upload
Parts:
- U406, U407, U408, U409: value SDRAM_512Mb(32Mx16) -> SDRAM_256Mb(16Mx16)
Connections:
- net EM1B0 is gone; now on net BANK0: U408.20 (BA0), U409.20 (BA0)
- net EM1B1 is gone; now on net BANK1: U408.21 (BA1), U409.21 (BA1)
- net EM0B0 renamed BANK0
- net EM0B1 renamed BANK1
Other:
- note added: "JN Notes: put row addresses 14..2 on the EMA bus and A16..15 on the bank select. Signal RAS (SDRAM BANKACTIVATE). Put column address 25..17 on the EMA bus and signal CAS. A26 is used to determine whether we are in the first 64MB or the second 64MB."
- note added: "This is Zorro 3 memory, so it is always treated as 32 bit memory and cannot be used by the Amiga 2000 chip set and cannot be used by anything on the Zorro 2 bus. It can only be used by the 68030."
- note removed: "JN Notes: put row address on the EMA bus and signal RAS. This is 68030 addresses A14:2. Put column address on the EMA bus and signal CAS. These are 68030 addresses A24:15."
- note removed: "This is Zorro 3 memory, so it is always treated as 32 bit memory and cannot be used by the Amiga 2000 chip set and cannot be used by anything on the Zoroo 2 bus. It can only be used by the 68030."
Changed lines of the file:
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@@
   (junction (at 105.41 148.59) (diameter 0) (color 0 0 0 0)
   )
+  (junction (at 71.12 191.77) (diameter 0) (color 0 0 0 0)
+  )
   (junction (at 115.57 57.15) (diameter 0) (color 0 0 0 0)
   )
@@
   (junction (at 105.41 219.71) (diameter 0) (color 0 0 0 0)
   )
+  (junction (at 67.31 194.31) (diameter 0) (color 0 0 0 0)
+  )
   (junction (at 107.95 57.15) (diameter 0) (color 0 0 0 0)
   )
@@
     (stroke (width 0) (type default) (color 0 0 0 0))
   )
-  (wire (pts (xy 156.21 252.73) (xy 30.48 252.73))
+  (wire (pts (xy 156.21 252.73) (xy 71.12 252.73))
     (stroke (width 0) (type default) (color 0 0 0 0))
   )
@@
     (stroke (width 0) (type default) (color 0 0 0 0))
   )
+  (wire (pts (xy 67.31 257.81) (xy 160.02 257.81))
+    (stroke (width 0) (type default) (color 0 0 0 0))
+  )
   (wire (pts (xy 100.33 57.15) (xy 102.87 57.15))
     (stroke (width 0) (type default) (color 0 0 0 0))
@@
     (stroke (width 0) (type default) (color 0 0 0 0))
   )
+  (wire (pts (xy 67.31 194.31) (xy 67.31 257.81))
+    (stroke (width 0) (type default) (color 0 0 0 0))
+  )
   (wire (pts (xy 209.55 219.71) (xy 212.09 219.71))
     (stroke (width 0) (type default) (color 0 0 0 0))
@@
     (stroke (width 0) (type default) (color 0 0 0 0))
   )
-  (wire (pts (xy 160.02 257.81) (xy 30.48 257.81))
-    (stroke (width 0) (type default) (color 0 0 0 0))
-  )
   (wire (pts (xy 320.675 90.805) (xy 314.325 90.805))
     (stroke (width 0) (type default) (color 0 0 0 0))
@@
     (stroke (width 0) (type default) (color 0 0 0 0))
   )
+  (wire (pts (xy 71.12 191.77) (xy 71.12 252.73))
+    (stroke (width 0) (type default) (color 0 0 0 0))
+  )
   (wire (pts (xy 229.87 86.36) (xy 236.22 86.36))
     (stroke (width 0) (type default) (color 0 0 0 0))
@@
     (effects (font (size 5.9944 5.9944)) (justify left bottom))
   )
-  (text "This is Zorro 3 memory, so it is always\ntreated as 32 bit memory and cannot be \nused by the Amiga 2000 chip set and cannot\nbe used by anything on the Zoroo 2 bus.\nIt can only be used by the 68030."
-    (at 274.955 155.575 0)
+  (text "This is Zorro 3 memory, so it is always\ntreated as 32 bit memory and cannot be \nused by the Amiga 2000 chip set and cannot\nbe used by anything on the Zorro 2 bus.\nIt can only be used by the 68030."
+    (at 146.685 37.465 0)
     (effects (font (size 3 3)) (justify left bottom))
   )
@@
     (effects (font (size 3.9878 3.9878)) (justify left bottom))
   )
-  (text "JN Notes: put row address on the EMA bus \nand signal RAS. This is 68030 addresses A14:2. \nPut column address on the EMA bus and signal \nCAS. These are 68030 addresses A24:15."
-    (at 274.32 132.08 0)
+  (text "JN Notes: put row addresses 14..2 on the EMA bus \nand A16..15 on the bank select. Signal RAS \n(SDRAM BANKACTIVATE). Put column address 25..17\non the EMA bus and signal CAS. A26 is used to \ndetermine whether we are in the first 64MB or\nthe second 64MB."
+    (at 273.05 147.955 0)
     (effects (font (size 2.9972 2.9972)) (justify left bottom))
   )
@@
     (effects (font (size 1.27 1.27)) (justify right bottom))
   )
-  (global_label "EM0B1" (shape input) (at 33.02 102.87 180) (fields_autoplaced)
-    (effects (font (size 1.27 1.27)) (justify right))
-    (property "Intersheet References" "${INTERSHEET_REFS}" (id 0) (at 0 0 0)
-      (effects (font (size 1.27 1.27)) hide)
-    )
-  )
-  (global_label "EM1B1" (shape input) (at 30.48 257.81 180) (fields_autoplaced)
+  (global_label "BANK1" (shape input) (at 33.02 102.87 180) (fields_autoplaced)
     (effects (font (size 1.27 1.27)) (justify right))
-    (property "Intersheet References" "${INTERSHEET_REFS}" (id 0) (at 0 0 0)
-      (effects (font (size 1.27 1.27)) hide)
+    (property "Intersheet References" "${INTERSHEET_REFS}" (id 0) (at 24.5272 102.7906 0)
+      (effects (font (size 1.27 1.27)) (justify right) hide)
     )
   )
@@
     )
   )
-  (global_label "EM1B0" (shape input) (at 30.48 252.73 180) (fields_autoplaced)
-    (effects (font (size 1.27 1.27)) (justify right))
-    (property "Intersheet References" "${INTERSHEET_REFS}" (id 0) (at 0 0 0)
-      (effects (font (size 1.27 1.27)) hide)
-    )
-  )
   (global_label "_RAS1" (shape input) (at 396.24 181.61 0) (fields_autoplaced)
     (effects (font (size 1.27 1.27)) (justify left))
@@
     )
   )
-  (global_label "EM0B0" (shape input) (at 33.02 100.33 180) (fields_autoplaced)
+  (global_label "BANK0" (shape input) (at 33.02 100.33 180) (fields_autoplaced)
     (effects (font (size 1.27 1.27)) (justify right))
-    (property "Intersheet References" "${INTERSHEET_REFS}" (id 0) (at 0 0 0)
-      (effects (font (size 1.27 1.27)) hide)
+    (property "Intersheet References" "${INTERSHEET_REFS}" (id 0) (at 24.5272 100.2506 0)
+      (effects (font (size 1.27 1.27)) (justify right) hide)
     )
   )
@@
     (in_bom yes) (on_board yes)
     (property "Reference" "U406" (id 0) (at 107.95 92.71 0))
-    (property "Value" "SDRAM_512Mb(32Mx16)" (id 1) (at 107.95 97.79 0))
+    (property "Value" "SDRAM_256Mb(16Mx16)" (id 1) (at 107.95 97.79 0))
     (property "Footprint" "Package_SO:TSOP-II-54_22.2x10.16mm_P0.8mm" (id 2) (at 107.95 92.71 0)
       (effects (font (size 1.27 1.27) italic) hide)
@@
     (in_bom yes) (on_board yes)
     (property "Reference" "U407" (id 0) (at 107.95 184.15 0))
-    (property "Value" "SDRAM_512Mb(32Mx16)" (id 1) (at 107.95 189.23 0))
+    (property "Value" "SDRAM_256Mb(16Mx16)" (id 1) (at 107.95 189.23 0))
     (property "Footprint" "Package_SO:TSOP-II-54_22.2x10.16mm_P0.8mm" (id 2) (at 107.95 184.15 0)
       (effects (font (size 1.27 1.27) italic) hide)
@@
     (in_bom yes) (on_board yes)
     (property "Reference" "U408" (id 0) (at 209.55 92.71 0))
-    (property "Value" "SDRAM_512Mb(32Mx16)" (id 1) (at 209.55 97.79 0))
+    (property "Value" "SDRAM_256Mb(16Mx16)" (id 1) (at 209.55 97.79 0))
     (property "Footprint" "Package_SO:TSOP-II-54_22.2x10.16mm_P0.8mm" (id 2) (at 209.55 92.71 0)
       (effects (font (size 1.27 1.27) italic) hide)
@@
     (in_bom yes) (on_board yes)
     (property "Reference" "U409" (id 0) (at 209.55 184.15 0))
-    (property "Value" "SDRAM_512Mb(32Mx16)" (id 1) (at 209.55 189.23 0))
+    (property "Value" "SDRAM_256Mb(16Mx16)" (id 1) (at 209.55 189.23 0))
     (property "Footprint" "Package_SO:TSOP-II-54_22.2x10.16mm_P0.8mm" (id 2) (at 209.55 184.15 0)
       (effects (font (size 1.27 1.27) italic) hide)

Commit message: Add files via upload
Connections:
- net EMA0: now also U406.26 (A3), U407.26 (A3), U408.31 (A6), U409.31 (A6); no longer U406.23 (A0), U407.23 (A0), U408.23 (A0), U409.23 (A0)
- net EMA1: now also U406.25 (A2), U407.25 (A2), U408.32 (A7), U409.32 (A7); no longer U406.24 (A1), U407.24 (A1), U408.24 (A1), U409.24 (A1)
- net EMA10: now also U406.33 (A8), U407.33 (A8), U408.29 (A4), U409.29 (A4); no longer U406.22 (A10), U407.22 (A10), U408.22 (A10), U409.22 (A10)
- net EMA11: now also U408.30 (A5), U409.30 (A5); no longer U408.35 (A11), U409.35 (A11)
- net EMA12: now also U408.24 (A1), U409.24 (A1); no longer U408.36 (A12), U409.36 (A12)
- net EMA2: now also U406.29 (A4), U407.29 (A4), U408.23 (A0), U409.23 (A0); no longer U406.25 (A2), U407.25 (A2), U408.25 (A2), U409.25 (A2)
- net EMA3: now also U406.30 (A5), U407.30 (A5), U408.22 (A10), U409.22 (A10); no longer U406.26 (A3), U407.26 (A3), U408.26 (A3), U409.26 (A3)
- net EMA4: now also U406.24 (A1), U407.24 (A1), U408.33 (A8), U409.33 (A8); no longer U406.29 (A4), U407.29 (A4), U408.29 (A4), U409.29 (A4)
- net EMA5: now also U406.23 (A0), U407.23 (A0), U408.35 (A11), U409.35 (A11); no longer U406.30 (A5), U407.30 (A5), U408.30 (A5), U409.30 (A5)
- net EMA6: now also U408.34 (A9), U409.34 (A9); no longer U408.31 (A6), U409.31 (A6)
- net EMA7: now also U408.36 (A12), U409.36 (A12); no longer U408.32 (A7), U409.32 (A7)
- net EMA8: now also U406.22 (A10), U407.22 (A10), U408.26 (A3), U409.26 (A3); no longer U406.33 (A8), U407.33 (A8), U408.33 (A8), U409.33 (A8)
- net EMA9: now also U408.25 (A2), U409.25 (A2); no longer U408.34 (A9), U409.34 (A9)
Changed lines of the file:
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@@
     (effects (font (size 2.9972 2.9972)) (justify left bottom))
   )
-  (label "EMA7" (at 182.88 175.26 0)
-    (effects (font (size 1.27 1.27)) (justify left bottom))
-  )
-  (label "EMA6" (at 182.88 81.28 0)
+  (label "EMA7" (at 182.88 187.96 0)
+    (effects (font (size 1.27 1.27)) (justify left bottom))
+  )
+  (label "EMA6" (at 182.88 88.9 0)
     (effects (font (size 1.27 1.27)) (justify left bottom))
   )
@@
     (effects (font (size 1.27 1.27)) (justify right bottom))
   )
-  (label "EMA1" (at 81.28 68.58 0)
+  (label "EMA1" (at 81.28 71.12 0)
     (effects (font (size 1.27 1.27)) (justify left bottom))
   )
@@
     (effects (font (size 1.27 1.27)) (justify left bottom))
   )
-  (label "EMA10" (at 182.88 91.44 0)
+  (label "EMA10" (at 182.88 76.2 0)
     (effects (font (size 1.27 1.27)) (justify left bottom))
   )
@@
     (effects (font (size 1.27 1.27)) (justify right bottom))
   )
-  (label "EMA5" (at 182.88 78.74 0)
+  (label "EMA5" (at 182.88 93.98 0)
     (effects (font (size 1.27 1.27)) (justify left bottom))
   )
@@
     (effects (font (size 1.27 1.27)) (justify right bottom))
   )
-  (label "EMA11" (at 182.88 185.42 0)
+  (label "EMA11" (at 182.88 170.18 0)
     (effects (font (size 1.27 1.27)) (justify left bottom))
   )
@@
     (effects (font (size 1.27 1.27)) (justify right bottom))
   )
-  (label "EMA9" (at 182.88 180.34 0)
+  (label "EMA9" (at 182.88 162.56 0)
     (effects (font (size 1.27 1.27)) (justify left bottom))
   )
@@
     (effects (font (size 1.27 1.27)) (justify left bottom))
   )
-  (label "EMA5" (at 81.28 170.18 0)
-    (effects (font (size 1.27 1.27)) (justify left bottom))
-  )
-  (label "EMA2" (at 81.28 71.12 0)
-    (effects (font (size 1.27 1.27)) (justify left bottom))
-  )
-  (label "EMA10" (at 81.28 182.88 0)
+  (label "EMA5" (at 81.28 157.48 0)
+    (effects (font (size 1.27 1.27)) (justify left bottom))
+  )
+  (label "EMA2" (at 81.28 76.2 0)
+    (effects (font (size 1.27 1.27)) (justify left bottom))
+  )
+  (label "EMA10" (at 81.28 177.8 0)
     (effects (font (size 1.27 1.27)) (justify left bottom))
   )
@@
     (effects (font (size 1.27 1.27)) (justify right bottom))
   )
-  (label "EMA4" (at 81.28 76.2 0)
+  (label "EMA4" (at 81.28 68.58 0)
     (effects (font (size 1.27 1.27)) (justify left bottom))
   )
@@
     (effects (font (size 1.27 1.27)) (justify right bottom))
   )
-  (label "EMA1" (at 182.88 160.02 0)
+  (label "EMA1" (at 182.88 175.26 0)
     (effects (font (size 1.27 1.27)) (justify left bottom))
   )
@@
     (effects (font (size 1.27 1.27)) (justify left bottom))
   )
-  (label "EMA0" (at 182.88 66.04 0)
-    (effects (font (size 1.27 1.27)) (justify left bottom))
-  )
-  (label "EMA12" (at 182.88 96.52 0)
+  (label "EMA0" (at 182.88 81.28 0)
+    (effects (font (size 1.27 1.27)) (justify left bottom))
+  )
+  (label "EMA12" (at 182.88 68.58 0)
     (effects (font (size 1.27 1.27)) (justify left bottom))
   )
@@
     (effects (font (size 1.27 1.27)) (justify right bottom))
   )
-  (label "EMA12" (at 182.88 187.96 0)
-    (effects (font (size 1.27 1.27)) (justify left bottom))
-  )
-  (label "EMA0" (at 81.28 66.04 0)
+  (label "EMA12" (at 182.88 160.02 0)
+    (effects (font (size 1.27 1.27)) (justify left bottom))
+  )
+  (label "EMA0" (at 81.28 73.66 0)
     (effects (font (size 1.27 1.27)) (justify left bottom))
   )
@@
     (effects (font (size 1.27 1.27)) (justify right bottom))
   )
-  (label "EMA7" (at 182.88 83.82 0)
+  (label "EMA7" (at 182.88 96.52 0)
     (effects (font (size 1.27 1.27)) (justify left bottom))
   )
@@
     (effects (font (size 1.27 1.27)) (justify right bottom))
   )
-  (label "EMA4" (at 182.88 76.2 0)
+  (label "EMA4" (at 182.88 86.36 0)
     (effects (font (size 1.27 1.27)) (justify left bottom))
   )
@@
     (effects (font (size 1.27 1.27)) (justify right bottom))
   )
-  (label "EMA4" (at 81.28 167.64 0)
+  (label "EMA4" (at 81.28 160.02 0)
     (effects (font (size 1.27 1.27)) (justify left bottom))
   )
@@
     (effects (font (size 1.27 1.27)) (justify right bottom))
   )
-  (label "EMA0" (at 182.88 157.48 0)
-    (effects (font (size 1.27 1.27)) (justify left bottom))
-  )
-  (label "EMA10" (at 182.88 182.88 0)
+  (label "EMA0" (at 182.88 172.72 0)
+    (effects (font (size 1.27 1.27)) (justify left bottom))
+  )
+  (label "EMA10" (at 182.88 167.64 0)
     (effects (font (size 1.27 1.27)) (justify left bottom))
   )
@@
     (effects (font (size 1.27 1.27)) (justify left bottom))
   )
-  (label "EMA5" (at 182.88 170.18 0)
+  (label "EMA5" (at 182.88 185.42 0)
     (effects (font (size 1.27 1.27)) (justify left bottom))
   )
@@
     (effects (font (size 1.27 1.27)) (justify right bottom))
   )
-  (label "EMA2" (at 182.88 71.12 0)
-    (effects (font (size 1.27 1.27)) (justify left bottom))
-  )
-  (label "EMA8" (at 81.28 86.36 0)
+  (label "EMA2" (at 182.88 66.04 0)
+    (effects (font (size 1.27 1.27)) (justify left bottom))
+  )
+  (label "EMA8" (at 81.28 91.44 0)
     (effects (font (size 1.27 1.27)) (justify left bottom))
   )
@@
     (effects (font (size 1.27 1.27)) (justify right bottom))
   )
-  (label "EMA3" (at 81.28 165.1 0)
+  (label "EMA3" (at 81.28 170.18 0)
     (effects (font (size 1.27 1.27)) (justify left bottom))
   )
@@
     (effects (font (size 1.27 1.27)) (justify right bottom))
   )
-  (label "EMA2" (at 182.88 162.56 0)
-    (effects (font (size 1.27 1.27)) (justify left bottom))
-  )
-  (label "EMA10" (at 81.28 91.44 0)
+  (label "EMA2" (at 182.88 157.48 0)
+    (effects (font (size 1.27 1.27)) (justify left bottom))
+  )
+  (label "EMA10" (at 81.28 86.36 0)
     (effects (font (size 1.27 1.27)) (justify left bottom))
   )
@@
     (effects (font (size 1.27 1.27)) (justify left bottom))
   )
-  (label "EMA8" (at 182.88 86.36 0)
+  (label "EMA8" (at 182.88 73.66 0)
     (effects (font (size 1.27 1.27)) (justify left bottom))
   )
@@
     (effects (font (size 1.27 1.27)) (justify left bottom))
   )
-  (label "EMA4" (at 182.88 167.64 0)
+  (label "EMA4" (at 182.88 177.8 0)
     (effects (font (size 1.27 1.27)) (justify left bottom))
   )
@@
     (effects (font (size 1.27 1.27)) (justify right bottom))
   )
-  (label "EMA2" (at 81.28 162.56 0)
+  (label "EMA2" (at 81.28 167.64 0)
     (effects (font (size 1.27 1.27)) (justify left bottom))
   )
@@
     (effects (font (size 1.27 1.27)) (justify left bottom))
   )
-  (label "EMA5" (at 81.28 78.74 0)
+  (label "EMA5" (at 81.28 66.04 0)
     (effects (font (size 1.27 1.27)) (justify left bottom))
   )
@@
     (effects (font (size 1.27 1.27)) (justify left bottom))
   )
-  (label "EMA8" (at 182.88 177.8 0)
+  (label "EMA8" (at 182.88 165.1 0)
     (effects (font (size 1.27 1.27)) (justify left bottom))
   )
@@
     (effects (font (size 1.27 1.27)) (justify right bottom))
   )
-  (label "EMA1" (at 81.28 160.02 0)
-    (effects (font (size 1.27 1.27)) (justify left bottom))
-  )
-  (label "EMA9" (at 182.88 88.9 0)
-    (effects (font (size 1.27 1.27)) (justify left bottom))
-  )
-  (label "EMA0" (at 81.28 157.48 0)
+  (label "EMA1" (at 81.28 162.56 0)
+    (effects (font (size 1.27 1.27)) (justify left bottom))
+  )
+  (label "EMA9" (at 182.88 71.12 0)
+    (effects (font (size 1.27 1.27)) (justify left bottom))
+  )
+  (label "EMA0" (at 81.28 165.1 0)
     (effects (font (size 1.27 1.27)) (justify left bottom))
   )
@@
     (effects (font (size 1.27 1.27)) (justify right bottom))
   )
-  (label "EMA8" (at 81.28 177.8 0)
+  (label "EMA8" (at 81.28 182.88 0)
     (effects (font (size 1.27 1.27)) (justify left bottom))
   )
@@
     (effects (font (size 1.27 1.27)) (justify left bottom))
   )
-  (label "EMA3" (at 182.88 165.1 0)
+  (label "EMA3" (at 182.88 182.88 0)
     (effects (font (size 1.27 1.27)) (justify left bottom))
   )
@@
     (effects (font (size 1.27 1.27)) (justify left bottom))
   )
-  (label "EMA11" (at 182.88 93.98 0)
+  (label "EMA11" (at 182.88 78.74 0)
     (effects (font (size 1.27 1.27)) (justify left bottom))
   )
@@
     (effects (font (size 1.27 1.27)) (justify left bottom))
   )
-  (label "EMA3" (at 182.88 73.66 0)
+  (label "EMA3" (at 182.88 91.44 0)
     (effects (font (size 1.27 1.27)) (justify left bottom))
   )
@@
     (effects (font (size 1.27 1.27)) (justify left bottom))
   )
-  (label "EMA1" (at 182.88 68.58 0)
-    (effects (font (size 1.27 1.27)) (justify left bottom))
-  )
-  (label "EMA3" (at 81.28 73.66 0)
-    (effects (font (size 1.27 1.27)) (justify left bottom))
-  )
-  (label "EMA6" (at 182.88 172.72 0)
-    (effects (font (size 1.27 1.27)) (justify left bottom))
-  )
+  (label "EMA1" (at 182.88 83.82 0)
+    (effects (font (size 1.27 1.27)) (justify left bottom))
+  )
+  (label "EMA3" (at 81.28 78.74 0)
+    (effects (font (size 1.27 1.27)) (justify left bottom))
+  )
+  (label "EMA6" (at 182.88 180.34 0)
+    (effects (font (size 1.27 1.27)) (justify left bottom))
+  )

Commit message: Add files via upload
Connections:
- net D16: no longer U407.2 (DQ0), U409.2 (DQ0)
- net D17: no longer U407.4 (DQ1), U409.4 (DQ1)
- net D18: no longer U407.5 (DQ2), U409.5 (DQ2)
- net D19: no longer U407.7 (DQ3), U409.7 (DQ3)
- net D20: no longer U407.8 (DQ4), U409.8 (DQ4)
- net D21: no longer U407.10 (DQ5), U409.10 (DQ5)
- net D22: no longer U407.11 (DQ6), U409.11 (DQ6)
- net D23: no longer U407.13 (DQ7), U409.13 (DQ7)
- net D24: no longer U407.42 (DQ8), U409.42 (DQ8)
- net D25: no longer U407.44 (DQ9), U409.44 (DQ9)
- net D26: no longer U407.45 (DQ10), U409.45 (DQ10)
- net D27: no longer U407.47 (DQ11), U409.47 (DQ11)
- net D28: no longer U407.48 (DQ12), U409.48 (DQ12)
- net D29: no longer U407.50 (DQ13), U409.50 (DQ13)
- net D30: no longer U407.51 (DQ14), U409.51 (DQ14)
- net D31: no longer U407.53 (DQ15), U409.53 (DQ15)
- net D0 renamed EMD0
- net D1 renamed EMD1
- net D10 renamed EMD10
- net D11 renamed EMD11
- net D12 renamed EMD12
- net D13 renamed EMD13
- net D14 renamed EMD14
- net D15 renamed EMD15
- net D2 renamed EMD2
- net D3 renamed EMD3
- net D4 renamed EMD4
- net D5 renamed EMD5
- net D6 renamed EMD6
- net D7 renamed EMD7
- net D8 renamed EMD8
- net D9 renamed EMD9
- new net EMD16: U407.2 (DQ0), U409.2 (DQ0)
- new net EMD17: U407.4 (DQ1), U409.4 (DQ1)
- new net EMD18: U407.5 (DQ2), U409.5 (DQ2)
- new net EMD19: U407.7 (DQ3), U409.7 (DQ3)
- new net EMD20: U407.8 (DQ4), U409.8 (DQ4)
- new net EMD21: U407.10 (DQ5), U409.10 (DQ5)
- new net EMD22: U407.11 (DQ6), U409.11 (DQ6)
- new net EMD23: U407.13 (DQ7), U409.13 (DQ7)
- new net EMD24: U407.42 (DQ8), U409.42 (DQ8)
- new net EMD25: U407.44 (DQ9), U409.44 (DQ9)
- new net EMD26: U407.45 (DQ10), U409.45 (DQ10)
- new net EMD27: U407.47 (DQ11), U409.47 (DQ11)
- new net EMD28: U407.48 (DQ12), U409.48 (DQ12)
- new net EMD29: U407.50 (DQ13), U409.50 (DQ13)
- new net EMD30: U407.51 (DQ14), U409.51 (DQ14)
- new net EMD31: U407.53 (DQ15), U409.53 (DQ15)

Commit message: Add files via upload
Other:
- note added: "HIGH_WORD"
- note added: "LOW_WORD"
- note added: "ZORRO 3 MEMORY"
- note removed: "EXPANDED MEMORY"
- note removed: "HIGH_BYTE"
- note removed: "LOW_BYTE"
Changed lines of the file:
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@@
     (stroke (width 0) (type default) (color 0 0 0 0))
   )
-  (text "EXPANDED MEMORY" (at 314.96 245.11 0)
+  (text "ZORRO 3 MEMORY" (at 314.96 245.11 0)
     (effects (font (size 5.9944 5.9944)) (justify left bottom))
   )
@@
     (effects (font (size 3 3)) (justify left bottom))
   )
-  (text "LOW_BYTE" (at 24.13 81.28 0)
+  (text "LOW_WORD" (at 24.13 81.28 0)
     (effects (font (size 2.9972 2.9972)) (justify left bottom))
   )
@@
     (effects (font (size 2.9972 2.9972)) (justify left bottom))
   )
-  (text "HIGH_BYTE" (at 24.13 180.975 0)
+  (text "HIGH_WORD" (at 24.13 180.975 0)
     (effects (font (size 2.9972 2.9972)) (justify left bottom))
   )

Commit message: Add files via upload
Parts:
- added C422, C423, C424, C425: 0.33uF, Capacitor_SMD:C_0805_2012Metric, symbol Device:C
Connections:
- net +3V3: now also C422.1, C423.1, C424.1, C425.1
- net GND: now also C422.2, C423.2, C424.2, C425.2
Other:
- moved on the sheet: C102, C103, C406, C407, C408, C409, C410, C411, C412, C413

Commit message: Add files via upload
Parts:
- added C426: 0.33uF, Capacitor_SMD:C_0805_2012Metric, symbol Device:C
Connections:
- net +3V3: now also C426.1
- net GND: now also C426.2
Other:
- moved on the sheet: C406, C407, C408, C409, C410, C411, C412, C413, C422, C423, C424, C425
