File: A2630-New-KiCAD/CPLD1.kicad_sch (KiCad schematic)
At the start: 17 parts, among them CN1 CPLD0, CN2 CPLD1, CN3 CPLD1, U600 XC9572XL-TQ100, U601 XC9572XL-TQ100, U602 XC9572XL-TQ100

Commit message: Add files via upload
Connections:
- net A22: now also U602.59 (P59)
- net A23: now also U602.60 (P60)
- net A24: now also U602.61 (P61)
- net A25: now also U602.63 (P63)
- net A26: now also U602.64 (P64)
- net A27: now also U602.65 (P65)
- net A28: now also U602.66 (P66)
- net A29: now also U602.67 (P67)
- net A30: now also U602.68 (P68)
- net A31: now also U602.70 (P70)
- net CPUCLK_A: now also U602.81 (P81)
- net _GRESET: now also U602.82 (P82)

Commit message: Add files via upload
Parts:
- added C607, C608, C609: 0.22uF, Capacitor_SMD:C_0805_2012Metric, symbol Device:C
Connections:
- net +3V3: now also C607.1, C608.1, C609.1
- net GND: now also C607.2, C608.2, C609.2
- no-connect marks 18 -> 22

Commit message: Add files via upload
Connections:
- net RESENB renamed RSTENB
Changed lines of the file:
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@@
     )
   )
-  (global_label "RESENB" (shape input) (at 110.49 170.815 0) (fields_autoplaced)
+  (global_label "RSTENB" (shape input) (at 110.49 170.815 0) (fields_autoplaced)
     (effects (font (size 1.27 1.27)) (justify left))
-    (property "Intersheet References" "${INTERSHEET_REFS}" (id 0) (at 0 0 0)
-      (effects (font (size 1.27 1.27)) hide)
+    (property "Intersheet References" "${INTERSHEET_REFS}" (id 0) (at 120.0109 170.7356 0)
+      (effects (font (size 1.27 1.27)) (justify left) hide)
     )
   )

Commit message: Add files via upload
Parts:
- removed R703: 47, Resistor_SMD:R_0805_2012Metric, symbol Device:R
Connections:
- net SN7MDIS is gone; now on net JMODE: U600.95 (P95)
- net _OE1 is gone; now on net _CPURESET: U601.14 (P14)
- net _WE1 is gone; now on net _MEMLOCK: U601.16 (P16)
- net A0: now also U601.63 (P63); no longer U601.32 (P32)
- net A1: now also U601.64 (P64); no longer U601.35 (P35)
- net A13: now also U601.71 (P71); no longer U601.52 (P52)
- net A14: now also U601.72 (P72); no longer U601.53 (P53)
- net A15: now also U601.74 (P74); no longer U601.54 (P54)
- net A16: now also U601.76 (P76); no longer U601.55 (P55)
- net A17: now also U601.77 (P77); no longer U601.56 (P56)
- net A18: now also U601.78 (P78); no longer U601.58 (P58)
- net A19: now also U601.79 (P79); no longer U601.59 (P59)
- net A2: now also U601.65 (P65); no longer U601.37 (P37)
- net A20: now also U601.81 (P81); no longer U601.60 (P60)
- net A21: now also U601.82 (P82); no longer U601.61 (P61)
- net A22: now also U601.85 (P85); no longer U601.63 (P63)
- net A23: now also U601.86 (P86); no longer U601.64 (P64)
- net A3: now also U601.66 (P66); no longer U601.41 (P41)
- net A4: now also U601.67 (P67); no longer U601.42 (P42)
- net A5: now also U601.68 (P68); no longer U601.49 (P49)
- net A6: now also U601.70 (P70); no longer U601.50 (P50)
- net AR_W: now also U601.36 (P36); no longer U601.79 (P79)
- net CPUCLK_A: now also U601.15 (P15); no longer U601.87 (P87)
- net D28: now also U601.8 (P8); no longer U601.65 (P65)
- net D29: now also U601.9 (P9); no longer U601.66 (P66)
- net D30: now also U601.10 (P10); no longer U601.67 (P67)
- net D31: now also U601.11 (P11); no longer U601.68 (P68)
- net EMDDIR: now also U601.54 (P54); no longer U601.23 (I/O/GCK2)
- net EXTSEL: now also U601.3 (I/O/GTS1); no longer U601.25 (P25)
- net FC0: now also U601.89 (P89); no longer U601.72 (P72)
- net FC1: now also U601.90 (P90); no longer U601.71 (P71)
- net FC2: now also U601.91 (P91); no longer U601.70 (P70)
- net JMODE: no longer U600.77 (P77)
- net MODE68K: now also U600.96 (P96); no longer U600.81 (P81)
- net OSMODE: now also U601.42 (P42); no longer U601.94 (P94)
- net PHANTOMHI: now also U601.6 (P6); no longer U601.91 (P91)
- net PHANTOMLO: now also U601.4 (I/O/GTS2); no longer U601.92 (P92)
- net ROMCLK: now also U601.99 (I/O/GSR); no longer U601.36 (P36)
- net RSTENB: now also U600.94 (P94); no longer U600.86 (P86)
- net R_W: now also U601.95 (P95); no longer U601.85 (P85)
- net SIZ0: now also U601.52 (P52); no longer U601.74 (P74)
- net SIZ1: now also U601.53 (P53); no longer U601.76 (P76)
- net _AS: now also U601.94 (P94); no longer U601.81 (P81)
- net _ASEN: now also U601.18 (P18); no longer U601.8 (P8)
- net _AVEC: now also U601.92 (P92); no longer U601.11 (P11)
- net _BERR: now also U601.13 (P13); no longer U601.78 (P78)
- net _BGACK: now also U601.1 (I/O/GTS3); no longer U601.86 (P86)
- net _CIIN: now also U601.87 (P87); no longer U601.97 (P97)
- net _CSROM: now also U601.97 (P97); no longer U601.90 (P90)
- net _CYCEND: now also U600.6 (P6), U601.25 (P25); no longer U601.10 (P10)
- net _DS: now also U601.93 (P93); no longer U601.82 (P82)
- net _DSEN: now also U601.20 (P20); no longer U601.6 (P6)
- net _EXTERN: now also U601.23 (I/O/GCK2); no longer U601.9 (P9)
- net _FPUCS: now also U601.96 (P96); no longer U601.77 (P77)
- net _LLBE: now also U601.55 (P55); no longer U601.22 (I/O/GCK1)
- net _LMBE: now also U601.56 (P56); no longer U601.20 (P20)
- net _MEMLOCK: no longer U601.12 (P12)
- net _MEMSEL: now also U601.17 (P17); no longer U601.96 (P96)
- net _OE0: now also U601.60 (P60); no longer U601.13 (P13)
- net _ONBOARD: now also U601.41 (P41); no longer U601.95 (P95)
- net _REGRESET: now also U600.97 (P97); no longer U600.58 (P58)
- net _RESET: no longer U601.93 (P93)
- net _S7MDISD: no longer U600.96 (P96)
- net _SENSE: now also U601.12 (P12); no longer U601.89 (P89)
- net _UMBE: now also U601.58 (P58); no longer U601.18 (P18)
- net _UUBE: now also U601.59 (P59); no longer U601.17 (P17)
- net _WE0: now also U601.61 (P61); no longer U601.15 (P15)
- net at R701.1: no longer U600.94 (P94)
- net at R705.1: no longer U600.97 (P97)
- no-connect marks 22 -> 17
Other:
- moved on the sheet: R701, R705

Commit message: Add files via upload
Connections:
- net AR_W: now also U601.27 (I/O/GCK3); no longer U601.36 (P36)
- net CONFIGED: now also U601.28 (P28); no longer U601.30 (P30)
- net OSMODE: now also U601.50 (P50); no longer U601.42 (P42)
- net TCK1: now also CN2.1 (Pin_1); no longer CN2.3 (Pin_3), CN3.1 (Pin_1), U602.48 (TCK)
- net TDI1: now also CN2.3 (Pin_3); no longer CN2.1 (Pin_1), CN3.3 (Pin_3), U602.45 (TDI)
- net TDO1: no longer CN3.4 (Pin_4), U602.83 (TDO)
- net TMS1: no longer CN3.2 (Pin_2), U602.47 (TMS)
- net TRISTATE: now also U601.29 (P29); no longer U601.33 (P33)
- net TWOMB: now also U601.39 (P39); no longer U601.28 (P28)
- net Z2AUTO: now also U601.40 (P40); no longer U601.29 (P29)
- net _ASEN: now also U601.17 (P17); no longer U601.18 (P18)
- net _CYCEND: no longer U600.6 (P6)
- net _LDS: now also U601.33 (P33); no longer U601.40 (P40)
- net _MEMSEL: now also U601.18 (P18); no longer U601.17 (P17)
- net _ONBOARD: now also U601.36 (P36); no longer U601.41 (P41)
- net _UDS: now also U601.30 (P30); no longer U601.39 (P39)
- new net TCK2: CN3.1 (Pin_1), U602.48 (TCK)
- new net TDI2: CN3.3 (Pin_3), U602.45 (TDI)
- new net TDO2: CN3.4 (Pin_4), U602.83 (TDO)
- new net TMS2: CN3.2 (Pin_2), U602.47 (TMS)
- no-connect marks 17 -> 18

Commit message: Add files via upload
Connections:
- net CDAC is gone; now on net _STERM: U600.87 (P87)
- net A1: now also U600.89 (P89); no longer U600.59 (P59)
- net A7M: now also U600.54 (P54); no longer U600.10 (P10)
- net ADDIR: now also U600.13 (P13); no longer U600.37 (P37)
- net AR_W: now also U600.52 (P52), U601.28 (P28); no longer U600.14 (P14), U601.27 (I/O/GCK3)
- net B2000: now also U600.42 (P42); no longer U600.82 (P82)
- net CONFIGED: now also U600.50 (P50), U601.27 (I/O/GCK3); no longer U600.33 (P33), U601.28 (P28)
- net CPUCLK_A: now also U600.67 (P67); no longer U600.91 (P91)
- net DRSEL: now also U600.14 (P14); no longer U600.35 (P35)
- net E: now also U600.36 (P36); no longer U600.61 (P61)
- net EXTSEL: now also U600.70 (P70); no longer U600.79 (P79)
- net FC0: now also U600.74 (P74); no longer U600.67 (P67)
- net FC1: now also U600.72 (P72); no longer U600.66 (P66)
- net FC2: now also U600.71 (P71); no longer U600.65 (P65)
- net MEMACCESS: now also U600.55 (P55), U601.41 (P41); no longer U600.30 (P30)
- net R_W: now also U600.86 (P86); no longer U600.15 (P15)
- net TCK0: now also CN1.1 (Pin_1); no longer CN1.3 (Pin_3)
- net TDI0: now also CN1.3 (Pin_3); no longer CN1.1 (Pin_1)
- net TRISTATE: now also U600.49 (P49); no longer U600.74 (P74)
- net _AAS: now also U600.22 (I/O/GCK1); no longer U600.20 (P20)
- net _ABG: now also U600.29 (P29); no longer U600.16 (P16)
- net _ABGACK: now also U600.30 (P30); no longer U600.17 (P17)
- net _ABR: now also U600.33 (P33); no longer U600.25 (P25)
- net _ADOEH: now also U600.15 (P15); no longer U600.42 (P42)
- net _ADOEL: now also U600.20 (P20); no longer U600.41 (P41)
- net _AS: now also U600.85 (P85); no longer U600.13 (P13)
- net _ASDELAY: now also U600.8 (P8); no longer U600.28 (P28)
- net _ASEN: now also U600.66 (P66); no longer U600.18 (P18)
- net _BGDIS: now also U600.58 (P58); no longer U600.56 (P56)
- net _BOSS: now also U600.6 (P6); no longer U600.76 (P76)
- net _C1: now also U600.17 (P17); no longer U600.11 (P11)
- net _C3: now also U600.18 (P18); no longer U600.12 (P12)
- net _CPURESET: now also U600.68 (P68); no longer U600.85 (P85)
- net _CYCEND: now also U600.60 (P60); no longer U600.52 (P52)
- net _DSACK0: now also U600.93 (P93); no longer U600.55 (P55)
- net _DSACK1: now also U600.92 (P92); no longer U600.54 (P54)
- net _DSACKDIS: now also U600.9 (P9); no longer U600.60 (P60)
- net _DSACKEN: now also U600.11 (P11); no longer U600.63 (P63)
- net _DSEN: now also U600.61 (P61), U601.23 (I/O/GCK2); no longer U600.29 (P29), U601.20 (P20)
- net _DTACK: now also U600.28 (P28); no longer U600.72 (P72)
- net _EXTERN: now also U600.65 (P65), U601.18 (P18); no longer U600.71 (P71), U601.23 (I/O/GCK2)
- net _IVMA: now also U600.41 (P41); no longer U600.70 (P70)
- net _LDS: now also U600.25 (P25); no longer U600.39 (P39)
- net _MEMSEL: now also U600.64 (P64), U601.20 (P20); no longer U600.50 (P50), U601.18 (P18)
- net _ONBOARD: now also U600.63 (P63), U601.22 (I/O/GCK1); no longer U600.64 (P64), U601.36 (P36)
- net _OVR: now also U600.39 (P39); no longer U600.49 (P49)
- net _RESET: now also U600.35 (P35); no longer U600.89 (P89)
- net _S7MDIS: now also U600.4 (I/O/GTS2); no longer U600.9 (P9)
- net _S7MDISD: now also U600.1 (I/O/GTS3)
- net _STERM: no longer U600.53 (P53)
- net _UDS: now also U600.23 (I/O/GCK2); no longer U600.36 (P36)
- net _VPA: now also U600.37 (P37); no longer U600.78 (P78)
- net at U600.3 (I/O/GTS1): now also R701.1
- net at R704.1: now also U600.10 (P10); no longer U600.8 (P8)
- net at R702.1: now also U600.16 (P16); no longer U600.92 (P92)
- net at R705.1: now also U600.12 (P12)
- new net _CDAC: U600.53 (P53)
- no-connect marks 18 -> 8
Other:
- moved on the sheet: R701, R702, R704, R705

Commit message: Add files via upload
Connections:
- net EMDDIR: now also U601.61 (P61); no longer U601.54 (P54)
- net SIZ0: now also U601.59 (P59); no longer U601.52 (P52)
- net SIZ1: now also U601.60 (P60); no longer U601.53 (P53)
- net _LLBE: now also U601.54 (P54); no longer U601.55 (P55)
- net _LMBE: now also U601.53 (P53); no longer U601.56 (P56)
- net _OE0: now also U601.52 (P52); no longer U601.60 (P60)
- net _UMBE: now also U601.56 (P56); no longer U601.58 (P58)
- net _UUBE: now also U601.55 (P55); no longer U601.59 (P59)
- net _WE0: now also U601.58 (P58); no longer U601.61 (P61)
Changed lines of the file:
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@@
     )
   )
-  (global_label "_UMBE" (shape output) (at 228.6 114.935 0) (fields_autoplaced)
-    (effects (font (size 1.27 1.27)) (justify left))
-    (property "Intersheet References" "${INTERSHEET_REFS}" (id 0) (at 388.62 212.09 0)
+  (global_label "_UMBE" (shape output) (at 228.6 112.395 0) (fields_autoplaced)
+    (effects (font (size 1.27 1.27)) (justify left))
+    (property "Intersheet References" "${INTERSHEET_REFS}" (id 0) (at 388.62 209.55 0)
       (effects (font (size 1.27 1.27)) hide)
     )
@@
     )
   )
-  (global_label "SIZ1" (shape input) (at 228.6 104.775 0) (fields_autoplaced)
-    (effects (font (size 1.27 1.27)) (justify left))
-    (property "Intersheet References" "${INTERSHEET_REFS}" (id 0) (at 0 -48.26 0)
+  (global_label "SIZ1" (shape input) (at 228.6 120.015 0) (fields_autoplaced)
+    (effects (font (size 1.27 1.27)) (justify left))
+    (property "Intersheet References" "${INTERSHEET_REFS}" (id 0) (at 0 -33.02 0)
       (effects (font (size 1.27 1.27)) hide)
     )
@@
     )
   )
-  (global_label "_OE0" (shape output) (at 228.6 120.015 0) (fields_autoplaced)
-    (effects (font (size 1.27 1.27)) (justify left))
-    (property "Intersheet References" "${INTERSHEET_REFS}" (id 0) (at 388.62 204.47 0)
+  (global_label "_OE0" (shape output) (at 228.6 102.235 0) (fields_autoplaced)
+    (effects (font (size 1.27 1.27)) (justify left))
+    (property "Intersheet References" "${INTERSHEET_REFS}" (id 0) (at 388.62 186.69 0)
       (effects (font (size 1.27 1.27)) hide)
     )
@@
     )
   )
-  (global_label "EMDDIR" (shape output) (at 228.6 107.315 0) (fields_autoplaced)
-    (effects (font (size 1.27 1.27)) (justify left))
-    (property "Intersheet References" "${INTERSHEET_REFS}" (id 0) (at 237.9394 107.2356 0)
+  (global_label "EMDDIR" (shape output) (at 228.6 122.555 0) (fields_autoplaced)
+    (effects (font (size 1.27 1.27)) (justify left))
+    (property "Intersheet References" "${INTERSHEET_REFS}" (id 0) (at 237.9394 122.4756 0)
       (effects (font (size 1.27 1.27)) (justify left) hide)
     )
@@
     )
   )
-  (global_label "_LLBE" (shape output) (at 228.6 109.855 0) (fields_autoplaced)
-    (effects (font (size 1.27 1.27)) (justify left))
-    (property "Intersheet References" "${INTERSHEET_REFS}" (id 0) (at 388.62 212.09 0)
+  (global_label "_LLBE" (shape output) (at 228.6 107.315 0) (fields_autoplaced)
+    (effects (font (size 1.27 1.27)) (justify left))
+    (property "Intersheet References" "${INTERSHEET_REFS}" (id 0) (at 388.62 209.55 0)
       (effects (font (size 1.27 1.27)) hide)
     )
@@
     )
   )
-  (global_label "SIZ0" (shape input) (at 228.6 102.235 0) (fields_autoplaced)
-    (effects (font (size 1.27 1.27)) (justify left))
-    (property "Intersheet References" "${INTERSHEET_REFS}" (id 0) (at 0 -48.26 0)
+  (global_label "SIZ0" (shape input) (at 228.6 117.475 0) (fields_autoplaced)
+    (effects (font (size 1.27 1.27)) (justify left))
+    (property "Intersheet References" "${INTERSHEET_REFS}" (id 0) (at 0 -33.02 0)
       (effects (font (size 1.27 1.27)) hide)
     )
@@
     )
   )
-  (global_label "_LMBE" (shape output) (at 228.6 112.395 0) (fields_autoplaced)
-    (effects (font (size 1.27 1.27)) (justify left))
-    (property "Intersheet References" "${INTERSHEET_REFS}" (id 0) (at 388.62 212.09 0)
+  (global_label "_LMBE" (shape output) (at 228.6 104.775 0) (fields_autoplaced)
+    (effects (font (size 1.27 1.27)) (justify left))
+    (property "Intersheet References" "${INTERSHEET_REFS}" (id 0) (at 388.62 204.47 0)
       (effects (font (size 1.27 1.27)) hide)
     )
@@
     )
   )
-  (global_label "_WE0" (shape output) (at 228.6 122.555 0) (fields_autoplaced)
-    (effects (font (size 1.27 1.27)) (justify left))
-    (property "Intersheet References" "${INTERSHEET_REFS}" (id 0) (at 388.62 212.09 0)
+  (global_label "_WE0" (shape output) (at 228.6 114.935 0) (fields_autoplaced)
+    (effects (font (size 1.27 1.27)) (justify left))
+    (property "Intersheet References" "${INTERSHEET_REFS}" (id 0) (at 388.62 204.47 0)
       (effects (font (size 1.27 1.27)) hide)
     )
@@
     )
   )
-  (global_label "_UUBE" (shape output) (at 228.6 117.475 0) (fields_autoplaced)
-    (effects (font (size 1.27 1.27)) (justify left))
-    (property "Intersheet References" "${INTERSHEET_REFS}" (id 0) (at 388.62 212.09 0)
-      (effects (font (size 1.27 1.27)) hide)
-    )
+  (global_label "_UUBE" (shape output) (at 228.6 109.855 0) (fields_autoplaced)
+    (effects (font (size 1.27 1.27)) (justify left))
+    (property "Intersheet References" "${INTERSHEET_REFS}" (id 0) (at 388.62 204.47 0)
+      (effects (font (size 1.27 1.27)) hide)
+    )

Commit message: Add files via upload
Parts:
- CN3: value CPLD1 -> CPLD2
Connections:
- no-connect marks 8 -> 20
