File: A2630-New-KiCAD/Power.kicad_sch (KiCad schematic)
At the start: 22 parts, among them U204 74HCT04, U300 74HCT05, U307 74HCT04, U606 74HCT244, U800 LM1117-3.3

Commit message: Add files via upload
Parts:
- added unit 5 of U307
- added unit 6 of U307
- added U507: 74HCT74, Package_SO:SOIC-14_3.9x8.7mm_P1.27mm, symbol 74xx:74LS74
Connections:
- net +5V: now also U507.10 (~{S}), U507.13 (~{R})
- net GND: now also U307.11, U307.13, U507.11 (C), U507.12 (D)
- no-connect marks 8 -> 12
Other:
- moved on the sheet: U204D, U300F, U307A, U307D, U606E, U606F, U606G, U606H

Commit message: Add files via upload
Parts:
- added H1, H2: MountingHole, MountingHole:MountingHole_3.2mm_M3_Pad, symbol Mechanical:MountingHole_Pad
Connections:
- net GND: now also H1.1, H2.1
Other:
- note added: "MOUNTING HOLES"
Changed lines of the file:
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@@
   (junction (at 159.385 33.655) (diameter 0) (color 0 0 0 0)
+  )
+  (junction (at 38.735 72.39) (diameter 0) (color 0 0 0 0)
   )
   (junction (at 81.915 34.925) (diameter 0) (color 0 0 0 0)
@@
     (stroke (width 0) (type default) (color 0 0 0 0))
   )
+  (wire (pts (xy 38.735 66.675) (xy 38.735 72.39))
+    (stroke (width 0) (type default) (color 0 0 0 0))
+  )
   (wire (pts (xy 151.765 41.275) (xy 144.145 41.275))
     (stroke (width 0) (type default) (color 0 0 0 0))
@@
     (stroke (width 0) (type default) (color 0 0 0 0))
   )
+  (polyline (pts (xy 66.675 86.995) (xy 66.675 55.88))
+    (stroke (width 0) (type default) (color 0 0 0 0))
+  )
   (polyline (pts (xy 23.495 20.955) (xy 23.495 52.705))
     (stroke (width 0) (type default) (color 0 0 0 0))
@@
     (stroke (width 0) (type default) (color 0 0 0 0))
   )
+  (polyline (pts (xy 23.495 86.995) (xy 66.675 86.995))
+    (stroke (width 0) (type default) (color 0 0 0 0))
+  )
   (wire (pts (xy 159.385 33.655) (xy 151.765 33.655))
     (stroke (width 0) (type default) (color 0 0 0 0))
   )
+  (polyline (pts (xy 23.495 55.88) (xy 23.495 86.995))
+    (stroke (width 0) (type default) (color 0 0 0 0))
+  )
   (wire (pts (xy 233.68 80.645) (xy 233.68 67.31))
     (stroke (width 0) (type default) (color 0 0 0 0))
@@
     (stroke (width 0) (type default) (color 0 0 0 0))
   )
+  (polyline (pts (xy 23.495 55.88) (xy 66.675 55.88))
+    (stroke (width 0) (type default) (color 0 0 0 0))
+  )
   (wire (pts (xy 189.865 33.655) (xy 203.835 33.655))
     (stroke (width 0) (type default) (color 0 0 0 0))
@@
   )
   (wire (pts (xy 114.3 41.275) (xy 121.92 41.275))
+    (stroke (width 0) (type default) (color 0 0 0 0))
+  )
+  (wire (pts (xy 38.735 72.39) (xy 38.735 78.74))
     (stroke (width 0) (type default) (color 0 0 0 0))
   )
@@
   (text "POWER AND SPARES" (at 179.07 176.53 0)
     (effects (font (size 5.9944 5.9944)) (justify left bottom))
+  )
+  (text "MOUNTING HOLES" (at 24.765 62.865 0)
+    (effects (font (size 3 3)) (justify left bottom))
   )
   (text "Come on down!" (at 211.455 164.465 180)
@@
     (pin "11")
   )
+  (symbol (lib_id "power:GND") (at 38.735 78.74 0) (unit 1)
+    (in_bom yes) (on_board yes) (fields_autoplaced)
+    (property "Reference" "#PWR0197" (id 0) (at 38.735 85.09 0)
+      (effects (font (size 1.27 1.27)) hide)
+    )
+    (property "Value" "GND" (id 1) (at 38.735 83.1834 0))
+    (property "Footprint" "" (id 2) (at 38.735 78.74 0)
+      (effects (font (size 1.27 1.27)) hide)
+    )
+    (property "Datasheet" "" (id 3) (at 38.735 78.74 0)
+      (effects (font (size 1.27 1.27)) hide)
+    )
+    (pin "1")
+  )
   (symbol (lib_id "74xx:74LS04") (at 265.43 79.502 0) (unit 6)
     (in_bom yes) (on_board yes)
@@
     (pin "12")
     (pin "13")
+  )
+  (symbol (lib_id "Mechanical:MountingHole_Pad") (at 41.275 66.675 270) (unit 1)
+    (in_bom yes) (on_board yes) (fields_autoplaced)
+    (property "Reference" "H1" (id 0) (at 45.085 65.8403 90)
+      (effects (font (size 1.27 1.27)) (justify left))
+    )
+    (property "Value" "MountingHole" (id 1) (at 45.085 68.3772 90)
+      (effects (font (size 1.27 1.27)) (justify left))
+    )
+    (property "Footprint" "MountingHole:MountingHole_3.2mm_M3_Pad" (id 2) (at 41.275 66.675 0)
+      (effects (font (size 1.27 1.27)) hide)
+    )
+    (property "Datasheet" "~" (id 3) (at 41.275 66.675 0)
+      (effects (font (size 1.27 1.27)) hide)
+    )
+    (pin "1")
   )
   (symbol (lib_id "74xx:74LS74") (at 241.3 123.19 0) (unit 2)
@@
     (pin "2")
   )
+  (symbol (lib_id "Mechanical:MountingHole_Pad") (at 41.275 72.39 270) (unit 1)
+    (in_bom yes) (on_board yes) (fields_autoplaced)
+    (property "Reference" "H2" (id 0) (at 45.085 71.5553 90)
+      (effects (font (size 1.27 1.27)) (justify left))
+    )
+    (property "Value" "MountingHole" (id 1) (at 45.085 74.0922 90)
+      (effects (font (size 1.27 1.27)) (justify left))
+    )
+    (property "Footprint" "MountingHole:MountingHole_3.2mm_M3_Pad" (id 2) (at 41.275 72.39 0)
+      (effects (font (size 0 0)) hide)
+    )
+    (property "Datasheet" "~" (id 3) (at 41.275 72.39 0)
+      (effects (font (size 1.27 1.27)) hide)
+    )
+    (pin "1")
+  )
   (symbol (lib_id "power:+5V") (at 265.43 111.76 0) (unit 1)

Commit message: Add files via upload
Parts:
- added C804: 47uF, Capacitor_THT:CP_Radial_D5.0mm_P2.00mm, symbol Device:CP
Connections:
- net +3V3: now also C804.1
- net GND: now also C804.2
Other:
- moved on the sheet: C800, C801, C802, C803, H1, H2, U800

Commit message: Add files via upload
Parts:
- added C805: 47uF, Capacitor_THT:CP_Radial_D5.0mm_P2.00mm, symbol Device:CP
Connections:
- net +3V3: now also C805.1
- net GND: now also C805.2
Changed lines of the file:
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@@
   (junction (at 233.68 94.615) (diameter 0) (color 0 0 0 0)
   )
+  (junction (at 107.315 70.485) (diameter 0) (color 0 0 0 0)
+  )
   (junction (at 182.88 41.275) (diameter 0) (color 0 0 0 0)
   )
@@
   )
   (junction (at 81.915 80.01) (diameter 0) (color 0 0 0 0)
+  )
+  (junction (at 94.615 80.01) (diameter 0) (color 0 0 0 0)
   )
   (junction (at 27.305 70.485) (diameter 0) (color 0 0 0 0)
@@
     (stroke (width 0) (type default) (color 0 0 0 0))
   )
+  (wire (pts (xy 94.615 70.485) (xy 107.315 70.485))
+    (stroke (width 0) (type default) (color 0 0 0 0))
+  )
   (wire (pts (xy 175.26 33.655) (xy 182.88 33.655))
     (stroke (width 0) (type default) (color 0 0 0 0))
@@
     (stroke (width 0) (type default) (color 0 0 0 0))
   )
-  (polyline (pts (xy 23.495 88.265) (xy 111.76 88.265))
+  (polyline (pts (xy 23.495 88.265) (xy 118.11 88.265))
     (stroke (width 0) (type default) (color 0 0 0 0))
   )
@@
     (stroke (width 0) (type default) (color 0 0 0 0))
   )
-  (polyline (pts (xy 111.76 56.515) (xy 23.495 56.515))
+  (polyline (pts (xy 118.11 56.515) (xy 23.495 56.515))
     (stroke (width 0) (type default) (color 0 0 0 0))
   )
@@
     (stroke (width 0) (type default) (color 0 0 0 0))
   )
-  (wire (pts (xy 94.615 70.485) (xy 94.615 67.31))
+  (wire (pts (xy 107.315 70.485) (xy 107.315 67.31))
     (stroke (width 0) (type default) (color 0 0 0 0))
   )
@@
     (stroke (width 0) (type default) (color 0 0 0 0))
   )
+  (wire (pts (xy 107.315 80.01) (xy 94.615 80.01))
+    (stroke (width 0) (type default) (color 0 0 0 0))
+  )
   (polyline (pts (xy 100.965 50.8) (xy 100.965 20.955))
     (stroke (width 0) (type default) (color 0 0 0 0))
@@
     (stroke (width 0) (type default) (color 0 0 0 0))
   )
-  (polyline (pts (xy 111.76 88.265) (xy 111.76 56.515))
+  (polyline (pts (xy 118.11 88.265) (xy 118.11 56.515))
     (stroke (width 0) (type default) (color 0 0 0 0))
   )
@@
   )
   (wire (pts (xy 189.865 41.275) (xy 203.835 41.275))
+    (stroke (width 0) (type default) (color 0 0 0 0))
+  )
+  (wire (pts (xy 107.315 78.105) (xy 107.315 80.01))
     (stroke (width 0) (type default) (color 0 0 0 0))
   )
@@
     (pin "1")
   )
-  (symbol (lib_id "power:+3.3V") (at 94.615 67.31 0) (unit 1)
-    (in_bom yes) (on_board yes)
-    (property "Reference" "#PWR0188" (id 0) (at 94.615 71.12 0)
-      (effects (font (size 1.27 1.27)) hide)
-    )
-    (property "Value" "+3.3V" (id 1) (at 94.996 62.9158 0))
-    (property "Footprint" "" (id 2) (at 94.615 67.31 0)
-      (effects (font (size 1.27 1.27)) hide)
-    )
-    (property "Datasheet" "" (id 3) (at 94.615 67.31 0)
+  (symbol (lib_id "power:+3.3V") (at 107.315 67.31 0) (unit 1)
+    (in_bom yes) (on_board yes)
+    (property "Reference" "#PWR0188" (id 0) (at 107.315 71.12 0)
+      (effects (font (size 1.27 1.27)) hide)
+    )
+    (property "Value" "+3.3V" (id 1) (at 107.696 62.9158 0))
+    (property "Footprint" "" (id 2) (at 107.315 67.31 0)
+      (effects (font (size 1.27 1.27)) hide)
+    )
+    (property "Datasheet" "" (id 3) (at 107.315 67.31 0)
       (effects (font (size 1.27 1.27)) hide)
     )
@@
     (pin "11")
   )
+  (symbol (lib_id "Device:CP") (at 107.315 74.295 0) (unit 1)
+    (in_bom yes) (on_board yes)
+    (property "Reference" "C805" (id 0) (at 110.3122 73.1266 0)
+      (effects (font (size 1.27 1.27)) (justify left))
+    )
+    (property "Value" "47uF" (id 1) (at 110.3122 75.438 0)
+      (effects (font (size 1.27 1.27)) (justify left))
+    )
+    (property "Footprint" "Capacitor_THT:CP_Radial_D5.0mm_P2.00mm" (id 2) (at 108.2802 78.105 0)
+      (effects (font (size 1.27 1.27)) hide)
+    )
+    (property "Datasheet" "~" (id 3) (at 107.315 74.295 0)
+      (effects (font (size 1.27 1.27)) hide)
+    )
+    (pin "1")
+    (pin "2")
+  )
   (symbol (lib_id "power:GND") (at 38.735 43.815 0) (unit 1)

Commit message: Add files via upload
Parts:
- C804, C805: value 47uF -> 10uF
Changed lines of the file:
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@@
       (effects (font (size 1.27 1.27)) (justify left))
     )
-    (property "Value" "47uF" (id 1) (at 110.3122 75.438 0)
+    (property "Value" "10uF" (id 1) (at 110.3122 75.438 0)
       (effects (font (size 1.27 1.27)) (justify left))
     )
@@
       (effects (font (size 1.27 1.27)) (justify left))
     )
-    (property "Value" "47uF" (id 1) (at 97.6122 75.438 0)
+    (property "Value" "10uF" (id 1) (at 97.6122 75.438 0)
       (effects (font (size 1.27 1.27)) (justify left))
     )

Commit message: Add files via upload
Parts:
- added CN4: CPLD3, Connector_PinHeader_2.54mm:PinHeader_1x06_P2.54mm_Vertical, symbol Connector_Generic:Conn_01x06
- added CN5: ATA/IDE, N2630:ATA_Header_2x20_P2.54mm, symbol Connector_Generic:Conn_02x20_Odd_Even
- added U603: XC9572XL-VQ64, Package_QFP:TQFP-64_10x10mm_P0.5mm, symbol CPLD_Xilinx:XC9572XL-VQ64
Connections:
- net +3V3: now also CN4.6 (Pin_6)
- net GND: now also CN4.5 (Pin_5), CN5.19 (Pin_19), CN5.2 (Pin_2), CN5.22 (Pin_22), CN5.24 (Pin_24), CN5.26 (Pin_26), CN5.30 (Pin_30), CN5.40 (Pin_40), U603.14 (GND), U603.21 (GND), U603.41 (GND), U603.54 (GND)
- new net A12: U603.11 (P11)
- new net A13: U603.12 (P12)
- new net A14: U603.13 (P13)
- new net A15: U603.15 (I/O/GCK1)
- new net A16: U603.16 (I/O/GCK2)
- new net A17: U603.17 (I/O/GCK3)
- new net A18: U603.18 (P18)
- new net A19: U603.19 (P19)
- new net A2: U603.8 (P8)
- new net A20: U603.20 (P20)
- new net A21: U603.23 (P23)
- new net A22: U603.1 (P1)
- new net A23: U603.4 (P4)
- new net A3: U603.9 (P9)
- new net A4: U603.10 (P10)
- new net CSEL: CN5.28 (Pin_28)
- new net D16: CN5.17 (Pin_17)
- new net D17: CN5.15 (Pin_15)
- new net D18: CN5.13 (Pin_13)
- new net D19: CN5.11 (Pin_11)
- new net D20: CN5.9 (Pin_9)
- new net D21: CN5.7 (Pin_7)
- new net D22: CN5.5 (Pin_5)
- new net D23: CN5.3 (Pin_3)
- new net D24: CN5.4 (Pin_4), U603.22 (P22)
- new net D25: CN5.6 (Pin_6), U603.24 (P24)
- new net D26: CN5.8 (Pin_8), U603.25 (P25)
- new net D27: CN5.10 (Pin_10), U603.27 (P27)
- new net D28: CN5.12 (Pin_12), U603.31 (P31)
- new net D29: CN5.14 (Pin_14), U603.32 (P32)
- new net D30: CN5.16 (Pin_16), U603.33 (P33)
- new net D31: CN5.18 (Pin_18), U603.34 (P34)
- new net DA0: CN5.35 (Pin_35), U603.7 (P7)
- new net DA1: CN5.33 (Pin_33), U603.58 (P58)
- new net DA2: CN5.36 (Pin_36), U603.59 (P59)
- new net DMARQ: CN5.21 (Pin_21)
- new net INTRQ: CN5.31 (Pin_31), U603.63 (P63)
- new net IORDY: CN5.27 (Pin_27), U603.44 (P44), U603.6 (P6)
- new net PDIAG: CN5.34 (Pin_34)
- new net TCK1: CN4.1 (Pin_1), U603.30 (TCK)
- new net TDI1: CN4.3 (Pin_3), U603.28 (TDI)
- new net TDO1: CN4.4 (Pin_4), U603.53 (TDO)
- new net TMS1: CN4.2 (Pin_2), U603.29 (TMS)
- new net _ACTIVE: CN5.39 (Pin_39)
- new net _AS: U603.48 (P48)
- new net _CS0: CN5.37 (Pin_37), U603.60 (P60)
- new net _CS1: CN5.38 (Pin_38), U603.61 (P61)
- new net _DIOR: CN5.25 (Pin_25), U603.45 (P45)
- new net _DIOW: CN5.23 (Pin_23), U603.46 (P46)
- new net _DMACK: CN5.29 (Pin_29)
- new net _DS: U603.47 (P47)
- new net _GRESET: CN5.1 (Pin_1)
- new net _INT2: U603.51 (P51)
- new net _IOCS16: CN5.32 (Pin_32)
- new net _OVR: U603.50 (P50)
- no-connect marks 12 -> 13
Other:
- note added: "GABRIELLE"
- note added: "GAYLE_ID is at $DE1000 110111100001000000000000 return $DF (11011111)"
- note added: "INTENA (enable ide interupts) $daa000 (110110101010000000000000) return $80 (set bit 7 to 1) to enable"
- moved on the sheet: C800, C801, C802, C803, C804, C805, U800

Commit message: Add files via upload
Parts:
- added C610, C611: 0.22uF, Capacitor_SMD:C_0805_2012Metric, symbol Device:C
- added CN6: LED, Connector_PinHeader_2.54mm:PinHeader_1x03_P2.54mm_Vertical, symbol Connector_Generic:Conn_01x03
- added R600: 2.7K, Resistor_SMD:R_0805_2012Metric, symbol Device:R
Connections:
- net +3V3: now also U603.26 (VCCIO), U603.3 (VCC), U603.37 (VCC), U603.55 (VCCIO), C610.1, C611.1
- net +5V: now also CN6.2 (Pin_2), R600.1
- net A12: now also U603.8 (P8); no longer U603.11 (P11)
- net A13: now also U603.7 (P7); no longer U603.12 (P12)
- net A14: now also U603.6 (P6); no longer U603.13 (P13)
- net A15: now also U603.5 (I/O/GTS1); no longer U603.15 (I/O/GCK1)
- net A16: now also U603.4 (P4); no longer U603.16 (I/O/GCK2)
- net A17: now also U603.15 (I/O/GCK1); no longer U603.17 (I/O/GCK3)
- net A18: now also U603.13 (P13); no longer U603.18 (P18)
- net A19: now also U603.12 (P12); no longer U603.19 (P19)
- net A2: now also U603.62 (P62); no longer U603.8 (P8)
- net A20: now also U603.11 (P11); no longer U603.20 (P20)
- net A21: now also U603.2 (I/O/GTS2); no longer U603.23 (P23)
- net A22: now also U603.10 (P10); no longer U603.1 (P1)
- net A23: now also U603.9 (P9); no longer U603.4 (P4)
- net A3: now also U603.63 (P63); no longer U603.9 (P9)
- net A4: now also U603.1 (P1); no longer U603.10 (P10)
- net D24: now also U603.18 (P18); no longer U603.22 (P22)
- net D25: now also U603.19 (P19); no longer U603.24 (P24)
- net D26: now also U603.22 (P22); no longer U603.25 (P25)
- net D27: now also U603.24 (P24); no longer U603.27 (P27)
- net D28: now also U603.25 (P25); no longer U603.31 (P31)
- net D29: now also U603.27 (P27); no longer U603.32 (P32)
- net D30: now also U603.31 (P31); no longer U603.33 (P33)
- net D31: now also U603.32 (P32); no longer U603.34 (P34)
- net DA0: now also U603.40 (P40); no longer U603.7 (P7)
- net DA1: now also U603.38 (P38); no longer U603.58 (P58)
- net DA2: now also U603.39 (P39); no longer U603.59 (P59)
- net GND: now also C610.2, C611.2
- net INTRQ: now also U603.36 (P36); no longer U603.63 (P63)
- net IORDY: now also U603.35 (P35); no longer U603.44 (P44), U603.6 (P6)
- net _ACTIVE: now also CN6.1 (Pin_1), CN6.3 (Pin_3), R600.2
- net _AS: now also U603.59 (P59); no longer U603.48 (P48)
- net _CS0: now also U603.43 (P43); no longer U603.60 (P60)
- net _CS1: now also U603.42 (P42); no longer U603.61 (P61)
- net _DIOR: now also U603.34 (P34); no longer U603.45 (P45)
- net _DIOW: now also U603.33 (P33); no longer U603.46 (P46)
- net _DS: now also U603.60 (P60); no longer U603.47 (P47)
- net _GRESET: now also U603.16 (I/O/GCK2)
- net _INT2: now also U603.57 (P57); no longer U603.51 (P51)
- net _OVR: now also U603.56 (P56); no longer U603.50 (P50)
- new net R_W: U603.58 (P58)
- no-connect marks 13 -> 26
Other:
- note removed: "GABRIELLE"
