File: A2630-New-KiCAD/Card Edge.kicad_sch (KiCad schematic)
At the start: 31 parts, among them CN700 Amiga-2000-CPU-Slot, J301 Jumper_NO_Small, J302 Jumper_NO_Small, J303 Jumper_NO_Small, J304 Jumper_NO_Small, J305 Jumper_NO_Small, U300 74HCT05, U307 74HCT04, U700 74HCT174, U701 74FCT646, U702 74FCT646, U703 74HCT245, U704 74HCT245, U705 74HCT245, U706 74HCT245, U707 74HCT245

Commit message: Add files via upload
Connections:
- net +5V: now also C700.1, U700.16 (VCC)
- net at R706.2, U700.1 (~{Mr}), U700.11 (D3)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: no longer C700.1, U700.16 (VCC)
Changed lines of the file:
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@@
   (junction (at 314.96 78.105) (diameter 0) (color 0 0 0 0)
   )
-  (junction (at 51.435 113.665) (diameter 0) (color 0 0 0 0)
-  )
   (junction (at 367.03 95.25) (diameter 0) (color 0 0 0 0)
   )
@@
   (junction (at 285.115 194.31) (diameter 0) (color 0 0 0 0)
   )
+  (junction (at 51.435 113.665) (diameter 0) (color 0 0 0 0)
+  )
   (junction (at 364.49 90.805) (diameter 0) (color 0 0 0 0)
   )
@@
   (junction (at 365.125 194.31) (diameter 0) (color 0 0 0 0)
   )
-  (junction (at 68.58 98.425) (diameter 0) (color 0 0 0 0)
-  )
   (junction (at 109.22 208.28) (diameter 0) (color 0 0 0 0)
   )
@@
     (stroke (width 0) (type default) (color 0 0 0 0))
   )
-  (wire (pts (xy 68.58 98.425) (xy 68.58 113.665))
-    (stroke (width 0) (type default) (color 0 0 0 0))
-  )
   (wire (pts (xy 102.235 233.68) (xy 115.57 233.68))
     (stroke (width 0) (type default) (color 0 0 0 0))
@@
     (stroke (width 0) (type default) (color 0 0 0 0))
   )
+  (wire (pts (xy 51.435 113.665) (xy 68.072 113.665))
+    (stroke (width 0) (type default) (color 0 0 0 0))
+  )
   (bus (pts (xy 205.74 184.15) (xy 205.74 186.69))
     (stroke (width 0) (type default) (color 0 0 0 0))
@@
     (stroke (width 0) (type default) (color 0 0 0 0))
   )
+  (wire (pts (xy 68.072 112.395) (xy 68.072 113.665))
+    (stroke (width 0) (type default) (color 0 0 0 0))
+  )
   (wire (pts (xy 104.775 214.63) (xy 24.13 214.63))
     (stroke (width 0) (type default) (color 0 0 0 0))
@@
     (stroke (width 0) (type default) (color 0 0 0 0))
   )
-  (wire (pts (xy 68.58 113.665) (xy 51.435 113.665))
-    (stroke (width 0) (type default) (color 0 0 0 0))
-  )
   (wire (pts (xy 329.565 224.155) (xy 342.9 224.155))
     (stroke (width 0) (type default) (color 0 0 0 0))
@@
       (effects (font (size 1.27 1.27)) hide)
     )
+    (pin "1")
+  )
+  (symbol (lib_id "power:+5V") (at 68.072 112.395 0) (unit 1)
+    (in_bom yes) (on_board yes)
+    (property "Reference" "#PWR0194" (id 0) (at 68.072 116.205 0)
+      (effects (font (size 1.27 1.27)) hide)
+    )
+    (property "Value" "+5V" (id 1) (at 68.453 108.0008 0))
+    (property "Footprint" "" (id 2) (at 68.072 112.395 0)
+      (effects (font (size 1.27 1.27)) hide)
+    )
+    (property "Datasheet" "" (id 3) (at 68.072 112.395 0)
+      (effects (font (size 1.27 1.27)) hide)
+    )

Commit message: Add files via upload
Parts:
- removed RN300: 3.3K, Resistor_THT:R_Array_SIP6, symbol Device:R_Network05
- added R302, R303, R304, R305, R306: 3.3k, Resistor_SMD:R_0805_2012Metric, symbol Device:R
Connections:
- net +3V3: now also R302.1, R303.1, R304.1, R305.1, R306.1
- net B2000: now also R303.2
- net OSMODE: now also R305.2
- net TWOMB: now also R302.2
- net Z2AUTO: now also R304.2
- net Z3AUTO: now also R306.2
Changed lines of the file:
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@@
   (junction (at 237.49 224.155) (diameter 0) (color 0 0 0 0)
   )
+  (junction (at 364.49 64.135) (diameter 0) (color 0 0 0 0)
+  )
   (junction (at 329.565 224.155) (diameter 0) (color 0 0 0 0)
   )
@@
   (junction (at 307.34 224.155) (diameter 0) (color 0 0 0 0)
   )
+  (junction (at 361.95 64.135) (diameter 0) (color 0 0 0 0)
+  )
   (junction (at 374.015 224.155) (diameter 0) (color 0 0 0 0)
   )
@@
   (junction (at 365.125 194.31) (diameter 0) (color 0 0 0 0)
   )
+  (junction (at 359.41 64.135) (diameter 0) (color 0 0 0 0)
+  )
   (junction (at 109.22 208.28) (diameter 0) (color 0 0 0 0)
   )
@@
   (junction (at 109.22 135.89) (diameter 0) (color 0 0 0 0)
   )
+  (junction (at 356.87 64.135) (diameter 0) (color 0 0 0 0)
+  )
   (junction (at 240.03 224.155) (diameter 0) (color 0 0 0 0)
   )
@@
     (stroke (width 0) (type default) (color 0 0 0 0))
   )
+  (wire (pts (xy 364.49 64.135) (xy 367.03 64.135))
+    (stroke (width 0) (type default) (color 0 0 0 0))
+  )
   (wire (pts (xy 299.085 98.425) (xy 307.975 98.425))
     (stroke (width 0) (type default) (color 0 0 0 0))
@@
     (stroke (width 0) (type default) (color 0 0 0 0))
   )
+  (wire (pts (xy 361.95 64.135) (xy 364.49 64.135))
+    (stroke (width 0) (type default) (color 0 0 0 0))
+  )
   (bus (pts (xy 134.62 165.1) (xy 134.62 166.37))
     (stroke (width 0) (type default) (color 0 0 0 0))
@@
     (stroke (width 0) (type default) (color 0 0 0 0))
   )
+  (wire (pts (xy 356.87 64.135) (xy 359.41 64.135))
+    (stroke (width 0) (type default) (color 0 0 0 0))
+  )
   (bus (pts (xy 205.74 233.045) (xy 205.74 235.585))
     (stroke (width 0) (type default) (color 0 0 0 0))
@@
     (stroke (width 0) (type default) (color 0 0 0 0))
   )
+  (wire (pts (xy 359.41 64.135) (xy 361.95 64.135))
+    (stroke (width 0) (type default) (color 0 0 0 0))
+  )
   (wire (pts (xy 356.87 77.47) (xy 381.635 77.47))
     (stroke (width 0) (type default) (color 0 0 0 0))
@@
     (stroke (width 0) (type default) (color 0 0 0 0))
   )
+  (wire (pts (xy 356.87 59.055) (xy 356.87 64.135))
+    (stroke (width 0) (type default) (color 0 0 0 0))
+  )
   (wire (pts (xy 214.63 161.925) (xy 394.335 161.925))
     (stroke (width 0) (type default) (color 0 0 0 0))
@@
     (pin "2")
   )
-  (symbol (lib_id "Device:R_Network05") (at 361.95 66.675 0) (unit 1)
-    (in_bom yes) (on_board yes)
-    (property "Reference" "RN300" (id 0) (at 369.2652 65.5066 0)
-      (effects (font (size 1.27 1.27)) (justify left))
-    )
-    (property "Value" "3.3K" (id 1) (at 369.2652 67.818 0)
-      (effects (font (size 1.27 1.27)) (justify left))
-    )
-    (property "Footprint" "Resistor_THT:R_Array_SIP6" (id 2) (at 371.475 66.675 90)
-      (effects (font (size 1.27 1.27)) hide)
-    )
-    (property "Datasheet" "http://www.vishay.com/docs/31509/csc.pdf" (id 3) (at 361.95 66.675 0)
-      (effects (font (size 1.27 1.27)) hide)
-    )
-    (pin "1")
-    (pin "2")
-    (pin "3")
-    (pin "4")
-    (pin "5")
-    (pin "6")
-  )
   (symbol (lib_id "N2630:74FCT646") (at 227.965 208.915 0) (unit 2)
     (in_bom yes) (on_board yes)
@@
     (pin "20")
   )
-  (symbol (lib_id "power:+3.3V") (at 356.87 61.595 0) (unit 1)
+  (symbol (lib_id "power:+3.3V") (at 356.87 59.055 0) (unit 1)
     (in_bom yes) (on_board yes)
-    (property "Reference" "#PWR0142" (id 0) (at 356.87 65.405 0)
+    (property "Reference" "#PWR0142" (id 0) (at 356.87 62.865 0)
       (effects (font (size 1.27 1.27)) hide)
     )
-    (property "Value" "+3.3V" (id 1) (at 357.251 57.2008 0))
-    (property "Footprint" "" (id 2) (at 356.87 61.595 0)
+    (property "Value" "+3.3V" (id 1) (at 357.251 54.6608 0))
+    (property "Footprint" "" (id 2) (at 356.87 59.055 0)
       (effects (font (size 1.27 1.27)) hide)
     )
-    (property "Datasheet" "" (id 3) (at 356.87 61.595 0)
+    (property "Datasheet" "" (id 3) (at 356.87 59.055 0)
       (effects (font (size 1.27 1.27)) hide)
     )
@@
     (pin "1")
   )
+  (symbol (lib_id "Device:R") (at 356.87 67.945 0) (unit 1)
+    (in_bom yes) (on_board yes)
+    (property "Reference" "R302" (id 0) (at 358.14 65.405 90)
+      (effects (font (size 1.27 1.27)) (justify left))
+    )
+    (property "Value" "3.3k" (id 1) (at 356.87 69.85 90)
+      (effects (font (size 1.27 1.27)) (justify left))
+    )
+    (property "Footprint" "Resistor_SMD:R_0805_2012Metric" (id 2) (at 355.092 67.945 90)
+      (effects (font (size 1.27 1.27)) hide)
+    )
+    (property "Datasheet" "~" (id 3) (at 356.87 67.945 0)
+      (effects (font (size 1.27 1.27)) hide)
+    )
+    (pin "1")
+    (pin "2")
+  )
+  (symbol (lib_id "Device:R") (at 364.49 67.945 0) (unit 1)
+    (in_bom yes) (on_board yes)
+    (property "Reference" "R305" (id 0) (at 365.76 65.405 90)
+      (effects (font (size 1.27 1.27)) (justify left))
+    )
+    (property "Value" "3.3k" (id 1) (at 364.49 69.85 90)
+      (effects (font (size 1.27 1.27)) (justify left))
+    )
+    (property "Footprint" "Resistor_SMD:R_0805_2012Metric" (id 2) (at 362.712 67.945 90)
+      (effects (font (size 1.27 1.27)) hide)
+    )
+    (property "Datasheet" "~" (id 3) (at 364.49 67.945 0)
+      (effects (font (size 1.27 1.27)) hide)
+    )
+    (pin "1")
+    (pin "2")
+  )
+  (symbol (lib_id "Device:R") (at 361.95 67.945 0) (unit 1)
+    (in_bom yes) (on_board yes)
+    (property "Reference" "R304" (id 0) (at 363.22 65.405 90)
+      (effects (font (size 1.27 1.27)) (justify left))
+    )
+    (property "Value" "3.3k" (id 1) (at 361.95 69.85 90)
+      (effects (font (size 1.27 1.27)) (justify left))
+    )
+    (property "Footprint" "Resistor_SMD:R_0805_2012Metric" (id 2) (at 360.172 67.945 90)
+      (effects (font (size 1.27 1.27)) hide)
+    )
+    (property "Datasheet" "~" (id 3) (at 361.95 67.945 0)
+      (effects (font (size 1.27 1.27)) hide)
+    )
+    (pin "1")
+    (pin "2")
+  )
+  (symbol (lib_id "Device:R") (at 359.41 67.945 0) (unit 1)
+    (in_bom yes) (on_board yes)
+    (property "Reference" "R303" (id 0) (at 360.68 65.405 90)
+      (effects (font (size 1.27 1.27)) (justify left))
+    )
+    (property "Value" "3.3k" (id 1) (at 359.41 69.85 90)
+      (effects (font (size 1.27 1.27)) (justify left))
+    )
+    (property "Footprint" "Resistor_SMD:R_0805_2012Metric" (id 2) (at 357.632 67.945 90)
+      (effects (font (size 1.27 1.27)) hide)
+    )
+    (property "Datasheet" "~" (id 3) (at 359.41 67.945 0)
+      (effects (font (size 1.27 1.27)) hide)
+    )
+    (pin "1")
+    (pin "2")
+  )
   (symbol (lib_id "power:+5V") (at 68.072 112.395 0) (unit 1)
     (in_bom yes) (on_board yes)
@@
     (pin "1")
   )
+  (symbol (lib_id "Device:R") (at 367.03 67.945 0) (unit 1)
+    (in_bom yes) (on_board yes)
+    (property "Reference" "R306" (id 0) (at 368.3 65.405 90)
+      (effects (font (size 1.27 1.27)) (justify left))
+    )
+    (property "Value" "3.3k" (id 1) (at 367.03 69.85 90)
+      (effects (font (size 1.27 1.27)) (justify left))
+    )
+    (property "Footprint" "Resistor_SMD:R_0805_2012Metric" (id 2) (at 365.252 67.945 90)
+      (effects (font (size 1.27 1.27)) hide)
+    )
+    (property "Datasheet" "~" (id 3) (at 367.03 67.945 0)
+      (effects (font (size 1.27 1.27)) hide)
+    )
+    (pin "1")
+    (pin "2")
+  )
 )

Commit message: Add files via upload
Connections:
- net 7M renamed IPLCLK
Changed lines of the file:
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@@
     )
   )
-  (global_label "7M" (shape input) (at 27.305 56.515 180) (fields_autoplaced)
+  (global_label "IPLCLK" (shape input) (at 27.305 56.515 180) (fields_autoplaced)
     (effects (font (size 1.27 1.27)) (justify right))
-    (property "Intersheet References" "${INTERSHEET_REFS}" (id 0) (at 0 0 0)
-      (effects (font (size 1.27 1.27)) hide)
+    (property "Intersheet References" "${INTERSHEET_REFS}" (id 0) (at 18.5098 56.4356 0)
+      (effects (font (size 1.27 1.27)) (justify right) hide)
     )
   )

Commit message: Add files via upload
Connections:
- net A7M: now reaches CN700.7
Changed lines of the file:
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@@
+    (stroke (width 0) (type default) (color 0 0 0 0))
+  )
+  (wire (pts (xy 102.235 139.7) (xy 93.345 139.7))
     (stroke (width 0) (type default) (color 0 0 0 0))
   )
@@
     (stroke (width 0) (type default) (color 0 0 0 0))
   )
+  (wire (pts (xy 93.345 139.7) (xy 93.345 132.715))
+    (stroke (width 0) (type default) (color 0 0 0 0))
+  )
   (wire (pts (xy 194.945 140.97) (xy 203.2 140.97))
     (stroke (width 0) (type default) (color 0 0 0 0))
@@
   )
   (wire (pts (xy 75.565 106.045) (xy 75.565 186.69))
+    (stroke (width 0) (type default) (color 0 0 0 0))
+  )
+  (wire (pts (xy 23.495 132.715) (xy 93.345 132.715))
     (stroke (width 0) (type default) (color 0 0 0 0))
   )
@@
     )
   )
+  (global_label "A7M" (shape output) (at 23.495 132.715 180) (fields_autoplaced)
+    (effects (font (size 1.27 1.27)) (justify right))
+    (property "Intersheet References" "${INTERSHEET_REFS}" (id 0) (at 17.4213 132.6356 0)
+      (effects (font (size 1.27 1.27)) (justify right) hide)
+    )
+  )

Commit message: Add files via upload
Connections:
- net _INT2: now reaches CN700.19
Changed lines of the file:
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@@
     (stroke (width 0) (type default) (color 0 0 0 0))
   )
-  (wire (pts (xy 104.775 156.21) (xy 23.495 156.21))
+  (wire (pts (xy 104.775 156.21) (xy 59.69 156.21))
     (stroke (width 0) (type default) (color 0 0 0 0))
   )
@@
     (stroke (width 0) (type default) (color 0 0 0 0))
   )
+  (wire (pts (xy 56.515 156.845) (xy 56.515 154.94))
+    (stroke (width 0) (type default) (color 0 0 0 0))
+  )
   (bus (pts (xy 262.89 85.725) (xy 262.89 88.265))
     (stroke (width 0) (type default) (color 0 0 0 0))
@@
     (stroke (width 0) (type default) (color 0 0 0 0))
   )
-  (wire (pts (xy 23.495 164.465) (xy 67.945 164.465))
+  (wire (pts (xy 23.495 169.545) (xy 67.945 169.545))
     (stroke (width 0) (type default) (color 0 0 0 0))
   )
@@
     (stroke (width 0) (type default) (color 0 0 0 0))
   )
-  (wire (pts (xy 70.485 161.925) (xy 23.495 161.925))
+  (wire (pts (xy 70.485 167.005) (xy 23.495 167.005))
+    (stroke (width 0) (type default) (color 0 0 0 0))
+  )
+  (wire (pts (xy 59.69 160.655) (xy 59.69 156.21))
     (stroke (width 0) (type default) (color 0 0 0 0))
   )
@@
     (stroke (width 0) (type default) (color 0 0 0 0))
   )
-  (wire (pts (xy 70.485 172.72) (xy 70.485 161.925))
+  (wire (pts (xy 70.485 172.72) (xy 70.485 167.005))
     (stroke (width 0) (type default) (color 0 0 0 0))
   )
@@
     (stroke (width 0) (type default) (color 0 0 0 0))
   )
-  (wire (pts (xy 23.495 159.385) (xy 73.025 159.385))
+  (wire (pts (xy 23.495 164.465) (xy 73.025 164.465))
     (stroke (width 0) (type default) (color 0 0 0 0))
   )
@@
     (stroke (width 0) (type default) (color 0 0 0 0))
   )
+  (wire (pts (xy 23.495 160.655) (xy 59.69 160.655))
+    (stroke (width 0) (type default) (color 0 0 0 0))
+  )
   (bus (pts (xy 310.515 83.185) (xy 310.515 85.725))
     (stroke (width 0) (type default) (color 0 0 0 0))
@@
     (stroke (width 0) (type default) (color 0 0 0 0))
   )
+  (wire (pts (xy 102.235 154.94) (xy 56.515 154.94))
+    (stroke (width 0) (type default) (color 0 0 0 0))
+  )
   (bus (pts (xy 310.515 46.355) (xy 310.515 48.895))
     (stroke (width 0) (type default) (color 0 0 0 0))
@@
     (stroke (width 0) (type default) (color 0 0 0 0))
   )
-  (wire (pts (xy 73.025 159.385) (xy 73.025 170.18))
+  (wire (pts (xy 73.025 164.465) (xy 73.025 170.18))
     (stroke (width 0) (type default) (color 0 0 0 0))
   )
@@
     (stroke (width 0) (type default) (color 0 0 0 0))
   )
+  (wire (pts (xy 22.86 156.845) (xy 56.515 156.845))
+    (stroke (width 0) (type default) (color 0 0 0 0))
+  )
   (wire (pts (xy 104.775 240.03) (xy 115.57 240.03))
     (stroke (width 0) (type default) (color 0 0 0 0))
@@
     (stroke (width 0) (type default) (color 0 0 0 0))
   )
-  (wire (pts (xy 67.945 164.465) (xy 67.945 175.26))
+  (wire (pts (xy 67.945 169.545) (xy 67.945 175.26))
     (stroke (width 0) (type default) (color 0 0 0 0))
   )
@@
     )
   )
-  (global_label "AFC1" (shape input) (at 23.495 161.925 180) (fields_autoplaced)
+  (global_label "AFC1" (shape input) (at 23.495 167.005 180) (fields_autoplaced)
     (effects (font (size 1.1938 1.1938)) (justify right))
-    (property "Intersheet References" "${INTERSHEET_REFS}" (id 0) (at 0 0 0)
+    (property "Intersheet References" "${INTERSHEET_REFS}" (id 0) (at 0 5.08 0)
       (effects (font (size 1.27 1.27)) hide)
     )
@@
     )
   )
-  (global_label "AFC0" (shape input) (at 23.495 159.385 180) (fields_autoplaced)
+  (global_label "_INT2" (shape input) (at 22.86 156.845 180) (fields_autoplaced)
+    (effects (font (size 1.27 1.27)) (justify right))
+    (property "Intersheet References" "${INTERSHEET_REFS}" (id 0) (at 15.4558 156.7656 0)
+      (effects (font (size 1.27 1.27)) (justify right) hide)
+    )
+  )
+  (global_label "AFC0" (shape input) (at 23.495 164.465 180) (fields_autoplaced)
     (effects (font (size 1.1938 1.1938)) (justify right))
-    (property "Intersheet References" "${INTERSHEET_REFS}" (id 0) (at 0 0 0)
+    (property "Intersheet References" "${INTERSHEET_REFS}" (id 0) (at 0 5.08 0)
       (effects (font (size 1.27 1.27)) hide)
     )
@@
     )
   )
-  (global_label "_BOSS" (shape input) (at 23.495 156.21 180) (fields_autoplaced)
+  (global_label "_BOSS" (shape input) (at 23.495 160.655 180) (fields_autoplaced)
     (effects (font (size 1.27 1.27)) (justify right))
-    (property "Intersheet References" "${INTERSHEET_REFS}" (id 0) (at 0 0 0)
+    (property "Intersheet References" "${INTERSHEET_REFS}" (id 0) (at 0 4.445 0)
       (effects (font (size 1.27 1.27)) hide)
     )
@@
     )
   )
-  (global_label "AFC2" (shape input) (at 23.495 164.465 180) (fields_autoplaced)
+  (global_label "AFC2" (shape input) (at 23.495 169.545 180) (fields_autoplaced)
     (effects (font (size 1.1938 1.1938)) (justify right))
-    (property "Intersheet References" "${INTERSHEET_REFS}" (id 0) (at 0 0 0)
-      (effects (font (size 1.27 1.27)) hide)
-    )
+    (property "Intersheet References" "${INTERSHEET_REFS}" (id 0) (at 0 5.08 0)
+      (effects (font (size 1.27 1.27)) hide)
+    )

Commit message: Add files via upload
Changed lines of the file:
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@@
   )
   (text "CARD EDGE AND\nINTERFACE LOGIC" (at 313.055 250.825 0)
-    (effects (font (size 5.5118 5.5118)) (justify left bottom))
+    (effects (font (size 5 5)) (justify left bottom))
   )
   (label "AA23" (at 265.43 48.895 0)

Commit message: Add files via upload
Connections:
- net _CDAC renamed CDAC
Other:
- note removed: "Seein' all the sights, many crazy nights"
Changed lines of the file:
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@@
     (stroke (width 0) (type default) (color 0 0 0 0))
-  )
-  (text "Seein' all the sights, many crazy nights" (at 312.42 234.315 0)
-    (effects (font (size 2.9972 2.9972)) (justify left bottom))
   )
   (text "Not all these jumpers will make it to the final version.\nJ301 - 2MEG Shorted/4MEG Open\nJ302 - A2000 Shorted/B2000 Open\nJ303 - Do not configure Z2 RAM Shorted/Autoconfigure Z2 RAM Open\nJ304 - AMIX Shorted/AmigaOS Open\nJ305 - Do not configure Z3 RAM Shorted/Autoconfigure Z3 RAM Open"
@@
     )
   )
-  (global_label "_CDAC" (shape output) (at 23.495 145.415 180) (fields_autoplaced)
-    (effects (font (size 1.27 1.27)) (justify right))
-    (property "Intersheet References" "${INTERSHEET_REFS}" (id 0) (at 0 0 0)
-      (effects (font (size 1.27 1.27)) hide)
-    )
-  )
+  (global_label "CDAC" (shape output) (at 23.495 145.415 180) (fields_autoplaced)
+    (effects (font (size 1.27 1.27)) (justify right))
+    (property "Intersheet References" "${INTERSHEET_REFS}" (id 0) (at 16.2722 145.3356 0)
+      (effects (font (size 1.27 1.27)) (justify right) hide)
+    )
+  )

Commit message: Add files via upload
Parts:
- U703, U704: footprint Package_SO:SOIC-24W_7.5x15.4mm_P1.27mm -> Package_SO:SOIC-20W_7.5x12.8mm_P1.27mm
Changed lines of the file:
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@@
     (property "Reference" "U704" (id 0) (at 182.245 211.0232 0))
     (property "Value" "74HCT245" (id 1) (at 182.245 213.3346 0))
-    (property "Footprint" "Package_SO:SOIC-24W_7.5x15.4mm_P1.27mm" (id 2) (at 182.245 230.505 0)
+    (property "Footprint" "Package_SO:SOIC-20W_7.5x12.8mm_P1.27mm" (id 2) (at 182.245 230.505 0)
       (effects (font (size 1.27 1.27)) hide)
     )
@@
     (property "Reference" "U703" (id 0) (at 182.245 169.7482 0))
     (property "Value" "74HCT245" (id 1) (at 182.245 172.0596 0))
-    (property "Footprint" "Package_SO:SOIC-24W_7.5x15.4mm_P1.27mm" (id 2) (at 182.245 189.23 0)
+    (property "Footprint" "Package_SO:SOIC-20W_7.5x12.8mm_P1.27mm" (id 2) (at 182.245 189.23 0)
       (effects (font (size 1.27 1.27)) hide)
     )
@@
       (effects (font (size 1.27 1.27)) (justify left))
     )
-    (property "Footprint" "Package_SO:SOIC-24W_7.5x15.4mm_P1.27mm" (id 2) (at 276.225 208.915 0)
+    (property "Footprint" "Package_SO:SOIC-20W_7.5x12.8mm_P1.27mm" (id 2) (at 276.225 208.915 0)
       (effects (font (size 1.27 1.27)) hide)
     )
@@
       (effects (font (size 1.27 1.27)) (justify left))
     )
-    (property "Footprint" "Package_SO:SOIC-24W_7.5x15.4mm_P1.27mm" (id 2) (at 298.45 208.915 0)
-      (effects (font (size 1.27 1.27)) hide)
-    )
+    (property "Footprint" "Package_SO:SOIC-20W_7.5x12.8mm_P1.27mm" (id 2) (at 298.45 208.915 0)
+      (effects (font (size 1.27 1.27)) hide)
+    )
