File: A2630-New-KiCAD/Processor.kicad_sch (KiCad schematic)
At the start: 50 parts, among them U200 MC68030FE, U201 MC68882, U204 74HCT04, X1 25MHz, X2 25MHz

Commit message: Add files via upload
Parts:
- removed RN101, RN102, RN103: 1K, Resistor_THT:R_Array_SIP9, symbol Device:R_Network08
- added R108, R109, R110, R111, R112, R113, R114, R115, R116, R117, R118, R119, R120, R121, R122, R123, R124, R125, R126, R127, R128, R129, R130, R131: 1K, Resistor_SMD:R_0805_2012Metric, symbol Device:R
Connections:
- net A0: now also R131.1
- net A1: now also R130.1
- net A10: now also R121.1
- net A11: now also R120.1
- net A12: now also R119.1
- net A13: now also R118.1
- net A14: now also R116.1
- net A15: now also R117.1
- net A16: now also R115.1
- net A17: now also R114.1
- net A18: now also R113.1
- net A19: now also R112.1
- net A2: now also R129.1
- net A20: now also R111.1
- net A21: now also R110.1
- net A22: now also R108.1
- net A23: now also R109.1
- net A3: now also R128.1
- net A4: now also R127.1
- net A5: now also R126.1
- net A6: now also R125.1
- net A7: now also R124.1
- net A8: now also R123.1
- net A9: now also R122.1
- net GND: now also R108.2, R109.2, R110.2, R111.2, R112.2, R113.2, R114.2, R115.2, R116.2, R117.2, R118.2, R119.2, R120.2, R121.2, R122.2, R123.2, R124.2, R125.2, R126.2, R127.2, R128.2, R129.2, R130.2, R131.2

Commit message: Add files via upload
Parts:
- removed R215: 47, Resistor_SMD:R_0805_2012Metric, symbol Device:R
Connections:
- net _ECS: no longer names the net of R221.1
- no-connect marks 7 -> 8
Changed lines of the file:
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@@
   (junction (at 144.145 132.08) (diameter 0) (color 0 0 0 0)
   )
-  (junction (at 282.575 19.05) (diameter 0) (color 0 0 0 0)
-  )
   (junction (at 96.52 120.65) (diameter 0) (color 0 0 0 0)
   )
@@
   (no_connect (at 247.015 123.19))
   (no_connect (at 247.015 101.6))
+  (no_connect (at 247.015 125.73))
   (no_connect (at 247.015 106.68))
   (no_connect (at 247.015 78.74))
@@
     (stroke (width 0) (type default) (color 0 0 0 0))
   )
-  (wire (pts (xy 262.89 125.73) (xy 282.575 125.73))
-    (stroke (width 0) (type default) (color 0 0 0 0))
-  )
   (bus (pts (xy 257.175 147.32) (xy 257.175 149.86))
     (stroke (width 0) (type default) (color 0 0 0 0))
@@
     (stroke (width 0) (type default) (color 0 0 0 0))
   )
-  (wire (pts (xy 282.575 19.05) (xy 282.575 125.73))
-    (stroke (width 0) (type default) (color 0 0 0 0))
-  )
   (wire (pts (xy 158.75 154.94) (xy 149.225 154.94))
     (stroke (width 0) (type default) (color 0 0 0 0))
@@
     (stroke (width 0) (type default) (color 0 0 0 0))
   )
-  (wire (pts (xy 247.015 125.73) (xy 255.27 125.73))
-    (stroke (width 0) (type default) (color 0 0 0 0))
-  )
   (bus (pts (xy 382.27 155.575) (xy 382.27 158.115))
     (stroke (width 0) (type default) (color 0 0 0 0))
@@
     (stroke (width 0) (type default) (color 0 0 0 0))
   )
-  (wire (pts (xy 299.72 19.05) (xy 282.575 19.05))
-    (stroke (width 0) (type default) (color 0 0 0 0))
-  )
   (wire (pts (xy 52.07 170.18) (xy 50.8 170.18))
     (stroke (width 0) (type default) (color 0 0 0 0))
@@
     (stroke (width 0) (type default) (color 0 0 0 0))
   )
-  (wire (pts (xy 29.21 19.05) (xy 282.575 19.05))
-    (stroke (width 0) (type default) (color 0 0 0 0))
-  )
   (wire (pts (xy 269.875 29.21) (xy 29.21 29.21))
     (stroke (width 0) (type default) (color 0 0 0 0))
@@
     )
   )
-  (global_label "_ECS" (shape output) (at 29.21 19.05 180) (fields_autoplaced)
-    (effects (font (size 1.27 1.27)) (justify right))
-    (property "Intersheet References" "${INTERSHEET_REFS}" (id 0) (at 0 0 0)
-      (effects (font (size 1.27 1.27)) hide)
-    )
-  )
   (global_label "_CBREQ" (shape output) (at 29.21 26.67 180) (fields_autoplaced)
     (effects (font (size 1.27 1.27)) (justify right))
@@
       (effects (font (size 1.27 1.27)) hide)
     )
-    (pin "1")
-    (pin "2")
-  )
-  (symbol (lib_id "Device:R") (at 259.08 125.73 90) (unit 1)
-    (in_bom yes) (on_board yes)
-    (property "Reference" "R215" (id 0) (at 259.08 127.635 90))
-    (property "Value" "47" (id 1) (at 259.08 125.73 90))
-    (property "Footprint" "Resistor_SMD:R_0805_2012Metric" (id 2) (at 259.08 127.508 90)
-      (effects (font (size 1.27 1.27)) hide)
-    )
-    (property "Datasheet" "~" (id 3) (at 259.08 125.73 0)
-      (effects (font (size 1.27 1.27)) hide)
-    )

Commit message: Add files via upload
Parts:
- removed R221: 1K, Resistor_SMD:R_0805_2012Metric, symbol Device:R
Changed lines of the file:
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@@
   (junction (at 143.256 167.64) (diameter 0) (color 0 0 0 0)
   )
-  (junction (at 299.72 128.27) (diameter 0) (color 0 0 0 0)
-  )
   (junction (at 131.445 113.03) (diameter 0) (color 0 0 0 0)
   )
@@
     (stroke (width 0) (type default) (color 0 0 0 0))
   )
-  (wire (pts (xy 299.72 120.65) (xy 299.72 19.05))
-    (stroke (width 0) (type default) (color 0 0 0 0))
-  )
   (wire (pts (xy 309.88 42.545) (xy 103.505 42.545))
     (stroke (width 0) (type default) (color 0 0 0 0))
@@
     (stroke (width 0) (type default) (color 0 0 0 0))
   )
-  (wire (pts (xy 299.72 128.27) (xy 302.26 128.27))
+  (wire (pts (xy 297.18 128.27) (xy 302.26 128.27))
     (stroke (width 0) (type default) (color 0 0 0 0))
   )
@@
     (stroke (width 0) (type default) (color 0 0 0 0))
   )
-  (wire (pts (xy 297.18 128.27) (xy 299.72 128.27))
-    (stroke (width 0) (type default) (color 0 0 0 0))
-  )
   (bus (pts (xy 168.275 172.72) (xy 168.275 175.26))
     (stroke (width 0) (type default) (color 0 0 0 0))
@@
       (effects (font (size 1.27 1.27)) hide)
     )
-    (pin "1")
-    (pin "2")
-  )
-  (symbol (lib_id "Device:R") (at 299.72 124.46 0) (unit 1)
-    (in_bom yes) (on_board yes)
-    (property "Reference" "R221" (id 0) (at 299.72 132.969 90))
-    (property "Value" "1K" (id 1) (at 299.72 124.46 90))
-    (property "Footprint" "Resistor_SMD:R_0805_2012Metric" (id 2) (at 297.942 124.46 90)
-      (effects (font (size 1.27 1.27)) hide)
-    )
-    (property "Datasheet" "~" (id 3) (at 299.72 124.46 0)
-      (effects (font (size 1.27 1.27)) hide)
-    )

Commit message: Add files via upload
Parts:
- removed RN200: 3.3K, Resistor_THT:R_Array_SIP10, symbol Device:R_Network09
- added R228, R229, R230, R231, R232, R233, R234, R235, R236: 3.3K, Resistor_SMD:R_0805_2012Metric, symbol Device:R
Connections:
- net +5V: now also R228.2, R229.2, R230.2, R231.2, R232.2, R233.2, R234.2, R235.2, R236.2
- net FC0: now also R234.1
- net FC1: now also R233.1
- net FC2: now also R232.1
- net R_W: now also R231.1
- net SIZ0: now also R236.1
- net SIZ1: now also R235.1
- net _AS: now also R230.1
- net _CPURESET: now also R228.1
- net _DS: now also R229.1

Commit message: Add files via upload
Parts:
- renumbered JP201 to J201, JP202 to J202
Changed lines of the file:
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@@
   (symbol (lib_id "Jumper:Jumper_3_Open") (at 56.515 189.23 90) (unit 1)
     (in_bom yes) (on_board yes)
-    (property "Reference" "JP201" (id 0) (at 54.3052 188.0616 90)
+    (property "Reference" "J201" (id 0) (at 54.3052 188.0616 90)
       (effects (font (size 1.27 1.27)) (justify left))
     )
@@
   (symbol (lib_id "Jumper:Jumper_3_Open") (at 125.095 252.73 90) (mirror x) (unit 1)
     (in_bom yes) (on_board yes)
-    (property "Reference" "JP202" (id 0) (at 122.8852 253.8984 90)
+    (property "Reference" "J202" (id 0) (at 122.8852 253.8984 90)
       (effects (font (size 1.27 1.27)) (justify left))
     )

Commit message: Add files via upload
Parts:
- added unit 4 of U204
Connections:
- net SIZ0: now also R235.1, U200.120 (SIZ0); no longer R236.1, U200.119 (SIZ1)
- net SIZ1: now also R236.1, U200.119 (SIZ1); no longer R235.1, U200.120 (SIZ0)
- net at C213.1, R211.2: now also U204.8; no longer R203.1
- new net: R203.1, U204.9
Other:
- moved on the sheet: C213, R211
Changed lines of the file:
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@@
   (junction (at 208.915 236.22) (diameter 0) (color 0 0 0 0)
   )
+  (junction (at 80.01 241.935) (diameter 0) (color 0 0 0 0)
+  )
   (junction (at 229.235 236.22) (diameter 0) (color 0 0 0 0)
   )
@@
   (junction (at 143.256 218.44) (diameter 0) (color 0 0 0 0)
   )
-  (junction (at 64.135 241.935) (diameter 0) (color 0 0 0 0)
-  )
   (junction (at 144.145 132.08) (diameter 0) (color 0 0 0 0)
   )
@@
     (stroke (width 0) (type default) (color 0 0 0 0))
   )
-  (wire (pts (xy 92.71 241.935) (xy 78.105 241.935))
+  (wire (pts (xy 92.71 241.935) (xy 89.535 241.935))
     (stroke (width 0) (type default) (color 0 0 0 0))
   )
@@
     (stroke (width 0) (type default) (color 0 0 0 0))
   )
-  (wire (pts (xy 70.485 241.935) (xy 64.135 241.935))
+  (wire (pts (xy 81.915 241.935) (xy 80.01 241.935))
     (stroke (width 0) (type default) (color 0 0 0 0))
   )
@@
     (stroke (width 0) (type default) (color 0 0 0 0))
   )
-  (wire (pts (xy 64.135 241.935) (xy 59.055 241.935))
+  (wire (pts (xy 59.055 241.935) (xy 60.96 241.935))
     (stroke (width 0) (type default) (color 0 0 0 0))
   )
@@
     (stroke (width 0) (type default) (color 0 0 0 0))
   )
+  (wire (pts (xy 76.2 241.935) (xy 80.01 241.935))
+    (stroke (width 0) (type default) (color 0 0 0 0))
+  )
   (wire (pts (xy 108.585 100.33) (xy 177.165 100.33))
     (stroke (width 0) (type default) (color 0 0 0 0))
@@
     )
   )
-  (global_label "SIZ0" (shape bidirectional) (at 29.21 140.97 180) (fields_autoplaced)
+  (global_label "SIZ0" (shape bidirectional) (at 29.21 138.43 180) (fields_autoplaced)
     (effects (font (size 1.27 1.27)) (justify right))
-    (property "Intersheet References" "${INTERSHEET_REFS}" (id 0) (at 0 0 0)
+    (property "Intersheet References" "${INTERSHEET_REFS}" (id 0) (at 0 -2.54 0)
       (effects (font (size 1.27 1.27)) hide)
     )
@@
     )
   )
-  (global_label "SIZ1" (shape bidirectional) (at 29.21 138.43 180) (fields_autoplaced)
+  (global_label "SIZ1" (shape bidirectional) (at 29.21 140.97 180) (fields_autoplaced)
     (effects (font (size 1.27 1.27)) (justify right))
-    (property "Intersheet References" "${INTERSHEET_REFS}" (id 0) (at 0 0 0)
+    (property "Intersheet References" "${INTERSHEET_REFS}" (id 0) (at 0 2.54 0)
       (effects (font (size 1.27 1.27)) hide)
     )
@@
     (pin "9")
   )
-  (symbol (lib_id "Device:R") (at 74.295 241.935 270) (unit 1)
+  (symbol (lib_id "Device:R") (at 85.725 241.935 270) (unit 1)
     (in_bom yes) (on_board yes)
-    (property "Reference" "R211" (id 0) (at 74.295 240.03 90))
-    (property "Value" "68" (id 1) (at 74.295 241.935 90))
-    (property "Footprint" "Resistor_SMD:R_0805_2012Metric" (id 2) (at 74.295 240.157 90)
+    (property "Reference" "R211" (id 0) (at 85.725 240.03 90))
+    (property "Value" "68" (id 1) (at 85.725 241.935 90))
+    (property "Footprint" "Resistor_SMD:R_0805_2012Metric" (id 2) (at 85.725 240.157 90)
       (effects (font (size 1.27 1.27)) hide)
     )
-    (property "Datasheet" "~" (id 3) (at 74.295 241.935 0)
+    (property "Datasheet" "~" (id 3) (at 85.725 241.935 0)
       (effects (font (size 1.27 1.27)) hide)
     )
@@
     (pin "2")
   )
-  (symbol (lib_id "Device:C") (at 64.135 245.745 0) (unit 1)
+  (symbol (lib_id "Device:C") (at 80.01 245.745 0) (unit 1)
     (in_bom yes) (on_board yes)
-    (property "Reference" "C213" (id 0) (at 67.056 244.5766 0)
+    (property "Reference" "C213" (id 0) (at 82.931 244.5766 0)
       (effects (font (size 1.27 1.27)) (justify left))
     )
-    (property "Value" "22pF" (id 1) (at 67.056 246.888 0)
+    (property "Value" "22pF" (id 1) (at 82.931 246.888 0)
       (effects (font (size 1.27 1.27)) (justify left))
     )
-    (property "Footprint" "Capacitor_SMD:C_0805_2012Metric" (id 2) (at 65.1002 249.555 0)
+    (property "Footprint" "Capacitor_SMD:C_0805_2012Metric" (id 2) (at 80.9752 249.555 0)
       (effects (font (size 1.27 1.27)) hide)
     )
-    (property "Datasheet" "~" (id 3) (at 64.135 245.745 0)
+    (property "Datasheet" "~" (id 3) (at 80.01 245.745 0)
       (effects (font (size 1.27 1.27)) hide)
     )
@@
     (pin "2")
   )
-  (symbol (lib_id "power:GND") (at 64.135 249.555 0) (unit 1)
+  (symbol (lib_id "power:GND") (at 80.01 249.555 0) (unit 1)
     (in_bom yes) (on_board yes)
-    (property "Reference" "#PWR0147" (id 0) (at 64.135 255.905 0)
+    (property "Reference" "#PWR0147" (id 0) (at 80.01 255.905 0)
       (effects (font (size 1.27 1.27)) hide)
     )
-    (property "Value" "GND" (id 1) (at 64.262 253.9492 0))
-    (property "Footprint" "" (id 2) (at 64.135 249.555 0)
+    (property "Value" "GND" (id 1) (at 80.137 253.9492 0))
+    (property "Footprint" "" (id 2) (at 80.01 249.555 0)
       (effects (font (size 1.27 1.27)) hide)
     )
-    (property "Datasheet" "" (id 3) (at 64.135 249.555 0)
+    (property "Datasheet" "" (id 3) (at 80.01 249.555 0)
       (effects (font (size 1.27 1.27)) hide)
     )
@@
     (pin "2")
   )
+  (symbol (lib_id "74xx:74HCT04") (at 68.58 241.935 0) (unit 4)
+    (in_bom yes) (on_board yes)
+    (property "Reference" "U204" (id 0) (at 68.58 233.8832 0))
+    (property "Value" "74HCT04" (id 1) (at 68.58 236.1946 0))
+    (property "Footprint" "Package_SO:SOIC-14_3.9x8.7mm_P1.27mm" (id 2) (at 68.58 241.935 0)
+      (effects (font (size 1.27 1.27)) hide)
+    )
+    (property "Datasheet" "https://assets.nexperia.com/documents/data-sheet/74HC_HCT04.pdf" (id 3) (at 68.58 241.935 0)
+      (effects (font (size 1.27 1.27)) hide)
+    )
+    (property "Digikey" "296-31832-1-ND" (id 4) (at 68.58 241.935 0)
+      (effects (font (size 1.27 1.27)) hide)
+    )
+    (pin "8")
+    (pin "9")
+  )
   (symbol (lib_id "Device:R") (at 147.066 180.34 270) (unit 1)
