File: A2630-New-KiCAD6/BaseMemory.kicad_sch (KiCad schematic)
At the start: 13 parts, among them U400 CY7C1061G, U401 CY7C1061G, U402 CY7C1061G, U403 CY7C1061G, U404 CY74FCT821T, U405 CY74FCT821T

Commit message: Add files via upload
Other:
- note added: "This is Zorro 2 memory, so it is always treated as 16 bit, even though it is 32 bits wide."
Changed lines of the file:
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@@
     (effects (font (size 2.9972 2.9972)) (justify left bottom))
+  )
+  (text "This is Zorro 2 memory, so it is \nalways treated as 16 bit, even \nthough it is 32 bits wide."
+    (at 50.8 45.085 0)
+    (effects (font (size 3 3)) (justify left bottom))
   )
   (text "BANK1" (at 273.558 48.387 180)
