File: A2630-New-KiCAD6/CPLD1.kicad_sch (KiCad schematic)
At the start: 17 parts, among them CN1 CPLD0, CN2 CPLD1, CN3 CPLD1, U600 XC9572XL-TQ100, U601 XC9572XL-TQ100, U602 XC9572XL-TQ100

Commit message: Add files via upload
Connections:
- net A22: now also U602.53 (P53)
- net A23: now also U602.54 (P54); no longer U602.53 (P53)
- net A24: now also U602.55 (P55); no longer U602.54 (P54)
- net A25: now also U602.56 (P56); no longer U602.55 (P55)
- net A26: now also U602.58 (P58); no longer U602.56 (P56)
- net _PRECHARGE: now reaches U602.72 (P72)
Other:
- note added: "When A23 is HIGH, we are in the second 64 MB memory space."
Changed lines of the file:
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@@
+    (stroke (width 0) (type default) (color 0 0 0 0))
+  )
+  (bus_entry (at 365.125 114.935) (size 2.54 -2.54)
     (stroke (width 0) (type default) (color 0 0 0 0))
   )
@@
     (stroke (width 0) (type default) (color 0 0 0 0))
   )
+  (bus (pts (xy 367.665 109.855) (xy 367.665 112.395))
+    (stroke (width 0) (type default) (color 0 0 0 0))
+  )
   (wire (pts (xy 361.95 188.595) (xy 346.075 188.595))
     (stroke (width 0) (type default) (color 0 0 0 0))
@@
     (stroke (width 0) (type default) (color 0 0 0 0))
   )
+  (wire (pts (xy 365.125 114.935) (xy 346.075 114.935))
+    (stroke (width 0) (type default) (color 0 0 0 0))
+  )
   (wire (pts (xy 113.03 207.645) (xy 108.585 207.645))
     (stroke (width 0) (type default) (color 0 0 0 0))
@@
     (stroke (width 0) (type default) (color 0 0 0 0))
   )
+  (wire (pts (xy 346.075 147.955) (xy 354.965 147.955))
+    (stroke (width 0) (type default) (color 0 0 0 0))
+  )
   (wire (pts (xy 78.74 241.935) (xy 71.12 241.935))
     (stroke (width 0) (type default) (color 0 0 0 0))
@@
   (wire (pts (xy 354.965 173.355) (xy 346.075 173.355))
     (stroke (width 0) (type default) (color 0 0 0 0))
+  )
+  (text "When A23 is HIGH, we are in the \nsecond 64 MB memory space."
+    (at 290.83 27.305 0)
+    (effects (font (size 4 4)) (justify left bottom))
   )
   (text "CPLDs" (at 341.63 245.745 180)
@@
     (effects (font (size 1.27 1.27)) (justify right bottom))
   )
+  (label "A26" (at 365.125 114.935 180)
+    (effects (font (size 1.27 1.27)) (justify right bottom))
+  )
   (label "TMS1" (at 361.95 186.055 180)
     (effects (font (size 1.27 1.27)) (justify right bottom))
@@
     (effects (font (size 1.27 1.27)) (justify right bottom))
   )
-  (label "A23" (at 365.125 104.775 180)
-    (effects (font (size 1.27 1.27)) (justify right bottom))
-  )
-  (label "A25" (at 365.125 109.855 180)
+  (label "A22" (at 365.125 104.775 180)
+    (effects (font (size 1.27 1.27)) (justify right bottom))
+  )
+  (label "A24" (at 365.125 109.855 180)
     (effects (font (size 1.27 1.27)) (justify right bottom))
   )
@@
     (effects (font (size 1.27 1.27)) (justify left bottom))
   )
-  (label "A24" (at 365.125 107.315 180)
+  (label "A23" (at 365.125 107.315 180)
     (effects (font (size 1.27 1.27)) (justify right bottom))
   )
@@
     (effects (font (size 1.27 1.27)) (justify left bottom))
   )
-  (label "A26" (at 365.125 112.395 180)
+  (label "A25" (at 365.125 112.395 180)
     (effects (font (size 1.27 1.27)) (justify right bottom))
   )
@@
     )
   )
+  (global_label "_PRECHARGE" (shape output) (at 354.965 147.955 0) (fields_autoplaced)
+    (effects (font (size 1.27 1.27)) (justify left))
+    (property "Intersheet References" "${INTERSHEET_REFS}" (id 0) (at 369.324 147.8756 0)
+      (effects (font (size 1.27 1.27)) (justify left) hide)
+    )
+  )
