File: A2630-New-KiCAD6/ExpansionMemory.kicad_sch (KiCad schematic)
At the start: 16 parts, among them U102 27C256, U103 27C256, U406 SDRAM_512Mb(32Mx16), U407 SDRAM_512Mb(32Mx16), U408 SDRAM_512Mb(32Mx16), U409 SDRAM_512Mb(32Mx16)

Commit message: Add files via upload
Other:
- note added: "TRIVIA: A31..24 is the autoconfig base address A1..0 are part of the sizing system for mem This leaves A23..A2 for actual addressing...22 bits. This is why the Amiga can only address 128 megabytes!"
- note added: "This is Zorro 3 memory, so it is always treated as 32 bit memory and cannot be used by the Amiga 2000 chip set and cannot be used by anything on the Zoroo 2 bus. It can only be used by the 68030."
Changed lines of the file:
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@@
     (effects (font (size 5.9944 5.9944)) (justify left bottom))
+  )
+  (text "This is Zorro 3 memory, so it is always\ntreated as 32 bit memory and cannot be \nused by the Amiga 2000 chip set and cannot\nbe used by anything on the Zoroo 2 bus.\nIt can only be used by the 68030."
+    (at 274.955 153.67 0)
+    (effects (font (size 3 3)) (justify left bottom))
   )
   (text "LOW_BYTE" (at 24.13 81.28 0)
@@
   (text "ROMs" (at 285.75 52.07 0)
     (effects (font (size 3.9878 3.9878)) (justify left bottom))
+  )
+  (text "TRIVIA:\nA31..24 is the autoconfig base address\nA1..0 are part of the sizing system for mem\nThis leaves A23..A2 for actual addressing...22 bits.\nThis is why the Amiga can only address 128 megabytes!"
+    (at 144.78 37.465 0)
+    (effects (font (size 3 3)) (justify left bottom))
   )
   (text "JN Notes: put row address on the EMA bus \nand signal RAS. This is 68030 addresses A14:2. \nPut column address on the EMA bus and signal \nCAS. These are 68030 addresses A24:15."
@@
     )
   )
-  (global_label "EMA(12..0)" (shape input) (at 34.29 27.94 180) (fields_autoplaced)
+  (global_label "EMA[12..0]" (shape input) (at 34.29 27.94 180) (fields_autoplaced)
     (effects (font (size 1.27 1.27)) (justify right))
-    (property "Intersheet References" "${INTERSHEET_REFS}" (id 0) (at 0 0 0)
-      (effects (font (size 1.27 1.27)) hide)
+    (property "Intersheet References" "${INTERSHEET_REFS}" (id 0) (at 21.7453 27.8606 0)
+      (effects (font (size 1.27 1.27)) (justify right) hide)
     )
   )
