File: A2630-New-KiCAD6/Logic.kicad_sch (KiCad schematic)
At the start: 24 parts, among them U300 74HCT05, U303 74HCT174, U307 74HCT04, U410 74LVC257, U411 74LVC257, U412 74LVC257, U413 74LVC257, U502 74HCT74, U503 74HCT74, U507 74HCT74, U606 74HCT244

Commit message: Add files via upload
Other:
- note added: "DISCRETE LOGIC STUFF"
- note removed: "DISCRETE LOGIC BITS"
Changed lines of the file:
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@@
     (effects (font (size 2.9972 2.9972)) (justify left bottom))
   )
-  (text "DISCRETE LOGIC BITS" (at 313.69 244.475 0)
+  (text "DISCRETE LOGIC STUFF" (at 313.69 244.475 0)
     (effects (font (size 5.9944 5.9944)) (justify left bottom))
   )
