File: A2630-New-KiCAD-Rev1/Power.kicad_sch (KiCad schematic)
At the start: 36 parts, among them CN4 CPLD3, CN5 ATA/IDE, CN6 LED, J600 IDE DISABLE, U204 74HCT04, U300 74HCT05, U307 74HCT04, U507 74HCT74, U603 XC9572XL-VQ64, U606 74HCT244, U800 LM1117-3.3

Commit message: Add files via upload
Connections:
- net A12: now also U603.5 (I/O/GTS1); no longer U603.8 (P8)
- net A13: now also U603.4 (P4); no longer U603.7 (P7)
- net A14: now also U603.63 (P63); no longer U603.6 (P6)
- net A15: now also U603.62 (P62); no longer U603.5 (I/O/GTS1)
- net A16: now also U603.60 (P60); no longer U603.4 (P4)
- net A2: now also U603.1 (P1); no longer U603.62 (P62)
- net A21: now also U603.59 (P59); no longer U603.2 (I/O/GTS2)
- net A3: now also U603.2 (I/O/GTS2); no longer U603.63 (P63)
- net A4: now also U603.58 (P58); no longer U603.1 (P1)
- net R_W: now also U603.6 (P6); no longer U603.58 (P58)
- net _AS: now also U603.7 (P7); no longer U603.59 (P59)
- net _DS: now also U603.8 (P8); no longer U603.60 (P60)
Changed lines of the file:
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@@
     (stroke (width 0) (type default) (color 0 0 0 0))
   )
-  (bus_entry (at 113.665 55.245) (size 2.54 2.54)
+  (bus_entry (at 113.665 111.125) (size 2.54 2.54)
     (stroke (width 0) (type default) (color 0 0 0 0))
   )
@@
     (stroke (width 0) (type default) (color 0 0 0 0))
   )
-  (bus_entry (at 113.665 100.965) (size 2.54 2.54)
-    (stroke (width 0) (type default) (color 0 0 0 0))
-  )
-  (bus_entry (at 113.665 103.505) (size 2.54 2.54)
+  (bus_entry (at 113.665 106.045) (size 2.54 2.54)
+    (stroke (width 0) (type default) (color 0 0 0 0))
+  )
+  (bus_entry (at 113.665 108.585) (size 2.54 2.54)
     (stroke (width 0) (type default) (color 0 0 0 0))
   )
@@
     (stroke (width 0) (type default) (color 0 0 0 0))
   )
+  (bus (pts (xy 113.665 108.585) (xy 113.665 111.125))
+    (stroke (width 0) (type default) (color 0 0 0 0))
+  )
   (wire (pts (xy 391.16 120.015) (xy 367.03 120.015))
     (stroke (width 0) (type default) (color 0 0 0 0))
@@
     (stroke (width 0) (type default) (color 0 0 0 0))
   )
-  (bus (pts (xy 113.665 103.505) (xy 113.665 116.205))
+  (bus (pts (xy 113.665 106.045) (xy 113.665 108.585))
     (stroke (width 0) (type default) (color 0 0 0 0))
   )
@@
     (stroke (width 0) (type default) (color 0 0 0 0))
   )
-  (bus (pts (xy 113.665 57.785) (xy 113.665 55.245))
-    (stroke (width 0) (type default) (color 0 0 0 0))
-  )
   (wire (pts (xy 88.265 107.315) (xy 98.425 107.315))
     (stroke (width 0) (type default) (color 0 0 0 0))
@@
     (stroke (width 0) (type default) (color 0 0 0 0))
   )
-  (wire (pts (xy 127.635 57.785) (xy 116.205 57.785))
+  (wire (pts (xy 127.635 113.665) (xy 116.205 113.665))
     (stroke (width 0) (type default) (color 0 0 0 0))
   )
@@
     (stroke (width 0) (type default) (color 0 0 0 0))
   )
-  (bus (pts (xy 113.665 98.425) (xy 113.665 100.965))
+  (bus (pts (xy 113.665 98.425) (xy 113.665 106.045))
     (stroke (width 0) (type default) (color 0 0 0 0))
   )
@@
     (stroke (width 0) (type default) (color 0 0 0 0))
   )
-  (wire (pts (xy 127.635 103.505) (xy 116.205 103.505))
+  (wire (pts (xy 127.635 108.585) (xy 116.205 108.585))
     (stroke (width 0) (type default) (color 0 0 0 0))
   )
@@
     (stroke (width 0) (type default) (color 0 0 0 0))
   )
-  (wire (pts (xy 121.92 108.585) (xy 127.635 108.585))
+  (wire (pts (xy 121.92 103.505) (xy 127.635 103.505))
     (stroke (width 0) (type default) (color 0 0 0 0))
   )
@@
     (stroke (width 0) (type default) (color 0 0 0 0))
   )
+  (bus (pts (xy 113.665 111.125) (xy 113.665 116.205))
+    (stroke (width 0) (type default) (color 0 0 0 0))
+  )
   (wire (pts (xy 53.34 104.775) (xy 53.34 102.235))
     (stroke (width 0) (type default) (color 0 0 0 0))
@@
     (stroke (width 0) (type default) (color 0 0 0 0))
   )
-  (wire (pts (xy 121.92 113.665) (xy 127.635 113.665))
+  (wire (pts (xy 121.92 57.785) (xy 127.635 57.785))
     (stroke (width 0) (type default) (color 0 0 0 0))
   )
@@
     (stroke (width 0) (type default) (color 0 0 0 0))
   )
-  (bus (pts (xy 113.665 100.965) (xy 113.665 103.505))
-    (stroke (width 0) (type default) (color 0 0 0 0))
-  )
   (wire (pts (xy 249.555 118.11) (xy 249.555 124.46))
     (stroke (width 0) (type default) (color 0 0 0 0))
@@
     (stroke (width 0) (type default) (color 0 0 0 0))
   )
-  (wire (pts (xy 121.92 111.125) (xy 127.635 111.125))
+  (wire (pts (xy 121.92 106.045) (xy 127.635 106.045))
     (stroke (width 0) (type default) (color 0 0 0 0))
   )
@@
     (stroke (width 0) (type default) (color 0 0 0 0))
   )
-  (wire (pts (xy 127.635 106.045) (xy 116.205 106.045))
+  (wire (pts (xy 127.635 111.125) (xy 116.205 111.125))
     (stroke (width 0) (type default) (color 0 0 0 0))
   )
@@
     (effects (font (size 1.27 1.27)) (justify right bottom))
   )
-  (label "A3" (at 116.205 121.285 0)
+  (label "A3" (at 116.205 95.885 0)
     (effects (font (size 1.27 1.27)) (justify left bottom))
   )
@@
     (effects (font (size 1.27 1.27)) (justify left bottom))
   )
-  (label "A15" (at 116.205 100.965 0)
+  (label "A15" (at 116.205 118.745 0)
     (effects (font (size 1.27 1.27)) (justify left bottom))
   )
@@
     (effects (font (size 1.27 1.27)) (justify right bottom))
   )
-  (label "A16" (at 116.205 98.425 0)
-    (effects (font (size 1.27 1.27)) (justify left bottom))
-  )
-  (label "A21" (at 116.205 95.885 0)
+  (label "A16" (at 116.205 113.665 0)
+    (effects (font (size 1.27 1.27)) (justify left bottom))
+  )
+  (label "A21" (at 116.205 111.125 0)
     (effects (font (size 1.27 1.27)) (justify left bottom))
   )
@@
     (effects (font (size 1.27 1.27)) (justify right bottom))
   )
-  (label "A14" (at 116.205 103.505 0)
+  (label "A14" (at 116.205 121.285 0)
     (effects (font (size 1.27 1.27)) (justify left bottom))
   )
@@
     (effects (font (size 1.27 1.27)) (justify right bottom))
   )
-  (label "A13" (at 116.205 106.045 0)
+  (label "A13" (at 116.205 98.425 0)
     (effects (font (size 1.27 1.27)) (justify left bottom))
   )
@@
     (effects (font (size 1.27 1.27)) (justify left bottom))
   )
-  (label "A4" (at 116.205 93.345 0)
+  (label "A4" (at 116.205 108.585 0)
     (effects (font (size 1.27 1.27)) (justify left bottom))
   )
@@
     (effects (font (size 1.27 1.27)) (justify left bottom))
   )
-  (label "A12" (at 116.205 57.785 0)
+  (label "A12" (at 116.205 100.965 0)
     (effects (font (size 1.27 1.27)) (justify left bottom))
   )
@@
     (effects (font (size 1.27 1.27)) (justify left bottom))
   )
-  (label "A2" (at 116.205 118.745 0)
+  (label "A2" (at 116.205 93.345 0)
     (effects (font (size 1.27 1.27)) (justify left bottom))
   )
@@
     )
   )
-  (global_label "R_W" (shape input) (at 121.92 108.585 180) (fields_autoplaced)
+  (global_label "R_W" (shape input) (at 121.92 103.505 180) (fields_autoplaced)
     (effects (font (size 1.27 1.27)) (justify right))
-    (property "Intersheet References" "${INTERSHEET_REFS}" (id 0) (at 115.9068 108.5056 0)
+    (property "Intersheet References" "${INTERSHEET_REFS}" (id 0) (at 115.9068 103.4256 0)
       (effects (font (size 1.27 1.27)) (justify right) hide)
     )
   )
-  (global_label "_AS" (shape input) (at 121.92 111.125 180) (fields_autoplaced)
+  (global_label "_AS" (shape input) (at 121.92 106.045 180) (fields_autoplaced)
     (effects (font (size 1.27 1.27)) (justify right))
-    (property "Intersheet References" "${INTERSHEET_REFS}" (id 0) (at 116.3301 111.2044 0)
+    (property "Intersheet References" "${INTERSHEET_REFS}" (id 0) (at 116.3301 106.1244 0)
       (effects (font (size 1.27 1.27)) (justify right) hide)
     )
@@
     )
   )
-  (global_label "_DS" (shape input) (at 121.92 113.665 180) (fields_autoplaced)
+  (global_label "_DS" (shape input) (at 121.92 57.785 180) (fields_autoplaced)
     (effects (font (size 1.27 1.27)) (justify right))
-    (property "Intersheet References" "${INTERSHEET_REFS}" (id 0) (at 116.1487 113.7444 0)
+    (property "Intersheet References" "${INTERSHEET_REFS}" (id 0) (at 116.1487 57.8644 0)
       (effects (font (size 1.27 1.27)) (justify right) hide)
     )

Commit message: Add files via upload
Parts:
- removed U204: 74HCT04, Package_SO:SOIC-14_3.9x8.7mm_P1.27mm, symbol 74xx:74HCT04
- removed U307: 74HCT04, Package_SO:SOIC-14_3.9x8.7mm_P1.27mm, symbol 74xx:74LS04
Connections:
- no-connect marks 27 -> 21
Other:
- moved on the sheet: U300C, U300F

Commit message: Add files via upload
Other:
- company: (none) -> Drawn By: Jason Neus
- title: (none) -> Amiga N2630

Commit message: Add files via upload
Parts:
- C800, C801: value 10uF -> (none); footprint Resistor_SMD:R_0805_2012Metric -> (none)
Changed lines of the file:
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@@
       (effects (font (size 1.27 1.27)) (justify left))
     )
-    (property "Value" "10uF" (id 1) (at 269.621 48.768 0)
+    (property "Value" "" (id 1) (at 269.621 48.768 0)
       (effects (font (size 1.27 1.27)) (justify left))
     )
-    (property "Footprint" "Resistor_SMD:R_0805_2012Metric" (id 2) (at 267.6652 51.435 0)
+    (property "Footprint" "" (id 2) (at 267.6652 51.435 0)
       (effects (font (size 1.27 1.27)) hide)
     )
@@
       (effects (font (size 1.27 1.27)) (justify left))
     )
-    (property "Value" "10uF" (id 1) (at 241.046 48.768 0)
+    (property "Value" "" (id 1) (at 241.046 48.768 0)
       (effects (font (size 1.27 1.27)) (justify left))
     )
-    (property "Footprint" "Resistor_SMD:R_0805_2012Metric" (id 2) (at 239.0902 51.435 0)
+    (property "Footprint" "" (id 2) (at 239.0902 51.435 0)
       (effects (font (size 1.27 1.27)) hide)
     )

Commit message: Add files via upload
Parts:
- C800, C801: value (none) -> 10uF; footprint (none) -> Capacitor_SMD:C_0805_2012Metric
- U507: value 74HCT74 -> (none)
Changed lines of the file:
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@@
       (effects (font (size 1.27 1.27)) (justify left))
     )
-    (property "Value" "" (id 1) (at 269.621 48.768 0)
-      (effects (font (size 1.27 1.27)) (justify left))
-    )
-    (property "Footprint" "" (id 2) (at 267.6652 51.435 0)
+    (property "Value" "10uF" (id 1) (at 269.621 48.768 0)
+      (effects (font (size 1.27 1.27)) (justify left))
+    )
+    (property "Footprint" "Capacitor_SMD:C_0805_2012Metric" (id 2) (at 267.6652 51.435 0)
       (effects (font (size 1.27 1.27)) hide)
     )
@@
       (effects (font (size 1.27 1.27)) (justify left))
     )
-    (property "Value" "" (id 1) (at 241.046 48.768 0)
-      (effects (font (size 1.27 1.27)) (justify left))
-    )
-    (property "Footprint" "" (id 2) (at 239.0902 51.435 0)
+    (property "Value" "10uF" (id 1) (at 241.046 48.768 0)
+      (effects (font (size 1.27 1.27)) (justify left))
+    )
+    (property "Footprint" "Capacitor_SMD:C_0805_2012Metric" (id 2) (at 239.0902 51.435 0)
       (effects (font (size 1.27 1.27)) hide)
     )
@@
     (in_bom yes) (on_board yes)
     (property "Reference" "U507" (id 0) (at 378.46 132.08 0))
-    (property "Value" "74HCT74" (id 1) (at 379.73 133.985 0))
+    (property "Value" "" (id 1) (at 379.73 133.985 0))
     (property "Footprint" "Package_SO:SOIC-14_3.9x8.7mm_P1.27mm" (id 2) (at 374.65 140.335 0)
       (effects (font (size 1.27 1.27)) hide)

Commit message: Add files via upload
Parts:
- U507: value (none) -> 74AHCT74
Changed lines of the file:
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@@
     (in_bom yes) (on_board yes)
     (property "Reference" "U507" (id 0) (at 378.46 132.08 0))
-    (property "Value" "" (id 1) (at 379.73 133.985 0))
+    (property "Value" "74AHCT74" (id 1) (at 379.73 133.985 0))
     (property "Footprint" "Package_SO:SOIC-14_3.9x8.7mm_P1.27mm" (id 2) (at 374.65 140.335 0)
       (effects (font (size 1.27 1.27)) hide)

Commit message: Add files via upload
Parts:
- removed unit 3 of U300
Changed lines of the file:
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@@
   (junction (at 292.735 86.36) (diameter 0) (color 0 0 0 0)
-  )
-  (junction (at 367.03 53.34) (diameter 0) (color 0 0 0 0)
   )
   (junction (at 367.03 111.125) (diameter 0) (color 0 0 0 0)
@@
     (stroke (width 0) (type default) (color 0 0 0 0))
   )
-  (wire (pts (xy 367.03 39.37) (xy 367.03 53.34))
-    (stroke (width 0) (type default) (color 0 0 0 0))
-  )
   (bus (pts (xy 113.665 75.565) (xy 113.665 95.885))
     (stroke (width 0) (type default) (color 0 0 0 0))
@@
     (stroke (width 0) (type default) (color 0 0 0 0))
   )
-  (wire (pts (xy 367.03 53.34) (xy 367.03 67.31))
+  (wire (pts (xy 367.03 39.37) (xy 367.03 67.31))
     (stroke (width 0) (type default) (color 0 0 0 0))
   )
@@
     (pin "1")
   )
-  (symbol (lib_id "74xx:74LS05") (at 374.65 53.34 0) (unit 3)
-    (in_bom yes) (on_board yes)
-    (property "Reference" "U300" (id 0) (at 374.65 45.72 0))
-    (property "Value" "74HCT05" (id 1) (at 374.65 48.26 0))
-    (property "Footprint" "Package_SO:SOIC-14_3.9x8.7mm_P1.27mm" (id 2) (at 374.65 53.34 0)
-      (effects (font (size 1.27 1.27)) hide)
-    )
-    (property "Datasheet" "http://www.ti.com/lit/gpn/sn74LS05" (id 3) (at 374.65 53.34 0)
-      (effects (font (size 1.27 1.27)) hide)
-    )
-    (pin "1")
-    (pin "2")
-    (pin "3")
-    (pin "4")
-    (pin "5")
-    (pin "6")
-    (pin "8")
-    (pin "9")
-    (pin "10")
-    (pin "11")
-    (pin "12")
-    (pin "13")
-    (pin "14")
-    (pin "7")
-  )
   (symbol (lib_id "Device:CP") (at 318.135 47.625 0) (unit 1)
