File: A2630-New-KiCAD-Rev1/ExpansionMemory.kicad_sch (KiCad schematic)
At the start: 21 parts, among them U102 27C256, U103 27C256, U406 SDRAM_256Mb(16Mx16), U407 SDRAM_256Mb(16Mx16), U408 SDRAM_256Mb(16Mx16), U409 SDRAM_256Mb(16Mx16)

Commit message: Add files via upload
Other:
- company: (none) -> Drawn By: Jason Neus
- title: (none) -> Amiga N2630
Changed lines of the file:
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@@
 (kicad_sch (version 20211123) (generator eeschema)
   (paper "B")
+  (title_block
+    (title "Amiga N2630")
+    (date "2022-03-25")
+    (rev "1.0")
+    (company "Drawn By: Jason Neus")
+  )
   (junction (at 346.075 29.21) (diameter 0) (color 0 0 0 0)
   )

Commit message: Add files via upload
Parts:
- U406, U407, U408, U409: value SDRAM_256Mb(16Mx16) -> (none)
Changed lines of the file:
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@@
     (in_bom yes) (on_board yes)
     (property "Reference" "U406" (id 0) (at 107.95 92.71 0))
-    (property "Value" "SDRAM_256Mb(16Mx16)" (id 1) (at 107.95 97.79 0))
+    (property "Value" "" (id 1) (at 107.95 97.79 0))
     (property "Footprint" "Package_SO:TSOP-II-54_22.2x10.16mm_P0.8mm" (id 2) (at 107.95 92.71 0)
       (effects (font (size 1.27 1.27) italic) hide)
@@
     (in_bom yes) (on_board yes)
     (property "Reference" "U407" (id 0) (at 107.95 184.15 0))
-    (property "Value" "SDRAM_256Mb(16Mx16)" (id 1) (at 107.95 189.23 0))
+    (property "Value" "" (id 1) (at 107.95 189.23 0))
     (property "Footprint" "Package_SO:TSOP-II-54_22.2x10.16mm_P0.8mm" (id 2) (at 107.95 184.15 0)
       (effects (font (size 1.27 1.27) italic) hide)
@@
     (in_bom yes) (on_board yes)
     (property "Reference" "U408" (id 0) (at 209.55 92.71 0))
-    (property "Value" "SDRAM_256Mb(16Mx16)" (id 1) (at 209.55 97.79 0))
+    (property "Value" "" (id 1) (at 209.55 97.79 0))
     (property "Footprint" "Package_SO:TSOP-II-54_22.2x10.16mm_P0.8mm" (id 2) (at 209.55 92.71 0)
       (effects (font (size 1.27 1.27) italic) hide)
@@
     (in_bom yes) (on_board yes)
     (property "Reference" "U409" (id 0) (at 209.55 184.15 0))
-    (property "Value" "SDRAM_256Mb(16Mx16)" (id 1) (at 209.55 189.23 0))
+    (property "Value" "" (id 1) (at 209.55 189.23 0))
     (property "Footprint" "Package_SO:TSOP-II-54_22.2x10.16mm_P0.8mm" (id 2) (at 209.55 184.15 0)
       (effects (font (size 1.27 1.27) italic) hide)

Commit message: Add files via upload
Parts:
- U406, U407, U408, U409: value (none) -> SDRAM(16Mx16)
Changed lines of the file:
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@@
     (in_bom yes) (on_board yes)
     (property "Reference" "U406" (id 0) (at 107.95 92.71 0))
-    (property "Value" "" (id 1) (at 107.95 97.79 0))
+    (property "Value" "SDRAM(16Mx16)" (id 1) (at 107.95 97.79 0))
     (property "Footprint" "Package_SO:TSOP-II-54_22.2x10.16mm_P0.8mm" (id 2) (at 107.95 92.71 0)
       (effects (font (size 1.27 1.27) italic) hide)
@@
     (in_bom yes) (on_board yes)
     (property "Reference" "U407" (id 0) (at 107.95 184.15 0))
-    (property "Value" "" (id 1) (at 107.95 189.23 0))
+    (property "Value" "SDRAM(16Mx16)" (id 1) (at 107.95 189.23 0))
     (property "Footprint" "Package_SO:TSOP-II-54_22.2x10.16mm_P0.8mm" (id 2) (at 107.95 184.15 0)
       (effects (font (size 1.27 1.27) italic) hide)
@@
     (in_bom yes) (on_board yes)
     (property "Reference" "U408" (id 0) (at 209.55 92.71 0))
-    (property "Value" "" (id 1) (at 209.55 97.79 0))
+    (property "Value" "SDRAM(16Mx16)" (id 1) (at 209.55 97.79 0))
     (property "Footprint" "Package_SO:TSOP-II-54_22.2x10.16mm_P0.8mm" (id 2) (at 209.55 92.71 0)
       (effects (font (size 1.27 1.27) italic) hide)
@@
     (in_bom yes) (on_board yes)
     (property "Reference" "U409" (id 0) (at 209.55 184.15 0))
-    (property "Value" "" (id 1) (at 209.55 189.23 0))
+    (property "Value" "SDRAM(16Mx16)" (id 1) (at 209.55 189.23 0))
     (property "Footprint" "Package_SO:TSOP-II-54_22.2x10.16mm_P0.8mm" (id 2) (at 209.55 184.15 0)
       (effects (font (size 1.27 1.27) italic) hide)

Commit message: Add files via upload
Other:
- company: Drawn By: Jason Neus -> (none)
Changed lines of the file:
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@@
   (title_block
     (title "Amiga N2630")
-    (date "2022-03-25")
+    (date "2022-04-24")
     (rev "1.0")
-    (company "Drawn By: Jason Neus")
   )
   (junction (at 346.075 29.21) (diameter 0) (color 0 0 0 0)

Commit message: Add files via upload
Connections:
- net EM0R_W renamed EM0WE
- net EM1R_W renamed EM1WE
Changed lines of the file:
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@@
     )
   )
-  (global_label "EM1R_W" (shape input) (at 396.24 175.26 0) (fields_autoplaced)
+  (global_label "EM1WE" (shape input) (at 396.24 175.26 0) (fields_autoplaced)
     (effects (font (size 1.27 1.27)) (justify left))
-    (property "Intersheet References" "${INTERSHEET_REFS}" (id 0) (at 0 0 0)
-      (effects (font (size 1.27 1.27)) hide)
+    (property "Intersheet References" "${INTERSHEET_REFS}" (id 0) (at 404.9747 175.1806 0)
+      (effects (font (size 1.27 1.27)) (justify left) hide)
     )
   )
@@
     )
   )
-  (global_label "EM0R_W" (shape input) (at 33.02 118.11 180) (fields_autoplaced)
+  (global_label "EM0WE" (shape input) (at 33.02 118.11 180) (fields_autoplaced)
     (effects (font (size 1.27 1.27)) (justify right))
-    (property "Intersheet References" "${INTERSHEET_REFS}" (id 0) (at 0 0 0)
-      (effects (font (size 1.27 1.27)) hide)
+    (property "Intersheet References" "${INTERSHEET_REFS}" (id 0) (at 24.2853 118.0306 0)
+      (effects (font (size 1.27 1.27)) (justify right) hide)
     )
   )

Commit message: Add files via upload
Other:
- note added: "This is Zorro 3 memory. It is exclusively for the 68030. It cannot be DMA'd from the Zorro 2 bus or Amiga chipset."
- note removed: "CKE..The next rising edge of the CLK signal is valid when CKE is high and invalid when it is low. When CKE is LOW, the device will be in power-down mode, clock suspend mode or self-refresh mode JN: Might be able to refresh one bank when the other is being accessed?"
- note removed: "JN Notes: put row addresses 14..2 on the EMA bus and A16..15 on the bank select. Signal RAS (SDRAM BANKACTIVATE). Put column address 25..17 on the EMA bus and signal CAS. A26 is used to determine whether we are in the first 64MB or the second 64MB."
- note removed: "This is Zorro 3 memory, so it is always treated as 32 bit memory and cannot be used by the Amiga 2000 chip set and cannot be used by anything on the Zorro 2 bus. It can only be used by the 68030."
Changed lines of the file:
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@@
   (title_block
     (title "Amiga N2630")
-    (date "2022-04-24")
+    (date "2022-05-02")
     (rev "1.0")
   )
@@
     (effects (font (size 5.9944 5.9944)) (justify left bottom))
   )
-  (text "This is Zorro 3 memory, so it is always\ntreated as 32 bit memory and cannot be \nused by the Amiga 2000 chip set and cannot\nbe used by anything on the Zorro 2 bus.\nIt can only be used by the 68030."
-    (at 146.685 37.465 0)
+  (text "This is Zorro 3 memory. It is exclusively\nfor the 68030. It cannot be DMA'd from the\nZorro 2 bus or Amiga chipset."
+    (at 281.94 144.78 0)
     (effects (font (size 3 3)) (justify left bottom))
   )
@@
     (effects (font (size 2.9972 2.9972)) (justify left bottom))
   )
-  (text "CKE..The next rising edge of the CLK signal is valid \nwhen CKE is high and invalid when it is low. When \nCKE is LOW, the device will be in power-down mode, \nclock suspend mode or self-refresh mode\nJN: Might be able to refresh one bank when the other is\nbeing accessed?"
-    (at 17.78 133.35 0)
-    (effects (font (size 1.27 1.27)) (justify left bottom))
-  )
   (text "BANK1" (at 203.2 45.72 0)
     (effects (font (size 2.9972 2.9972)) (justify left bottom))
@@
     (effects (font (size 3.9878 3.9878)) (justify left bottom))
   )
-  (text "JN Notes: put row addresses 14..2 on the EMA bus \nand A16..15 on the bank select. Signal RAS \n(SDRAM BANKACTIVATE). Put column address 25..17\non the EMA bus and signal CAS. A26 is used to \ndetermine whether we are in the first 64MB or\nthe second 64MB."
-    (at 273.05 147.955 0)
-    (effects (font (size 2.9972 2.9972)) (justify left bottom))
-  )
   (text "HIGH_WORD" (at 24.13 180.975 0)
