File: A2630-New-KiCAD-Rev1/N2360.kicad_sch (KiCad schematic)
At the start: 0 parts

Commit message: Add files via upload
Other:
- company: Drawn By: Jason Neus -> (none)
Changed lines of the file:
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@@
   (title_block
     (title "Amiga N2630")
-    (date "2022-03-25")
+    (date "2022-04-24")
     (rev "1.0")
-    (company "Drawn By: Jason Neus")
   )
   (image (at 144.145 59.69)

Commit message: Add files via upload
Other:
- sheet Base Memory renamed Base Memory, Spares
- sheet Logic renamed Logic, IDE, Power
- removed sheet IDE, Power, and Spares
