File: A2630-New-KiCAD-Rev1/Processor.kicad_sch (KiCad schematic)
At the start: 77 parts, among them J201 25/28, J202 25/FPU, U200 MC68030FE, U201 MC68882, U204 74HCT04, X1 25MHz, X2 25MHz

Commit message: Add files via upload
Other:
- company: (none) -> Drawn By: Jason Neus
- title: N2630 -> Amiga N2630
Changed lines of the file:
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@@
   (paper "B")
   (title_block
-    (title "N2630")
+    (title "Amiga N2630")
+    (date "2022-03-25")
     (rev "1.0")
+    (company "Drawn By: Jason Neus")
   )
   (junction (at 143.256 187.96) (diameter 0) (color 0 0 0 0)

Commit message: Add files via upload
Parts:
- U200: value MC68030FE -> (none); footprint Package_QFP:PQFP-132_24x24mm_P0.635mm -> (none)
Changed lines of the file:
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@@
       (effects (font (size 1.524 1.524)))
     )
-    (property "Value" "MC68030FE" (id 1) (at 212.09 55.9562 0)
+    (property "Value" "" (id 1) (at 212.09 55.9562 0)
       (effects (font (size 1.524 1.524)))
     )
-    (property "Footprint" "Package_QFP:PQFP-132_24x24mm_P0.635mm" (id 2) (at 212.09 53.2638 0)
+    (property "Footprint" "" (id 2) (at 212.09 53.2638 0)
       (effects (font (size 1.524 1.524)) hide)
     )

Commit message: Add files via upload
Parts:
- U200: value (none) -> MC68030FE; footprint (none) -> N2630:MC68030FE-PQFP-132
Changed lines of the file:
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@@
       (effects (font (size 1.524 1.524)))
     )
-    (property "Value" "" (id 1) (at 212.09 55.9562 0)
+    (property "Value" "MC68030FE" (id 1) (at 212.09 55.9562 0)
       (effects (font (size 1.524 1.524)))
     )
-    (property "Footprint" "" (id 2) (at 212.09 53.2638 0)
+    (property "Footprint" "N2630:MC68030FE-PQFP-132" (id 2) (at 212.09 53.2638 0)
       (effects (font (size 1.524 1.524)) hide)
     )

Commit message: Add files via upload
Parts:
- U204: value 74HCT04 -> (none)
Changed lines of the file:
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@@
     (in_bom yes) (on_board yes)
     (property "Reference" "U204" (id 0) (at 73.025 181.1782 0))
-    (property "Value" "74HCT04" (id 1) (at 73.025 183.4896 0))
+    (property "Value" "" (id 1) (at 73.025 183.4896 0))
     (property "Footprint" "Package_SO:SOIC-14_3.9x8.7mm_P1.27mm" (id 2) (at 73.025 189.23 0)
       (effects (font (size 1.27 1.27)) hide)
@@
     (in_bom yes) (on_board yes)
     (property "Reference" "U204" (id 0) (at 88.265 212.2932 0))
-    (property "Value" "74HCT04" (id 1) (at 88.265 214.6046 0))
+    (property "Value" "" (id 1) (at 88.265 214.6046 0))
     (property "Footprint" "Package_SO:SOIC-14_3.9x8.7mm_P1.27mm" (id 2) (at 88.265 220.345 0)
       (effects (font (size 1.27 1.27)) hide)
@@
     (in_bom yes) (on_board yes)
     (property "Reference" "U204" (id 0) (at 88.265 154.5082 0))
-    (property "Value" "74HCT04" (id 1) (at 88.265 156.8196 0))
+    (property "Value" "" (id 1) (at 88.265 156.8196 0))
     (property "Footprint" "Package_SO:SOIC-14_3.9x8.7mm_P1.27mm" (id 2) (at 88.265 162.56 0)
       (effects (font (size 1.27 1.27)) hide)
@@
       (effects (font (size 1.27 1.27)) (justify left))
     )
-    (property "Value" "74HCT04" (id 1) (at 50.165 59.055 90)
+    (property "Value" "" (id 1) (at 50.165 59.055 90)
       (effects (font (size 1.27 1.27)) (justify left))
     )
@@
     (in_bom yes) (on_board yes)
     (property "Reference" "U204" (id 0) (at 68.58 233.8832 0))
-    (property "Value" "74HCT04" (id 1) (at 68.58 236.1946 0))
+    (property "Value" "" (id 1) (at 68.58 236.1946 0))
     (property "Footprint" "Package_SO:SOIC-14_3.9x8.7mm_P1.27mm" (id 2) (at 68.58 241.935 0)
       (effects (font (size 1.27 1.27)) hide)

Commit message: Add files via upload
Parts:
- U204: value (none) -> 74AHCT04
Changed lines of the file:
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@@
     (in_bom yes) (on_board yes)
     (property "Reference" "U204" (id 0) (at 73.025 181.1782 0))
-    (property "Value" "" (id 1) (at 73.025 183.4896 0))
+    (property "Value" "74AHCT04" (id 1) (at 73.025 183.4896 0))
     (property "Footprint" "Package_SO:SOIC-14_3.9x8.7mm_P1.27mm" (id 2) (at 73.025 189.23 0)
       (effects (font (size 1.27 1.27)) hide)
@@
     (in_bom yes) (on_board yes)
     (property "Reference" "U204" (id 0) (at 88.265 212.2932 0))
-    (property "Value" "" (id 1) (at 88.265 214.6046 0))
+    (property "Value" "74AHCT04" (id 1) (at 88.265 214.6046 0))
     (property "Footprint" "Package_SO:SOIC-14_3.9x8.7mm_P1.27mm" (id 2) (at 88.265 220.345 0)
       (effects (font (size 1.27 1.27)) hide)
@@
     (in_bom yes) (on_board yes)
     (property "Reference" "U204" (id 0) (at 88.265 154.5082 0))
-    (property "Value" "" (id 1) (at 88.265 156.8196 0))
+    (property "Value" "74AHCT04" (id 1) (at 88.265 156.8196 0))
     (property "Footprint" "Package_SO:SOIC-14_3.9x8.7mm_P1.27mm" (id 2) (at 88.265 162.56 0)
       (effects (font (size 1.27 1.27)) hide)
@@
       (effects (font (size 1.27 1.27)) (justify left))
     )
-    (property "Value" "" (id 1) (at 50.165 59.055 90)
+    (property "Value" "74AHCT04" (id 1) (at 50.165 59.055 90)
       (effects (font (size 1.27 1.27)) (justify left))
     )
@@
     (in_bom yes) (on_board yes)
     (property "Reference" "U204" (id 0) (at 68.58 233.8832 0))
-    (property "Value" "" (id 1) (at 68.58 236.1946 0))
+    (property "Value" "74AHCT04" (id 1) (at 68.58 236.1946 0))
     (property "Footprint" "Package_SO:SOIC-14_3.9x8.7mm_P1.27mm" (id 2) (at 68.58 241.935 0)
       (effects (font (size 1.27 1.27)) hide)

Commit message: Add files via upload
Other:
- company: Drawn By: Jason Neus -> (none)
Changed lines of the file:
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@@
   (title_block
     (title "Amiga N2630")
-    (date "2022-03-25")
+    (date "2022-04-24")
     (rev "1.0")
-    (company "Drawn By: Jason Neus")
   )
   (junction (at 143.256 187.96) (diameter 0) (color 0 0 0 0)
