File: A2630-New-KiCAD-Rev11/BaseMemory.kicad_sch (KiCad schematic)
At the start: 13 parts, among them U300 74HCT05, U400 SDRAM_32Mb(2Mx16), U401 SDRAM_32Mb(2Mx16), U507 74AHCT74, U606 74HCT244

Commit message: Add files via upload
Parts:
- removed unit 3 of U300
- removed U507: 74AHCT74, Package_SO:SOIC-14_3.9x8.7mm_P1.27mm, symbol 74xx:74LS74
Connections:
- no-connect marks 8 -> 5
Changed lines of the file:
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@@
   (title_block
     (title "Amiga N2630")
-    (date "2022-05-20")
+    (date "2022-05-25")
     (rev "1.1")
   )
-  (junction (at 337.82 144.78) (diameter 0) (color 0 0 0 0)
-  )
   (junction (at 171.45 253.365) (diameter 0) (color 0 0 0 0)
   )
@@
   (junction (at 337.82 101.6) (diameter 0) (color 0 0 0 0)
   )
-  (junction (at 337.82 57.15) (diameter 0) (color 0 0 0 0)
-  )
   (junction (at 121.92 138.684) (diameter 0) (color 0 0 0 0)
   )
@@
   (junction (at 111.76 214.249) (diameter 0) (color 0 0 0 0)
   )
-  (junction (at 337.82 142.24) (diameter 0) (color 0 0 0 0)
-  )
   (junction (at 66.04 193.294) (diameter 0) (color 0 0 0 0)
   )
@@
   (junction (at 185.42 231.14) (diameter 0) (color 0 0 0 0)
   )
-  (junction (at 369.57 135.255) (diameter 0) (color 0 0 0 0)
-  )
   (junction (at 193.04 253.365) (diameter 0) (color 0 0 0 0)
   )
-  (no_connect (at 353.06 147.32))
-  (no_connect (at 353.06 57.15))
   (no_connect (at 353.06 71.755))
   (no_connect (at 353.06 115.57))
   (no_connect (at 353.06 88.265))
-  (no_connect (at 353.06 142.24))
   (no_connect (at 353.06 101.6))
   (no_connect (at 353.06 43.815))
@@
     (stroke (width 0) (type default) (color 0 0 0 0))
   )
-  (wire (pts (xy 337.82 57.15) (xy 337.82 71.755))
-    (stroke (width 0) (type default) (color 0 0 0 0))
-  )
   (wire (pts (xy 116.84 138.684) (xy 116.84 143.764))
     (stroke (width 0) (type default) (color 0 0 0 0))
@@
     (stroke (width 0) (type default) (color 0 0 0 0))
   )
-  (wire (pts (xy 337.82 43.815) (xy 337.82 57.15))
+  (wire (pts (xy 337.82 43.815) (xy 337.82 71.755))
     (stroke (width 0) (type default) (color 0 0 0 0))
   )
@@
     (stroke (width 0) (type default) (color 0 0 0 0))
   )
-  (wire (pts (xy 337.82 144.78) (xy 337.82 154.305))
+  (wire (pts (xy 337.82 115.57) (xy 337.82 154.305))
     (stroke (width 0) (type default) (color 0 0 0 0))
   )
@@
     (stroke (width 0) (type default) (color 0 0 0 0))
   )
-  (wire (pts (xy 369.57 135.255) (xy 369.57 152.4))
-    (stroke (width 0) (type default) (color 0 0 0 0))
-  )
   (bus (pts (xy 156.845 183.134) (xy 156.845 180.594))
     (stroke (width 0) (type default) (color 0 0 0 0))
@@
     (stroke (width 0) (type default) (color 0 0 0 0))
   )
-  (wire (pts (xy 337.82 142.24) (xy 337.82 144.78))
-    (stroke (width 0) (type default) (color 0 0 0 0))
-  )
   (wire (pts (xy 139.7 88.519) (xy 154.305 88.519))
     (stroke (width 0) (type default) (color 0 0 0 0))
@@
     (stroke (width 0) (type default) (color 0 0 0 0))
   )
-  (wire (pts (xy 345.44 137.16) (xy 345.44 135.255))
-    (stroke (width 0) (type default) (color 0 0 0 0))
-  )
-  (wire (pts (xy 345.44 152.4) (xy 369.57 152.4))
-    (stroke (width 0) (type default) (color 0 0 0 0))
-  )
   (wire (pts (xy 89.535 99.949) (xy 99.06 99.949))
     (stroke (width 0) (type default) (color 0 0 0 0))
@@
     (stroke (width 0) (type default) (color 0 0 0 0))
   )
-  (wire (pts (xy 369.57 133.35) (xy 369.57 135.255))
-    (stroke (width 0) (type default) (color 0 0 0 0))
-  )
   (wire (pts (xy 116.84 41.529) (xy 119.38 41.529))
     (stroke (width 0) (type default) (color 0 0 0 0))
@@
     (stroke (width 0) (type default) (color 0 0 0 0))
   )
-  (wire (pts (xy 345.44 135.255) (xy 369.57 135.255))
-    (stroke (width 0) (type default) (color 0 0 0 0))
-  )
   (wire (pts (xy 139.7 188.214) (xy 154.305 188.214))
     (stroke (width 0) (type default) (color 0 0 0 0))
@@
   )
   (wire (pts (xy 66.04 239.014) (xy 66.04 193.294))
-    (stroke (width 0) (type default) (color 0 0 0 0))
-  )
-  (wire (pts (xy 337.82 115.57) (xy 337.82 142.24))
     (stroke (width 0) (type default) (color 0 0 0 0))
   )
@@
     (pin "1")
   )
-  (symbol (lib_id "power:+5V") (at 369.57 133.35 0) (unit 1)
-    (in_bom yes) (on_board yes) (fields_autoplaced)
-    (property "Reference" "#PWR0196" (id 0) (at 369.57 137.16 0)
-      (effects (font (size 1.27 1.27)) hide)
-    )
-    (property "Value" "+5V" (id 1) (at 369.57 129.7742 0))
-    (property "Footprint" "" (id 2) (at 369.57 133.35 0)
-      (effects (font (size 1.27 1.27)) hide)
-    )
-    (property "Datasheet" "" (id 3) (at 369.57 133.35 0)
-      (effects (font (size 1.27 1.27)) hide)
-    )
-    (pin "1")
-  )
   (symbol (lib_id "Device:C") (at 185.42 241.3 0) (unit 1)
     (in_bom yes) (on_board yes)
@@
     (pin "10")
     (pin "20")
-  )
-  (symbol (lib_id "74xx:74LS05") (at 345.44 57.15 0) (unit 3)
-    (in_bom yes) (on_board yes)
-    (property "Reference" "U300" (id 0) (at 345.44 49.53 0))
-    (property "Value" "74HCT05" (id 1) (at 345.44 52.07 0))
-    (property "Footprint" "Package_SO:SOIC-14_3.9x8.7mm_P1.27mm" (id 2) (at 345.44 57.15 0)
-      (effects (font (size 1.27 1.27)) hide)
-    )
-    (property "Datasheet" "http://www.ti.com/lit/gpn/sn74LS05" (id 3) (at 345.44 57.15 0)
-      (effects (font (size 1.27 1.27)) hide)
-    )
-    (pin "1")
-    (pin "2")
-    (pin "3")
-    (pin "4")
-    (pin "5")
-    (pin "6")
-    (pin "8")
-    (pin "9")
-    (pin "10")
-    (pin "11")
-    (pin "12")
-    (pin "13")
-    (pin "14")
-    (pin "7")
   )
   (symbol (lib_id "power:GND") (at 348.615 189.23 0) (unit 1)
@@
     (pin "20")
   )
-  (symbol (lib_id "74xx:74LS74") (at 345.44 144.78 0) (unit 2)
-    (in_bom yes) (on_board yes)
-    (property "Reference" "U507" (id 0) (at 349.25 136.525 0))
-    (property "Value" "74AHCT74" (id 1) (at 350.52 138.43 0))
-    (property "Footprint" "Package_SO:SOIC-14_3.9x8.7mm_P1.27mm" (id 2) (at 345.44 144.78 0)
-      (effects (font (size 1.27 1.27)) hide)
-    )
-    (property "Datasheet" "74xx/74hc_hct74.pdf" (id 3) (at 345.44 144.78 0)
-      (effects (font (size 1.27 1.27)) hide)
-    )
-    (pin "1")
-    (pin "2")
-    (pin "3")
-    (pin "4")
-    (pin "5")
-    (pin "6")
-    (pin "10")
-    (pin "11")
-    (pin "12")
-    (pin "13")
-    (pin "8")
-    (pin "9")
-    (pin "14")
-    (pin "7")
-  )
   (symbol (lib_id "power:+3.3V") (at 171.45 227.965 0) (unit 1)
