File: A2630-New-KiCAD-Rev11/Card Edge.kicad_sch (KiCad schematic)
At the start: 33 parts, among them CN700 Amiga-2000-CPU-Slot, J302 Jumper_NO_Small, J303 Jumper_NO_Small, J304 Jumper_NO_Small, J305 Z3 DISABLE, U204 74AHCT04, U300 74HCT05, U700 74HCT174, U701 74FCT646, U702 74FCT646, U703 74HCT245, U704 74HCT245, U705 74HCT245, U706 74HCT245, U707 74HCT245

Commit message: Add files via upload
Parts:
- removed R700: 1k, Resistor_SMD:R_0805_2012Metric, symbol Device:R
- removed U204: 74AHCT04, Package_SO:SOIC-14_3.9x8.7mm_P1.27mm, symbol 74xx:74LS04
- removed U300: 74HCT05, Package_SO:SOIC-14_3.9x8.7mm_P1.27mm, symbol 74xx:74LS05
- added U300: 74HCT05, Package_SO:SOIC-14_3.9x8.7mm_P1.27mm, symbol 74xx:74LS05
Connections:
- net _BERR: now also CN700.46
- net _COPCFG: now reaches CN700.11
- net _COPCFG: now also U300.6
- new net CONFIGED: U300.5
