File: A2630-New-KiCAD-Rev11/ExpansionMemory.kicad_sch (KiCad schematic)
At the start: 31 parts, among them J400 Jumper_NO_Small, J401 Jumper_NO_Small, J402 Jumper_NO_Small, J403 Jumper_NO_Small, J404 Jumper_NO_Small, U102 27C256, U103 27C256, U406 SDRAM(16Mx16), U407 SDRAM(16Mx16), U408 SDRAM(16Mx16), U409 SDRAM(16Mx16)

Commit message: Add files via upload
Changed lines of the file:
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@@
   (title_block
     (title "Amiga N2630")
-    (date "2022-05-20")
+    (date "2022-05-25")
     (rev "1.1")
   )
@@
     )
   )
-  (global_label "D[31..0]" (shape bidirectional) (at 290.195 110.49 180) (fields_autoplaced)
+  (global_label "D[31..0]" (shape bidirectional) (at 292.1 29.21 180) (fields_autoplaced)
     (effects (font (size 1.27 1.27)) (justify right))
-    (property "Intersheet References" "${INTERSHEET_REFS}" (id 0) (at 0 0 0)
+    (property "Intersheet References" "${INTERSHEET_REFS}" (id 0) (at 1.905 -81.28 0)
       (effects (font (size 1.27 1.27)) hide)
     )
@@
     )
   )
-  (global_label "A[31..0]" (shape input) (at 292.1 29.21 180) (fields_autoplaced)
+  (global_label "A[31..0]" (shape input) (at 290.195 110.49 180) (fields_autoplaced)
     (effects (font (size 1.27 1.27)) (justify right))
-    (property "Intersheet References" "${INTERSHEET_REFS}" (id 0) (at 0 0 0)
+    (property "Intersheet References" "${INTERSHEET_REFS}" (id 0) (at -1.905 81.28 0)
       (effects (font (size 1.27 1.27)) hide)
     )
