File: A2630-New-KiCAD-Rev11/Logic.kicad_sch (KiCad schematic)
At the start: 56 parts, among them CN5 ATA/IDE, CN6 LED, U204 74AHCT04, U300 74HCT05, U303 74HCT174, U418 74LVC245, U419 74LVC245, U420 74LVC245, U421 74LVC245, U502 74HCT74, U503 74HCT74, U507 74AHCT74, U606 74HCT244, U700 74HCT245, U701 74HCT245, U800 LM1117-3.3

Commit message: Add files via upload
Connections:
- net D16: now also U700.9 (A7); no longer U700.11 (B7)
- net D17: now also U700.8 (A6); no longer U700.12 (B6)
- net D18: now also U700.7 (A5); no longer U700.13 (B5)
- net D19: now also U700.6 (A4); no longer U700.14 (B4)
- net D20: now also U700.5 (A3); no longer U700.15 (B3)
- net D21: now also U700.4 (A2); no longer U700.16 (B2)
- net D22: now also U700.3 (A1); no longer U700.17 (B1)
- net D23: now also U700.2 (A0); no longer U700.18 (B0)
- net D24: now also U701.2 (A0); no longer U701.18 (B0)
- net D25: now also U701.3 (A1); no longer U701.17 (B1)
- net D26: now also U701.4 (A2); no longer U701.16 (B2)
- net D27: now also U701.5 (A3); no longer U701.15 (B3)
- net D28: now also U701.6 (A4); no longer U701.14 (B4)
- net D29: now also U701.7 (A5); no longer U701.13 (B5)
- net D30: now also U701.8 (A6); no longer U701.12 (B6)
- net D31: now also U701.9 (A7); no longer U701.11 (B7)
- net IDED0: now also U700.11 (B7); no longer U700.9 (A7)
- net IDED1: now also U700.12 (B6); no longer U700.8 (A6)
- net IDED10: now also U701.16 (B2); no longer U701.4 (A2)
- net IDED11: now also U701.15 (B3); no longer U701.5 (A3)
- net IDED12: now also U701.14 (B4); no longer U701.6 (A4)
- net IDED13: now also U701.13 (B5); no longer U701.7 (A5)
- net IDED14: now also U701.12 (B6); no longer U701.8 (A6)
- net IDED15: now also U701.11 (B7); no longer U701.9 (A7)
- net IDED2: now also U700.13 (B5); no longer U700.7 (A5)
- net IDED3: now also U700.14 (B4); no longer U700.6 (A4)
- net IDED4: now also U700.15 (B3); no longer U700.5 (A3)
- net IDED5: now also U700.16 (B2); no longer U700.4 (A2)
- net IDED6: now also U700.17 (B1); no longer U700.3 (A1)
- net IDED7: now also U700.18 (B0); no longer U700.2 (A0)
- net IDED8: now also U701.18 (B0); no longer U701.2 (A0)
- net IDED9: now also U701.17 (B1); no longer U701.3 (A1)
- net R_W renamed IDEDIR
Other:
- moved on the sheet: CN6, R600

Commit message: Add files via upload
Parts:
- removed C502, C503, C507: 0.22uf, Capacitor_SMD:C_0805_2012Metric, symbol Device:C
- removed R503, R504, R505, R506: 1K, Resistor_SMD:R_0805_2012Metric, symbol Device:R
- removed unit 1 of U300
- removed unit 5 of U300
- removed U502, U503: 74HCT74, Package_SO:SOIC-14_3.9x8.7mm_P1.27mm, symbol 74xx:74LS74
- removed U507: 74AHCT74, Package_SO:SOIC-14_3.9x8.7mm_P1.27mm, symbol 74xx:74LS74
- added R405: 1K, Resistor_SMD:R_0805_2012Metric, symbol Device:R
- renumbered C700 to C900, C701 to C901, U700 to U900, U701 to U901
Connections:
- net +3V3: now also R405.1
- net D16: now also U900.8 (A6); no longer U900.9 (A7)
- net D17: now also U900.6 (A4); no longer U900.8 (A6)
- net D18: now also U900.4 (A2); no longer U900.7 (A5)
- net D19: now also U900.2 (A0); no longer U900.6 (A4)
- net D20: now also U901.8 (A6); no longer U900.5 (A3)
- net D21: now also U901.6 (A4); no longer U900.4 (A2)
- net D22: now also U901.4 (A2); no longer U900.3 (A1)
- net D23: now also U901.2 (A0); no longer U900.2 (A0)
- net D24: now also U901.3 (A1); no longer U901.2 (A0)
- net D25: now also U901.5 (A3); no longer U901.3 (A1)
- net D26: now also U901.7 (A5); no longer U901.4 (A2)
- net D27: now also U901.9 (A7); no longer U901.5 (A3)
- net D28: now also U900.3 (A1); no longer U901.6 (A4)
- net D29: now also U900.5 (A3); no longer U901.7 (A5)
- net D30: now also U900.7 (A5); no longer U901.8 (A6)
- net D31: now also U900.9 (A7); no longer U901.9 (A7)
- net IDED0: now also U900.12 (B6); no longer U900.11 (B7)
- net IDED1: now also U900.14 (B4); no longer U900.12 (B6)
- net IDED10: now also U901.13 (B5); no longer U901.16 (B2)
- net IDED11: now also U901.11 (B7); no longer U901.15 (B3)
- net IDED12: now also U900.17 (B1); no longer U901.14 (B4)
- net IDED13: now also U900.15 (B3); no longer U901.13 (B5)
- net IDED14: now also U900.13 (B5); no longer U901.12 (B6)
- net IDED15: now also U900.11 (B7); no longer U901.11 (B7)
- net IDED2: now also U900.16 (B2); no longer U900.13 (B5)
- net IDED3: now also U900.18 (B0); no longer U900.14 (B4)
- net IDED4: now also U901.12 (B6); no longer U900.15 (B3)
- net IDED5: now also U901.14 (B4); no longer U900.16 (B2)
- net IDED6: now also U901.16 (B2); no longer U900.17 (B1)
- net IDED7: now also U901.18 (B0); no longer U900.18 (B0)
- net IDED8: now also U901.17 (B1); no longer U901.18 (B0)
- net IDED9: now also U901.15 (B3); no longer U901.17 (B1)
- new net _Z3CONFIGED: R405.2
- no-connect marks 8 -> 5
Other:
- note removed: "BUS GRANT ENABLE/DISABLE"
- note removed: "DSACK FOR 16 BIT CYCLES"
- note removed: "STATE MACHINE"
