File: A2630-New-KiCAD-Rev11/Processor.kicad_sch (KiCad schematic)
At the start: 77 parts, among them J201 25/28, J202 25/FPU, U200 MC68030FE, U201 MC68882, U204 74AHCT04, X1 25MHz, X2 25MHz

Commit message: Add files via upload
Parts:
- removed R115, R116, R117, R118, R119, R120, R121, R122, R123, R124, R125, R126, R127, R128, R129, R130: 1K, Resistor_SMD:R_0805_2012Metric, symbol Device:R
- added RN108, RN109: 1K, Resistor_THT:R_Array_SIP9, symbol Device:R_Network08
Connections:
- net A1: now also RN108.2 (R1)
- net A10: now also RN108.6 (R5)
- net A11: now also RN109.3 (R2)
- net A12: now also RN108.5 (R4)
- net A13: now also RN109.8 (R7)
- net A14: now also RN108.8 (R7)
- net A15: now also RN108.9 (R8)
- net A16: now also RN109.9 (R8)
- net A2: now also RN109.2 (R1)
- net A3: now also RN108.3 (R2)
- net A4: now also RN108.4 (R3)
- net A5: now also RN109.4 (R3)
- net A6: now also RN109.5 (R4)
- net A7: now also RN109.6 (R5)
- net A8: now also RN109.7 (R6)
- net A9: now also RN108.7 (R6)
- net GND: now also RN108.1 (common), RN109.1 (common)
- net _CPURESET: no longer R228.1
- net _HALT: now also R228.1
Other:
- moved on the sheet: R100, R101, R102, R103, R104, R105, R106, R107, R108, R109, R110, R111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
