File: A2630-New-KiCAD-Rev2/BaseMemory.kicad_sch (KiCad schematic)
At the start: 13 parts, among them U300 74HCT05, U400 SDRAM_32Mb(2Mx16), U401 SDRAM_32Mb(2Mx16), U606 74HCT244

Commit message: Add files via upload
Parts:
- added U204: 74AHCT04, Package_SO:SOIC-14_3.9x8.7mm_P1.27mm, symbol 74xx:74HCT04
- added unit 1 of U300
- added unit 4 of U300
- added unit 5 of U300
- U902: value (none) -> 74HCT125; footprint (none) -> Package_SO:SOIC-14_3.9x8.7mm_P1.27mm
Connections:
- net GND: now also U204.5, U300.1, U300.11, U300.9
- no-connect marks 6 -> 10
Other:
- moved on the sheet: H1, H2, U606E, U606F, U606G, U606H, U902D

Commit message: Add files via upload
Parts:
- U400, U401: value SDRAM_32Mb(2Mx16) -> SDRAM(2Mx16)
Changed lines of the file:
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@@
     (in_bom yes) (on_board yes)
     (property "Reference" "U400" (id 0) (at 119.38 79.629 0))
-    (property "Value" "SDRAM_32Mb(2Mx16)" (id 1) (at 119.38 84.709 0))
+    (property "Value" "SDRAM(2Mx16)" (id 1) (at 119.38 84.709 0))
     (property "Footprint" "Package_SO:TSOP-II-54_22.2x10.16mm_P0.8mm" (id 2) (at 119.38 79.629 0)
       (effects (font (size 1.27 1.27) italic) hide)
@@
     (in_bom yes) (on_board yes)
     (property "Reference" "U401" (id 0) (at 119.38 176.784 0))
-    (property "Value" "SDRAM_32Mb(2Mx16)" (id 1) (at 119.38 181.864 0))
+    (property "Value" "SDRAM(2Mx16)" (id 1) (at 119.38 181.864 0))
     (property "Footprint" "Package_SO:TSOP-II-54_22.2x10.16mm_P0.8mm" (id 2) (at 119.38 176.784 0)
       (effects (font (size 1.27 1.27) italic) hide)
