File: A2630-New-KiCAD-Rev2/CPLD1.kicad_sch (KiCad schematic)
At the start: 19 parts, among them CN600 CPLD0, CN601 CPLD1, CN602 CPLD2, J600 IDE DISABLE, U600 XC9572XL-VQ64, U601 XC95144XL-TQ144, U602 XC95144XL-TQ144

Commit message: Add files via upload
Connections:
- net _RAS is gone; now on net EMA6: U602.102 (P102)
- net BANK0: now also U602.94 (P94); no longer U602.79 (P79)
- net BANK1: now also U602.96 (P96); no longer U602.81 (P81)
- net EMA0: now also U602.101 (P101); no longer U602.76 (P76)
- net EMA1: now also U602.103 (P103); no longer U602.78 (P78)
- net EMA10: now also U602.98 (P98); no longer U602.92 (P92)
- net EMA12: now also U602.91 (P91); no longer U602.94 (P94)
- net EMA2: now also U602.105 (P105); no longer U602.80 (P80)
- net EMA3: now also U602.107 (P107); no longer U602.82 (P82)
- net EMA4: now also U602.106 (P106); no longer U602.83 (P83)
- net EMA5: now also U602.104 (P104); no longer U602.85 (P85)
- net EMA6: no longer U602.86 (P86)
- net EMA7: now also U602.100 (P100); no longer U602.87 (P87)
- net EMA8: now also U602.97 (P97); no longer U602.88 (P88)
- net EMA9: now also U602.95 (P95); no longer U602.91 (P91)
- net EMCLKE: now also U602.87 (P87); no longer U602.101 (P101)
- net EMWE: now also U602.85 (P85); no longer U602.104 (P104)
- net IDEDIR: now also U602.111 (P111); no longer U602.105 (P105)
- net MODE68K: now also U601.69 (P69)
- net REF: now also U602.3 (I/O/GTS4); no longer U602.130 (P130)
- net REFACKZ3: now also U602.2 (I/O/GTS3); no longer U602.129 (P129)
- net _EM0CS: now also U602.92 (P92); no longer U602.103 (P103)
- net _EM1CS: now also U602.81 (P81); no longer U602.77 (P77)
- net _EMCAS: now also U602.86 (P86); no longer U602.100 (P100)
- net _EMLLBE: now also U602.79 (P79); no longer U602.95 (P95)
- net _EMLMBE: now also U602.80 (P80); no longer U602.97 (P97)
- net _EMUMBE: now also U602.82 (P82); no longer U602.98 (P98)
- net _EMUUBE: now also U602.83 (P83); no longer U602.96 (P96)
- net _IDERST: now reaches U602.112 (P112)
- net ROMCLK: no longer names the net of U601.2 (I/O/GTS3)
- new net _EMRAS: U602.88 (P88)
- no-connect marks 29 -> 30

Commit message: Add files via upload
Connections:
- net CDAC is gone; now on net ADDIR: U600.31 (P31)
- net A0: now also U600.56 (P56)
- net ADDIR: no longer U601.54 (P54)
- net CONFIGED: now also U600.64 (I/O/GSR)
- net FC1: now also U600.60 (P60); no longer U600.59 (P59)
- net GND: now also J600.1 (A); no longer J600.2 (B)
- net J400: now also U602.131 (P131); no longer U600.8 (P8)
- net J401: now also U602.130 (P130); no longer U600.6 (P6)
- net J402: now also U602.129 (P129); no longer U600.5 (I/O/GTS1)
- net J404: now also U602.118 (P118)
- net MODE68K: now also U602.113 (P113); no longer U602.131 (P131)
- net SIZ0: now also U600.62 (P62)
- net SIZ1: now also U600.63 (P63)
- net TRISTATE: no longer U601.34 (P34)
- net _BERR: now also U600.5 (I/O/GTS1)
- net _CPURESET: now also U600.59 (P59); no longer U600.58 (P58)
- net _EXTERN: no longer U601.27 (P27)
- net _HALT: now also U600.58 (P58), U601.40 (P40); no longer U600.56 (P56)
- net _IDEDIS: now also J600.2 (B); no longer J600.1 (A)
- net _LDS: now also U600.35 (P35)
- net _ONBOARD: no longer U601.28 (P28)
- net _STERM: now also U600.8 (P8)
- net _UDS: now also U600.36 (P36)
- net 68KMODE: now reaches U600.61 (P61)
- net _ASEN: no longer names the net of U601.31 (P31)
- removed net _CYCEND: U600.35 (P35), U601.40 (P40)
- net _DSEN: no longer names the net of U601.39 (P39)
- net _DSEN: no longer U600.36 (P36)
- new net _BG: U600.6 (P6)
- no-connect marks 30 -> 24
Other:
- moved on the sheet: J600

Commit message: Add files via upload
Connections:
- net CONFIGED: now also U600.8 (P8); no longer U600.64 (I/O/GSR)
- net J404: now also U602.136 (P136); no longer U602.118 (P118)
- net SIZ0: now also U600.63 (P63); no longer U600.62 (P62)
- net SIZ1: now also U600.62 (P62); no longer U600.63 (P63)
- net _BERR: now also U600.64 (I/O/GSR); no longer U600.5 (I/O/GTS1)
- net _HALT: now also U601.2 (I/O/GTS3); no longer U601.40 (P40)
- net _OVR: no longer U602.136 (P136)
- net _STERM: now also U600.5 (I/O/GTS1); no longer U600.8 (P8)
- net Z3AUTO renamed _Z3DIS
- no-connect marks 24 -> 35
Changed lines of the file:
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@@
   (title_block
     (title "Amiga N2630")
-    (date "2022-05-26")
+    (date "2022-05-31")
     (rev "2.0 QFP")
   )
@@
   (no_connect (at 226.695 67.31))
   (no_connect (at 226.695 64.77))
+  (no_connect (at 226.695 69.85))
   (no_connect (at 300.355 104.775))
+  (no_connect (at 160.655 97.79))
+  (no_connect (at 160.655 92.71))
+  (no_connect (at 160.655 90.17))
+  (no_connect (at 160.655 87.63))
   (no_connect (at 160.655 113.03))
   (no_connect (at 160.655 115.57))
+  (no_connect (at 300.355 175.895))
+  (no_connect (at 366.395 94.615))
   (no_connect (at 160.655 153.67))
   (no_connect (at 160.655 146.05))
@@
   (no_connect (at 366.395 137.795))
   (no_connect (at 366.395 135.255))
-  (no_connect (at 160.655 105.41))
+  (no_connect (at 160.655 151.13))
+  (no_connect (at 160.655 156.21))
+  (no_connect (at 160.655 158.75))
+  (no_connect (at 160.655 179.07))
+  (no_connect (at 160.655 176.53))
+  (no_connect (at 160.655 181.61))
   (no_connect (at 366.395 132.715))
-  (no_connect (at 375.285 94.615))
   (bus_entry (at 281.305 137.795) (size -2.54 -2.54)
     (stroke (width 0) (type default) (color 0 0 0 0))
@@
     (stroke (width 0) (type default) (color 0 0 0 0))
   )
-  (wire (pts (xy 160.655 156.21) (xy 151.765 156.21))
-    (stroke (width 0) (type default) (color 0 0 0 0))
-  )
   (bus (pts (xy 287.02 125.095) (xy 287.02 127.635))
     (stroke (width 0) (type default) (color 0 0 0 0))
@@
     (stroke (width 0) (type default) (color 0 0 0 0))
   )
-  (wire (pts (xy 151.765 90.17) (xy 160.655 90.17))
-    (stroke (width 0) (type default) (color 0 0 0 0))
-  )
   (wire (pts (xy 53.975 137.795) (xy 37.465 137.795))
     (stroke (width 0) (type default) (color 0 0 0 0))
@@
     (stroke (width 0) (type default) (color 0 0 0 0))
   )
-  (wire (pts (xy 288.925 175.895) (xy 300.355 175.895))
-    (stroke (width 0) (type default) (color 0 0 0 0))
-  )
   (wire (pts (xy 281.305 86.995) (xy 300.355 86.995))
     (stroke (width 0) (type default) (color 0 0 0 0))
@@
     (stroke (width 0) (type default) (color 0 0 0 0))
   )
-  (wire (pts (xy 160.655 92.71) (xy 151.765 92.71))
-    (stroke (width 0) (type default) (color 0 0 0 0))
-  )
   (bus (pts (xy 387.985 66.675) (xy 387.985 69.215))
     (stroke (width 0) (type default) (color 0 0 0 0))
@@
     (stroke (width 0) (type default) (color 0 0 0 0))
   )
-  (wire (pts (xy 160.655 87.63) (xy 151.765 87.63))
-    (stroke (width 0) (type default) (color 0 0 0 0))
-  )
   (wire (pts (xy 323.215 224.155) (xy 320.675 224.155))
     (stroke (width 0) (type default) (color 0 0 0 0))
@@
     (stroke (width 0) (type default) (color 0 0 0 0))
   )
-  (wire (pts (xy 160.655 151.13) (xy 151.765 151.13))
-    (stroke (width 0) (type default) (color 0 0 0 0))
-  )
   (wire (pts (xy 226.695 161.29) (xy 240.03 161.29))
     (stroke (width 0) (type default) (color 0 0 0 0))
@@
     (stroke (width 0) (type default) (color 0 0 0 0))
   )
-  (wire (pts (xy 151.765 176.53) (xy 160.655 176.53))
-    (stroke (width 0) (type default) (color 0 0 0 0))
-  )
   (wire (pts (xy 281.305 153.035) (xy 300.355 153.035))
     (stroke (width 0) (type default) (color 0 0 0 0))
@@
     (stroke (width 0) (type default) (color 0 0 0 0))
   )
-  (wire (pts (xy 151.765 97.79) (xy 160.655 97.79))
-    (stroke (width 0) (type default) (color 0 0 0 0))
-  )
   (wire (pts (xy 160.655 80.01) (xy 151.765 80.01))
     (stroke (width 0) (type default) (color 0 0 0 0))
@@
     (stroke (width 0) (type default) (color 0 0 0 0))
   )
-  (wire (pts (xy 226.695 69.85) (xy 236.22 69.85))
-    (stroke (width 0) (type default) (color 0 0 0 0))
-  )
   (bus (pts (xy 278.765 147.955) (xy 278.765 150.495))
     (stroke (width 0) (type default) (color 0 0 0 0))
@@
     (stroke (width 0) (type default) (color 0 0 0 0))
   )
-  (wire (pts (xy 151.765 158.75) (xy 160.655 158.75))
+  (wire (pts (xy 152.4 105.41) (xy 160.655 105.41))
     (stroke (width 0) (type default) (color 0 0 0 0))
   )
@@
     (stroke (width 0) (type default) (color 0 0 0 0))
   )
-  (wire (pts (xy 151.765 179.07) (xy 160.655 179.07))
-    (stroke (width 0) (type default) (color 0 0 0 0))
-  )
   (wire (pts (xy 300.355 188.595) (xy 288.925 188.595))
     (stroke (width 0) (type default) (color 0 0 0 0))
@@
     (stroke (width 0) (type default) (color 0 0 0 0))
   )
-  (wire (pts (xy 375.285 94.615) (xy 366.395 94.615))
-    (stroke (width 0) (type default) (color 0 0 0 0))
-  )
   (wire (pts (xy 226.695 166.37) (xy 251.46 166.37))
     (stroke (width 0) (type default) (color 0 0 0 0))
@@
     (stroke (width 0) (type default) (color 0 0 0 0))
   )
-  (wire (pts (xy 154.432 181.61) (xy 160.655 181.61))
-    (stroke (width 0) (type default) (color 0 0 0 0))
-  )
   (wire (pts (xy 385.445 59.055) (xy 366.395 59.055))
     (stroke (width 0) (type default) (color 0 0 0 0))
@@
     (effects (font (size 1.27 1.27)) (justify right bottom))
   )
-  (global_label "SIZ1" (shape input) (at 37.465 160.655 180) (fields_autoplaced)
+  (global_label "SIZ0" (shape input) (at 37.465 160.655 180) (fields_autoplaced)
     (effects (font (size 1.27 1.27)) (justify right))
     (property "Intersheet References" "${INTERSHEET_REFS}" (id 0) (at 30.9075 160.5756 0)
@@
     )
   )
-  (global_label "_OVR" (shape output) (at 288.29 201.295 180) (fields_autoplaced)
-    (effects (font (size 1.27 1.27)) (justify right))
-    (property "Intersheet References" "${INTERSHEET_REFS}" (id 0) (at 281.3091 201.3744 0)
-      (effects (font (size 1.27 1.27)) (justify right) hide)
-    )
-  )
   (global_label "_ADOEL" (shape output) (at 37.465 109.855 180) (fields_autoplaced)
     (effects (font (size 1.27 1.27)) (justify right))
@@
     )
   )
-  (global_label "IORDY" (shape output) (at 375.285 109.855 0) (fields_autoplaced)
+  (global_label "IORDY" (shape input) (at 375.285 109.855 0) (fields_autoplaced)
     (effects (font (size 1.27 1.27)) (justify left))
     (property "Intersheet References" "${INTERSHEET_REFS}" (id 0) (at 383.173 109.7756 0)
@@
     )
   )
-  (global_label "INTRQ" (shape output) (at 375.285 112.395 0) (fields_autoplaced)
+  (global_label "INTRQ" (shape input) (at 375.285 112.395 0) (fields_autoplaced)
     (effects (font (size 1.27 1.27)) (justify left))
     (property "Intersheet References" "${INTERSHEET_REFS}" (id 0) (at 383.1125 112.3156 0)
@@
     )
   )
-  (global_label "_STERM" (shape input) (at 37.465 97.155 180) (fields_autoplaced)
+  (global_label "_STERM" (shape input) (at 37.465 140.335 180) (fields_autoplaced)
     (effects (font (size 1.27 1.27)) (justify right))
-    (property "Intersheet References" "${INTERSHEET_REFS}" (id 0) (at 28.1256 97.0756 0)
+    (property "Intersheet References" "${INTERSHEET_REFS}" (id 0) (at 28.1256 140.2556 0)
       (effects (font (size 1.27 1.27)) (justify right) hide)
     )
@@
     )
   )
-  (global_label "SIZ0" (shape input) (at 37.465 158.115 180) (fields_autoplaced)
+  (global_label "SIZ1" (shape input) (at 37.465 158.115 180) (fields_autoplaced)
     (effects (font (size 1.27 1.27)) (justify right))
     (property "Intersheet References" "${INTERSHEET_REFS}" (id 0) (at 30.9075 158.0356 0)
@@
     )
   )
-  (global_label "Z3AUTO" (shape input) (at 288.29 211.455 180) (fields_autoplaced)
+  (global_label "_Z3DIS" (shape input) (at 288.29 211.455 180) (fields_autoplaced)
     (effects (font (size 1.2954 1.2954)) (justify right))
-    (property "Intersheet References" "${INTERSHEET_REFS}" (id 0) (at 8.89 30.48 0)
-      (effects (font (size 1.27 1.27)) hide)
+    (property "Intersheet References" "${INTERSHEET_REFS}" (id 0) (at 279.3191 211.3741 0)
+      (effects (font (size 1.2954 1.2954)) (justify right) hide)
     )
   )
@@
     )
   )
-  (global_label "CONFIGED" (shape input) (at 37.465 163.195 180) (fields_autoplaced)
+  (global_label "CONFIGED" (shape input) (at 37.465 97.155 180) (fields_autoplaced)
     (effects (font (size 1.27 1.27)) (justify right))
-    (property "Intersheet References" "${INTERSHEET_REFS}" (id 0) (at 25.8275 163.1156 0)
+    (property "Intersheet References" "${INTERSHEET_REFS}" (id 0) (at 25.8275 97.0756 0)
       (effects (font (size 1.27 1.27)) (justify right) hide)
     )
@@
     )
   )
-  (global_label "J404" (shape input) (at 288.925 175.895 180) (fields_autoplaced)
+  (global_label "J404" (shape input) (at 288.29 201.295 180) (fields_autoplaced)
     (effects (font (size 1.27 1.27)) (justify right))
-    (property "Intersheet References" "${INTERSHEET_REFS}" (id 0) (at 282.0046 175.8156 0)
+    (property "Intersheet References" "${INTERSHEET_REFS}" (id 0) (at 281.3696 201.2156 0)
       (effects (font (size 1.27 1.27)) (justify right) hide)
     )
@@
     )
   )
-  (global_label "_HALT" (shape input) (at 151.765 158.75 180) (fields_autoplaced)
+  (global_label "_HALT" (shape input) (at 152.4 105.41 180) (fields_autoplaced)
     (effects (font (size 1.27 1.27)) (justify right))
-    (property "Intersheet References" "${INTERSHEET_REFS}" (id 0) (at 144.0584 158.6706 0)
+    (property "Intersheet References" "${INTERSHEET_REFS}" (id 0) (at 144.6934 105.3306 0)
       (effects (font (size 1.27 1.27)) (justify right) hide)
     )
@@
     )
   )
-  (global_label "_BERR" (shape input) (at 37.465 140.335 180) (fields_autoplaced)
+  (global_label "_BERR" (shape output) (at 37.465 163.195 180) (fields_autoplaced)
     (effects (font (size 1.27 1.27)) (justify right))
-    (property "Intersheet References" "${INTERSHEET_REFS}" (id 0) (at 29.2141 140.2556 0)
+    (property "Intersheet References" "${INTERSHEET_REFS}" (id 0) (at 29.2141 163.1156 0)
       (effects (font (size 1.27 1.27)) (justify right) hide)
     )
