File: A2630-New-KiCAD-Rev2/Card Edge.kicad_sch (KiCad schematic)
At the start: 31 parts, among them CN700 Amiga-2000-CPU-Slot, J302 Jumper_NO_Small, J303 Jumper_NO_Small, J304 Jumper_NO_Small, J305 Z3 DISABLE, U300 74HCT05, U700 74HCT174, U701 74FCT646, U702 74FCT646, U703 74HCT245, U704 74HCT245, U705 74HCT245, U706 74HCT245, U707 74HCT245

Commit message: Add files via upload
Connections:
- net GND: now also J305.1; no longer J305.2
- net Z3AUTO: now also J305.2; no longer J305.1
Other:
- moved on the sheet: J305
Changed lines of the file:
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@@
     (pin "2")
   )
-  (symbol (lib_id "Device:Jumper_NO_Small") (at 349.25 95.25 180) (unit 1)
+  (symbol (lib_id "Device:Jumper_NO_Small") (at 349.25 95.25 0) (unit 1)
     (in_bom yes) (on_board yes)
-    (property "Reference" "J305" (id 0) (at 349.25 97.6122 0))
-    (property "Value" "Z3 DISABLE" (id 1) (at 349.25 97.6376 0)
+    (property "Reference" "J305" (id 0) (at 349.25 92.8878 0))
+    (property "Value" "Z3 DISABLE" (id 1) (at 349.25 92.8624 0)
       (effects (font (size 1.27 1.27)) hide)
     )

Commit message: Add files via upload
Connections:
- net CDAC: no longer names the net of CN700.15
- net Z3AUTO renamed _Z3DIS
Changed lines of the file:
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@@
   (title_block
     (title "Amiga N2630")
-    (date "2022-05-26")
+    (date "2022-05-31")
     (rev "2.0 QFP")
   )
@@
     (stroke (width 0) (type default) (color 0 0 0 0))
   )
-  (wire (pts (xy 23.368 149.86) (xy 102.235 149.86))
-    (stroke (width 0) (type default) (color 0 0 0 0))
-  )
   (wire (pts (xy 114.935 152.4) (xy 114.935 160.02))
     (stroke (width 0) (type default) (color 0 0 0 0))
@@
     )
   )
-  (global_label "CDAC" (shape output) (at 23.368 149.86 180) (fields_autoplaced)
-    (effects (font (size 1.27 1.27)) (justify right))
-    (property "Intersheet References" "${INTERSHEET_REFS}" (id 0) (at 16.1452 149.7806 0)
-      (effects (font (size 1.27 1.27)) (justify right) hide)
-    )
-  )
   (global_label "OSMODE" (shape output) (at 381.635 90.805 0) (fields_autoplaced)
     (effects (font (size 1.2954 1.2954)) (justify left))
@@
     )
   )
-  (global_label "Z3AUTO" (shape output) (at 381.635 95.25 0) (fields_autoplaced)
+  (global_label "_Z3DIS" (shape output) (at 381.635 95.25 0) (fields_autoplaced)
     (effects (font (size 1.2954 1.2954)) (justify left))
-    (property "Intersheet References" "${INTERSHEET_REFS}" (id 0) (at 0 0 0)
-      (effects (font (size 1.27 1.27)) hide)
+    (property "Intersheet References" "${INTERSHEET_REFS}" (id 0) (at 390.6059 95.1691 0)
+      (effects (font (size 1.2954 1.2954)) (justify left) hide)
     )
   )
