File: A2630-New-KiCAD-Rev2/Logic.kicad_sch (KiCad schematic)
At the start: 47 parts, among them CN5 ATA/IDE, CN6 LED, U204 74AHCT04, U300 74HCT05, U418 74LVC245, U419 74LVC245, U420 74LVC245, U421 74LVC245, U606 74HCT244, U800 LM1117-3.3, U900 74HCT245, U901 74HCT245

Commit message: Add files via upload
Parts:
- U902: value (none) -> 74HCT125; footprint (none) -> Package_SO:SOIC-14_3.9x8.7mm_P1.27mm
- renumbered R1 to R406
Connections:
- net _RESET renamed _IDERST
Changed lines of the file:
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@@
     (title "Amiga N2630")
     (date "2022-05-26")
-    (rev "2.0")
+    (rev "2.0 QFP")
   )
   (junction (at 340.487 113.284) (diameter 0) (color 0 0 0 0)
@@
     )
   )
-  (global_label "_RESET" (shape input) (at 247.523 94.615 180) (fields_autoplaced)
+  (global_label "_IDERST" (shape input) (at 247.523 94.615 180) (fields_autoplaced)
     (effects (font (size 1.27 1.27)) (justify right))
-    (property "Intersheet References" "${INTERSHEET_REFS}" (id 0) (at 238.4859 94.5356 0)
+    (property "Intersheet References" "${INTERSHEET_REFS}" (id 0) (at 237.7602 94.5356 0)
       (effects (font (size 1.27 1.27)) (justify right) hide)
     )
@@
     (in_bom yes) (on_board yes) (fields_autoplaced)
     (property "Reference" "U902" (id 0) (at 226.06 137.2702 0))
-    (property "Value" "" (id 1) (at 226.06 139.8071 0))
-    (property "Footprint" "" (id 2) (at 226.06 144.78 0)
+    (property "Value" "74HCT125" (id 1) (at 226.06 139.8071 0))
+    (property "Footprint" "Package_SO:SOIC-14_3.9x8.7mm_P1.27mm" (id 2) (at 226.06 144.78 0)
       (effects (font (size 1.27 1.27)) hide)
     )
@@
   (symbol (lib_id "Device:R") (at 178.435 55.499 0) (unit 1)
     (in_bom yes) (on_board yes)
-    (property "Reference" "R1" (id 0) (at 180.213 54.3306 0)
+    (property "Reference" "R406" (id 0) (at 180.213 54.3306 0)
       (effects (font (size 1.27 1.27)) (justify left))
     )
@@
       (effects (font (size 1.27 1.27)) (justify left))
     )
-    (property "Value" "" (id 1) (at 174.625 248.285 90)
+    (property "Value" "74HCT125" (id 1) (at 174.625 248.285 90)
       (effects (font (size 1.27 1.27)) (justify left))
     )
-    (property "Footprint" "" (id 2) (at 177.8 243.84 0)
+    (property "Footprint" "Package_SO:SOIC-14_3.9x8.7mm_P1.27mm" (id 2) (at 177.8 243.84 0)
       (effects (font (size 1.27 1.27)) hide)
     )
@@
     (in_bom yes) (on_board yes) (fields_autoplaced)
     (property "Reference" "U902" (id 0) (at 318.135 143.6354 0))
-    (property "Value" "" (id 1) (at 318.135 146.1723 0))
-    (property "Footprint" "" (id 2) (at 318.135 137.795 0)
+    (property "Value" "74HCT125" (id 1) (at 318.135 146.1723 0))
+    (property "Footprint" "Package_SO:SOIC-14_3.9x8.7mm_P1.27mm" (id 2) (at 318.135 137.795 0)
       (effects (font (size 1.27 1.27)) hide)
     )
@@
     (in_bom yes) (on_board yes) (fields_autoplaced)
     (property "Reference" "U902" (id 0) (at 225.425 113.7752 0))
-    (property "Value" "" (id 1) (at 225.425 116.3121 0))
-    (property "Footprint" "" (id 2) (at 225.425 121.285 0)
+    (property "Value" "74HCT125" (id 1) (at 225.425 116.3121 0))
+    (property "Footprint" "Package_SO:SOIC-14_3.9x8.7mm_P1.27mm" (id 2) (at 225.425 121.285 0)
       (effects (font (size 1.27 1.27)) hide)
     )
