File: A2630-New-KiCAD-Rev2-PGA/Card Edge.kicad_sch (KiCad schematic)
At the start: 31 parts, among them CN700 Amiga-2000-CPU-Slot, J302 Jumper_NO_Small, J303 Jumper_NO_Small, J304 Jumper_NO_Small, J305 Z3 DISABLE, U300 74HCT05, U700 74HCT174, U701 74FCT646, U702 74FCT646, U703 74HCT245, U704 74HCT245, U705 74HCT245, U706 74HCT245, U707 74HCT245

Commit message: Add files via upload
Connections:
- net GND: now also U700.11 (D3), U700.13 (D4), U700.14 (D5)
- new net: R706.2, U700.1 (~{Mr})
Changed lines of the file:
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@@
   (junction (at 320.04 41.275) (diameter 0) (color 0 0 0 0)
   )
-  (junction (at 68.58 76.962) (diameter 0) (color 0 0 0 0)
-  )
   (junction (at 237.49 224.155) (diameter 0) (color 0 0 0 0)
   )
@@
   (junction (at 178.435 165.735) (diameter 0) (color 0 0 0 0)
   )
-  (junction (at 68.58 93.345) (diameter 0) (color 0 0 0 0)
-  )
   (junction (at 307.34 194.31) (diameter 0) (color 0 0 0 0)
   )
@@
   (junction (at 240.03 224.155) (diameter 0) (color 0 0 0 0)
   )
-  (junction (at 68.58 83.185) (diameter 0) (color 0 0 0 0)
-  )
   (junction (at 298.45 194.31) (diameter 0) (color 0 0 0 0)
   )
+  (junction (at 68.58 93.345) (diameter 0) (color 0 0 0 0)
+  )
   (junction (at 240.03 243.84) (diameter 0) (color 0 0 0 0)
   )
@@
     (stroke (width 0) (type default) (color 0 0 0 0))
   )
+  (wire (pts (xy 88.392 93.345) (xy 88.392 95.25))
+    (stroke (width 0) (type default) (color 0 0 0 0))
+  )
   (wire (pts (xy 102.235 142.24) (xy 91.44 142.24))
     (stroke (width 0) (type default) (color 0 0 0 0))
@@
     (stroke (width 0) (type default) (color 0 0 0 0))
   )
-  (wire (pts (xy 68.58 76.835) (xy 68.58 76.962))
-    (stroke (width 0) (type default) (color 0 0 0 0))
-  )
   (wire (pts (xy 252.095 224.155) (xy 261.62 224.155))
     (stroke (width 0) (type default) (color 0 0 0 0))
@@
     (stroke (width 0) (type default) (color 0 0 0 0))
   )
-  (wire (pts (xy 68.58 76.962) (xy 68.58 83.185))
-    (stroke (width 0) (type default) (color 0 0 0 0))
-  )
   (wire (pts (xy 314.96 116.84) (xy 314.96 78.105))
     (stroke (width 0) (type default) (color 0 0 0 0))
@@
     (stroke (width 0) (type default) (color 0 0 0 0))
   )
+  (wire (pts (xy 68.58 93.345) (xy 88.392 93.345))
+    (stroke (width 0) (type default) (color 0 0 0 0))
+  )
   (wire (pts (xy 102.235 154.94) (xy 56.515 154.94))
     (stroke (width 0) (type default) (color 0 0 0 0))
@@
     (stroke (width 0) (type default) (color 0 0 0 0))
   )
-  (wire (pts (xy 68.58 93.345) (xy 68.58 83.185))
-    (stroke (width 0) (type default) (color 0 0 0 0))
-  )
   (bus (pts (xy 262.89 61.595) (xy 262.89 83.185))
     (stroke (width 0) (type default) (color 0 0 0 0))
@@
     (stroke (width 0) (type default) (color 0 0 0 0))
   )
+  (wire (pts (xy 68.58 76.962) (xy 68.58 83.185))
+    (stroke (width 0) (type default) (color 0 0 0 0))
+  )
   (wire (pts (xy 367.03 95.25) (xy 381.635 95.25))
     (stroke (width 0) (type default) (color 0 0 0 0))
@@
   (symbol (lib_id "Device:R") (at 364.49 67.945 0) (unit 1)
     (in_bom yes) (on_board yes)
-    (property "Reference" "R305" (id 0) (at 365.76 65.405 90)
+    (property "Reference" "R305" (id 0) (at 364.49 63.5 90)
       (effects (font (size 1.27 1.27)) (justify left))
     )
@@
   (symbol (lib_id "Device:R") (at 361.95 67.945 0) (unit 1)
     (in_bom yes) (on_board yes)
-    (property "Reference" "R304" (id 0) (at 363.22 65.405 90)
+    (property "Reference" "R304" (id 0) (at 361.95 63.5 90)
       (effects (font (size 1.27 1.27)) (justify left))
     )
@@
   (symbol (lib_id "Device:R") (at 359.41 67.945 0) (unit 1)
     (in_bom yes) (on_board yes)
-    (property "Reference" "R303" (id 0) (at 360.68 65.405 90)
+    (property "Reference" "R303" (id 0) (at 359.41 63.5 90)
       (effects (font (size 1.27 1.27)) (justify left))
     )
@@
     (pin "2")
   )
+  (symbol (lib_id "power:GND") (at 88.392 95.25 0) (unit 1)
+    (in_bom yes) (on_board yes) (fields_autoplaced)
+    (property "Reference" "#PWR?" (id 0) (at 88.392 101.6 0)
+      (effects (font (size 1.27 1.27)) hide)
+    )
+    (property "Value" "GND" (id 1) (at 88.392 99.6934 0))
+    (property "Footprint" "" (id 2) (at 88.392 95.25 0)
+      (effects (font (size 1.27 1.27)) hide)
+    )
+    (property "Datasheet" "" (id 3) (at 88.392 95.25 0)
+      (effects (font (size 1.27 1.27)) hide)
+    )
+    (pin "1")
+  )
   (symbol (lib_id "power:+5V") (at 68.072 112.395 0) (unit 1)
     (in_bom yes) (on_board yes)
@@
   (symbol (lib_id "Device:R") (at 367.03 67.945 0) (unit 1)
     (in_bom yes) (on_board yes)
-    (property "Reference" "R306" (id 0) (at 368.3 65.405 90)
+    (property "Reference" "R306" (id 0) (at 367.03 63.5 90)
       (effects (font (size 1.27 1.27)) (justify left))
     )

Commit message: Add files via upload
Parts:
- added C719: 10uF, Capacitor_THT:CP_Radial_D5.0mm_P2.00mm, symbol Device:CP1
Connections:
- net +5V: now also C719.1
- net GND: now also C719.2
Changed lines of the file:
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@@
   (junction (at 252.095 243.84) (diameter 0) (color 0 0 0 0)
   )
+  (junction (at 263.525 243.84) (diameter 0) (color 0 0 0 0)
+  )
   (junction (at 365.125 194.31) (diameter 0) (color 0 0 0 0)
   )
@@
   (junction (at 237.49 194.31) (diameter 0) (color 0 0 0 0)
   )
+  (junction (at 275.082 224.155) (diameter 0) (color 0 0 0 0)
+  )
   (junction (at 227.965 224.155) (diameter 0) (color 0 0 0 0)
   )
@@
     (stroke (width 0) (type default) (color 0 0 0 0))
   )
+  (wire (pts (xy 263.525 243.84) (xy 275.082 243.84))
+    (stroke (width 0) (type default) (color 0 0 0 0))
+  )
   (bus (pts (xy 158.75 80.645) (xy 158.75 83.185))
     (stroke (width 0) (type default) (color 0 0 0 0))
@@
     (stroke (width 0) (type default) (color 0 0 0 0))
   )
-  (wire (pts (xy 263.525 224.155) (xy 276.225 224.155))
+  (wire (pts (xy 263.525 224.155) (xy 275.082 224.155))
     (stroke (width 0) (type default) (color 0 0 0 0))
   )
@@
     (stroke (width 0) (type default) (color 0 0 0 0))
   )
+  (wire (pts (xy 275.082 224.155) (xy 276.225 224.155))
+    (stroke (width 0) (type default) (color 0 0 0 0))
+  )
   (wire (pts (xy 364.49 90.805) (xy 381.635 90.805))
     (stroke (width 0) (type default) (color 0 0 0 0))
@@
     (stroke (width 0) (type default) (color 0 0 0 0))
   )
+  (wire (pts (xy 275.082 229.87) (xy 275.082 224.155))
+    (stroke (width 0) (type default) (color 0 0 0 0))
+  )
   (bus (pts (xy 158.75 65.405) (xy 158.75 67.945))
     (stroke (width 0) (type default) (color 0 0 0 0))
@@
     (stroke (width 0) (type default) (color 0 0 0 0))
   )
+  (wire (pts (xy 275.082 243.84) (xy 275.082 237.49))
+    (stroke (width 0) (type default) (color 0 0 0 0))
+  )
   (bus (pts (xy 404.495 24.765) (xy 310.515 24.765))
     (stroke (width 0) (type default) (color 0 0 0 0))
@@
     (pin "1")
   )
+  (symbol (lib_id "Device:CP1") (at 275.082 233.68 180) (unit 1)
+    (in_bom yes) (on_board yes)
+    (property "Reference" "C719" (id 0) (at 278.003 232.5116 0)
+      (effects (font (size 1.27 1.27)) (justify right))
+    )
+    (property "Value" "10uF" (id 1) (at 278.003 234.823 0)
+      (effects (font (size 1.27 1.27)) (justify right))
+    )
+    (property "Footprint" "Capacitor_THT:CP_Radial_D5.0mm_P2.00mm" (id 2) (at 275.082 233.68 0)
+      (effects (font (size 1.27 1.27)) hide)
+    )
+    (property "Datasheet" "~" (id 3) (at 275.082 233.68 0)
+      (effects (font (size 1.27 1.27)) hide)
+    )
+    (pin "1")
+    (pin "2")
+  )
   (symbol (lib_id "Device:R") (at 364.49 67.945 0) (unit 1)
     (in_bom yes) (on_board yes)
@@
   (symbol (lib_id "power:GND") (at 88.392 95.25 0) (unit 1)
     (in_bom yes) (on_board yes) (fields_autoplaced)
-    (property "Reference" "#PWR?" (id 0) (at 88.392 101.6 0)
+    (property "Reference" "#PWR04" (id 0) (at 88.392 101.6 0)
       (effects (font (size 1.27 1.27)) hide)
     )
