File: A2630-New-KiCAD-Rev21-PGA/Card Edge.kicad_sch (KiCad schematic)
At the start: 32 parts, among them CN700 Amiga-2000-CPU-Slot, J302 Jumper_NO_Small, J303 Jumper_NO_Small, J304 Jumper_NO_Small, J305 Z3 DISABLE, U300 74HCT05, U700 74HCT174, U701 74FCT646, U702 74FCT646, U703 74HCT245, U704 74HCT245, U705 74HCT245, U706 74HCT245, U707 74HCT245

Commit message: Add files via upload
Parts:
- R706: value 1k -> 1K
Changed lines of the file:
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@@
       (effects (font (size 1.27 1.27)) (justify left))
     )
-    (property "Value" "1k" (id 1) (at 70.358 74.295 0)
+    (property "Value" "1K" (id 1) (at 70.358 74.295 0)
       (effects (font (size 1.27 1.27)) (justify left))
     )

Commit message: Add files via upload
Parts:
- CN700: now left out of the parts list
Changed lines of the file:
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@@
   )
   (symbol (lib_id "N2630:Amiga-2000-CPU-Slot") (at 103.505 185.42 0) (unit 1)
-    (in_bom yes) (on_board yes)
+    (in_bom no) (on_board yes)
     (property "Reference" "CN700" (id 0) (at 100.965 128.905 0)
       (effects (font (size 1.27 1.27)) (justify left))

Commit message: Add files via upload
Connections:
- net _AIPL0: now reaches CN700.40, U700.6 (D2)
- net _AIPL1: now reaches CN700.42, U700.4 (D1)
- net _AIPL2: now reaches CN700.44, U700.3 (D0)
Changed lines of the file:
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@@
     (effects (font (size 1.2954 1.2954)) (justify right bottom))
+  )
+  (label "_AIPL2" (at 64.135 106.045 0)
+    (effects (font (size 1.27 1.27)) (justify left bottom))
   )
   (label "D21" (at 161.29 125.73 0)
@@
   (label "A18" (at 307.975 59.055 180)
     (effects (font (size 1.2954 1.2954)) (justify right bottom))
+  )
+  (label "_AIPL0" (at 64.135 100.965 0)
+    (effects (font (size 1.27 1.27)) (justify left bottom))
   )
   (label "_COPCFG" (at 52.578 139.7 0)
@@
     (effects (font (size 1.2954 1.2954)) (justify left bottom))
   )
+  (label "_AIPL1" (at 64.135 103.505 0)
+    (effects (font (size 1.27 1.27)) (justify left bottom))
+  )
   (label "AD8" (at 132.715 241.3 180)

Commit message: Add files via upload
Parts:
- U300: value 74HCT05 -> 74HCT04
Connections:
- net GND: now also U701.1 (CPAB), U702.1 (CPAB)
- net _BOSS: no longer U705.19 (CE), U706.19 (CE), U707.19 (CE)
- net 7M: now reaches U701.23 (CPBA)
- net 7M: now also U702.23 (CPBA)
- net _BGACK renamed AADIR
- new net _AAENA: U705.19 (CE), U706.19 (CE), U707.19 (CE)
Changed lines of the file:
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@@
   (junction (at 109.22 177.8) (diameter 0) (color 0 0 0 0)
   )
+  (junction (at 141.478 132.207) (diameter 0) (color 0 0 0 0)
+  )
   (junction (at 261.62 194.31) (diameter 0) (color 0 0 0 0)
   )
@@
   (junction (at 240.03 243.84) (diameter 0) (color 0 0 0 0)
   )
+  (junction (at 149.987 75.565) (diameter 0) (color 0 0 0 0)
+  )
   (junction (at 261.62 224.155) (diameter 0) (color 0 0 0 0)
   )
@@
     (stroke (width 0) (type default) (color 0 0 0 0))
   )
+  (wire (pts (xy 169.545 130.81) (xy 164.338 130.81))
+    (stroke (width 0) (type default) (color 0 0 0 0))
+  )
   (wire (pts (xy 109.22 135.89) (xy 109.22 147.32))
     (stroke (width 0) (type default) (color 0 0 0 0))
@@
     (stroke (width 0) (type default) (color 0 0 0 0))
   )
+  (wire (pts (xy 164.338 130.81) (xy 164.338 132.207))
+    (stroke (width 0) (type default) (color 0 0 0 0))
+  )
   (wire (pts (xy 169.545 225.425) (xy 161.29 225.425))
     (stroke (width 0) (type default) (color 0 0 0 0))
@@
     (stroke (width 0) (type default) (color 0 0 0 0))
   )
+  (wire (pts (xy 26.67 50.546) (xy 149.987 50.546))
+    (stroke (width 0) (type default) (color 0 0 0 0))
+  )
   (wire (pts (xy 298.45 219.075) (xy 298.45 224.155))
     (stroke (width 0) (type default) (color 0 0 0 0))
@@
     (stroke (width 0) (type default) (color 0 0 0 0))
   )
+  (wire (pts (xy 149.987 50.546) (xy 149.987 75.565))
+    (stroke (width 0) (type default) (color 0 0 0 0))
+  )
   (bus (pts (xy 310.515 83.185) (xy 310.515 85.725))
     (stroke (width 0) (type default) (color 0 0 0 0))
@@
     (stroke (width 0) (type default) (color 0 0 0 0))
   )
+  (wire (pts (xy 141.478 74.295) (xy 164.211 74.295))
+    (stroke (width 0) (type default) (color 0 0 0 0))
+  )
   (wire (pts (xy 299.085 61.595) (xy 307.975 61.595))
     (stroke (width 0) (type default) (color 0 0 0 0))
@@
     (stroke (width 0) (type default) (color 0 0 0 0))
   )
+  (wire (pts (xy 149.987 75.565) (xy 170.18 75.565))
+    (stroke (width 0) (type default) (color 0 0 0 0))
+  )
   (wire (pts (xy 351.79 205.105) (xy 351.79 194.31))
     (stroke (width 0) (type default) (color 0 0 0 0))
@@
     (stroke (width 0) (type default) (color 0 0 0 0))
   )
+  (wire (pts (xy 164.211 74.295) (xy 164.211 73.025))
+    (stroke (width 0) (type default) (color 0 0 0 0))
+  )
   (bus (pts (xy 262.89 46.355) (xy 262.89 48.895))
     (stroke (width 0) (type default) (color 0 0 0 0))
@@
     (stroke (width 0) (type default) (color 0 0 0 0))
   )
+  (wire (pts (xy 141.478 132.207) (xy 141.478 74.295))
+    (stroke (width 0) (type default) (color 0 0 0 0))
+  )
   (bus (pts (xy 31.75 100.965) (xy 31.75 103.505))
     (stroke (width 0) (type default) (color 0 0 0 0))
@@
     (stroke (width 0) (type default) (color 0 0 0 0))
   )
+  (wire (pts (xy 141.478 132.207) (xy 164.338 132.207))
+    (stroke (width 0) (type default) (color 0 0 0 0))
+  )
   (wire (pts (xy 119.38 234.95) (xy 119.38 245.11))
     (stroke (width 0) (type default) (color 0 0 0 0))
@@
     (stroke (width 0) (type default) (color 0 0 0 0))
   )
+  (wire (pts (xy 141.478 132.207) (xy 141.478 134.874))
+    (stroke (width 0) (type default) (color 0 0 0 0))
+  )
   (wire (pts (xy 364.49 71.755) (xy 364.49 90.805))
     (stroke (width 0) (type default) (color 0 0 0 0))
@@
     (stroke (width 0) (type default) (color 0 0 0 0))
   )
+  (wire (pts (xy 164.211 73.025) (xy 170.18 73.025))
+    (stroke (width 0) (type default) (color 0 0 0 0))
+  )
   (wire (pts (xy 153.035 104.775) (xy 179.07 104.775))
     (stroke (width 0) (type default) (color 0 0 0 0))
@@
     (stroke (width 0) (type default) (color 0 0 0 0))
   )
+  (wire (pts (xy 149.987 133.35) (xy 169.545 133.35))
+    (stroke (width 0) (type default) (color 0 0 0 0))
+  )
   (bus (pts (xy 158.75 238.125) (xy 158.75 259.715))
     (stroke (width 0) (type default) (color 0 0 0 0))
@@
     (stroke (width 0) (type default) (color 0 0 0 0))
   )
+  (wire (pts (xy 149.987 75.565) (xy 149.987 133.35))
+    (stroke (width 0) (type default) (color 0 0 0 0))
+  )
   (bus (pts (xy 158.75 230.505) (xy 158.75 233.045))
     (stroke (width 0) (type default) (color 0 0 0 0))
@@
     )
   )
+  (global_label "7M" (shape input) (at 26.67 50.546 180) (fields_autoplaced)
+    (effects (font (size 1.27 1.27)) (justify right))
+    (property "Intersheet References" "${INTERSHEET_REFS}" (id 0) (at 21.6848 50.6254 0)
+      (effects (font (size 1.27 1.27)) (justify right) hide)
+    )
+  )
   (global_label "B2000" (shape output) (at 381.635 81.915 0) (fields_autoplaced)
     (effects (font (size 1.2954 1.2954)) (justify left))
@@
     )
   )
-  (global_label "_BGACK" (shape input) (at 404.495 41.275 0) (fields_autoplaced)
+  (global_label "AADIR" (shape input) (at 404.495 41.275 0) (fields_autoplaced)
     (effects (font (size 1.2954 1.2954)) (justify left))
-    (property "Intersheet References" "${INTERSHEET_REFS}" (id 0) (at 0 0 0)
-      (effects (font (size 1.27 1.27)) hide)
+    (property "Intersheet References" "${INTERSHEET_REFS}" (id 0) (at 412.2938 41.1941 0)
+      (effects (font (size 1.2954 1.2954)) (justify left) hide)
     )
   )
@@
     )
   )
-  (global_label "_BOSS" (shape input) (at 404.495 38.735 0) (fields_autoplaced)
+  (global_label "_AAENA" (shape input) (at 404.495 38.735 0) (fields_autoplaced)
     (effects (font (size 1.2954 1.2954)) (justify left))
-    (property "Intersheet References" "${INTERSHEET_REFS}" (id 0) (at 0 0 0)
-      (effects (font (size 1.27 1.27)) hide)
+    (property "Intersheet References" "${INTERSHEET_REFS}" (id 0) (at 413.7126 38.6541 0)
+      (effects (font (size 1.2954 1.2954)) (justify left) hide)
     )
   )
@@
     (pin "1")
   )
+  (symbol (lib_id "power:GND") (at 141.478 134.874 0) (unit 1)
+    (in_bom yes) (on_board yes) (fields_autoplaced)
+    (property "Reference" "#PWR?" (id 0) (at 141.478 141.224 0)
+      (effects (font (size 1.27 1.27)) hide)
+    )
+    (property "Value" "GND" (id 1) (at 141.478 139.3174 0))
+    (property "Footprint" "" (id 2) (at 141.478 134.874 0)
+      (effects (font (size 1.27 1.27)) hide)
+    )
+    (property "Datasheet" "" (id 3) (at 141.478 134.874 0)
+      (effects (font (size 1.27 1.27)) hide)
+    )
+    (pin "1")
+  )
   (symbol (lib_id "Device:R") (at 367.03 67.945 0) (unit 1)
     (in_bom yes) (on_board yes)
@@
     (in_bom yes) (on_board yes)
     (property "Reference" "U300" (id 0) (at 44.831 132.08 0))
-    (property "Value" "74HCT05" (id 1) (at 44.831 134.62 0))
+    (property "Value" "74HCT04" (id 1) (at 44.831 134.62 0))
     (property "Footprint" "Package_SO:SOIC-14_3.9x8.7mm_P1.27mm" (id 2) (at 44.831 139.7 0)
       (effects (font (size 1.27 1.27)) hide)

Commit message: Add files via upload
Parts:
- added unit 5 of U300
- added unit 4 of U300
Connections:
- net _BERR: now also U300.8; no longer CN700.46
- new net: U300.10, U300.9
- new net _ABERR: CN700.46, U300.11
Changed lines of the file:
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@@
   (title_block
     (title "Amiga N2630")
-    (date "2022-06-05")
+    (date "2022-07-21")
     (rev "2.1 QFP")
   )
@@
     (stroke (width 0) (type default) (color 0 0 0 0))
   )
-  (wire (pts (xy 72.39 183.134) (xy 72.39 187.96))
-    (stroke (width 0) (type default) (color 0 0 0 0))
-  )
   (bus (pts (xy 310.515 51.435) (xy 310.515 53.975))
     (stroke (width 0) (type default) (color 0 0 0 0))
@@
     (stroke (width 0) (type default) (color 0 0 0 0))
   )
+  (wire (pts (xy 72.39 179.959) (xy 72.39 187.96))
+    (stroke (width 0) (type default) (color 0 0 0 0))
+  )
   (wire (pts (xy 240.03 224.155) (xy 252.095 224.155))
     (stroke (width 0) (type default) (color 0 0 0 0))
@@
     (stroke (width 0) (type default) (color 0 0 0 0))
   )
+  (wire (pts (xy 23.622 179.959) (xy 32.385 179.959))
+    (stroke (width 0) (type default) (color 0 0 0 0))
+  )
   (wire (pts (xy 118.11 236.22) (xy 118.11 247.015))
     (stroke (width 0) (type default) (color 0 0 0 0))
@@
     (stroke (width 0) (type default) (color 0 0 0 0))
   )
+  (wire (pts (xy 62.865 179.959) (xy 72.39 179.959))
+    (stroke (width 0) (type default) (color 0 0 0 0))
+  )
   (wire (pts (xy 237.49 205.105) (xy 237.49 194.31))
     (stroke (width 0) (type default) (color 0 0 0 0))
@@
     (stroke (width 0) (type default) (color 0 0 0 0))
   )
-  (wire (pts (xy 24.13 183.134) (xy 72.39 183.134))
-    (stroke (width 0) (type default) (color 0 0 0 0))
-  )
   (wire (pts (xy 273.685 137.16) (xy 265.43 137.16))
     (stroke (width 0) (type default) (color 0 0 0 0))
@@
     (effects (font (size 1.2954 1.2954)) (justify left bottom))
   )
+  (label "_ABERR" (at 72.263 179.959 180)
+    (effects (font (size 1.27 1.27)) (justify right bottom))
+  )
   (label "AD5" (at 203.2 125.73 180)
     (effects (font (size 1.2954 1.2954)) (justify right bottom))
@@
     (effects (font (size 1.2954 1.2954)) (justify left bottom))
   )
-  (global_label "_BERR" (shape output) (at 24.13 183.134 180) (fields_autoplaced)
+  (global_label "_BERR" (shape output) (at 23.622 179.959 180) (fields_autoplaced)
     (effects (font (size 1.2954 1.2954)) (justify right))
-    (property "Intersheet References" "${INTERSHEET_REFS}" (id 0) (at 0 -0.381 0)
+    (property "Intersheet References" "${INTERSHEET_REFS}" (id 0) (at -0.508 -3.556 0)
       (effects (font (size 1.27 1.27)) hide)
     )
@@
     )
   )
-  (global_label "_HALT" (shape output) (at 24.13 200.66 180) (fields_autoplaced)
+  (global_label "_HALT" (shape bidirectional) (at 24.13 200.66 180) (fields_autoplaced)
     (effects (font (size 1.27 1.27)) (justify right))
-    (property "Intersheet References" "${INTERSHEET_REFS}" (id 0) (at 0 0 0)
-      (effects (font (size 1.27 1.27)) hide)
+    (property "Intersheet References" "${INTERSHEET_REFS}" (id 0) (at 16.4234 200.5806 0)
+      (effects (font (size 1.27 1.27)) (justify right) hide)
     )
   )
@@
     (pin "2")
   )
+  (symbol (lib_id "74xx:74LS05") (at 55.245 179.959 180) (unit 5)
+    (in_bom yes) (on_board yes)
+    (property "Reference" "U300" (id 0) (at 55.245 187.579 0))
+    (property "Value" "74HCT04" (id 1) (at 55.245 185.039 0))
+    (property "Footprint" "Package_SO:SOIC-14_3.9x8.7mm_P1.27mm" (id 2) (at 55.245 179.959 0)
+      (effects (font (size 1.27 1.27)) hide)
+    )
+    (property "Datasheet" "http://www.ti.com/lit/gpn/sn74LS05" (id 3) (at 55.245 179.959 0)
+      (effects (font (size 1.27 1.27)) hide)
+    )
+    (pin "1")
+    (pin "2")
+    (pin "3")
+    (pin "4")
+    (pin "5")
+    (pin "6")
+    (pin "8")
+    (pin "9")
+    (pin "10")
+    (pin "11")
+    (pin "12")
+    (pin "13")
+    (pin "14")
+    (pin "7")
+  )
   (symbol (lib_id "Device:R") (at 364.49 67.945 0) (unit 1)
     (in_bom yes) (on_board yes)
@@
   (symbol (lib_id "power:GND") (at 141.478 134.874 0) (unit 1)
     (in_bom yes) (on_board yes) (fields_autoplaced)
-    (property "Reference" "#PWR?" (id 0) (at 141.478 141.224 0)
+    (property "Reference" "#PWR0153" (id 0) (at 141.478 141.224 0)
       (effects (font (size 1.27 1.27)) hide)
     )
@@
     (pin "2")
   )
+  (symbol (lib_id "74xx:74LS05") (at 40.005 179.959 180) (unit 4)
+    (in_bom yes) (on_board yes)
+    (property "Reference" "U300" (id 0) (at 40.005 187.579 0))
+    (property "Value" "74HCT04" (id 1) (at 40.005 185.039 0))
+    (property "Footprint" "Package_SO:SOIC-14_3.9x8.7mm_P1.27mm" (id 2) (at 40.005 179.959 0)
+      (effects (font (size 1.27 1.27)) hide)
+    )
+    (property "Datasheet" "http://www.ti.com/lit/gpn/sn74LS05" (id 3) (at 40.005 179.959 0)
+      (effects (font (size 1.27 1.27)) hide)
+    )
+    (pin "1")
+    (pin "2")
+    (pin "3")
+    (pin "4")
+    (pin "5")
+    (pin "6")
+    (pin "8")
+    (pin "9")
+    (pin "10")
+    (pin "11")
+    (pin "12")
+    (pin "13")
+    (pin "14")
+    (pin "7")
+  )
   (symbol (lib_id "74xx:74LS05") (at 44.831 139.7 0) (unit 3)
