File: A2630-New-KiCAD-Rev21-PGA/ExpansionMemory.kicad_sch (KiCad schematic)
At the start: 31 parts, among them J400 Jumper_NO_Small, J401 Jumper_NO_Small, J402 Jumper_NO_Small, J403 Jumper_NO_Small, J404 Jumper_NO_Small, U102 27C256, U103 27C256, U406 SDRAM(16Mx16), U407 SDRAM(16Mx16), U408 SDRAM(16Mx16), U409 SDRAM(16Mx16)

Commit message: Add files via upload
Connections:
- net A16: no longer names the net of U103.1 (VPP)
- net A16: no longer U102.1 (VPP)
- no-connect marks 0 -> 2
Changed lines of the file:
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@@
   (junction (at 212.09 219.71) (diameter 0) (color 0 0 0 0)
   )
+  (no_connect (at 366.395 88.265))
+  (no_connect (at 320.675 88.265))
   (bus_entry (at 81.28 157.48) (size -2.54 -2.54)
     (stroke (width 0) (type default) (color 0 0 0 0))
@@
     (stroke (width 0) (type default) (color 0 0 0 0))
   )
-  (bus_entry (at 361.315 88.265) (size -2.54 -2.54)
-    (stroke (width 0) (type default) (color 0 0 0 0))
-  )
   (bus_entry (at 361.315 52.705) (size -2.54 -2.54)
     (stroke (width 0) (type default) (color 0 0 0 0))
@@
     (stroke (width 0) (type default) (color 0 0 0 0))
   )
-  (bus_entry (at 315.595 88.265) (size -2.54 -2.54)
-    (stroke (width 0) (type default) (color 0 0 0 0))
-  )
   (bus_entry (at 315.595 50.165) (size -2.54 -2.54)
     (stroke (width 0) (type default) (color 0 0 0 0))
@@
     (stroke (width 0) (type default) (color 0 0 0 0))
   )
-  (bus (pts (xy 358.775 85.725) (xy 358.775 110.49))
+  (bus (pts (xy 358.775 80.645) (xy 358.775 110.49))
     (stroke (width 0) (type default) (color 0 0 0 0))
   )
@@
     (stroke (width 0) (type default) (color 0 0 0 0))
   )
-  (wire (pts (xy 320.675 88.265) (xy 315.595 88.265))
-    (stroke (width 0) (type default) (color 0 0 0 0))
-  )
   (wire (pts (xy 398.145 210.185) (xy 406.4 210.185))
     (stroke (width 0) (type default) (color 0 0 0 0))
@@
     (stroke (width 0) (type default) (color 0 0 0 0))
   )
-  (bus (pts (xy 358.775 80.645) (xy 358.775 85.725))
-    (stroke (width 0) (type default) (color 0 0 0 0))
-  )
   (wire (pts (xy 209.55 151.13) (xy 209.55 148.59))
     (stroke (width 0) (type default) (color 0 0 0 0))
@@
     (stroke (width 0) (type default) (color 0 0 0 0))
   )
-  (wire (pts (xy 366.395 88.265) (xy 361.315 88.265))
-    (stroke (width 0) (type default) (color 0 0 0 0))
-  )
   (wire (pts (xy 366.395 65.405) (xy 361.315 65.405))
     (stroke (width 0) (type default) (color 0 0 0 0))
@@
     (stroke (width 0) (type default) (color 0 0 0 0))
   )
-  (bus (pts (xy 313.055 85.725) (xy 313.055 107.95))
+  (bus (pts (xy 313.055 80.645) (xy 313.055 107.95))
     (stroke (width 0) (type default) (color 0 0 0 0))
   )
@@
   )
   (wire (pts (xy 133.35 231.14) (xy 30.48 231.14))
-    (stroke (width 0) (type default) (color 0 0 0 0))
-  )
-  (bus (pts (xy 313.055 80.645) (xy 313.055 85.725))
     (stroke (width 0) (type default) (color 0 0 0 0))
   )
@@
     (effects (font (size 1.27 1.27)) (justify left bottom))
   )
-  (label "A16" (at 361.315 88.265 0)
-    (effects (font (size 1.27 1.27)) (justify left bottom))
-  )
   (label "EMA7" (at 182.88 83.82 0)
     (effects (font (size 1.27 1.27)) (justify left bottom))
@@
     (effects (font (size 1.27 1.27)) (justify left bottom))
   )
-  (label "A16" (at 315.595 88.265 0)
-    (effects (font (size 1.27 1.27)) (justify left bottom))
-  )
