File: A2630-New-KiCAD-Rev21-PGA/N2360.kicad_sch (KiCad schematic)
At the start: 0 parts

Commit message: Add files via upload
Other:
- note added: "CHANGED ROUTE OF _BG UPDATED BLOCK DIAGRAM CONNECTED _ONBOARD BETWEEN U600 & 601"
- note removed: "CHANGED ROUTE OF _BG UPDATED BLOCK DIAGRAM"
Changed lines of the file:
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@@
     )
   )
-  (text "CHANGED ROUTE OF _BG\nUPDATED BLOCK DIAGRAM" (at 32.385 227.965 0)
+  (text "CHANGED ROUTE OF _BG\nUPDATED BLOCK DIAGRAM\nCONNECTED _ONBOARD BETWEEN U600 & 601"
+    (at 32.385 227.965 0)
     (effects (font (size 2 2)) (justify left bottom))
   )
@@
     )
     (path "/00000000-0000-0000-0000-0000634ecc15/00000000-0000-0000-0000-00006353b771"
-      (reference "C300") (unit 1) (value "0.22uf") (footprint "Capacitor_SMD:C_0805_2012Metric")
+      (reference "C300") (unit 1) (value "0.22uF") (footprint "Capacitor_SMD:C_0805_2012Metric")
     )
     (path "/00000000-0000-0000-0000-000061d9c8dc/00000000-0000-0000-0000-000062f57967"
@@
     )
     (path "/00000000-0000-0000-0000-0000634ecc15/e3a5749a-06b1-4652-8d14-c1188ceff788"
-      (reference "C418") (unit 1) (value "0.22uf") (footprint "Capacitor_SMD:C_0805_2012Metric")
+      (reference "C418") (unit 1) (value "0.22uF") (footprint "Capacitor_SMD:C_0805_2012Metric")
     )
     (path "/00000000-0000-0000-0000-0000634ecc15/f5409630-eb22-4a5f-83e0-a76f7645f97a"
-      (reference "C419") (unit 1) (value "0.22uf") (footprint "Capacitor_SMD:C_0805_2012Metric")
+      (reference "C419") (unit 1) (value "0.22uF") (footprint "Capacitor_SMD:C_0805_2012Metric")
     )
     (path "/00000000-0000-0000-0000-0000634ecc15/92b829ac-b135-4d17-a413-fe66f5f0b73a"
-      (reference "C420") (unit 1) (value "0.22uf") (footprint "Capacitor_SMD:C_0805_2012Metric")
+      (reference "C420") (unit 1) (value "0.22uF") (footprint "Capacitor_SMD:C_0805_2012Metric")
     )
     (path "/00000000-0000-0000-0000-0000634ecc15/94826e71-e4c9-47cd-9978-67efa513fa1e"
-      (reference "C421") (unit 1) (value "0.22uf") (footprint "Capacitor_SMD:C_0805_2012Metric")
+      (reference "C421") (unit 1) (value "0.22uF") (footprint "Capacitor_SMD:C_0805_2012Metric")
     )
     (path "/00000000-0000-0000-0000-000061d9c8dc/47237a30-5dd2-4ae9-9ffc-945423ba4f5f"
@@
     )
     (path "/00000000-0000-0000-0000-0000634ecc15/00000000-0000-0000-0000-00006353d849"
-      (reference "C606") (unit 1) (value "0.22uf") (footprint "Capacitor_SMD:C_0805_2012Metric")
+      (reference "C606") (unit 1) (value "0.22uF") (footprint "Capacitor_SMD:C_0805_2012Metric")
     )
     (path "/00000000-0000-0000-0000-000062089831/7fe9de19-9c81-40a2-a5bf-845f55fe22c0"
@@
     )
     (path "/00000000-0000-0000-0000-0000634ecc15/e2cede5f-1a19-467f-9f46-a0e8e0a1caae"
-      (reference "C900") (unit 1) (value "0.22uf") (footprint "Capacitor_SMD:C_0805_2012Metric")
+      (reference "C900") (unit 1) (value "0.22uF") (footprint "Capacitor_SMD:C_0805_2012Metric")
     )
     (path "/00000000-0000-0000-0000-0000634ecc15/975ee057-ed5e-43b5-9db5-9030e0584272"
-      (reference "C901") (unit 1) (value "0.22uf") (footprint "Capacitor_SMD:C_0805_2012Metric")
+      (reference "C901") (unit 1) (value "0.22uF") (footprint "Capacitor_SMD:C_0805_2012Metric")
     )
     (path "/00000000-0000-0000-0000-0000634ecc15/52c6e3e6-d3c1-4d90-b616-c66a78fd0aa3"
-      (reference "C902") (unit 1) (value "0.22uf") (footprint "Capacitor_SMD:C_0805_2012Metric")
+      (reference "C902") (unit 1) (value "0.22uF") (footprint "Capacitor_SMD:C_0805_2012Metric")
     )
     (path "/00000000-0000-0000-0000-0000634ecc15/530da3a7-2703-4790-b4ff-b781e3a8b1bf"
@@
     )
     (path "/00000000-0000-0000-0000-000061df74a0/00000000-0000-0000-0000-000062551812"
-      (reference "R706") (unit 1) (value "1k") (footprint "Resistor_SMD:R_0805_2012Metric")
+      (reference "R706") (unit 1) (value "1K") (footprint "Resistor_SMD:R_0805_2012Metric")
     )
     (path "/00000000-0000-0000-0000-000061d79ebc/00000000-0000-0000-0000-000062dfcaac"

Commit message: Add files via upload
Other:
- note added: "CHANGED ROUTE OF _BG UPDATED BLOCK DIAGRAM CONNECTED _ONBOARD BETWEEN U600 & 601 Fixed A2 Crazy Trace CONNECT MODE68K U601 AND U600 TODO: REMOVE A16 FROM ROMs"
- note removed: "CHANGED ROUTE OF _BG UPDATED BLOCK DIAGRAM CONNECTED _ONBOARD BETWEEN U600 & 601"
Changed lines of the file:
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@@
     )
   )
-  (text "CHANGED ROUTE OF _BG\nUPDATED BLOCK DIAGRAM\nCONNECTED _ONBOARD BETWEEN U600 & 601"
+  (text "CHANGED ROUTE OF _BG\nUPDATED BLOCK DIAGRAM\nCONNECTED _ONBOARD BETWEEN U600 & 601\nFixed A2 Crazy Trace\nCONNECT MODE68K U601 AND U600\n\nTODO: REMOVE A16 FROM ROMs"
     (at 32.385 227.965 0)
     (effects (font (size 2 2)) (justify left bottom))

Commit message: Add files via upload
Other:
- note removed: "CHANGED ROUTE OF _BG UPDATED BLOCK DIAGRAM CONNECTED _ONBOARD BETWEEN U600 & 601 Fixed A2 Crazy Trace CONNECT MODE68K U601 AND U600 TODO: REMOVE A16 FROM ROMs"
Changed lines of the file:
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@@
   (title_block
     (title "Amiga N2630")
-    (date "2022-06-05")
+    (date "2022-07-21")
     (rev "2.1 QFP")
   )
@@
     )
   )
-  (text "CHANGED ROUTE OF _BG\nUPDATED BLOCK DIAGRAM\nCONNECTED _ONBOARD BETWEEN U600 & 601\nFixed A2 Crazy Trace\nCONNECT MODE68K U601 AND U600\n\nTODO: REMOVE A16 FROM ROMs"
-    (at 32.385 227.965 0)
-    (effects (font (size 2 2)) (justify left bottom))
-  )
   (text "AMIGA N2630" (at 314.452 245.618 0)
     (effects (font (size 6 6)) (justify left bottom))
@@
       (reference "#PWR0148") (unit 1) (value "GND") (footprint "")
     )
-    (path "/00000000-0000-0000-0000-0000634ecc15/13040080-f24d-4f78-98a5-6c5df98b58c3"
-      (reference "#PWR0149") (unit 1) (value "+3.3V") (footprint "")
-    )
     (path "/00000000-0000-0000-0000-0000634ecc15/7a5ce3d5-cb25-428c-a9ca-16ea991a720b"
       (reference "#PWR0150") (unit 1) (value "+3.3V") (footprint "")
     )
+    (path "/00000000-0000-0000-0000-0000634ecc15/8604977b-2d6f-42be-81b7-a944e68d0b8b"
+      (reference "#PWR0151") (unit 1) (value "+3.3V") (footprint "")
+    )
+    (path "/00000000-0000-0000-0000-0000634ecc15/609e499a-8e19-4a2a-87f6-e6af7657800e"
+      (reference "#PWR0152") (unit 1) (value "+3.3V") (footprint "")
+    )
+    (path "/00000000-0000-0000-0000-000061df74a0/9481eb72-b44f-4908-8d19-cced640e09b3"
+      (reference "#PWR0153") (unit 1) (value "GND") (footprint "")
+    )
     (path "/00000000-0000-0000-0000-000061d79ebc/00000000-0000-0000-0000-00006289d1a9"
       (reference "#PWR0154") (unit 1) (value "GND") (footprint "")
@@
       (reference "#PWR0202") (unit 1) (value "+5V") (footprint "")
     )
-    (path "/00000000-0000-0000-0000-0000634ecc15/609e499a-8e19-4a2a-87f6-e6af7657800e"
-      (reference "#PWR?") (unit 1) (value "+3.3V") (footprint "")
-    )
-    (path "/00000000-0000-0000-0000-0000634ecc15/8604977b-2d6f-42be-81b7-a944e68d0b8b"
-      (reference "#PWR?") (unit 1) (value "+3.3V") (footprint "")
-    )
-    (path "/00000000-0000-0000-0000-000061df74a0/9481eb72-b44f-4908-8d19-cced640e09b3"
-      (reference "#PWR?") (unit 1) (value "GND") (footprint "")
-    )
     (path "/00000000-0000-0000-0000-000061d9c8dc/00000000-0000-0000-0000-000062b32a4c"
       (reference "C102") (unit 1) (value "0.22uF") (footprint "Capacitor_SMD:C_0805_2012Metric")
@@
     )
     (path "/00000000-0000-0000-0000-0000634ecc15/30ec9d1e-2a98-4009-b845-2064a986995f"
-      (reference "C800") (unit 1) (value "10uF") (footprint "Capacitor_SMD:C_0805_2012Metric")
+      (reference "C800") (unit 1) (value "4.7uF") (footprint "Capacitor_SMD:C_0805_2012Metric")
     )
     (path "/00000000-0000-0000-0000-0000634ecc15/76906a90-dd2f-433d-9ed8-d6dbd9d32c95"
-      (reference "C801") (unit 1) (value "10uF") (footprint "Capacitor_SMD:C_0805_2012Metric")
+      (reference "C801") (unit 1) (value "4.7uF") (footprint "Capacitor_SMD:C_0805_2012Metric")
     )
     (path "/00000000-0000-0000-0000-0000634ecc15/f2151f95-5542-4651-959d-6fd31f1b4bee"
@@
       (reference "H2") (unit 1) (value "MountingHole") (footprint "MountingHole:MountingHole_3.2mm_M3_Pad")
     )
-    (path "/00000000-0000-0000-0000-000061d79ebc/00000000-0000-0000-0000-000062a4690d"
-      (reference "J201") (unit 1) (value "25/28") (footprint "Connector_PinHeader_2.54mm:PinHeader_1x03_P2.54mm_Vertical")
-    )
     (path "/00000000-0000-0000-0000-000061d79ebc/00000000-0000-0000-0000-000062dd28db"
       (reference "J202") (unit 1) (value "25/FPU") (footprint "Connector_PinHeader_2.54mm:PinHeader_1x03_P2.54mm_Vertical")
@@
       (reference "J600") (unit 1) (value "IDE DISABLE") (footprint "Connector_PinHeader_2.54mm:PinHeader_1x02_P2.54mm_Vertical")
     )
+    (path "/00000000-0000-0000-0000-0000634ecc15/48041955-8198-42aa-a14d-ce9b4e3a0712"
+      (reference "JT1") (unit 1) (value "MODE68K") (footprint "Connector_PinHeader_2.54mm:PinHeader_1x01_P2.54mm_Vertical")
+    )
+    (path "/00000000-0000-0000-0000-0000634ecc15/1537ebc2-e72e-42b4-96ec-efba3861d976"
+      (reference "JT2") (unit 1) (value "SMDIS") (footprint "Connector_PinHeader_2.54mm:PinHeader_1x01_P2.54mm_Vertical")
+    )
+    (path "/00000000-0000-0000-0000-0000634ecc15/5067e930-3dba-451e-b140-ca23f8021b8b"
+      (reference "JT3") (unit 1) (value "_Z3CONFIGED") (footprint "Connector_PinHeader_2.54mm:PinHeader_1x01_P2.54mm_Vertical")
+    )
+    (path "/00000000-0000-0000-0000-0000634ecc15/e98e8195-a7f3-4e9b-8a86-36f69e8f3306"
+      (reference "JT4") (unit 1) (value "_IDEACCESS") (footprint "Connector_PinHeader_2.54mm:PinHeader_1x01_P2.54mm_Vertical")
+    )
+    (path "/00000000-0000-0000-0000-0000634ecc15/8fbb9a3b-f5e2-41fc-9f64-e00ee746a6fc"
+      (reference "JT5") (unit 1) (value "_MEMZ3") (footprint "Connector_PinHeader_2.54mm:PinHeader_1x01_P2.54mm_Vertical")
+    )
+    (path "/00000000-0000-0000-0000-0000634ecc15/6ae21b3f-cea8-419f-beb7-82f679998203"
+      (reference "JT6") (unit 1) (value "_MEMZ2") (footprint "Connector_PinHeader_2.54mm:PinHeader_1x01_P2.54mm_Vertical")
+    )
     (path "/00000000-0000-0000-0000-000061d79ebc/00000000-0000-0000-0000-00006219f0d8"
       (reference "R100") (unit 1) (value "1K") (footprint "Resistor_SMD:R_0805_2012Metric")
@@
       (reference "R406") (unit 1) (value "1K") (footprint "Resistor_SMD:R_0805_2012Metric")
     )
+    (path "/00000000-0000-0000-0000-0000634ecc15/90bd6186-5f60-4ae5-b203-7bbff3c3c1b9"
+      (reference "R407") (unit 1) (value "1K") (footprint "Resistor_SMD:R_0805_2012Metric")
+    )
+    (path "/00000000-0000-0000-0000-0000634ecc15/69078552-a4bf-409b-a23e-b338d843736f"
+      (reference "R408") (unit 1) (value "1K") (footprint "Resistor_SMD:R_0805_2012Metric")
+    )
     (path "/00000000-0000-0000-0000-0000634ecc15/00000000-0000-0000-0000-000061f93d08"
       (reference "R501") (unit 1) (value "1K") (footprint "Resistor_SMD:R_0805_2012Metric")
     )
-    (path "/00000000-0000-0000-0000-0000634ecc15/00000000-0000-0000-0000-000061fa2cd0"
-      (reference "R502") (unit 1) (value "1K") (footprint "Resistor_SMD:R_0805_2012Metric")
-    )
     (path "/00000000-0000-0000-0000-0000634ecc15/91731142-a9d3-44a8-91a6-3290133282f0"
       (reference "R600") (unit 1) (value "2.7K") (footprint "Resistor_SMD:R_0805_2012Metric")
@@
       (reference "R601") (unit 1) (value "1K") (footprint "Resistor_SMD:R_0805_2012Metric")
     )
-    (path "/00000000-0000-0000-0000-000062089831/00000000-0000-0000-0000-000062581d0a"
-      (reference "R704") (unit 1) (value "47") (footprint "Resistor_SMD:R_0805_2012Metric")
-    )
     (path "/00000000-0000-0000-0000-000061df74a0/00000000-0000-0000-0000-000062551812"
       (reference "R706") (unit 1) (value "1K") (footprint "Resistor_SMD:R_0805_2012Metric")
     )
-    (path "/00000000-0000-0000-0000-0000634ecc15/69078552-a4bf-409b-a23e-b338d843736f"
-      (reference "R?") (unit 1) (value "1K") (footprint "Resistor_SMD:R_0805_2012Metric")
-    )
-    (path "/00000000-0000-0000-0000-0000634ecc15/90bd6186-5f60-4ae5-b203-7bbff3c3c1b9"
-      (reference "R?") (unit 1) (value "1K") (footprint "Resistor_SMD:R_0805_2012Metric")
-    )
     (path "/00000000-0000-0000-0000-000061d79ebc/00000000-0000-0000-0000-000062dfcaac"
       (reference "RN104") (unit 1) (value "1K") (footprint "Resistor_THT:R_Array_SIP9")
@@
       (reference "U300") (unit 3) (value "74HCT04") (footprint "Package_SO:SOIC-14_3.9x8.7mm_P1.27mm")
     )
-    (path "/00000000-0000-0000-0000-000061fbe594/a754946d-d9d1-4add-9c28-05c026e18446"
+    (path "/00000000-0000-0000-0000-000061df74a0/d74f4ee6-5adb-461b-a1a5-e4055c430c1e"
       (reference "U300") (unit 4) (value "74HCT04") (footprint "Package_SO:SOIC-14_3.9x8.7mm_P1.27mm")
     )
-    (path "/00000000-0000-0000-0000-000061fbe594/df70592e-8649-40b6-916d-9b96a20e646d"
+    (path "/00000000-0000-0000-0000-000061df74a0/34c6d825-453c-40c8-b0a5-4465fafff44d"
       (reference "U300") (unit 5) (value "74HCT04") (footprint "Package_SO:SOIC-14_3.9x8.7mm_P1.27mm")
     )
@@
       (reference "U707") (unit 2) (value "74HCT245") (footprint "Package_SO:SOIC-20W_7.5x12.8mm_P1.27mm")
     )
-    (path "/00000000-0000-0000-0000-0000634ecc15/1e5e16f9-5aa2-4346-a822-d95e3d0e48d2"
-      (reference "U800") (unit 1) (value "LM1117-3.3") (footprint "Package_TO_SOT_SMD:SOT-223")
+    (path "/00000000-0000-0000-0000-0000634ecc15/52e7a18e-88ef-4efc-a1e7-fbb103097843"
+      (reference "U800") (unit 1) (value "AP7361C-33ER") (footprint "Package_TO_SOT_SMD:SOT-223-3_TabPin2")
     )
     (path "/00000000-0000-0000-0000-0000634ecc15/78e793bf-b02d-4adb-8811-ecc0735d5003"
