File: A2630-New-KiCAD-Rev21-PGA/Processor.kicad_sch (KiCad schematic)
At the start: 58 parts, among them J201 25/28, J202 25/FPU, U200 MC68030, U201 MC68882, U204 74AHCT04, X1 25MHz, X2 25MHz

Commit message: Add files via upload
Parts:
- removed J201: 25/28, Connector_PinHeader_2.54mm:PinHeader_1x03_P2.54mm_Vertical, symbol Jumper:Jumper_3_Open
Connections:
- net at R204.1: now also U204.1
Changed lines of the file:
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@@
   (title_block
     (title "Amiga N2630")
-    (date "2022-06-05")
+    (date "2022-07-21")
     (rev "2.1 QFP")
   )
@@
     (stroke (width 0) (type default) (color 0 0 0 0))
   )
-  (wire (pts (xy 56.515 182.88) (xy 56.515 177.8))
-    (stroke (width 0) (type default) (color 0 0 0 0))
-  )
   (bus (pts (xy 382.27 84.455) (xy 382.27 86.995))
     (stroke (width 0) (type default) (color 0 0 0 0))
@@
     (stroke (width 0) (type default) (color 0 0 0 0))
   )
-  (wire (pts (xy 56.515 195.58) (xy 56.515 200.025))
-    (stroke (width 0) (type default) (color 0 0 0 0))
-  )
   (wire (pts (xy 374.015 122.555) (xy 379.73 122.555))
     (stroke (width 0) (type default) (color 0 0 0 0))
@@
     (stroke (width 0) (type default) (color 0 0 0 0))
   )
-  (wire (pts (xy 56.515 177.8) (xy 59.69 177.8))
-    (stroke (width 0) (type default) (color 0 0 0 0))
-  )
   (wire (pts (xy 41.275 234.315) (xy 41.275 229.87))
     (stroke (width 0) (type default) (color 0 0 0 0))
@@
     (stroke (width 0) (type default) (color 0 0 0 0))
   )
-  (wire (pts (xy 65.405 189.23) (xy 60.325 189.23))
+  (wire (pts (xy 65.405 189.23) (xy 59.69 189.23))
     (stroke (width 0) (type default) (color 0 0 0 0))
   )
@@
     (stroke (width 0) (type default) (color 0 0 0 0))
   )
-  (wire (pts (xy 56.515 200.025) (xy 24.765 200.025))
-    (stroke (width 0) (type default) (color 0 0 0 0))
-  )
   (wire (pts (xy 259.715 134.62) (xy 263.525 134.62))
     (stroke (width 0) (type default) (color 0 0 0 0))
@@
     (stroke (width 0) (type default) (color 0 0 0 0))
   )
-  (wire (pts (xy 59.69 177.8) (xy 59.69 170.18))
+  (wire (pts (xy 59.69 189.23) (xy 59.69 170.18))
     (stroke (width 0) (type default) (color 0 0 0 0))
   )
@@
     )
   )
-  (global_label "28M" (shape input) (at 24.765 200.025 180) (fields_autoplaced)
-    (effects (font (size 1.27 1.27)) (justify right))
-    (property "Intersheet References" "${INTERSHEET_REFS}" (id 0) (at 0 0 0)
-      (effects (font (size 1.27 1.27)) hide)
-    )
-  )
   (global_label "_AVEC" (shape input) (at 29.21 31.75 180) (fields_autoplaced)
     (effects (font (size 1.27 1.27)) (justify right))
@@
     (pin "1")
   )
-  (symbol (lib_id "Jumper:Jumper_3_Open") (at 56.515 189.23 90) (unit 1)
-    (in_bom yes) (on_board yes)
-    (property "Reference" "J201" (id 0) (at 54.3052 188.0616 90)
-      (effects (font (size 1.27 1.27)) (justify left))
-    )
-    (property "Value" "25/28" (id 1) (at 54.3052 190.373 90)
-      (effects (font (size 1.27 1.27)) (justify left))
-    )
-    (property "Footprint" "Connector_PinHeader_2.54mm:PinHeader_1x03_P2.54mm_Vertical" (id 2) (at 56.515 189.23 0)
-      (effects (font (size 1.27 1.27)) hide)
-    )
-    (property "Datasheet" "~" (id 3) (at 56.515 189.23 0)
-      (effects (font (size 1.27 1.27)) hide)
-    )
-    (pin "1")
-    (pin "2")
-    (pin "3")
-  )
   (symbol (lib_id "N2630:CXO_DIP8") (at 43.815 241.935 0) (unit 1)
