File: A2630-New-KiCAD-Rev21-PGA/CPLD1.kicad_sch (KiCad schematic)
At the start: 19 parts, among them CN600 CPLD0, CN601 CPLD1, CN602 CPLD2, J600 IDE DISABLE, U600 XC9572XL-VQ64, U601 XC95144XL-TQ144, U602 XC95144XL-TQ144

Commit message: Add files via upload
Connections:
- net 68KMODE is gone; now on net MODE68K: U600.61 (P61)
Changed lines of the file:
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@@
     )
   )
-  (global_label "68KMODE" (shape input) (at 37.465 155.575 180) (fields_autoplaced)
+  (global_label "MODE68K" (shape input) (at 37.465 155.575 180) (fields_autoplaced)
     (effects (font (size 1.27 1.27)) (justify right))
     (property "Intersheet References" "${INTERSHEET_REFS}" (id 0) (at 26.2508 155.4956 0)

Commit message: Add files via upload
Connections:
- net CONFIGED: no longer U600.8 (P8)
- net _BOSS: now also U601.26 (P26)
- net 7M: now reaches U600.42 (P42)
- net AADIR: now reaches U601.39 (P39)
- net _AAENA: now reaches U601.40 (P40)
- net _IDEACCESS: now reaches U601.5 (I/O/GTS1)
- net _IDEACCESS: now also U602.6 (I/O/GTS2)
- net _MEMZ3: now reaches U601.57 (P57)
- net _MEMZ3: now also U602.10 (P10)
- net _EMENA: now reaches U601.68 (P68)
- net EXTSEL renamed SMDIS
- net SMDIS: no longer U602.10 (P10)
- net MEMACCESS renamed _MEMZ2
- net Z3CONFIGED renamed _Z3CONFIGED
- no-connect marks 35 -> 28

Commit message: Add files via upload
Parts:
- removed R704: 47, Resistor_SMD:R_0805_2012Metric, symbol Device:R
Connections:
- net IPLCLK: now also U600.8 (P8)
- net J403: now also U600.5 (I/O/GTS1); no longer U600.4 (P4)
- net J404: now also U600.4 (P4); no longer U600.2 (I/O/GTS2)
- net REF: now also U601.25 (P25); no longer U601.24 (P24)
- net REFACKZ2: now also U601.26 (P26); no longer U601.25 (P25)
- net SMDIS: now also U601.23 (P23); no longer U601.22 (P22)
- net _BERR: now also U601.24 (P24); no longer U601.23 (P23)
- net _BG: now also U600.7 (P7); no longer U600.6 (P6)
- net _BGACK: now also U601.22 (P22); no longer U601.21 (P21)
- net _BOSS: now also U601.21 (P21); no longer U601.26 (P26)
- net _DS: now also U600.2 (I/O/GTS2)
- net _GRESET: now also U601.66 (P66)
- net _IDEACCESS: now also U602.32 (I/O/GCK2); no longer U602.6 (I/O/GTS2)
- net _MEMZ3: now also U601.58 (P58); no longer U601.57 (P57)
- net _OVR: now also U602.6 (I/O/GTS2)
- net _STERM: now also U600.6 (P6); no longer U600.5 (I/O/GTS1)
- net _ONBOARD: no longer names the net of U600.40 (P40)
- net _ONBOARD: no longer U601.28 (P28)
- no-connect marks 28 -> 27

Commit message: Add files via upload
Connections:
- net J404: now also U601.27 (P27)
- no-connect marks 27 -> 26
Changed lines of the file:
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@@
   (title_block
     (title "Amiga N2630")
-    (date "2022-07-21")
-    (rev "2.1 QFP")
+    (date "2022-07-22")
+    (rev "2.1")
   )
   (junction (at 93.98 234.315) (diameter 0) (color 0 0 0 0)
@@
   (no_connect (at 160.655 115.57))
   (no_connect (at 160.655 97.79))
-  (no_connect (at 160.655 90.17))
   (no_connect (at 300.355 175.895))
   (no_connect (at 366.395 94.615))
@@
     (stroke (width 0) (type default) (color 0 0 0 0))
   )
+  (wire (pts (xy 151.892 90.17) (xy 160.655 90.17))
+    (stroke (width 0) (type default) (color 0 0 0 0))
+  )
   (bus (pts (xy 254 186.69) (xy 254 189.23))
     (stroke (width 0) (type default) (color 0 0 0 0))
@@
     )
   )
-  (global_label "_RESET" (shape output) (at 103.505 97.155 0) (fields_autoplaced)
+  (global_label "_RESET" (shape bidirectional) (at 103.505 97.155 0) (fields_autoplaced)
     (effects (font (size 1.27 1.27)) (justify left))
-    (property "Intersheet References" "${INTERSHEET_REFS}" (id 0) (at -6.985 -76.2 0)
-      (effects (font (size 1.27 1.27)) hide)
+    (property "Intersheet References" "${INTERSHEET_REFS}" (id 0) (at 112.5421 97.0756 0)
+      (effects (font (size 1.27 1.27)) (justify left) hide)
     )
   )
@@
     )
   )
+  (global_label "J404" (shape input) (at 151.892 90.17 180) (fields_autoplaced)
+    (effects (font (size 1.27 1.27)) (justify right))
+    (property "Intersheet References" "${INTERSHEET_REFS}" (id 0) (at 144.9716 90.0906 0)
+      (effects (font (size 1.27 1.27)) (justify right) hide)
+    )
+  )

Commit message: Add files via upload
Connections:
- net REFACKZ2 renamed _REFACKZ2
- net REFACKZ3 renamed _REFACKZ3
Changed lines of the file:
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@@
     )
   )
-  (global_label "REFACKZ3" (shape output) (at 275.59 92.71 180) (fields_autoplaced)
-    (effects (font (size 1.27 1.27)) (justify right))
-    (property "Intersheet References" "${INTERSHEET_REFS}" (id 0) (at 263.7106 92.6306 0)
+  (global_label "_REFACKZ3" (shape output) (at 275.59 92.71 180) (fields_autoplaced)
+    (effects (font (size 1.27 1.27)) (justify right))
+    (property "Intersheet References" "${INTERSHEET_REFS}" (id 0) (at 262.7429 92.6306 0)
       (effects (font (size 1.27 1.27)) (justify right) hide)
     )
@@
     )
   )
-  (global_label "REFACKZ2" (shape input) (at 103.505 135.255 0) (fields_autoplaced)
-    (effects (font (size 1.27 1.27)) (justify left))
-    (property "Intersheet References" "${INTERSHEET_REFS}" (id 0) (at 115.3844 135.3344 0)
+  (global_label "_REFACKZ2" (shape input) (at 103.505 135.255 0) (fields_autoplaced)
+    (effects (font (size 1.27 1.27)) (justify left))
+    (property "Intersheet References" "${INTERSHEET_REFS}" (id 0) (at 116.3521 135.1756 0)
       (effects (font (size 1.27 1.27)) (justify left) hide)
     )
@@
     )
   )
-  (global_label "REFACKZ2" (shape output) (at 151.765 87.63 180) (fields_autoplaced)
-    (effects (font (size 1.27 1.27)) (justify right))
-    (property "Intersheet References" "${INTERSHEET_REFS}" (id 0) (at 139.8856 87.5506 0)
+  (global_label "_REFACKZ2" (shape output) (at 151.765 87.63 180) (fields_autoplaced)
+    (effects (font (size 1.27 1.27)) (justify right))
+    (property "Intersheet References" "${INTERSHEET_REFS}" (id 0) (at 138.9179 87.5506 0)
       (effects (font (size 1.27 1.27)) (justify right) hide)
     )
@@
     )
   )
-  (global_label "REFACKZ3" (shape input) (at 103.505 147.955 0) (fields_autoplaced)
-    (effects (font (size 1.27 1.27)) (justify left))
-    (property "Intersheet References" "${INTERSHEET_REFS}" (id 0) (at 115.3844 148.0344 0)
-      (effects (font (size 1.27 1.27)) (justify left) hide)
-    )
+  (global_label "_REFACKZ3" (shape input) (at 103.505 147.955 0) (fields_autoplaced)
+    (effects (font (size 1.27 1.27)) (justify left))
+    (property "Intersheet References" "${INTERSHEET_REFS}" (id 0) (at 116.3521 147.8756 0)
+      (effects (font (size 1.27 1.27)) (justify left) hide)
+    )

Commit message: Add files via upload
Connections:
- net _REFACKZ2 renamed REFACKZ2
- net _REFACKZ3 renamed REFACKZ3
- net _Z3CONFIGED renamed Z3CONFIGED
Changed lines of the file:
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@@
     )
   )
-  (global_label "_REFACKZ3" (shape output) (at 275.59 92.71 180) (fields_autoplaced)
-    (effects (font (size 1.27 1.27)) (justify right))
-    (property "Intersheet References" "${INTERSHEET_REFS}" (id 0) (at 262.7429 92.6306 0)
+  (global_label "REFACKZ3" (shape output) (at 275.59 92.71 180) (fields_autoplaced)
+    (effects (font (size 1.27 1.27)) (justify right))
+    (property "Intersheet References" "${INTERSHEET_REFS}" (id 0) (at 263.7106 92.6306 0)
       (effects (font (size 1.27 1.27)) (justify right) hide)
     )
@@
     )
   )
-  (global_label "_REFACKZ2" (shape input) (at 103.505 135.255 0) (fields_autoplaced)
-    (effects (font (size 1.27 1.27)) (justify left))
-    (property "Intersheet References" "${INTERSHEET_REFS}" (id 0) (at 116.3521 135.1756 0)
+  (global_label "REFACKZ2" (shape input) (at 103.505 135.255 0) (fields_autoplaced)
+    (effects (font (size 1.27 1.27)) (justify left))
+    (property "Intersheet References" "${INTERSHEET_REFS}" (id 0) (at 115.3844 135.1756 0)
       (effects (font (size 1.27 1.27)) (justify left) hide)
     )
@@
     )
   )
-  (global_label "_REFACKZ2" (shape output) (at 151.765 87.63 180) (fields_autoplaced)
-    (effects (font (size 1.27 1.27)) (justify right))
-    (property "Intersheet References" "${INTERSHEET_REFS}" (id 0) (at 138.9179 87.5506 0)
+  (global_label "REFACKZ2" (shape output) (at 151.765 87.63 180) (fields_autoplaced)
+    (effects (font (size 1.27 1.27)) (justify right))
+    (property "Intersheet References" "${INTERSHEET_REFS}" (id 0) (at 139.8856 87.5506 0)
       (effects (font (size 1.27 1.27)) (justify right) hide)
     )
@@
     )
   )
-  (global_label "_Z3CONFIGED" (shape input) (at 240.03 138.43 0) (fields_autoplaced)
-    (effects (font (size 1.27 1.27)) (justify left))
-    (property "Intersheet References" "${INTERSHEET_REFS}" (id 0) (at 255.0542 138.3506 0)
+  (global_label "Z3CONFIGED" (shape input) (at 240.03 138.43 0) (fields_autoplaced)
+    (effects (font (size 1.27 1.27)) (justify left))
+    (property "Intersheet References" "${INTERSHEET_REFS}" (id 0) (at 254.0866 138.3506 0)
       (effects (font (size 1.27 1.27)) (justify left) hide)
     )
@@
     )
   )
-  (global_label "_REFACKZ3" (shape input) (at 103.505 147.955 0) (fields_autoplaced)
-    (effects (font (size 1.27 1.27)) (justify left))
-    (property "Intersheet References" "${INTERSHEET_REFS}" (id 0) (at 116.3521 147.8756 0)
+  (global_label "REFACKZ3" (shape input) (at 103.505 147.955 0) (fields_autoplaced)
+    (effects (font (size 1.27 1.27)) (justify left))
+    (property "Intersheet References" "${INTERSHEET_REFS}" (id 0) (at 115.3844 147.8756 0)
       (effects (font (size 1.27 1.27)) (justify left) hide)
     )
@@
     )
   )
-  (global_label "_Z3CONFIGED" (shape output) (at 375.158 130.175 0) (fields_autoplaced)
-    (effects (font (size 1.27 1.27)) (justify left))
-    (property "Intersheet References" "${INTERSHEET_REFS}" (id 0) (at 390.1822 130.0956 0)
-      (effects (font (size 1.27 1.27)) (justify left) hide)
-    )
+  (global_label "Z3CONFIGED" (shape output) (at 375.158 130.175 0) (fields_autoplaced)
+    (effects (font (size 1.27 1.27)) (justify left))
+    (property "Intersheet References" "${INTERSHEET_REFS}" (id 0) (at 389.2146 130.0956 0)
+      (effects (font (size 1.27 1.27)) (justify left) hide)
+    )
