File: A2630-New-KiCAD-Rev23-PGA/BaseMemory.kicad_sch (KiCad schematic)
At the start: 46 parts, among them U204 74AHCT04, U300 74HCT04, U400 SDRAM(4Mx16), U401 SDRAM(4Mx16), U606 74HCT244, U902 74HCT125

Commit message: Add files via upload
Parts:
- removed U204: 74AHCT04, Package_SO:SOIC-14_3.9x8.7mm_P1.27mm, symbol 74xx:74HCT04
- removed unit 1 of U300
- C427, C428, C429, C430, C431, C432: value 0.33uF -> 0.1uF
Changed lines of the file:
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@@
   (junction (at 360.045 102.235) (diameter 0) (color 0 0 0 0)
   )
-  (junction (at 337.82 98.425) (diameter 0) (color 0 0 0 0)
-  )
   (junction (at 207.264 43.688) (diameter 0) (color 0 0 0 0)
-  )
-  (junction (at 337.82 57.15) (diameter 0) (color 0 0 0 0)
   )
   (junction (at 123.952 138.557) (diameter 0) (color 0 0 0 0)
@@
     (stroke (width 0) (type default) (color 0 0 0 0))
   )
-  (wire (pts (xy 337.82 43.815) (xy 337.82 57.15))
-    (stroke (width 0) (type default) (color 0 0 0 0))
-  )
   (wire (pts (xy 96.012 202.057) (xy 96.012 223.647))
     (stroke (width 0) (type default) (color 0 0 0 0))
@@
     (stroke (width 0) (type default) (color 0 0 0 0))
   )
-  (wire (pts (xy 337.82 57.15) (xy 337.82 98.425))
+  (wire (pts (xy 337.82 43.815) (xy 337.82 108.585))
     (stroke (width 0) (type default) (color 0 0 0 0))
   )
@@
   )
   (bus (pts (xy 156.337 62.992) (xy 156.337 60.452))
-    (stroke (width 0) (type default) (color 0 0 0 0))
-  )
-  (wire (pts (xy 337.82 98.425) (xy 337.82 108.585))
     (stroke (width 0) (type default) (color 0 0 0 0))
   )
@@
       (effects (font (size 1.27 1.27)) (justify left))
     )
-    (property "Value" "0.33uF" (id 1) (at 179.832 249.428 90)
+    (property "Value" "0.1uF" (id 1) (at 179.832 249.428 90)
       (effects (font (size 1.27 1.27)) (justify left))
     )
@@
     (pin "1")
     (pin "2")
-  )
-  (symbol (lib_id "74xx:74LS05") (at 345.44 57.15 0) (unit 1)
-    (in_bom yes) (on_board yes)
-    (property "Reference" "U300" (id 0) (at 345.44 49.53 0))
-    (property "Value" "74HCT04" (id 1) (at 345.44 52.07 0))
-    (property "Footprint" "Package_SO:SOIC-14_3.9x8.7mm_P1.27mm" (id 2) (at 345.44 57.15 0)
-      (effects (font (size 1.27 1.27)) hide)
-    )
-    (property "Datasheet" "http://www.ti.com/lit/gpn/sn74LS05" (id 3) (at 345.44 57.15 0)
-      (effects (font (size 1.27 1.27)) hide)
-    )
-    (pin "1")
-    (pin "2")
-    (pin "3")
-    (pin "4")
-    (pin "5")
-    (pin "6")
-    (pin "8")
-    (pin "9")
-    (pin "10")
-    (pin "11")
-    (pin "12")
-    (pin "13")
-    (pin "14")
-    (pin "7")
   )
   (symbol (lib_id "74xx:74LS125") (at 367.665 102.235 0) (unit 4)
@@
       (effects (font (size 1.27 1.27)) (justify left))
     )
-    (property "Value" "0.33uF" (id 1) (at 209.677 249.428 90)
+    (property "Value" "0.1uF" (id 1) (at 209.677 249.428 90)
       (effects (font (size 1.27 1.27)) (justify left))
     )
@@
       (effects (font (size 1.27 1.27)) (justify left))
     )
-    (property "Value" "0.33uF" (id 1) (at 172.847 249.428 90)
+    (property "Value" "0.1uF" (id 1) (at 172.847 249.428 90)
       (effects (font (size 1.27 1.27)) (justify left))
     )
@@
     (pin "1")
   )
-  (symbol (lib_id "74xx:74HCT04") (at 345.44 98.425 0) (unit 3)
-    (in_bom yes) (on_board yes)
-    (property "Reference" "U204" (id 0) (at 345.44 90.3732 0))
-    (property "Value" "74AHCT04" (id 1) (at 345.44 92.6846 0))
-    (property "Footprint" "Package_SO:SOIC-14_3.9x8.7mm_P1.27mm" (id 2) (at 345.44 98.425 0)
-      (effects (font (size 1.27 1.27)) hide)
-    )
-    (property "Datasheet" "https://assets.nexperia.com/documents/data-sheet/74HC_HCT04.pdf" (id 3) (at 345.44 98.425 0)
-      (effects (font (size 1.27 1.27)) hide)
-    )
-    (property "Digikey" "296-31832-1-ND" (id 4) (at 345.44 98.425 0)
-      (effects (font (size 1.27 1.27)) hide)
-    )
-    (pin "1")
-    (pin "2")
-    (pin "3")
-    (pin "4")
-    (pin "5")
-    (pin "6")
-    (pin "8")
-    (pin "9")
-    (pin "10")
-    (pin "11")
-    (pin "12")
-    (pin "13")
-    (pin "14")
-    (pin "7")
-  )
   (symbol (lib_id "Device:R") (at 189.23 39.878 0) (unit 1)
     (in_bom yes) (on_board yes)
@@
       (effects (font (size 1.27 1.27)) (justify left))
     )
-    (property "Value" "0.33uF" (id 1) (at 186.817 249.428 90)
+    (property "Value" "0.1uF" (id 1) (at 186.817 249.428 90)
       (effects (font (size 1.27 1.27)) (justify left))
     )
@@
       (effects (font (size 1.27 1.27)) (justify left))
     )
-    (property "Value" "0.33uF" (id 1) (at 202.057 249.428 90)
+    (property "Value" "0.1uF" (id 1) (at 202.057 249.428 90)
       (effects (font (size 1.27 1.27)) (justify left))
     )
@@
       (effects (font (size 1.27 1.27)) (justify left))
     )
-    (property "Value" "0.33uF" (id 1) (at 194.437 249.428 90)
+    (property "Value" "0.1uF" (id 1) (at 194.437 249.428 90)
       (effects (font (size 1.27 1.27)) (justify left))
     )

Commit message: Add files via upload
Parts:
- added U204: 74AHCT04, Package_SO:SOIC-14_3.9x8.7mm_P1.27mm, symbol 74xx:74HCT04
Connections:
- net EMD2: now also R418.1; no longer R410.1
- net EMD3: now also R411.1; no longer R418.1
- net EMD4: now also R419.1; no longer R411.1
- net EMD5: now also R410.1; no longer R419.1
- net GND: now also U204.5; no longer U400.36 (A12), U401.36 (A12)
- new net ZMA12: U400.36 (A12), U401.36 (A12)
- no-connect marks 8 -> 7
Changed lines of the file:
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@@
   (title_block
     (title "Amiga N2630")
-    (date "2022-08-20")
-    (rev "2.2")
+    (date "2022-09-09")
+    (rev "2.3")
   )
   (junction (at 170.942 253.238) (diameter 0) (color 0 0 0 0)
@@
   (junction (at 243.078 43.688) (diameter 0) (color 0 0 0 0)
   )
+  (junction (at 337.82 63.246) (diameter 0) (color 0 0 0 0)
+  )
   (junction (at 170.942 231.013) (diameter 0) (color 0 0 0 0)
   )
@@
   (junction (at 217.424 43.688) (diameter 0) (color 0 0 0 0)
   )
+  (no_connect (at 353.06 63.246))
   (no_connect (at 375.285 102.235))
   (no_connect (at 375.285 43.815))
@@
   (no_connect (at 375.285 73.66))
   (no_connect (at 353.06 43.815))
-  (no_connect (at 353.06 98.425))
-  (no_connect (at 353.06 57.15))
+  (bus_entry (at 78.232 83.312) (size -2.54 -2.54)
+    (stroke (width 0) (type default) (color 0 0 0 0))
+  )
   (bus_entry (at 222.504 30.734) (size 2.54 -2.54)
     (stroke (width 0) (type default) (color 0 0 0 0))
@@
     (stroke (width 0) (type default) (color 0 0 0 0))
   )
+  (wire (pts (xy 91.5924 180.467) (xy 98.552 180.467))
+    (stroke (width 0) (type default) (color 0 0 0 0))
+  )
   (wire (pts (xy 78.232 65.532) (xy 98.552 65.532))
     (stroke (width 0) (type default) (color 0 0 0 0))
@@
     (stroke (width 0) (type default) (color 0 0 0 0))
   )
-  (wire (pts (xy 65.532 80.264) (xy 71.628 80.264))
-    (stroke (width 0) (type default) (color 0 0 0 0))
-  )
   (wire (pts (xy 360.045 108.585) (xy 337.82 108.585))
     (stroke (width 0) (type default) (color 0 0 0 0))
@@
     (stroke (width 0) (type default) (color 0 0 0 0))
   )
+  (wire (pts (xy 78.232 83.312) (xy 98.552 83.312))
+    (stroke (width 0) (type default) (color 0 0 0 0))
+  )
   (wire (pts (xy 91.5924 177.927) (xy 98.552 177.927))
     (stroke (width 0) (type default) (color 0 0 0 0))
@@
     (stroke (width 0) (type default) (color 0 0 0 0))
   )
-  (wire (pts (xy 98.552 83.312) (xy 71.628 83.312))
-    (stroke (width 0) (type default) (color 0 0 0 0))
-  )
   (bus (pts (xy 156.337 73.152) (xy 156.337 70.612))
     (stroke (width 0) (type default) (color 0 0 0 0))
@@
     (stroke (width 0) (type default) (color 0 0 0 0))
   )
-  (wire (pts (xy 337.82 43.815) (xy 337.82 108.585))
+  (wire (pts (xy 337.82 43.815) (xy 337.82 63.246))
     (stroke (width 0) (type default) (color 0 0 0 0))
   )
@@
     (stroke (width 0) (type default) (color 0 0 0 0))
   )
-  (wire (pts (xy 82.042 180.467) (xy 98.552 180.467))
-    (stroke (width 0) (type default) (color 0 0 0 0))
-  )
   (wire (pts (xy 207.264 30.734) (xy 207.264 36.068))
     (stroke (width 0) (type default) (color 0 0 0 0))
@@
     (stroke (width 0) (type default) (color 0 0 0 0))
   )
+  (bus (pts (xy 75.692 78.232) (xy 75.692 80.772))
+    (stroke (width 0) (type default) (color 0 0 0 0))
+  )
   (wire (pts (xy 177.927 231.013) (xy 170.942 231.013))
     (stroke (width 0) (type default) (color 0 0 0 0))
@@
     (stroke (width 0) (type default) (color 0 0 0 0))
   )
-  (wire (pts (xy 71.628 83.312) (xy 71.628 80.264))
-    (stroke (width 0) (type default) (color 0 0 0 0))
-  )
   (bus (pts (xy 156.337 147.447) (xy 156.337 88.392))
     (stroke (width 0) (type default) (color 0 0 0 0))
@@
   )
   (wire (pts (xy 113.792 138.557) (xy 113.792 143.637))
+    (stroke (width 0) (type default) (color 0 0 0 0))
+  )
+  (wire (pts (xy 337.82 63.246) (xy 337.82 108.585))
     (stroke (width 0) (type default) (color 0 0 0 0))
   )
@@
     (effects (font (size 1.27 1.27)) (justify right bottom))
   )
-  (label "EMD3" (at 186.69 30.734 270)
+  (label "EMD2" (at 186.69 30.734 270)
     (effects (font (size 1.27 1.27)) (justify right bottom))
   )
@@
     (effects (font (size 1.27 1.27)) (justify right bottom))
   )
+  (label "ZMA12" (at 91.5924 180.467 0)
+    (effects (font (size 1.27 1.27)) (justify left bottom))
+  )
   (label "EMD19" (at 153.797 57.912 180)
     (effects (font (size 1.27 1.27)) (justify right bottom))
@@
     (effects (font (size 1.27 1.27)) (justify right bottom))
   )
-  (label "EMD2" (at 166.116 30.734 270)
+  (label "EMD5" (at 166.116 30.734 270)
     (effects (font (size 1.27 1.27)) (justify right bottom))
   )
@@
     (effects (font (size 1.27 1.27)) (justify left bottom))
   )
-  (label "EMD5" (at 189.23 30.734 270)
+  (label "ZMA12" (at 88.392 83.312 0)
+    (effects (font (size 1.27 1.27)) (justify left bottom))
+  )
+  (label "EMD4" (at 189.23 30.734 270)
     (effects (font (size 1.27 1.27)) (justify right bottom))
   )
@@
     (effects (font (size 1.27 1.27)) (justify right bottom))
   )
-  (label "EMD4" (at 168.656 30.734 270)
+  (label "EMD3" (at 168.656 30.734 270)
     (effects (font (size 1.27 1.27)) (justify right bottom))
   )
@@
     )
   )
-  (global_label "ZMA[11..0]" (shape input) (at 37.084 28.702 180) (fields_autoplaced)
+  (global_label "ZMA[12..0]" (shape input) (at 37.084 28.702 180) (fields_autoplaced)
     (effects (font (size 1.27 1.27)) (justify right))
     (property "Intersheet References" "${INTERSHEET_REFS}" (id 0) (at 24.4788 28.6226 0)
@@
     (pin "2")
   )
-  (symbol (lib_id "power:GND") (at 82.042 180.467 0) (unit 1)
-    (in_bom yes) (on_board yes) (fields_autoplaced)
-    (property "Reference" "#PWR0160" (id 0) (at 82.042 186.817 0)
-      (effects (font (size 1.27 1.27)) hide)
-    )
-    (property "Value" "GND" (id 1) (at 82.042 184.9104 0))
-    (property "Footprint" "" (id 2) (at 82.042 180.467 0)
-      (effects (font (size 1.27 1.27)) hide)
-    )
-    (property "Datasheet" "" (id 3) (at 82.042 180.467 0)
-      (effects (font (size 1.27 1.27)) hide)
-    )
-    (pin "1")
-  )
-  (symbol (lib_id "74xx:74LS05") (at 345.44 43.815 0) (unit 6)
-    (in_bom yes) (on_board yes)
-    (property "Reference" "U300" (id 0) (at 345.44 36.195 0))
-    (property "Value" "74HCT04" (id 1) (at 345.44 38.735 0))
-    (property "Footprint" "Package_SO:SOIC-14_3.9x8.7mm_P1.27mm" (id 2) (at 345.44 43.815 0)
-      (effects (font (size 1.27 1.27)) hide)
-    )
-    (property "Datasheet" "http://www.ti.com/lit/gpn/sn74LS05" (id 3) (at 345.44 43.815 0)
+  (symbol (lib_id "74xx:74HCT04") (at 345.44 63.246 0) (unit 3)
+    (in_bom yes) (on_board yes)
+    (property "Reference" "U204" (id 0) (at 345.44 55.1942 0))
+    (property "Value" "74AHCT04" (id 1) (at 345.44 57.5056 0))
+    (property "Footprint" "Package_SO:SOIC-14_3.9x8.7mm_P1.27mm" (id 2) (at 345.44 63.246 0)
+      (effects (font (size 1.27 1.27)) hide)
+    )
+    (property "Datasheet" "https://assets.nexperia.com/documents/data-sheet/74HC_HCT04.pdf" (id 3) (at 345.44 63.246 0)
+      (effects (font (size 1.27 1.27)) hide)
+    )
+    (property "Digikey" "296-31832-1-ND" (id 4) (at 345.44 63.246 0)
       (effects (font (size 1.27 1.27)) hide)
     )
@@
     (pin "7")
   )
-  (symbol (lib_id "power:GND") (at 65.532 80.264 0) (unit 1)
-    (in_bom yes) (on_board yes) (fields_autoplaced)
-    (property "Reference" "#PWR0149" (id 0) (at 65.532 86.614 0)
-      (effects (font (size 1.27 1.27)) hide)
-    )
-    (property "Value" "GND" (id 1) (at 65.532 84.7074 0))
-    (property "Footprint" "" (id 2) (at 65.532 80.264 0)
-      (effects (font (size 1.27 1.27)) hide)
-    )
-    (property "Datasheet" "" (id 3) (at 65.532 80.264 0)
-      (effects (font (size 1.27 1.27)) hide)
-    )
-    (pin "1")
+  (symbol (lib_id "74xx:74LS05") (at 345.44 43.815 0) (unit 6)
+    (in_bom yes) (on_board yes)
+    (property "Reference" "U300" (id 0) (at 345.44 36.195 0))
+    (property "Value" "74HCT04" (id 1) (at 345.44 38.735 0))
+    (property "Footprint" "Package_SO:SOIC-14_3.9x8.7mm_P1.27mm" (id 2) (at 345.44 43.815 0)
+      (effects (font (size 1.27 1.27)) hide)
+    )
+    (property "Datasheet" "http://www.ti.com/lit/gpn/sn74LS05" (id 3) (at 345.44 43.815 0)
+      (effects (font (size 1.27 1.27)) hide)
+    )
+    (pin "1")
+    (pin "2")
+    (pin "3")
+    (pin "4")
+    (pin "5")
+    (pin "6")
+    (pin "8")
+    (pin "9")
+    (pin "10")
+    (pin "11")
+    (pin "12")
+    (pin "13")
+    (pin "14")
+    (pin "7")
   )
 )
