File: A2630-New-KiCAD-Rev23-PGA/Card Edge.kicad_sch (KiCad schematic)
At the start: 32 parts, among them CN700 Amiga-2000-CPU-Slot, J302 Jumper_NO_Small, J303 Jumper_NO_Small, J304 Jumper_NO_Small, J305 Z3 DISABLE, U300 74HCT04, U700 74HCT174, U701 74FCT646, U702 74FCT646, U703 74HCT245, U704 74HCT245, U705 74HCT245, U706 74HCT245, U707 74HCT245

Commit message: Add files via upload
Parts:
- C700, C701, C702, C703, C704, C705, C706, C707: value 0.22uF -> 0.1uF
Connections:
- net CDAC: now reaches CN700.15
Other:
- note added: "J302 - A2000 Shorted/B2000 Open J303 - Do not configure Z2 RAM Shorted/Autoconfigure Z2 RAM Open J304 - AMIX Shorted/AmigaOS Open J305 - Do not configure Z3 RAM Shorted/Autoconfigure Z3 RAM Open"
- note removed: "Not all these jumpers will make it to the final version. J301 - 2MEG Shorted/4MEG Open J302 - A2000 Shorted/B2000 Open J303 - Do not configure Z2 RAM Shorted/Autoconfigure Z2 RAM Open J304 - AMIX Shorted/AmigaOS Open J305 - Do not configure Z3 RAM Shorted/Autoconfigure Z3 RAM Open"
