File: A2630-New-KiCAD-Rev23-PGA/Processor.kicad_sch (KiCad schematic)
At the start: 57 parts, among them J202 25/FPU, U200 MC68030, U201 MC68882, U204 74AHCT04, X1 25MHz, X2 25MHz

Commit message: Add files via upload
Parts:
- added R206: 68, Resistor_SMD:R_0805_2012Metric, symbol Device:R
- added unit 3 of U204
- added unit 2 of U204
- C204: value 0.22uF -> 0.1uF
Connections:
- net at U204.11, U204.13, U204.2: now also U204.3
- new net: U204.4, U204.5
- new net: R206.1, U204.6
- new net _CPUCLK_A: R206.2
Changed lines of the file:
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@@
   (junction (at 41.275 253.365) (diameter 0) (color 0 0 0 0)
   )
+  (junction (at 80.645 189.2554) (diameter 0) (color 0 0 0 0)
+  )
   (junction (at 80.645 189.23) (diameter 0) (color 0 0 0 0)
   )
@@
     (stroke (width 0) (type default) (color 0 0 0 0))
   )
-  (wire (pts (xy 80.645 189.23) (xy 80.645 220.345))
+  (wire (pts (xy 80.645 189.23) (xy 80.645 189.2554))
     (stroke (width 0) (type default) (color 0 0 0 0))
   )
@@
     (stroke (width 0) (type default) (color 0 0 0 0))
   )
+  (wire (pts (xy 117.602 189.2554) (xy 111.125 189.2554))
+    (stroke (width 0) (type default) (color 0 0 0 0))
+  )
   (bus (pts (xy 168.275 167.64) (xy 168.275 170.18))
     (stroke (width 0) (type default) (color 0 0 0 0))
@@
     (stroke (width 0) (type default) (color 0 0 0 0))
   )
+  (wire (pts (xy 80.645 189.2554) (xy 80.645 220.345))
+    (stroke (width 0) (type default) (color 0 0 0 0))
+  )
   (wire (pts (xy 224.155 236.22) (xy 234.315 236.22))
     (stroke (width 0) (type default) (color 0 0 0 0))
@@
     (stroke (width 0) (type default) (color 0 0 0 0))
   )
+  (wire (pts (xy 117.602 206.502) (xy 117.602 189.2554))
+    (stroke (width 0) (type default) (color 0 0 0 0))
+  )
   (wire (pts (xy 263.525 170.18) (xy 259.715 170.18))
     (stroke (width 0) (type default) (color 0 0 0 0))
@@
     (stroke (width 0) (type default) (color 0 0 0 0))
   )
+  (wire (pts (xy 65.024 206.502) (xy 117.602 206.502))
+    (stroke (width 0) (type default) (color 0 0 0 0))
+  )
   (wire (pts (xy 276.225 114.3) (xy 289.56 114.3))
     (stroke (width 0) (type default) (color 0 0 0 0))
@@
     (stroke (width 0) (type default) (color 0 0 0 0))
   )
+  (wire (pts (xy 30.48 206.502) (xy 57.404 206.502))
+    (stroke (width 0) (type default) (color 0 0 0 0))
+  )
   (wire (pts (xy 247.015 96.52) (xy 263.525 96.52))
     (stroke (width 0) (type default) (color 0 0 0 0))
@@
     )
   )
+  (global_label "_CPUCLK_A" (shape output) (at 30.48 206.502 180) (fields_autoplaced)
+    (effects (font (size 1.27 1.27)) (justify right))
+    (property "Intersheet References" "${INTERSHEET_REFS}" (id 0) (at 17.6934 206.4226 0)
+      (effects (font (size 1.27 1.27)) (justify right) hide)
+    )
+  )
   (global_label "_BR" (shape input) (at 29.21 78.74 180) (fields_autoplaced)
     (effects (font (size 1.27 1.27)) (justify right))
@@
       (effects (font (size 1.27 1.27)) (justify left))
     )
-    (property "Value" "0.22uF" (id 1) (at 60.325 55.245 0)
+    (property "Value" "0.1uF" (id 1) (at 60.325 55.245 0)
       (effects (font (size 1.27 1.27)) (justify left))
     )
@@
   (symbol (lib_id "Device:R") (at 55.245 241.935 270) (unit 1)
     (in_bom yes) (on_board yes)
-    (property "Reference" "R203" (id 0) (at 55.245 236.6772 90))
-    (property "Value" "68" (id 1) (at 55.245 238.9886 90))
+    (property "Reference" "R203" (id 0) (at 55.372 239.776 90))
+    (property "Value" "68" (id 1) (at 55.372 242.062 90))
     (property "Footprint" "Resistor_SMD:R_0805_2012Metric" (id 2) (at 55.245 240.157 90)
       (effects (font (size 1.27 1.27)) hide)
@@
     (pin "2")
   )
+  (symbol (lib_id "74xx:74HCT04") (at 103.505 189.2554 0) (unit 3)
+    (in_bom yes) (on_board yes)
+    (property "Reference" "U204" (id 0) (at 103.505 181.2036 0))
+    (property "Value" "74AHCT04" (id 1) (at 103.505 183.515 0))
+    (property "Footprint" "Package_SO:SOIC-14_3.9x8.7mm_P1.27mm" (id 2) (at 103.505 189.2554 0)
+      (effects (font (size 1.27 1.27)) hide)
+    )
+    (property "Datasheet" "https://assets.nexperia.com/documents/data-sheet/74HC_HCT04.pdf" (id 3) (at 103.505 189.2554 0)
+      (effects (font (size 1.27 1.27)) hide)
+    )
+    (property "Digikey" "296-31832-1-ND" (id 4) (at 103.505 189.2554 0)
+      (effects (font (size 1.27 1.27)) hide)
+    )
+    (pin "1")
+    (pin "2")
+    (pin "3")
+    (pin "4")
+    (pin "5")
+    (pin "6")
+    (pin "8")
+    (pin "9")
+    (pin "10")
+    (pin "11")
+    (pin "12")
+    (pin "13")
+    (pin "14")
+    (pin "7")
+  )
   (symbol (lib_id "Device:R") (at 144.145 148.59 0) (unit 1)
     (in_bom yes) (on_board yes)
@@
     (pin "9")
   )
+  (symbol (lib_id "74xx:74LS04") (at 88.265 189.2554 0) (unit 2)
+    (in_bom yes) (on_board yes)
+    (property "Reference" "U204" (id 0) (at 88.265 197.3072 0))
+    (property "Value" "74AHCT04" (id 1) (at 88.265 194.9958 0))
+    (property "Footprint" "Package_SO:SOIC-14_3.9x8.7mm_P1.27mm" (id 2) (at 88.265 189.2554 0)
+      (effects (font (size 1.27 1.27)) hide)
+    )
+    (property "Datasheet" "http://www.ti.com/lit/gpn/sn74LS04" (id 3) (at 88.265 189.2554 0)
+      (effects (font (size 1.27 1.27)) hide)
+    )
+    (pin "1")
+    (pin "2")
+    (pin "3")
+    (pin "4")
+    (pin "5")
+    (pin "6")
+    (pin "8")
+    (pin "9")
+    (pin "10")
+    (pin "11")
+    (pin "12")
+    (pin "13")
+    (pin "14")
+    (pin "7")
+  )
+  (symbol (lib_id "Device:R") (at 61.214 206.502 270) (unit 1)
+    (in_bom yes) (on_board yes)
+    (property "Reference" "R206" (id 0) (at 61.214 204.597 90))
+    (property "Value" "68" (id 1) (at 61.214 206.502 90))
+    (property "Footprint" "Resistor_SMD:R_0805_2012Metric" (id 2) (at 61.214 204.724 90)
+      (effects (font (size 1.27 1.27)) hide)
+    )
+    (property "Datasheet" "~" (id 3) (at 61.214 206.502 0)
+      (effects (font (size 1.27 1.27)) hide)
+    )
+    (pin "1")
+    (pin "2")
+  )
   (symbol (lib_id "Device:R") (at 126.365 148.59 0) (unit 1)

Commit message: Add files via upload
Parts:
- removed unit 3 of U204
Connections:
- net at U204.4: now also R206.1
- net _CPUCLK_A renamed CPUCLK_B
Other:
- moved on the sheet: R206
Changed lines of the file:
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@@
   (title_block
     (title "Amiga N2630")
-    (date "2022-08-20")
-    (rev "2.2")
+    (date "2022-09-09")
+    (rev "2.3")
   )
   (junction (at 342.9 71.755) (diameter 0) (color 0 0 0 0)
@@
     (stroke (width 0) (type default) (color 0 0 0 0))
   )
-  (wire (pts (xy 117.602 189.2554) (xy 111.125 189.2554))
-    (stroke (width 0) (type default) (color 0 0 0 0))
-  )
   (bus (pts (xy 168.275 167.64) (xy 168.275 170.18))
     (stroke (width 0) (type default) (color 0 0 0 0))
@@
     (stroke (width 0) (type default) (color 0 0 0 0))
   )
+  (wire (pts (xy 117.602 189.2554) (xy 117.602 206.4766))
+    (stroke (width 0) (type default) (color 0 0 0 0))
+  )
   (bus (pts (xy 382.27 155.575) (xy 382.27 158.115))
     (stroke (width 0) (type default) (color 0 0 0 0))
@@
     (stroke (width 0) (type default) (color 0 0 0 0))
   )
+  (wire (pts (xy 95.885 189.2554) (xy 117.602 189.2554))
+    (stroke (width 0) (type default) (color 0 0 0 0))
+  )
   (wire (pts (xy 139.065 144.78) (xy 139.065 127))
     (stroke (width 0) (type default) (color 0 0 0 0))
@@
     (stroke (width 0) (type default) (color 0 0 0 0))
   )
-  (wire (pts (xy 117.602 206.502) (xy 117.602 189.2554))
-    (stroke (width 0) (type default) (color 0 0 0 0))
-  )
   (wire (pts (xy 263.525 170.18) (xy 259.715 170.18))
     (stroke (width 0) (type default) (color 0 0 0 0))
@@
     (stroke (width 0) (type default) (color 0 0 0 0))
   )
-  (wire (pts (xy 65.024 206.502) (xy 117.602 206.502))
-    (stroke (width 0) (type default) (color 0 0 0 0))
-  )
   (wire (pts (xy 276.225 114.3) (xy 289.56 114.3))
     (stroke (width 0) (type default) (color 0 0 0 0))
@@
     (stroke (width 0) (type default) (color 0 0 0 0))
   )
+  (wire (pts (xy 66.04 206.4766) (xy 117.602 206.4766))
+    (stroke (width 0) (type default) (color 0 0 0 0))
+  )
   (wire (pts (xy 259.715 134.62) (xy 263.525 134.62))
     (stroke (width 0) (type default) (color 0 0 0 0))
@@
     (stroke (width 0) (type default) (color 0 0 0 0))
   )
-  (wire (pts (xy 30.48 206.502) (xy 57.404 206.502))
+  (wire (pts (xy 29.21 206.756) (xy 58.42 206.4766))
     (stroke (width 0) (type default) (color 0 0 0 0))
   )
@@
     )
   )
-  (global_label "_CPUCLK_A" (shape output) (at 30.48 206.502 180) (fields_autoplaced)
+  (global_label "CPUCLK_B" (shape output) (at 29.21 206.756 180) (fields_autoplaced)
     (effects (font (size 1.27 1.27)) (justify right))
-    (property "Intersheet References" "${INTERSHEET_REFS}" (id 0) (at 17.6934 206.4226 0)
+    (property "Intersheet References" "${INTERSHEET_REFS}" (id 0) (at 17.2096 206.6766 0)
       (effects (font (size 1.27 1.27)) (justify right) hide)
     )
@@
     (pin "2")
   )
-  (symbol (lib_id "74xx:74HCT04") (at 103.505 189.2554 0) (unit 3)
-    (in_bom yes) (on_board yes)
-    (property "Reference" "U204" (id 0) (at 103.505 181.2036 0))
-    (property "Value" "74AHCT04" (id 1) (at 103.505 183.515 0))
-    (property "Footprint" "Package_SO:SOIC-14_3.9x8.7mm_P1.27mm" (id 2) (at 103.505 189.2554 0)
-      (effects (font (size 1.27 1.27)) hide)
-    )
-    (property "Datasheet" "https://assets.nexperia.com/documents/data-sheet/74HC_HCT04.pdf" (id 3) (at 103.505 189.2554 0)
-      (effects (font (size 1.27 1.27)) hide)
-    )
-    (property "Digikey" "296-31832-1-ND" (id 4) (at 103.505 189.2554 0)
-      (effects (font (size 1.27 1.27)) hide)
-    )
-    (pin "1")
-    (pin "2")
-    (pin "3")
-    (pin "4")
-    (pin "5")
-    (pin "6")
-    (pin "8")
-    (pin "9")
-    (pin "10")
-    (pin "11")
-    (pin "12")
-    (pin "13")
-    (pin "14")
-    (pin "7")
-  )
   (symbol (lib_id "Device:R") (at 144.145 148.59 0) (unit 1)
     (in_bom yes) (on_board yes)
@@
     (pin "7")
   )
-  (symbol (lib_id "Device:R") (at 61.214 206.502 270) (unit 1)
+  (symbol (lib_id "Device:R") (at 62.23 206.4766 270) (unit 1)
     (in_bom yes) (on_board yes)
-    (property "Reference" "R206" (id 0) (at 61.214 204.597 90))
-    (property "Value" "68" (id 1) (at 61.214 206.502 90))
-    (property "Footprint" "Resistor_SMD:R_0805_2012Metric" (id 2) (at 61.214 204.724 90)
+    (property "Reference" "R206" (id 0) (at 62.23 204.5716 90))
+    (property "Value" "68" (id 1) (at 62.23 206.4766 90))
+    (property "Footprint" "Resistor_SMD:R_0805_2012Metric" (id 2) (at 62.23 204.6986 90)
       (effects (font (size 1.27 1.27)) hide)
     )
-    (property "Datasheet" "~" (id 3) (at 61.214 206.502 0)
+    (property "Datasheet" "~" (id 3) (at 62.23 206.4766 0)
       (effects (font (size 1.27 1.27)) hide)
     )
