File: A2630-New-KiCAD-Rev23-PGA/jumpers.kicad_sch (KiCad schematic)
At the start: 0 parts

Commit message: Add files via upload
Other:
- note added: "MOVE NOISE RES _AS, _DS, R_W CLOSER TO CONSUMING LOGIC."
Changed lines of the file:
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@@
     )
+  )
+  (text "MOVE NOISE RES _AS, _DS, R_W CLOSER \nTO CONSUMING LOGIC."
+    (at 117.602 174.244 0)
+    (effects (font (size 5 5)) (justify left bottom))
   )
   (text "JUMPER SETTINGS" (at 313.69 243.586 0)

Commit message: Add files via upload
Other:
- note added: "NOTE: J401 and J402 have no effect if J400 is open."
- note removed: "MOVE NOISE RES _AS, _DS, R_W CLOSER TO CONSUMING LOGIC."
