File: A2630-New-KiCAD-Rev30-PGA/BaseMemory.kicad_sch (KiCad schematic)
At the start: 26 parts, among them SW1 MODE, U204 74AHCT04, U300 74HCT04, U400 SDRAM(4Mx16), U401 SDRAM(4Mx16), U606 74HCT244, U902 74HCT125

Commit message: Add files via upload
Parts:
- removed U902: 74HCT125, Package_SO:SOIC-14_3.9x8.7mm_P1.27mm, symbol 74xx:74LS125
- added C200, C201, C202, C206, C208, C214, C215, C216, C218, C219, C220: 0.1uF, Capacitor_SMD:C_0805_2012Metric, symbol Device:C
- added C205: 330pF, Capacitor_SMD:C_0805_2012Metric, symbol Device:C
- added C209: 0.22uF, Capacitor_SMD:C_0805_2012Metric, symbol Device:C
- added C800, C801: 4.7uF, Capacitor_SMD:C_0805_2012Metric, symbol Device:C
- added C802, C804, C805: 10uF, Capacitor_THT:CP_Radial_D5.0mm_P2.00mm, symbol Device:CP
- added C803: 47uF, Capacitor_THT:CP_Radial_D5.0mm_P2.00mm, symbol Device:CP
- added U800: AP7361C-33ER, Package_TO_SOT_SMD:SOT-223-3_TabPin2, symbol Regulator_Linear:AP7361C-33E
Connections:
- net +3V3: now also C800.1, C802.1, C803.1, C804.1, C805.1, U800.2 (VO)
- net GND: now also C200.2, C201.2, C202.2, C205.2, C206.2, C208.2, C209.2, C214.2, C215.2, C216.2, C218.2, C219.2, C220.2, C800.2, C801.2, C802.2, C803.2, C804.2, C805.2, U800.1 (GND)
- new net +5V: C200.1, C201.1, C202.1, C205.1, C206.1, C208.1, C209.1, C214.1, C215.1, C216.1, C218.1, C219.1, C220.1, C801.1, U800.3 (VI)
- no-connect marks 7 -> 6
Other:
- note added: "+3.3V"
- note added: "CPU/FPU DECOUPLING"
- note added: "ZORRO 2 MEMORY, SPARES, POWER"
- note removed: "ZORRO 2 MEMORY SPARES"
- moved on the sheet: JT1, JT2, JT4, JT5, JT6

Commit message: Add files via upload
Parts:
- removed U204: 74AHCT04, Package_SO:SOIC-14_3.9x8.7mm_P1.27mm, symbol 74xx:74HCT04
- removed U300: 74HCT04, Package_SO:SOIC-14_3.9x8.7mm_P1.27mm, symbol 74xx:74LS05
- added U300: 74HCT05, Package_SO:SOIC-14_3.9x8.7mm_P1.27mm, symbol 74xx:74LS05
Connections:
- net GND: now also U300.11, U300.9
Changed lines of the file:
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@@
   (title_block
     (title "Amiga N2630")
-    (date "2022-12-01")
+    (date "2022-12-04")
     (rev "3.0")
   )
@@
   (junction (at 287.274 92.837) (diameter 0) (color 0 0 0 0)
   )
-  (junction (at 337.82 63.246) (diameter 0) (color 0 0 0 0)
-  )
   (junction (at 170.942 231.013) (diameter 0) (color 0 0 0 0)
   )
@@
   (junction (at 350.266 185.42) (diameter 0) (color 0 0 0 0)
   )
+  (junction (at 337.82 57.277) (diameter 0) (color 0 0 0 0)
+  )
   (junction (at 264.795 135.636) (diameter 0) (color 0 0 0 0)
   )
@@
   (junction (at 192.532 253.238) (diameter 0) (color 0 0 0 0)
   )
-  (no_connect (at 353.06 63.246))
+  (no_connect (at 353.06 57.277))
   (no_connect (at 375.285 43.815))
   (no_connect (at 375.285 87.63))
@@
     (stroke (width 0) (type default) (color 0 0 0 0))
   )
+  (wire (pts (xy 337.82 57.277) (xy 337.82 108.585))
+    (stroke (width 0) (type default) (color 0 0 0 0))
+  )
   (bus (pts (xy 156.337 177.927) (xy 156.337 175.387))
     (stroke (width 0) (type default) (color 0 0 0 0))
@@
     (stroke (width 0) (type default) (color 0 0 0 0))
   )
-  (wire (pts (xy 337.82 43.815) (xy 337.82 63.246))
-    (stroke (width 0) (type default) (color 0 0 0 0))
-  )
   (bus (pts (xy 156.337 180.467) (xy 156.337 177.927))
     (stroke (width 0) (type default) (color 0 0 0 0))
@@
     (stroke (width 0) (type default) (color 0 0 0 0))
   )
-  (wire (pts (xy 337.82 63.246) (xy 337.82 108.585))
-    (stroke (width 0) (type default) (color 0 0 0 0))
-  )
   (polyline (pts (xy 332.74 123.19) (xy 375.92 123.19))
     (stroke (width 0) (type default) (color 0 0 0 0))
@@
     (stroke (width 0) (type default) (color 0 0 0 0))
   )
+  (wire (pts (xy 337.82 43.815) (xy 337.82 57.277))
+    (stroke (width 0) (type default) (color 0 0 0 0))
+  )
   (bus (pts (xy 156.337 62.992) (xy 156.337 60.452))
     (stroke (width 0) (type default) (color 0 0 0 0))
@@
     (pin "9")
   )
+  (symbol (lib_id "74xx:74LS05") (at 345.44 57.277 0) (unit 5)
+    (in_bom yes) (on_board yes) (fields_autoplaced)
+    (property "Reference" "U300" (id 0) (at 345.44 49.7672 0))
+    (property "Value" "74HCT05" (id 1) (at 345.44 52.3041 0))
+    (property "Footprint" "Package_SO:SOIC-14_3.9x8.7mm_P1.27mm" (id 2) (at 345.44 57.277 0)
+      (effects (font (size 1.27 1.27)) hide)
+    )
+    (property "Datasheet" "http://www.ti.com/lit/gpn/sn74LS05" (id 3) (at 345.44 57.277 0)
+      (effects (font (size 1.27 1.27)) hide)
+    )
+    (pin "1")
+    (pin "2")
+    (pin "3")
+    (pin "4")
+    (pin "5")
+    (pin "6")
+    (pin "8")
+    (pin "9")
+    (pin "10")
+    (pin "11")
+    (pin "12")
+    (pin "13")
+    (pin "14")
+    (pin "7")
+  )
   (symbol (lib_id "Switch:SW_SPDT") (at 336.55 204.724 0) (unit 1)
     (in_bom yes) (on_board yes) (fields_autoplaced)
@@
     (pin "1")
   )
+  (symbol (lib_id "74xx:74LS05") (at 345.44 43.815 0) (unit 4)
+    (in_bom yes) (on_board yes) (fields_autoplaced)
+    (property "Reference" "U300" (id 0) (at 345.44 36.3052 0))
+    (property "Value" "74HCT05" (id 1) (at 345.44 38.8421 0))
+    (property "Footprint" "Package_SO:SOIC-14_3.9x8.7mm_P1.27mm" (id 2) (at 345.44 43.815 0)
+      (effects (font (size 1.27 1.27)) hide)
+    )
+    (property "Datasheet" "http://www.ti.com/lit/gpn/sn74LS05" (id 3) (at 345.44 43.815 0)
+      (effects (font (size 1.27 1.27)) hide)
+    )
+    (pin "1")
+    (pin "2")
+    (pin "3")
+    (pin "4")
+    (pin "5")
+    (pin "6")
+    (pin "8")
+    (pin "9")
+    (pin "10")
+    (pin "11")
+    (pin "12")
+    (pin "13")
+    (pin "14")
+    (pin "7")
+  )
   (symbol (lib_id "Device:C") (at 219.71 96.647 0) (unit 1)
     (in_bom yes) (on_board yes)
@@
     (pin "2")
   )
-  (symbol (lib_id "74xx:74HCT04") (at 345.44 63.246 0) (unit 3)
-    (in_bom yes) (on_board yes)
-    (property "Reference" "U204" (id 0) (at 345.44 55.1942 0))
-    (property "Value" "74AHCT04" (id 1) (at 345.44 57.5056 0))
-    (property "Footprint" "Package_SO:SOIC-14_3.9x8.7mm_P1.27mm" (id 2) (at 345.44 63.246 0)
-      (effects (font (size 1.27 1.27)) hide)
-    )
-    (property "Datasheet" "https://assets.nexperia.com/documents/data-sheet/74HC_HCT04.pdf" (id 3) (at 345.44 63.246 0)
-      (effects (font (size 1.27 1.27)) hide)
-    )
-    (property "Digikey" "296-31832-1-ND" (id 4) (at 345.44 63.246 0)
-      (effects (font (size 1.27 1.27)) hide)
-    )
-    (pin "1")
-    (pin "2")
-    (pin "3")
-    (pin "4")
-    (pin "5")
-    (pin "6")
-    (pin "8")
-    (pin "9")
-    (pin "10")
-    (pin "11")
-    (pin "12")
-    (pin "13")
-    (pin "14")
-    (pin "7")
-  )
-  (symbol (lib_id "74xx:74LS05") (at 345.44 43.815 0) (unit 6)
-    (in_bom yes) (on_board yes)
-    (property "Reference" "U300" (id 0) (at 345.44 36.195 0))
-    (property "Value" "74HCT04" (id 1) (at 345.44 38.735 0))
-    (property "Footprint" "Package_SO:SOIC-14_3.9x8.7mm_P1.27mm" (id 2) (at 345.44 43.815 0)
-      (effects (font (size 1.27 1.27)) hide)
-    )
-    (property "Datasheet" "http://www.ti.com/lit/gpn/sn74LS05" (id 3) (at 345.44 43.815 0)
-      (effects (font (size 1.27 1.27)) hide)
-    )
-    (pin "1")
-    (pin "2")
-    (pin "3")
-    (pin "4")
-    (pin "5")
-    (pin "6")
-    (pin "8")
-    (pin "9")
-    (pin "10")
-    (pin "11")
-    (pin "12")
-    (pin "13")
-    (pin "14")
-    (pin "7")
-  )
 )

Commit message: Exclude non-BOM items.
Parts:
- R600, R601, SW1: now left out of the parts list
Changed lines of the file:
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@@
   (title_block
     (title "Amiga N2630")
-    (date "2022-12-04")
+    (date "2023-01-23")
     (rev "3.0")
   )
@@
   )
   (symbol (lib_id "Device:R") (at 355.346 194.31 0) (unit 1)
-    (in_bom yes) (on_board yes)
+    (in_bom no) (on_board yes)
     (property "Reference" "R601" (id 0) (at 356.616 191.77 90)
       (effects (font (size 1.27 1.27)) (justify left))
@@
   )
   (symbol (lib_id "Switch:SW_SPDT") (at 336.55 204.724 0) (unit 1)
-    (in_bom yes) (on_board yes) (fields_autoplaced)
+    (in_bom no) (on_board yes) (fields_autoplaced)
     (property "Reference" "SW1" (id 0) (at 336.55 198.1032 0))
     (property "Value" "MODE" (id 1) (at 336.55 200.6401 0))
@@
   )
   (symbol (lib_id "Device:R") (at 350.266 194.31 0) (unit 1)
-    (in_bom yes) (on_board yes)
+    (in_bom no) (on_board yes)
     (property "Reference" "R600" (id 0) (at 351.536 191.77 90)
       (effects (font (size 1.27 1.27)) (justify left))
