File: A2630-New-KiCAD-Rev30-PGA/Card Edge.kicad_sch (KiCad schematic)
At the start: 32 parts, among them CN700 Amiga-2000-CPU-Slot, J302 Jumper_NO_Small, J304 Jumper_NO_Small, J403 Jumper_NO_Small, J405 Z3 DISABLE, U300 74HCT04, U700 74HCT174, U701 74FCT646, U702 74FCT646, U703 74HCT245, U704 74HCT245, U705 74HCT245, U706 74HCT245, U707 74HCT245

Commit message: Add files via upload
Parts:
- added C720: 10uF, Capacitor_THT:CP_Radial_D5.0mm_P2.00mm, symbol Device:CP1
Connections:
- net +5V: now also C720.1
- net GND: now also C720.2
Changed lines of the file:
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@@
   (title_block
     (title "Amiga N2630")
-    (date "2022-11-24")
+    (date "2022-11-26")
     (rev "3.0")
   )
@@
   (junction (at 365.76 99.695) (diameter 0) (color 0 0 0 0)
   )
+  (junction (at 275.082 243.84) (diameter 0) (color 0 0 0 0)
+  )
   (junction (at 109.22 238.76) (diameter 0) (color 0 0 0 0)
   )
@@
   (junction (at 342.9 224.155) (diameter 0) (color 0 0 0 0)
   )
+  (junction (at 286.385 224.155) (diameter 0) (color 0 0 0 0)
+  )
   (junction (at 341.63 95.25) (diameter 0) (color 0 0 0 0)
   )
@@
     (stroke (width 0) (type default) (color 0 0 0 0))
   )
+  (wire (pts (xy 286.385 229.87) (xy 286.385 224.155))
+    (stroke (width 0) (type default) (color 0 0 0 0))
+  )
   (wire (pts (xy 104.775 156.21) (xy 59.69 156.21))
     (stroke (width 0) (type default) (color 0 0 0 0))
@@
     (stroke (width 0) (type default) (color 0 0 0 0))
   )
+  (wire (pts (xy 286.385 243.84) (xy 286.385 237.49))
+    (stroke (width 0) (type default) (color 0 0 0 0))
+  )
   (bus (pts (xy 134.62 177.8) (xy 134.62 180.34))
     (stroke (width 0) (type default) (color 0 0 0 0))
@@
     (stroke (width 0) (type default) (color 0 0 0 0))
   )
-  (wire (pts (xy 285.115 224.155) (xy 298.45 224.155))
+  (wire (pts (xy 285.115 224.155) (xy 286.385 224.155))
     (stroke (width 0) (type default) (color 0 0 0 0))
   )
@@
     (stroke (width 0) (type default) (color 0 0 0 0))
   )
+  (wire (pts (xy 286.385 224.155) (xy 298.45 224.155))
+    (stroke (width 0) (type default) (color 0 0 0 0))
+  )
   (wire (pts (xy 215.9 194.31) (xy 227.965 194.31))
     (stroke (width 0) (type default) (color 0 0 0 0))
@@
     (stroke (width 0) (type default) (color 0 0 0 0))
   )
+  (wire (pts (xy 275.082 243.84) (xy 286.385 243.84))
+    (stroke (width 0) (type default) (color 0 0 0 0))
+  )
   (wire (pts (xy 227.965 198.755) (xy 227.965 194.31))
     (stroke (width 0) (type default) (color 0 0 0 0))
@@
     (pin "7")
   )
+  (symbol (lib_id "Device:CP1") (at 286.385 233.68 180) (unit 1)
+    (in_bom yes) (on_board yes)
+    (property "Reference" "C720" (id 0) (at 289.306 232.5116 0)
+      (effects (font (size 1.27 1.27)) (justify right))
+    )
+    (property "Value" "10uF" (id 1) (at 289.306 234.823 0)
+      (effects (font (size 1.27 1.27)) (justify right))
+    )
+    (property "Footprint" "Capacitor_THT:CP_Radial_D5.0mm_P2.00mm" (id 2) (at 286.385 233.68 0)
+      (effects (font (size 1.27 1.27)) hide)
+    )
+    (property "Datasheet" "~" (id 3) (at 286.385 233.68 0)
+      (effects (font (size 1.27 1.27)) hide)
+    )
+    (pin "1")
+    (pin "2")
+  )
   (symbol (lib_id "74xx:74LS05") (at 44.831 139.7 0) (unit 3)

Commit message: Add files via upload
Parts:
- removed unit 5 of U300
- removed unit 4 of U300
- added R303: 1K, Resistor_SMD:R_0805_2012Metric, symbol Device:R
- added U204: 74AHCT04, Package_SO:SOIC-14_3.9x8.7mm_P1.27mm, symbol 74xx:74HCT04
- added unit 6 of U300
- U300: value 74HCT04 -> 74HCT05
- renumbered R303 to R304, R304 to R305, R305 to R306
Connections:
- net +5V: now also R303.1
- net _ABERR: now also U204.5
- net _BERR: now also U300.12
- net _COPCFG: now also R303.2
- new net: U204.6, U300.13
Changed lines of the file:
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@@
   (title_block
     (title "Amiga N2630")
-    (date "2022-12-01")
+    (date "2022-12-04")
     (rev "3.0")
   )
@@
   (junction (at 365.76 99.695) (diameter 0) (color 0 0 0 0)
   )
+  (junction (at 68.072 113.665) (diameter 0) (color 0 0 0 0)
+  )
   (junction (at 275.082 243.84) (diameter 0) (color 0 0 0 0)
   )
@@
   (junction (at 109.22 208.28) (diameter 0) (color 0 0 0 0)
   )
+  (junction (at 68.199 113.538) (diameter 0) (color 0 0 0 0)
+  )
   (junction (at 363.22 95.25) (diameter 0) (color 0 0 0 0)
   )
   (junction (at 149.86 201.93) (diameter 0) (color 0 0 0 0)
   )
+  (junction (at 68.072 113.538) (diameter 0) (color 0 0 0 0)
+  )
   (junction (at 237.49 194.31) (diameter 0) (color 0 0 0 0)
   )
@@
   (junction (at 320.675 194.31) (diameter 0) (color 0 0 0 0)
   )
+  (junction (at 68.072 139.7) (diameter 0) (color 0 0 0 0)
+  )
   (junction (at 153.035 199.39) (diameter 0) (color 0 0 0 0)
   )
@@
     (stroke (width 0) (type default) (color 0 0 0 0))
   )
-  (wire (pts (xy 52.451 139.7) (xy 90.678 139.7))
+  (wire (pts (xy 52.451 139.7) (xy 68.072 139.7))
     (stroke (width 0) (type default) (color 0 0 0 0))
   )
@@
     (stroke (width 0) (type default) (color 0 0 0 0))
   )
-  (wire (pts (xy 68.072 112.395) (xy 68.072 113.665))
+  (wire (pts (xy 68.072 112.395) (xy 68.072 113.538))
     (stroke (width 0) (type default) (color 0 0 0 0))
   )
@@
     (stroke (width 0) (type default) (color 0 0 0 0))
   )
+  (wire (pts (xy 68.072 113.538) (xy 68.072 113.665))
+    (stroke (width 0) (type default) (color 0 0 0 0))
+  )
   (wire (pts (xy 90.678 139.7) (xy 90.678 144.78))
     (stroke (width 0) (type default) (color 0 0 0 0))
@@
     (stroke (width 0) (type default) (color 0 0 0 0))
   )
+  (wire (pts (xy 68.072 139.7) (xy 90.678 139.7))
+    (stroke (width 0) (type default) (color 0 0 0 0))
+  )
   (wire (pts (xy 265.43 103.505) (xy 273.685 103.505))
     (stroke (width 0) (type default) (color 0 0 0 0))
@@
     (stroke (width 0) (type default) (color 0 0 0 0))
   )
+  (wire (pts (xy 68.072 113.665) (xy 68.072 132.08))
+    (stroke (width 0) (type default) (color 0 0 0 0))
+  )
   (wire (pts (xy 194.945 233.045) (xy 203.2 233.045))
     (stroke (width 0) (type default) (color 0 0 0 0))
@@
     (stroke (width 0) (type default) (color 0 0 0 0))
   )
+  (wire (pts (xy 68.072 113.538) (xy 68.199 113.538))
+    (stroke (width 0) (type default) (color 0 0 0 0))
+  )
   (wire (pts (xy 91.44 129.794) (xy 91.44 142.24))
     (stroke (width 0) (type default) (color 0 0 0 0))
@@
     (pin "2")
   )
-  (symbol (lib_id "74xx:74LS05") (at 55.245 179.959 180) (unit 5)
+  (symbol (lib_id "Device:R") (at 68.072 135.89 0) (unit 1)
     (in_bom yes) (on_board yes)
-    (property "Reference" "U300" (id 0) (at 55.245 187.579 0))
-    (property "Value" "74HCT04" (id 1) (at 55.245 185.039 0))
-    (property "Footprint" "Package_SO:SOIC-14_3.9x8.7mm_P1.27mm" (id 2) (at 55.245 179.959 0)
+    (property "Reference" "R303" (id 0) (at 69.85 134.7216 0)
+      (effects (font (size 1.27 1.27)) (justify left))
+    )
+    (property "Value" "1K" (id 1) (at 69.85 137.033 0)
+      (effects (font (size 1.27 1.27)) (justify left))
+    )
+    (property "Footprint" "Resistor_SMD:R_0805_2012Metric" (id 2) (at 66.294 135.89 90)
       (effects (font (size 1.27 1.27)) hide)
     )
-    (property "Datasheet" "http://www.ti.com/lit/gpn/sn74LS05" (id 3) (at 55.245 179.959 0)
+    (property "Datasheet" "~" (id 3) (at 68.072 135.89 0)
+      (effects (font (size 1.27 1.27)) hide)
+    )
+    (pin "1")
+    (pin "2")
+  )
+  (symbol (lib_id "74xx:74LS05") (at 44.831 139.7 0) (unit 3)
+    (in_bom yes) (on_board yes)
+    (property "Reference" "U300" (id 0) (at 44.831 134.747 0))
+    (property "Value" "74HCT05" (id 1) (at 44.831 132.2101 0))
+    (property "Footprint" "Package_SO:SOIC-14_3.9x8.7mm_P1.27mm" (id 2) (at 44.831 139.7 0)
+      (effects (font (size 1.27 1.27)) hide)
+    )
+    (property "Datasheet" "http://www.ti.com/lit/gpn/sn74LS05" (id 3) (at 44.831 139.7 0)
       (effects (font (size 1.27 1.27)) hide)
     )
@@
   (symbol (lib_id "Device:R") (at 365.76 76.835 0) (unit 1)
     (in_bom yes) (on_board yes)
-    (property "Reference" "R305" (id 0) (at 365.76 72.39 90)
+    (property "Reference" "R306" (id 0) (at 365.76 72.39 90)
       (effects (font (size 1.27 1.27)) (justify left))
     )
@@
   (symbol (lib_id "Device:R") (at 363.22 76.835 0) (unit 1)
     (in_bom yes) (on_board yes)
-    (property "Reference" "R304" (id 0) (at 363.22 72.39 90)
+    (property "Reference" "R305" (id 0) (at 363.22 72.39 90)
       (effects (font (size 1.27 1.27)) (justify left))
     )
@@
   (symbol (lib_id "Device:R") (at 360.68 76.835 0) (unit 1)
     (in_bom yes) (on_board yes)
-    (property "Reference" "R303" (id 0) (at 360.68 72.39 90)
+    (property "Reference" "R304" (id 0) (at 360.68 72.39 90)
       (effects (font (size 1.27 1.27)) (justify left))
     )
@@
     (pin "1")
   )
+  (symbol (lib_id "74xx:74HCT04") (at 55.245 179.959 180) (unit 3)
+    (in_bom yes) (on_board yes)
+    (property "Reference" "U204" (id 0) (at 55.372 184.785 0))
+    (property "Value" "74AHCT04" (id 1) (at 55.499 187.0202 0))
+    (property "Footprint" "Package_SO:SOIC-14_3.9x8.7mm_P1.27mm" (id 2) (at 55.245 179.959 0)
+      (effects (font (size 1.27 1.27)) hide)
+    )
+    (property "Datasheet" "https://assets.nexperia.com/documents/data-sheet/74HC_HCT04.pdf" (id 3) (at 55.245 179.959 0)
+      (effects (font (size 1.27 1.27)) hide)
+    )
+    (property "Digikey" "296-31832-1-ND" (id 4) (at 55.245 179.959 0)
+      (effects (font (size 1.27 1.27)) hide)
+    )
+    (pin "1")
+    (pin "2")
+    (pin "3")
+    (pin "4")
+    (pin "5")
+    (pin "6")
+    (pin "8")
+    (pin "9")
+    (pin "10")
+    (pin "11")
+    (pin "12")
+    (pin "13")
+    (pin "14")
+    (pin "7")
+  )
   (symbol (lib_id "power:+5V") (at 68.072 112.395 0) (unit 1)
     (in_bom yes) (on_board yes)
@@
     (pin "1")
   )
-  (symbol (lib_id "Device:R") (at 368.3 76.835 0) (unit 1)
-    (in_bom yes) (on_board yes)
-    (property "Reference" "R405" (id 0) (at 368.3 72.39 90)
-      (effects (font (size 1.27 1.27)) (justify left))
-    )
-    (property "Value" "1K" (id 1) (at 368.3 78.74 90)
-      (effects (font (size 1.27 1.27)) (justify left))
-    )
-    (property "Footprint" "Resistor_SMD:R_0805_2012Metric" (id 2) (at 366.522 76.835 90)
-      (effects (font (size 1.27 1.27)) hide)
-    )
-    (property "Datasheet" "~" (id 3) (at 368.3 76.835 0)
-      (effects (font (size 1.27 1.27)) hide)
-    )
-    (pin "1")
-    (pin "2")
-  )
-  (symbol (lib_id "74xx:74LS05") (at 40.005 179.959 180) (unit 4)
+  (symbol (lib_id "74xx:74LS05") (at 40.005 179.959 180) (unit 6)
     (in_bom yes) (on_board yes)
-    (property "Reference" "U300" (id 0) (at 40.005 187.579 0))
-    (property "Value" "74HCT04" (id 1) (at 40.005 185.039 0))
+    (property "Reference" "U300" (id 0) (at 40.005 184.912 0))
+    (property "Value" "74HCT05" (id 1) (at 40.005 187.4489 0))
     (property "Footprint" "Package_SO:SOIC-14_3.9x8.7mm_P1.27mm" (id 2) (at 40.005 179.959 0)
       (effects (font (size 1.27 1.27)) hide)
@@
     (pin "7")
   )
-  (symbol (lib_id "Device:CP1") (at 286.385 233.68 180) (unit 1)
+  (symbol (lib_id "Device:R") (at 368.3 76.835 0) (unit 1)
     (in_bom yes) (on_board yes)
-    (property "Reference" "C720" (id 0) (at 289.306 232.5116 0)
-      (effects (font (size 1.27 1.27)) (justify right))
+    (property "Reference" "R405" (id 0) (at 368.3 72.39 90)
+      (effects (font (size 1.27 1.27)) (justify left))
     )
-    (property "Value" "10uF" (id 1) (at 289.306 234.823 0)
-      (effects (font (size 1.27 1.27)) (justify right))
+    (property "Value" "1K" (id 1) (at 368.3 78.74 90)
+      (effects (font (size 1.27 1.27)) (justify left))
     )
-    (property "Footprint" "Capacitor_THT:CP_Radial_D5.0mm_P2.00mm" (id 2) (at 286.385 233.68 0)
+    (property "Footprint" "Resistor_SMD:R_0805_2012Metric" (id 2) (at 366.522 76.835 90)
       (effects (font (size 1.27 1.27)) hide)
     )
-    (property "Datasheet" "~" (id 3) (at 286.385 233.68 0)
+    (property "Datasheet" "~" (id 3) (at 368.3 76.835 0)
       (effects (font (size 1.27 1.27)) hide)
     )
@@
     (pin "2")
   )
-  (symbol (lib_id "74xx:74LS05") (at 44.831 139.7 0) (unit 3)
+  (symbol (lib_id "Device:CP1") (at 286.385 233.68 180) (unit 1)
     (in_bom yes) (on_board yes)
-    (property "Reference" "U300" (id 0) (at 44.831 132.08 0))
-    (property "Value" "74HCT04" (id 1) (at 44.831 134.62 0))
-    (property "Footprint" "Package_SO:SOIC-14_3.9x8.7mm_P1.27mm" (id 2) (at 44.831 139.7 0)
+    (property "Reference" "C720" (id 0) (at 289.306 232.5116 0)
+      (effects (font (size 1.27 1.27)) (justify right))
+    )
+    (property "Value" "10uF" (id 1) (at 289.306 234.823 0)
+      (effects (font (size 1.27 1.27)) (justify right))
+    )
+    (property "Footprint" "Capacitor_THT:CP_Radial_D5.0mm_P2.00mm" (id 2) (at 286.385 233.68 0)
       (effects (font (size 1.27 1.27)) hide)
     )
-    (property "Datasheet" "http://www.ti.com/lit/gpn/sn74LS05" (id 3) (at 44.831 139.7 0)
+    (property "Datasheet" "~" (id 3) (at 286.385 233.68 0)
       (effects (font (size 1.27 1.27)) hide)
     )
     (pin "1")
     (pin "2")
-    (pin "3")
-    (pin "4")
-    (pin "5")
-    (pin "6")
-    (pin "8")
-    (pin "9")
-    (pin "10")
-    (pin "11")
-    (pin "12")
-    (pin "13")
-    (pin "14")
-    (pin "7")
   )
 )
