File: A2630-New-KiCAD-Rev30-PGA/N2360.kicad_sch (KiCad schematic)
At the start: 0 parts

Commit message: Add files via upload
Other:
- sheet Base Memory, Spares renamed Base Memory, Spares, Power
- sheet Logic, IDE, Power renamed Logic, IDE
