File: KiCAD/A2630-New-KiCAD-Rev401-PLCC/ExpansionMemory.kicad_sch (KiCad schematic)
At the start: 29 parts, among them U102 27C256, U103 27C256, U406 SDRAM(16Mx16), U407 SDRAM(16Mx16), U408 SDRAM(16Mx16), U409 SDRAM(16Mx16)

Commit message: Revision 4.1.0
Other:
- title: Amiga N2630 -> Amiga N2630 MC68882 PLCC
