File: KiCAD/A2630-New-KiCAD-Rev401-PLCC/Processor.kicad_sch (KiCad schematic)
At the start: 60 parts, among them J202 25/FPU, U200 MC68030, U201 MC68882, U204 74AHCT04, X1 25MHz, X2 50MHz

Commit message: Revision 4.1.0
Parts:
- U200: footprint N2630:MC68030-PGA -> N2630 Libraries:MC68030-PGA
Other:
- title: Amiga N2630 -> Amiga N2630 MC68882 PLCC
